Commit message: new bullet world

File: packages/suturo_urdf_publisher/urdf/hsrb_lab.urdf.xacro (robot description, xacro)
@@ -1,7 +1,8 @@
 <?xml version="1.0"?>
 <robot name="hsrb_lab" xmlns:xacro="http://ros.org/wiki/xacro">
-    <xacro:include filename="$(find suturo_urdf_publisher)/urdf/hsr_table.urdf.xacro"/>
-    <xacro:include filename="$(find suturo_urdf_publisher)/urdf/hsrb_lab_walls.urdf.xacro"/>
-    <xacro:include filename="$(find suturo_urdf_publisher)/urdf/hsr_shelf.urdf.xacro"/>
+    <xacro:include filename="$(find cram_hsrb_lab_demo)/launch/hsr_table.urdf.xacro"/>
+    <xacro:include filename="$(find cram_hsrb_lab_demo)/launch/hsrb_lab_walls.urdf.xacro"/>
+    <xacro:include filename="$(find cram_hsrb_lab_demo)/launch/hsr_shelf.urdf.xacro"/>
+    <xacro:include filename="$(find cram_hsrb_lab_demo)/launch/hsr_small_shelf.urdf.xacro"/>
     <xacro:include filename="$(find iai_kitchen)/urdf_obj/IAI_tables.urdf.xacro"/>
     <xacro:property name="pi" value="3.1415926535897931" />
@@ -9,5 +10,5 @@
     <xacro:property name="simulated" value="true" />
     <xacro:property name="data"
-    value="${load_yaml('$(find suturo_urdf_publisher)/urdf/yaml/semantic_map_manual_data.yaml')}" />
+    value="${load_yaml('$(find cram_hsrb_lab_demo)/resource/semantic_map_manual_data.yaml')}" />
     <xacro:property name="table_x"
         value="${data['robocup_table']['x_pos']}" />
@@ -22,4 +23,16 @@
     <xacro:property name="table_height"
         value="${data['robocup_table']['height']}" />
+    <xacro:property name="small_table_x"
+        value="${data['robocup_small_table']['x_pos']}" />
+    <xacro:property name="small_table_y"
+        value="${data['robocup_small_table']['y_pos']}" />
+    <xacro:property name="small_table_z_rot"
+        value="${data['robocup_small_table']['z_rot']}" />
+    <xacro:property name="small_table_depth"
+        value="${data['robocup_small_table']['depth']}" />
+    <xacro:property name="small_table_width"
+        value="${data['robocup_small_table']['width']}" />
+    <xacro:property name="small_table_height"
+        value="${data['robocup_small_table']['height']}" />
     <xacro:property name="shelf_x"
         value="${data['robocup_shelf']['x_pos']}" />
@@ -38,4 +51,20 @@
     <xacro:property name="num_floors"
         value="${data['robocup_shelf']['num_floors']}" />
+    <xacro:property name="shelf_2_x"
+        value="${data['robocup_shelf_2']['x_pos']}" />
+    <xacro:property name="shelf_2_y"
+        value="${data['robocup_shelf_2']['y_pos']}" />
+    <xacro:property name="shelf_2_z_rot"
+        value="${data['robocup_shelf_2']['z_rot']}" />
+    <xacro:property name="shelf_2_depth"
+        value="${data['robocup_shelf_2']['depth']}" />
+    <xacro:property name="shelf_2_width"
+        value="${data['robocup_shelf_2']['width']}" />
+    <xacro:property name="shelf_2_height"
+        value="${data['robocup_shelf_2']['height']}" />
+    <xacro:property name="shelf_2_floors_height"
+        value="${data['robocup_shelf_2']['floors_height']}" />
+    <xacro:property name="num_floors_2"
+        value="${data['robocup_shelf_2']['num_floors']}" />
     <xacro:if value="${simulated}">
         <link name="world"/>
@@ -50,18 +79,28 @@
     <robocup_shelf name="shelf" parent="room_link"
     size_x="${shelf_depth}" size_y="${shelf_width}" size_z="${shelf_height}" floors_height="${shelf_floors_height}">
-    <origin xyz="-0.1 -0.3 0" rpy="0 0 -${half_pi}" />
+    <origin xyz="0.0 -0.1 0" rpy="0 0 -${half_pi}" />
     </robocup_shelf>
     <robocup_table name="table" parent="room_link" size_x="${table_depth}" size_y="${table_width}" size_z="${table_height}" >
-        <origin xyz="-3 0 0" rpy="0 0 ${table_z_rot}" />
+        <origin xyz="-2.5 0.2 0" rpy="0 0 ${table_z_rot}" />
       </robocup_table>
     <!-- OTHER-->
+       <robocup_table name="table_2" parent="room_link" size_x="${table_depth}" size_y="${table_width}" size_z="${table_height}" >
+        <origin xyz="-1.7025 1.2 0" rpy="0 0 ${pi}" />
+      </robocup_table>
+       <robocup_table name="table_3" parent="room_link" size_x="${small_table_depth}" size_y="${small_table_width}" size_z="${small_table_height}" >
+        <origin xyz="2.3 1 0" rpy="0 0 ${pi}" />
+      </robocup_table>
+      <robocup_small_shelf name="shelf_small" parent="room_link"
+        size_x="${shelf_2_depth}" size_y="${shelf_2_width}" size_z="${shelf_2_height}" floors_height="${shelf_2_floors_height}">
+        <origin xyz="-0.95 -0.1 0" rpy="0 0 -${half_pi}" />
+      </robocup_small_shelf>
     <iai_table_1 name="table_area" parent="room_link">
-        <origin xyz="1.85 2.15 0" rpy="0 0 ${pi}" />
+        <origin xyz="2.35 2.35 0" rpy="0 0 ${pi}" />
     </iai_table_1>
     <iai_table_1 name="table_area_2" parent="room_link">
-        <origin xyz="-0.35 2.15 0" rpy="0 0 ${pi}" />
+        <origin xyz="0.25 2.35 0" rpy="0 0 ${pi}" />
     </iai_table_1>
     <hsr_lab_walls parent="room_link">
-        <origin xyz="-0.5 1 0" rpy="0 0 0" />
+        <origin xyz="0 1.2 0" rpy="0 0 0" />
     </hsr_lab_walls>
 </robot>

Commit message: switch to inorder and remove redef pi

File: packages/suturo_urdf_publisher/urdf/hsrb_lab.urdf.xacro (robot description, xacro)
@@ -6,5 +6,5 @@
     <xacro:include filename="$(find suturo_urdf_publisher)/urdf/hsr_small_shelf.urdf.xacro"/>
     <xacro:include filename="$(find suturo_urdf_publisher)/urdf/IAI_tables.urdf.xacro"/>
-    <xacro:property name="pi" value="3.1415926535897931" />
+    <!--<xacro:property name="pi" value="3.1415926535897931" /> -->
     <xacro:property name="half_pi" value="1.570796327" />
     <xacro:property name="simulated" value="true" />

Commit message: minor changes in the urdf

File: packages/suturo_urdf_publisher/urdf/hsrb_lab.urdf.xacro (robot description, xacro)
@@ -1,14 +1,14 @@
 <?xml version="1.0"?>
 <robot name="hsrb_lab" xmlns:xacro="http://ros.org/wiki/xacro">
-    <xacro:include filename="$(find suturo_urdf_publisher)/urdf/hsr_table.urdf.xacro"/>
-    <xacro:include filename="$(find suturo_urdf_publisher)/urdf/hsrb_lab_walls.urdf.xacro"/>
-    <xacro:include filename="$(find suturo_urdf_publisher)/urdf/hsr_shelf.urdf.xacro"/>
-    <xacro:include filename="$(find suturo_urdf_publisher)/urdf/hsr_small_shelf.urdf.xacro"/>
-    <xacro:include filename="$(find suturo_urdf_publisher)/urdf/IAI_tables.urdf.xacro"/>
-    <!--<xacro:property name="pi" value="3.1415926535897931" /> -->
+    <xacro:include filename="$(find cram_hsrb_lab_demo)/launch/hsr_table.urdf.xacro"/>
+    <xacro:include filename="$(find cram_hsrb_lab_demo)/launch/hsrb_lab_walls.urdf.xacro"/>
+    <xacro:include filename="$(find cram_hsrb_lab_demo)/launch/hsr_shelf.urdf.xacro"/>
+    <xacro:include filename="$(find cram_hsrb_lab_demo)/launch/hsr_small_shelf.urdf.xacro"/>
+    <xacro:include filename="$(find iai_kitchen)/urdf_obj/IAI_tables.urdf.xacro"/>
+    <xacro:property name="pi" value="3.1415926535897931" />
     <xacro:property name="half_pi" value="1.570796327" />
     <xacro:property name="simulated" value="true" />
     <xacro:property name="data"
-    value="${load_yaml('$(find suturo_urdf_publisher)/urdf/yaml/semantic_map_manual_data.yaml')}" />
+    value="${load_yaml('$(find cram_hsrb_lab_demo)/resource/semantic_map_manual_data.yaml')}" />
     <xacro:property name="table_x"
         value="${data['robocup_table']['x_pos']}" />
@@ -86,5 +86,5 @@
     <!-- OTHER-->
        <robocup_table name="table_2" parent="room_link" size_x="${table_depth}" size_y="${table_width}" size_z="${table_height}" >
-        <origin xyz="-1.7025 1.2 0" rpy="0 0 ${pi}" />
+        <origin xyz="-1.6 1.2 0" rpy="0 0 ${pi}" />
       </robocup_table>
        <robocup_table name="table_3" parent="room_link" size_x="${small_table_depth}" size_y="${small_table_width}" size_z="${small_table_height}" >

Commit message: commited wrong changes

File: packages/suturo_urdf_publisher/urdf/hsrb_lab.urdf.xacro (robot description, xacro)
@@ -1,14 +1,13 @@
 <?xml version="1.0"?>
 <robot name="hsrb_lab" xmlns:xacro="http://ros.org/wiki/xacro">
-    <xacro:include filename="$(find cram_hsrb_lab_demo)/launch/hsr_table.urdf.xacro"/>
-    <xacro:include filename="$(find cram_hsrb_lab_demo)/launch/hsrb_lab_walls.urdf.xacro"/>
-    <xacro:include filename="$(find cram_hsrb_lab_demo)/launch/hsr_shelf.urdf.xacro"/>
-    <xacro:include filename="$(find cram_hsrb_lab_demo)/launch/hsr_small_shelf.urdf.xacro"/>
-    <xacro:include filename="$(find iai_kitchen)/urdf_obj/IAI_tables.urdf.xacro"/>
+    <xacro:include filename="$(find suturo_urdf_publisher)/urdf/hsr_table.urdf.xacro"/>
+    <xacro:include filename="$(find suturo_urdf_publisher)/urdf/hsrb_lab_walls.urdf.xacro"/>
+    <xacro:include filename="$(find suturo_urdf_publisher)/urdf/hsr_shelf.urdf.xacro"/>
+    <xacro:include filename="$(find suturo_urdf_publisher)/urdf/IAI_tables.urdf.xacro"/>
     <xacro:property name="pi" value="3.1415926535897931" />
     <xacro:property name="half_pi" value="1.570796327" />
     <xacro:property name="simulated" value="true" />
     <xacro:property name="data"
-    value="${load_yaml('$(find cram_hsrb_lab_demo)/resource/semantic_map_manual_data.yaml')}" />
+    value="${load_yaml('$(find suturo_urdf_publisher)/urdf/yaml/semantic_map_manual_data.yaml')}" />
     <xacro:property name="table_x"
         value="${data['robocup_table']['x_pos']}" />
@@ -23,16 +22,4 @@
     <xacro:property name="table_height"
         value="${data['robocup_table']['height']}" />
-    <xacro:property name="small_table_x"
-        value="${data['robocup_small_table']['x_pos']}" />
-    <xacro:property name="small_table_y"
-        value="${data['robocup_small_table']['y_pos']}" />
-    <xacro:property name="small_table_z_rot"
-        value="${data['robocup_small_table']['z_rot']}" />
-    <xacro:property name="small_table_depth"
-        value="${data['robocup_small_table']['depth']}" />
-    <xacro:property name="small_table_width"
-        value="${data['robocup_small_table']['width']}" />
-    <xacro:property name="small_table_height"
-        value="${data['robocup_small_table']['height']}" />
     <xacro:property name="shelf_x"
         value="${data['robocup_shelf']['x_pos']}" />
@@ -51,20 +38,4 @@
     <xacro:property name="num_floors"
         value="${data['robocup_shelf']['num_floors']}" />
-    <xacro:property name="shelf_2_x"
-        value="${data['robocup_shelf_2']['x_pos']}" />
-    <xacro:property name="shelf_2_y"
-        value="${data['robocup_shelf_2']['y_pos']}" />
-    <xacro:property name="shelf_2_z_rot"
-        value="${data['robocup_shelf_2']['z_rot']}" />
-    <xacro:property name="shelf_2_depth"
-        value="${data['robocup_shelf_2']['depth']}" />
-    <xacro:property name="shelf_2_width"
-        value="${data['robocup_shelf_2']['width']}" />
-    <xacro:property name="shelf_2_height"
-        value="${data['robocup_shelf_2']['height']}" />
-    <xacro:property name="shelf_2_floors_height"
-        value="${data['robocup_shelf_2']['floors_height']}" />
-    <xacro:property name="num_floors_2"
-        value="${data['robocup_shelf_2']['num_floors']}" />
     <xacro:if value="${simulated}">
         <link name="world"/>
@@ -79,28 +50,21 @@
     <robocup_shelf name="shelf" parent="room_link"
     size_x="${shelf_depth}" size_y="${shelf_width}" size_z="${shelf_height}" floors_height="${shelf_floors_height}">
-    <origin xyz="0.0 -0.1 0" rpy="0 0 -${half_pi}" />
+    <origin xyz="-0.1 -0.3 0" rpy="0 0 -${half_pi}" />
     </robocup_shelf>
     <robocup_table name="table" parent="room_link" size_x="${table_depth}" size_y="${table_width}" size_z="${table_height}" >
-        <origin xyz="-2.5 0.2 0" rpy="0 0 ${table_z_rot}" />
+        <origin xyz="-3 0 0" rpy="0 0 ${table_z_rot}" />
+      </robocup_table>
+      <robocup_table name="table_2" parent="room_link" size_x="${table_depth}" size_y="${table_width}" size_z="${table_height}" >
+        <origin xyz="-1.6 1.2 0" rpy="0 0 ${pi}" />
       </robocup_table>
     <!-- OTHER-->
-       <robocup_table name="table_2" parent="room_link" size_x="${table_depth}" size_y="${table_width}" size_z="${table_height}" >
-        <origin xyz="-1.6 1.2 0" rpy="0 0 ${pi}" />
-      </robocup_table>
-       <robocup_table name="table_3" parent="room_link" size_x="${small_table_depth}" size_y="${small_table_width}" size_z="${small_table_height}" >
-        <origin xyz="2.3 1 0" rpy="0 0 ${pi}" />
-      </robocup_table>
-      <robocup_small_shelf name="shelf_small" parent="room_link"
-        size_x="${shelf_2_depth}" size_y="${shelf_2_width}" size_z="${shelf_2_height}" floors_height="${shelf_2_floors_height}">
-        <origin xyz="-0.95 -0.1 0" rpy="0 0 -${half_pi}" />
-      </robocup_small_shelf>
     <iai_table_1 name="table_area" parent="room_link">
-        <origin xyz="2.35 2.35 0" rpy="0 0 ${pi}" />
+        <origin xyz="1.85 2.15 0" rpy="0 0 ${pi}" />
     </iai_table_1>
     <iai_table_1 name="table_area_2" parent="room_link">
-        <origin xyz="0.25 2.35 0" rpy="0 0 ${pi}" />
+        <origin xyz="-0.35 2.15 0" rpy="0 0 ${pi}" />
     </iai_table_1>
     <hsr_lab_walls parent="room_link">
-        <origin xyz="0 1.2 0" rpy="0 0 0" />
+        <origin xyz="-0.5 1 0" rpy="0 0 0" />
     </hsr_lab_walls>
 </robot>

Commit message: changes urdf

File: packages/suturo_urdf_publisher/urdf/hsrb_lab.urdf.xacro (robot description, xacro)
@@ -4,4 +4,5 @@
     <xacro:include filename="$(find suturo_urdf_publisher)/urdf/hsrb_lab_walls.urdf.xacro"/>
     <xacro:include filename="$(find suturo_urdf_publisher)/urdf/hsr_shelf.urdf.xacro"/>
+    <xacro:include filename="$(find suturo_urdf_publisher)/urdf/hsr_small_shelf.urdf.xacro"/>
     <xacro:include filename="$(find suturo_urdf_publisher)/urdf/IAI_tables.urdf.xacro"/>
     <xacro:property name="pi" value="3.1415926535897931" />
@@ -9,5 +10,5 @@
     <xacro:property name="simulated" value="true" />
     <xacro:property name="data"
-    value="${load_yaml('$(find suturo_urdf_publisher)/urdf/yaml/semantic_map_manual_data.yaml')}" />
+    value="${load_yaml('$(find cram_hsrb_lab_demo)/resource/semantic_map_manual_data.yaml')}" />
     <xacro:property name="table_x"
         value="${data['robocup_table']['x_pos']}" />
@@ -22,4 +23,16 @@
     <xacro:property name="table_height"
         value="${data['robocup_table']['height']}" />
+    <xacro:property name="small_table_x"
+        value="${data['robocup_small_table']['x_pos']}" />
+    <xacro:property name="small_table_y"
+        value="${data['robocup_small_table']['y_pos']}" />
+    <xacro:property name="small_table_z_rot"
+        value="${data['robocup_small_table']['z_rot']}" />
+    <xacro:property name="small_table_depth"
+        value="${data['robocup_small_table']['depth']}" />
+    <xacro:property name="small_table_width"
+        value="${data['robocup_small_table']['width']}" />
+    <xacro:property name="small_table_height"
+        value="${data['robocup_small_table']['height']}" />
     <xacro:property name="shelf_x"
         value="${data['robocup_shelf']['x_pos']}" />
@@ -38,4 +51,20 @@
     <xacro:property name="num_floors"
         value="${data['robocup_shelf']['num_floors']}" />
+    <xacro:property name="shelf_2_x"
+        value="${data['robocup_shelf_2']['x_pos']}" />
+    <xacro:property name="shelf_2_y"
+        value="${data['robocup_shelf_2']['y_pos']}" />
+    <xacro:property name="shelf_2_z_rot"
+        value="${data['robocup_shelf_2']['z_rot']}" />
+    <xacro:property name="shelf_2_depth"
+        value="${data['robocup_shelf_2']['depth']}" />
+    <xacro:property name="shelf_2_width"
+        value="${data['robocup_shelf_2']['width']}" />
+    <xacro:property name="shelf_2_height"
+        value="${data['robocup_shelf_2']['height']}" />
+    <xacro:property name="shelf_2_floors_height"
+        value="${data['robocup_shelf_2']['floors_height']}" />
+    <xacro:property name="num_floors_2"
+        value="${data['robocup_shelf_2']['num_floors']}" />
     <xacro:if value="${simulated}">
         <link name="world"/>
@@ -50,21 +79,28 @@
     <robocup_shelf name="shelf" parent="room_link"
     size_x="${shelf_depth}" size_y="${shelf_width}" size_z="${shelf_height}" floors_height="${shelf_floors_height}">
-    <origin xyz="-0.1 -0.3 0" rpy="0 0 -${half_pi}" />
+    <origin xyz="0.0 -0.1 0" rpy="0 0 -${half_pi}" />
     </robocup_shelf>
     <robocup_table name="table" parent="room_link" size_x="${table_depth}" size_y="${table_width}" size_z="${table_height}" >
-        <origin xyz="-3 0 0" rpy="0 0 ${table_z_rot}" />
+        <origin xyz="-2.5 0.2 0" rpy="0 0 ${table_z_rot}" />
       </robocup_table>
-      <robocup_table name="table_2" parent="room_link" size_x="${table_depth}" size_y="${table_width}" size_z="${table_height}" >
+    <!-- OTHER-->
+       <robocup_table name="table_2" parent="room_link" size_x="${table_depth}" size_y="${table_width}" size_z="${table_height}" >
         <origin xyz="-1.6 1.2 0" rpy="0 0 ${pi}" />
       </robocup_table>
-    <!-- OTHER-->
+       <robocup_table name="table_3" parent="room_link" size_x="${small_table_depth}" size_y="${small_table_width}" size_z="${small_table_height}" >
+        <origin xyz="2.3 1 0" rpy="0 0 ${pi}" />
+      </robocup_table>
+      <robocup_small_shelf name="shelf_small" parent="room_link"
+        size_x="${shelf_2_depth}" size_y="${shelf_2_width}" size_z="${shelf_2_height}" floors_height="${shelf_2_floors_height}">
+        <origin xyz="-0.95 -0.1 0" rpy="0 0 -${half_pi}" />
+      </robocup_small_shelf>
     <iai_table_1 name="table_area" parent="room_link">
-        <origin xyz="1.85 2.15 0" rpy="0 0 ${pi}" />
+        <origin xyz="2.35 2.35 0" rpy="0 0 ${pi}" />
     </iai_table_1>
     <iai_table_1 name="table_area_2" parent="room_link">
-        <origin xyz="-0.35 2.15 0" rpy="0 0 ${pi}" />
+        <origin xyz="0.25 2.35 0" rpy="0 0 ${pi}" />
     </iai_table_1>
     <hsr_lab_walls parent="room_link">
-        <origin xyz="-0.5 1 0" rpy="0 0 0" />
+        <origin xyz="0 1.2 0" rpy="0 0 0" />
     </hsr_lab_walls>
 </robot>

Commit message: moved the map 12cm in y direction

File: packages/suturo_urdf_publisher/urdf/hsrb_lab.urdf.xacro (robot description, xacro)
@@ -70,5 +70,5 @@
         <link name="world"/>
         <joint name="world_room_joint" type="fixed">
-            <origin xyz="0.0 0.0 0 " rpy="0 0 0" />
+            <origin xyz="0.0 0.12 0 " rpy="0 0 0" />
             <parent link="world"/>
             <child link="room_link"/>

Commit message: moved shelf about 10 cm in x direction

File: packages/suturo_urdf_publisher/urdf/hsrb_lab.urdf.xacro (robot description, xacro)
@@ -79,5 +79,5 @@
     <robocup_shelf name="shelf" parent="room_link"
     size_x="${shelf_depth}" size_y="${shelf_width}" size_z="${shelf_height}" floors_height="${shelf_floors_height}">
-    <origin xyz="0.0 -0.1 0" rpy="0 0 -${half_pi}" />
+    <origin xyz="0.1 -0.1 0" rpy="0 0 -${half_pi}" />
     </robocup_shelf>
     <robocup_table name="table" parent="room_link" size_x="${table_depth}" size_y="${table_width}" size_z="${table_height}" >

Commit message: update urdf for new map

File: packages/suturo_urdf_publisher/urdf/hsrb_lab.urdf.xacro (robot description, xacro)
@@ -70,5 +70,5 @@
         <link name="world"/>
         <joint name="world_room_joint" type="fixed">
-            <origin xyz="0.0 0.12 0 " rpy="0 0 0" />
+            <origin xyz="0.0 0 0 " rpy="0 0 0" />
             <parent link="world"/>
             <child link="room_link"/>

Commit message: urdf back to old map

File: packages/suturo_urdf_publisher/urdf/hsrb_lab.urdf.xacro (robot description, xacro)
@@ -70,5 +70,5 @@
         <link name="world"/>
         <joint name="world_room_joint" type="fixed">
-            <origin xyz="0.0 0 0 " rpy="0 0 0" />
+            <origin xyz="0.0 0.12 0 " rpy="0 0 0" />
             <parent link="world"/>
             <child link="room_link"/>
