Commit message: small shelf for robosim

File: packages/suturo_urdf_publisher/urdf/robocup_sim.urdf.xacro (robot description, xacro)
@@ -23,16 +23,4 @@
     <xacro:property name="table_height"
         value="${data['robocup_table']['height']}" />
-    <xacro:property name="small_table_x"
-        value="${data['robocup_small_table']['x_pos']}" />
-    <xacro:property name="small_table_y"
-        value="${data['robocup_small_table']['y_pos']}" />
-    <xacro:property name="small_table_z_rot"
-        value="${data['robocup_small_table']['z_rot']}" />
-    <xacro:property name="small_table_depth"
-        value="${data['robocup_small_table']['depth']}" />
-    <xacro:property name="small_table_width"
-        value="${data['robocup_small_table']['width']}" />
-    <xacro:property name="small_table_height"
-        value="${data['robocup_small_table']['height']}" />
     <xacro:property name="shelf_x"
         value="${data['robocup_shelf']['x_pos']}" />
@@ -85,20 +73,8 @@
       </robocup_table>
     <!-- OTHER-->
-       <robocup_table name="table_2" parent="room_link" size_x="${table_depth}" size_y="${table_width}" size_z="${table_height}" >
-        <origin xyz="-1.6 1.2 0" rpy="0 0 ${pi}" />
-      </robocup_table>
-       <robocup_table name="table_3" parent="room_link" size_x="${small_table_depth}" size_y="${small_table_width}" size_z="${small_table_height}" >
-        <origin xyz="2.3 1 0" rpy="0 0 ${pi}" />
-      </robocup_table>
       <robocup_small_shelf name="shelf_small" parent="room_link"
         size_x="${shelf_2_depth}" size_y="${shelf_2_width}" size_z="${shelf_2_height}" floors_height="${shelf_2_floors_height}">
         <origin xyz="-0.95 -0.1 0" rpy="0 0 -${half_pi}" />
       </robocup_small_shelf>
-    <iai_table_1 name="table_area" parent="room_link">
-        <origin xyz="2.35 2.35 0" rpy="0 0 ${pi}" />
-    </iai_table_1>
-    <iai_table_1 name="table_area_2" parent="room_link">
-        <origin xyz="0.25 2.35 0" rpy="0 0 ${pi}" />
-    </iai_table_1>
     <hsr_lab_walls parent="room_link">
         <origin xyz="0 1.2 0" rpy="0 0 0" />

File: packages/suturo_urdf_publisher/urdf/robocup_sim_small_shelf.urdf.xacro (robot description, xacro)
@@ -3,7 +3,4 @@
   <material name="shelf_small_grey">
     <color rgba="0.7 0.7 0.8 1"/>
-  </material>
-  <material name="shelf_door_grey">
-    <color rgba="0.9 0.9 0.98 1"/>
   </material>
   <macro name="robocup_small_shelf" params="name parent *origin size_x size_y size_z floors_height">
@@ -40,8 +37,4 @@
       <origin xyz="${size_x/2} ${size_y} ${size_z/2}" rpy="0 0 0"/>
     </robocup_small_shelf_piece>
-    <robocup_small_shelf_door name="${name}_door_left" parent="${name}_left_side"
-      size_x="0.01" size_y="${size_y/2}" size_z="${size_z}" offset_x="${size_x}">
-      <origin xyz="0 ${size_y*0.75} ${size_z/2}" rpy="0 0 0"/>
-    </robocup_small_shelf_door>
     <!-- FLOORS -->
     <xacro:if value="${num_floors > 0}">
@@ -96,29 +89,3 @@
     </joint>
   </macro>
-  <macro name="robocup_small_shelf_door" params="name parent *origin box_z_offset=0.0 size_x size_y size_z offset_x">
-    <!-- LINK -->
-    <link name="${name}_door">
-      <visual>
-        <material name="shelf_door_grey"/>
-        <origin xyz="0 0 ${box_z_offset}" rpy="0 0 0" />
-        <geometry>
-          <box size="${size_x} ${size_y} ${size_z}" />
-        </geometry>
-      </visual>
-      <collision>
-        <origin xyz="0 0 ${box_z_offset}" rpy="0 0 0" />
-        <geometry>
-          <box size="${size_x} ${size_y} ${size_z}" />
-        </geometry>
-      </collision>
-    </link>
-    <!-- JOINT -->
-    <joint name="${name}_door_joint" type="revolute">
-      <origin xyz="${offset_x/-2} ${size_y/-2} 0" rpy="0 0 3.1416"/>
-      <axis xyz="0 0 1" />
-      <parent link="${parent}_piece"/>
-      <child link="${name}_door"/>
-      <limit effort="30" velocity="1.0" lower="0.0" upper="1.91986" />
-    </joint>
-  </macro>
 </robot>
