Commit message: work on urdf

File: packages/suturo_urdf_publisher/urdf/robocup_sim_t1.urdf.xacro (robot description, xacro)
@@ -2,7 +2,7 @@
 <robot name="hsrb_lab" xmlns:xacro="http://ros.org/wiki/xacro">
     <xacro:include filename="$(find suturo_urdf_publisher)/urdf/hsr_table.urdf.xacro"/>
-    <xacro:include filename="$(find suturo_urdf_publisher)/urdf/hsrb_lab_walls.urdf.xacro"/>
-    <xacro:include filename="$(find suturo_urdf_publisher)/urdf/hsr_shelf.urdf.xacro"/>
-    <xacro:include filename="$(find suturo_urdf_publisher)/urdf/hsr_small_shelf.urdf.xacro"/>
+    <xacro:include filename="$(find suturo_urdf_publisher)/urdf/robocup_sim_walls.urdf.xacro"/>
+    <xacro:include filename="$(find suturo_urdf_publisher)/urdf/robocup_sim_shelf.urdf.xacro"/>
+    <xacro:include filename="$(find suturo_urdf_publisher)/urdf/robocup_sim_small_shelf.urdf.xacro"/>
     <xacro:include filename="$(find suturo_urdf_publisher)/urdf/IAI_tables.urdf.xacro"/>
     <xacro:property name="pi" value="3.1415926535897931" />
@@ -58,5 +58,5 @@
         <link name="world"/>
         <joint name="world_room_joint" type="fixed">
-            <origin xyz="0.0 0.12 0 " rpy="0 0 0" />
+            <origin xyz="0.0 0.0 0 " rpy="0 0 0" />
             <parent link="world"/>
             <child link="room_link"/>
@@ -67,5 +67,5 @@
     <robocup_shelf name="shelf" parent="room_link"
     size_x="${shelf_depth}" size_y="${shelf_width}" size_z="${shelf_height}" floors_height="${shelf_floors_height}">
-    <origin xyz="0.1 -0.1 0" rpy="0 0 -${half_pi}" />
+    <origin xyz="${shelf_x} ${shelf_y} 0" rpy="0 0 -${half_pi}" />
     </robocup_shelf>
     <robocup_table name="table" parent="room_link" size_x="${table_depth}" size_y="${table_width}" size_z="${table_height}" >
@@ -75,8 +75,8 @@
       <robocup_small_shelf name="shelf_small" parent="room_link"
         size_x="${shelf_2_depth}" size_y="${shelf_2_width}" size_z="${shelf_2_height}" floors_height="${shelf_2_floors_height}">
-        <origin xyz="-0.95 -0.1 0" rpy="0 0 -${half_pi}" />
+        <origin xyz="${shelf_2_x} ${shelf_2_y} 0" rpy="0 0 -${half_pi}" />
       </robocup_small_shelf>
     <hsr_lab_walls parent="room_link">
-        <origin xyz="0 1.2 0" rpy="0 0 0" />
+        <origin xyz="0 0 0" rpy="0 0 0" />
     </hsr_lab_walls>
 </robot>

File: packages/suturo_urdf_publisher/urdf/robocup_sim_t2.urdf.xacro (robot description, xacro)
@@ -58,5 +58,5 @@
         <link name="world"/>
         <joint name="world_room_joint" type="fixed">
-            <origin xyz="0.0 0.12 0 " rpy="0 0 0" />
+            <origin xyz="0.0 0.0 0 " rpy="0 0 0" />
             <parent link="world"/>
             <child link="room_link"/>
@@ -67,5 +67,5 @@
     <robocup_shelf name="shelf" parent="room_link"
     size_x="${shelf_depth}" size_y="${shelf_width}" size_z="${shelf_height}" floors_height="${shelf_floors_height}">
-    <origin xyz="0.1 -0.1 0" rpy="0 0 -${half_pi}" />
+    <origin xyz="${shelf_x} ${shelf_y} 0" rpy="0 0 -${half_pi}" />
     </robocup_shelf>
     <robocup_table name="table" parent="room_link" size_x="${table_depth}" size_y="${table_width}" size_z="${table_height}" >
@@ -75,8 +75,8 @@
       <robocup_small_shelf name="shelf_small" parent="room_link"
         size_x="${shelf_2_depth}" size_y="${shelf_2_width}" size_z="${shelf_2_height}" floors_height="${shelf_2_floors_height}">
-        <origin xyz="-0.95 -0.1 0" rpy="0 0 -${half_pi}" />
+        <origin xyz="${shelf_2_x} ${shelf_2_y} 0" rpy="0 0 -${half_pi}" />
       </robocup_small_shelf>
     <hsr_lab_walls parent="room_link">
-        <origin xyz="0 1.2 0" rpy="0 0 0" />
+        <origin xyz="0 0 0" rpy="0 0 0" />
     </hsr_lab_walls>
 </robot>

Commit message: rotate shelfs

File: packages/suturo_urdf_publisher/urdf/robocup_sim_t1.urdf.xacro (robot description, xacro)
@@ -67,5 +67,5 @@
     <robocup_shelf name="shelf" parent="room_link"
     size_x="${shelf_depth}" size_y="${shelf_width}" size_z="${shelf_height}" floors_height="${shelf_floors_height}">
-    <origin xyz="${shelf_x} ${shelf_y} 0" rpy="0 0 -${half_pi}" />
+    <origin xyz="${shelf_x} ${shelf_y} 0" rpy="0 0 ${shelf_z_rot}" />
     </robocup_shelf>
     <robocup_table name="table" parent="room_link" size_x="${table_depth}" size_y="${table_width}" size_z="${table_height}" >
@@ -75,5 +75,5 @@
       <robocup_small_shelf name="shelf_small" parent="room_link"
         size_x="${shelf_2_depth}" size_y="${shelf_2_width}" size_z="${shelf_2_height}" floors_height="${shelf_2_floors_height}">
-        <origin xyz="${shelf_2_x} ${shelf_2_y} 0" rpy="0 0 -${half_pi}" />
+        <origin xyz="${shelf_2_x} ${shelf_2_y} 0" rpy="0 0 ${shelf_2_z_rot}" />
       </robocup_small_shelf>
     <hsr_lab_walls parent="room_link">

Commit message: place table1

File: packages/suturo_urdf_publisher/urdf/robocup_sim_t1.urdf.xacro (robot description, xacro)
@@ -70,5 +70,5 @@
     </robocup_shelf>
     <robocup_table name="table" parent="room_link" size_x="${table_depth}" size_y="${table_width}" size_z="${table_height}" >
-        <origin xyz="-2.5 0.2 0" rpy="0 0 ${table_z_rot}" />
+        <origin xyz="${table_x} ${table_y} 0" rpy="0 0 ${table_z_rot}" />
       </robocup_table>
     <!-- OTHER-->
