Commit message: sim walls urdf

File: packages/suturo_urdf_publisher/urdf/robocup_sim_walls.urdf.xacro (robot description, xacro)
@@ -8,5 +8,5 @@
         <origin xyz="0 0 0.35" rpy="0 0 0" />
         <geometry>
-            <box size="4 0.15 0.7" />
+            <box size="1.75 0.15 0.7" />
         </geometry>
       </visual>
@@ -14,5 +14,5 @@
         <origin xyz="0 0 0.35" rpy="0 0 0" />
         <geometry>
-            <box size="4 0.15 0.7" />
+            <box size="1.75 0.15 0.7" />
         </geometry>
       </collision>
@@ -23,5 +23,5 @@
         <origin xyz="0 0 0.35" rpy="0 0 0" />
         <geometry>
-            <box size="5 0.15 0.7" />
+            <box size="2.25 0.15 0.7" />
         </geometry>
      </visual>
@@ -29,5 +29,5 @@
         <origin xyz="0 0 0.35" rpy="0 0 0" />
         <geometry>
-            <box size="5 0.15 0.7" />
+            <box size="2.25 0.15 0.7" />
         </geometry>
       </collision>
@@ -39,5 +39,5 @@
         <origin xyz="0 0 0.35" rpy="0 0 0" />
         <geometry>
-            <box size="4 0.15 0.7" />
+            <box size="1.35 0.15 0.7" />
         </geometry>
      </visual>
@@ -45,5 +45,5 @@
         <origin xyz="0 0 0.35" rpy="0 0 0" />
         <geometry>
-            <box size="4 0.15 0.7" />
+            <box size="1.35 0.15 0.7" />
         </geometry>
       </collision>
@@ -54,5 +54,5 @@
         <origin xyz="0 0 0.35" rpy="0 0 0" />
         <geometry>
-            <box size="5 0.15 0.7" />
+            <box size="2.24 0.15 0.7" />
         </geometry>
      </visual>
@@ -60,5 +60,80 @@
         <origin xyz="0 0 0.35" rpy="0 0 0" />
         <geometry>
-            <box size="5 0.15 0.7" />
+            <box size="2.24 0.15 0.7" />
+        </geometry>
+      </collision>
+    </link>
+    <link name="hsr_lab_wall_5">
+      <sphere_inertia radius="0" mass="0"/>
+      <visual>
+        <origin xyz="0 0 0.35" rpy="0 0 0" />
+        <geometry>
+            <box size="3.25 0.15 0.7" />
+        </geometry>
+     </visual>
+      <collision>
+        <origin xyz="0 0 0.35" rpy="0 0 0" />
+        <geometry>
+            <box size="3.25 0.15 0.7" />
+        </geometry>
+      </collision>
+    </link>
+    <link name="hsr_lab_wall_6">
+      <sphere_inertia radius="0" mass="0"/>
+      <visual>
+        <origin xyz="0 0 0.35" rpy="0 0 0" />
+        <geometry>
+            <box size="4.7 0.15 0.7" />
+        </geometry>
+     </visual>
+      <collision>
+        <origin xyz="0 0 0.35" rpy="0 0 0" />
+        <geometry>
+            <box size="4.7 0.15 0.7" />
+        </geometry>
+      </collision>
+    </link>
+    <link name="hsr_lab_wall_7">
+      <sphere_inertia radius="0" mass="0"/>
+      <visual>
+        <origin xyz="0 0 0.35" rpy="0 0 0" />
+        <geometry>
+            <box size="4.3 0.15 0.7" />
+        </geometry>
+     </visual>
+      <collision>
+        <origin xyz="0 0 0.35" rpy="0 0 0" />
+        <geometry>
+            <box size="4.3 0.15 0.7" />
+        </geometry>
+      </collision>
+    </link>
+    <link name="hsr_lab_wall_8">
+      <sphere_inertia radius="0" mass="0"/>
+      <visual>
+        <origin xyz="0 0 0.35" rpy="0 0 0" />
+        <geometry>
+            <box size="0.75 0.15 0.7" />
+        </geometry>
+     </visual>
+      <collision>
+        <origin xyz="0 0 0.35" rpy="0 0 0" />
+        <geometry>
+            <box size="0.75 0.15 0.7" />
+        </geometry>
+      </collision>
+    </link>
+    <link name="hsr_lab_wall_9">
+      <sphere_inertia radius="0" mass="0"/>
+      <visual>
+        <origin xyz="0 0 0.35" rpy="0 0 0" />
+        <geometry>
+            <box size="0.1 0.15 0.7" />
+        </geometry>
+     </visual>
+      <collision>
+        <origin xyz="0 0 0.35" rpy="0 0 0" />
+        <geometry>
+            <box size="0.1 0.15 0.7" />
         </geometry>
       </collision>
@@ -72,23 +147,48 @@
     </joint>
     <joint name="wall_1_joint" type="fixed">
-      <origin xyz="2.5 0.25 0" rpy="0 -0 1.5708" />
+      <origin xyz="0 -0.5 0" rpy="0 -0 1.5708" />
       <parent link="kitchen_walls"/>
       <child link="hsr_lab_wall_1"/>
     </joint>
     <joint name="wall_2_joint" type="fixed">
-        <origin xyz="0 2.25 0" rpy="0 -0 3.14159" />
+        <origin xyz="-2.25 -0.94 0" rpy="0 -0 3.14159" />
       <parent link="kitchen_walls"/>
       <child link="hsr_lab_wall_2"/>
     </joint>
     <joint name="wall_3_joint" type="fixed">
-        <origin xyz="-2.5 0.25 0" rpy="0 0 -1.5708" />
+        <origin xyz="1.75 -0.5 0" rpy="0 0 -1.5708" />
       <parent link="kitchen_walls"/>
       <child link="hsr_lab_wall_3"/>
     </joint>
-    <joint name="wall__joint" type="fixed">
+    <joint name="wall_4_joint" type="fixed">
         <origin xyz="0 -1.75 0" rpy="0 -0 0.000157" />
       <parent link="kitchen_walls"/>
       <child link="hsr_lab_wall_4"/>
     </joint>
+    <joint name="wall_5_joint" type="fixed">
+        <origin xyz="-2.35 4.55 0" rpy="0 -0 0.000157" />
+      <parent link="kitchen_walls"/>
+      <child link="hsr_lab_wall_5"/>
+    </joint>
+    <joint name="wall_6_joint" type="fixed">
+        <origin xyz="-2.35 5.15 0" rpy="0 -0 0.000157" />
+      <parent link="kitchen_walls"/>
+      <child link="hsr_lab_wall_6"/>
+    </joint>
+    <joint name="wall_7_joint" type="fixed">
+        <origin xyz="2.5 5.15 0" rpy="0 -0 0.000157" />
+      <parent link="kitchen_walls"/>
+      <child link="hsr_lab_wall_7"/>
+    </joint>
+    <joint name="wall_8_joint" type="fixed">
+        <origin xyz="1.75 0.85 0" rpy="0 -0 0.000157" />
+      <parent link="kitchen_walls"/>
+      <child link="hsr_lab_wall_8"/>
+    </joint>
+    <joint name="wall_9_joint" type="fixed">
+        <origin xyz="-2.35 1.5 0" rpy="0 -0 0.000157" />
+      <parent link="kitchen_walls"/>
+      <child link="hsr_lab_wall_9"/>
+    </joint>
   </macro>
 </robot>

Commit message: fix for walls?

File: packages/suturo_urdf_publisher/urdf/robocup_sim_walls.urdf.xacro (robot description, xacro)
@@ -152,40 +152,40 @@
     </joint>
     <joint name="wall_2_joint" type="fixed">
-        <origin xyz="-2.25 -0.94 0" rpy="0 -0 3.14159" />
+        <origin xyz="-2.25 -0.94 0" rpy="0 -0 1.5708" />
       <parent link="kitchen_walls"/>
       <child link="hsr_lab_wall_2"/>
     </joint>
     <joint name="wall_3_joint" type="fixed">
-        <origin xyz="1.75 -0.5 0" rpy="0 0 -1.5708" />
+        <origin xyz="1.75 -0.5 0" rpy="0 0 3.14159" />
       <parent link="kitchen_walls"/>
       <child link="hsr_lab_wall_3"/>
     </joint>
     <joint name="wall_4_joint" type="fixed">
-        <origin xyz="0 -1.75 0" rpy="0 -0 0.000157" />
+        <origin xyz="0 -1.75 0" rpy="0 -0 3.14159" />
       <parent link="kitchen_walls"/>
       <child link="hsr_lab_wall_4"/>
     </joint>
     <joint name="wall_5_joint" type="fixed">
-        <origin xyz="-2.35 4.55 0" rpy="0 -0 0.000157" />
+        <origin xyz="-2.35 4.55 0" rpy="0 -0 3.14159" />
       <parent link="kitchen_walls"/>
       <child link="hsr_lab_wall_5"/>
     </joint>
     <joint name="wall_6_joint" type="fixed">
-        <origin xyz="-2.35 5.15 0" rpy="0 -0 0.000157" />
+        <origin xyz="-2.35 5.15 0" rpy="0 -0 1.5798" />
       <parent link="kitchen_walls"/>
       <child link="hsr_lab_wall_6"/>
     </joint>
     <joint name="wall_7_joint" type="fixed">
-        <origin xyz="2.5 5.15 0" rpy="0 -0 0.000157" />
+        <origin xyz="2.5 5.15 0" rpy="0 -0 3.14159" />
       <parent link="kitchen_walls"/>
       <child link="hsr_lab_wall_7"/>
     </joint>
     <joint name="wall_8_joint" type="fixed">
-        <origin xyz="1.75 0.85 0" rpy="0 -0 0.000157" />
+        <origin xyz="1.75 0.85 0" rpy="0 -0 1.5798" />
       <parent link="kitchen_walls"/>
       <child link="hsr_lab_wall_8"/>
     </joint>
     <joint name="wall_9_joint" type="fixed">
-        <origin xyz="-2.35 1.5 0" rpy="0 -0 0.000157" />
+        <origin xyz="-2.35 1.5 0" rpy="0 -0 1.5798" />
       <parent link="kitchen_walls"/>
       <child link="hsr_lab_wall_9"/>

Commit message: rotation for walls 1-3

File: packages/suturo_urdf_publisher/urdf/robocup_sim_walls.urdf.xacro (robot description, xacro)
@@ -147,15 +147,15 @@
     </joint>
     <joint name="wall_1_joint" type="fixed">
-      <origin xyz="0 -0.5 0" rpy="0 -0 1.5708" />
+      <origin xyz="0 -0.5 0" rpy="0 -0 3.14159" />
       <parent link="kitchen_walls"/>
       <child link="hsr_lab_wall_1"/>
     </joint>
     <joint name="wall_2_joint" type="fixed">
-        <origin xyz="-2.25 -0.94 0" rpy="0 -0 1.5708" />
+        <origin xyz="-2.25 -0.94 0" rpy="0 3.14159" />
       <parent link="kitchen_walls"/>
       <child link="hsr_lab_wall_2"/>
     </joint>
     <joint name="wall_3_joint" type="fixed">
-        <origin xyz="1.75 -0.5 0" rpy="0 0 3.14159" />
+        <origin xyz="1.75 -0.5 0" rpy="0 0 -1.5798" />
       <parent link="kitchen_walls"/>
       <child link="hsr_lab_wall_3"/>

Commit message: added missing argument

File: packages/suturo_urdf_publisher/urdf/robocup_sim_walls.urdf.xacro (robot description, xacro)
@@ -152,10 +152,10 @@
     </joint>
     <joint name="wall_2_joint" type="fixed">
-        <origin xyz="-2.25 -0.94 0" rpy="0 3.14159" />
+        <origin xyz="-2.25 -0.94 0" rpy="0 -0 3.14159" />
       <parent link="kitchen_walls"/>
       <child link="hsr_lab_wall_2"/>
     </joint>
     <joint name="wall_3_joint" type="fixed">
-        <origin xyz="1.75 -0.5 0" rpy="0 0 -1.5798" />
+        <origin xyz="1.75 -0.5 0" rpy="0 -0 -1.5798" />
       <parent link="kitchen_walls"/>
       <child link="hsr_lab_wall_3"/>

Commit message: rotation and size walls 1-4

File: packages/suturo_urdf_publisher/urdf/robocup_sim_walls.urdf.xacro (robot description, xacro)
@@ -8,5 +8,5 @@
         <origin xyz="0 0 0.35" rpy="0 0 0" />
         <geometry>
-            <box size="1.75 0.15 0.7" />
+            <box size="2 0.15 0.7" />
         </geometry>
       </visual>
@@ -14,5 +14,5 @@
         <origin xyz="0 0 0.35" rpy="0 0 0" />
         <geometry>
-            <box size="1.75 0.15 0.7" />
+            <box size="2 0.15 0.7" />
         </geometry>
       </collision>
@@ -23,5 +23,5 @@
         <origin xyz="0 0 0.35" rpy="0 0 0" />
         <geometry>
-            <box size="2.25 0.15 0.7" />
+            <box size="3 0.15 0.7" />
         </geometry>
      </visual>
@@ -29,5 +29,5 @@
         <origin xyz="0 0 0.35" rpy="0 0 0" />
         <geometry>
-            <box size="2.25 0.15 0.7" />
+            <box size="3 0.15 0.7" />
         </geometry>
       </collision>
@@ -147,20 +147,20 @@
     </joint>
     <joint name="wall_1_joint" type="fixed">
-      <origin xyz="0 -0.5 0" rpy="0 -0 3.14159" />
+      <origin xyz="0.75 -0.5 0" rpy="0 -0 0" />
       <parent link="kitchen_walls"/>
       <child link="hsr_lab_wall_1"/>
     </joint>
     <joint name="wall_2_joint" type="fixed">
-        <origin xyz="-2.25 -0.94 0" rpy="0 -0 3.14159" />
+        <origin xyz="-1.75 -0.94 0" rpy="0 -0 0" />
       <parent link="kitchen_walls"/>
       <child link="hsr_lab_wall_2"/>
     </joint>
     <joint name="wall_3_joint" type="fixed">
-        <origin xyz="1.75 -0.5 0" rpy="0 -0 -1.5798" />
+        <origin xyz="1.75 -0.5 0" rpy="0 -0 1.5798" />
       <parent link="kitchen_walls"/>
       <child link="hsr_lab_wall_3"/>
     </joint>
     <joint name="wall_4_joint" type="fixed">
-        <origin xyz="0 -1.75 0" rpy="0 -0 3.14159" />
+        <origin xyz="-2.25 -1.75 0" rpy="0 -0 -1.5798" />
       <parent link="kitchen_walls"/>
       <child link="hsr_lab_wall_4"/>

Commit message: fix for wall 1-4?

File: packages/suturo_urdf_publisher/urdf/robocup_sim_walls.urdf.xacro (robot description, xacro)
@@ -8,5 +8,5 @@
         <origin xyz="0 0 0.35" rpy="0 0 0" />
         <geometry>
-            <box size="2 0.15 0.7" />
+            <box size="1.75 0.15 0.7" />
         </geometry>
       </visual>
@@ -14,5 +14,5 @@
         <origin xyz="0 0 0.35" rpy="0 0 0" />
         <geometry>
-            <box size="2 0.15 0.7" />
+            <box size="1.75 0.15 0.7" />
         </geometry>
       </collision>
@@ -23,5 +23,5 @@
         <origin xyz="0 0 0.35" rpy="0 0 0" />
         <geometry>
-            <box size="3 0.15 0.7" />
+            <box size="2.25 0.15 0.7" />
         </geometry>
      </visual>
@@ -29,5 +29,5 @@
         <origin xyz="0 0 0.35" rpy="0 0 0" />
         <geometry>
-            <box size="3 0.15 0.7" />
+            <box size="2.25 0.15 0.7" />
         </geometry>
       </collision>
@@ -147,10 +147,10 @@
     </joint>
     <joint name="wall_1_joint" type="fixed">
-      <origin xyz="0.75 -0.5 0" rpy="0 -0 0" />
+      <origin xyz="0 -0.5 0" rpy="0 -0 0" />
       <parent link="kitchen_walls"/>
       <child link="hsr_lab_wall_1"/>
     </joint>
     <joint name="wall_2_joint" type="fixed">
-        <origin xyz="-1.75 -0.94 0" rpy="0 -0 0" />
+        <origin xyz="-2.25 -0.5 0" rpy="0 -0 0" />
       <parent link="kitchen_walls"/>
       <child link="hsr_lab_wall_2"/>
@@ -162,5 +162,5 @@
     </joint>
     <joint name="wall_4_joint" type="fixed">
-        <origin xyz="-2.25 -1.75 0" rpy="0 -0 -1.5798" />
+        <origin xyz="-2.25 -1.75 0" rpy="0 -0 1.5798" />
       <parent link="kitchen_walls"/>
       <child link="hsr_lab_wall_4"/>

Commit message: walls ...

File: packages/suturo_urdf_publisher/urdf/robocup_sim_walls.urdf.xacro (robot description, xacro)
@@ -8,5 +8,5 @@
         <origin xyz="0 0 0.35" rpy="0 0 0" />
         <geometry>
-            <box size="1.75 0.15 0.7" />
+            <box size="2 0.15 0.7" />
         </geometry>
       </visual>
@@ -14,5 +14,5 @@
         <origin xyz="0 0 0.35" rpy="0 0 0" />
         <geometry>
-            <box size="1.75 0.15 0.7" />
+            <box size="2 0.15 0.7" />
         </geometry>
       </collision>
@@ -39,5 +39,5 @@
         <origin xyz="0 0 0.35" rpy="0 0 0" />
         <geometry>
-            <box size="1.35 0.15 0.7" />
+            <box size="6 0.15 0.7" />
         </geometry>
      </visual>
@@ -45,5 +45,5 @@
         <origin xyz="0 0 0.35" rpy="0 0 0" />
         <geometry>
-            <box size="1.35 0.15 0.7" />
+            <box size="6 0.15 0.7" />
         </geometry>
       </collision>
@@ -94,34 +94,4 @@
       </collision>
     </link>
-    <link name="hsr_lab_wall_7">
-      <sphere_inertia radius="0" mass="0"/>
-      <visual>
-        <origin xyz="0 0 0.35" rpy="0 0 0" />
-        <geometry>
-            <box size="4.3 0.15 0.7" />
-        </geometry>
-     </visual>
-      <collision>
-        <origin xyz="0 0 0.35" rpy="0 0 0" />
-        <geometry>
-            <box size="4.3 0.15 0.7" />
-        </geometry>
-      </collision>
-    </link>
-    <link name="hsr_lab_wall_8">
-      <sphere_inertia radius="0" mass="0"/>
-      <visual>
-        <origin xyz="0 0 0.35" rpy="0 0 0" />
-        <geometry>
-            <box size="0.75 0.15 0.7" />
-        </geometry>
-     </visual>
-      <collision>
-        <origin xyz="0 0 0.35" rpy="0 0 0" />
-        <geometry>
-            <box size="0.75 0.15 0.7" />
-        </geometry>
-      </collision>
-    </link>
     <link name="hsr_lab_wall_9">
       <sphere_inertia radius="0" mass="0"/>
@@ -147,20 +117,20 @@
     </joint>
     <joint name="wall_1_joint" type="fixed">
-      <origin xyz="0 -0.5 0" rpy="0 -0 0" />
+      <origin xyz="1 -0.94 0" rpy="0 -0 0" />
       <parent link="kitchen_walls"/>
       <child link="hsr_lab_wall_1"/>
     </joint>
     <joint name="wall_2_joint" type="fixed">
-        <origin xyz="-2.25 -0.5 0" rpy="0 -0 0" />
+        <origin xyz="-2.25 -0.94 0" rpy="0 -0 0" />
       <parent link="kitchen_walls"/>
       <child link="hsr_lab_wall_2"/>
     </joint>
     <joint name="wall_3_joint" type="fixed">
-        <origin xyz="1.75 -0.5 0" rpy="0 -0 1.5798" />
+        <origin xyz="2.5 -0.94 0" rpy="0 -0 1.5798" />
       <parent link="kitchen_walls"/>
       <child link="hsr_lab_wall_3"/>
     </joint>
     <joint name="wall_4_joint" type="fixed">
-        <origin xyz="-2.25 -1.75 0" rpy="0 -0 1.5798" />
+        <origin xyz="-2.25 -0.5 0" rpy="0 -0 1.5798" />
       <parent link="kitchen_walls"/>
       <child link="hsr_lab_wall_4"/>
@@ -176,14 +146,4 @@
       <child link="hsr_lab_wall_6"/>
     </joint>
-    <joint name="wall_7_joint" type="fixed">
-        <origin xyz="2.5 5.15 0" rpy="0 -0 3.14159" />
-      <parent link="kitchen_walls"/>
-      <child link="hsr_lab_wall_7"/>
-    </joint>
-    <joint name="wall_8_joint" type="fixed">
-        <origin xyz="1.75 0.85 0" rpy="0 -0 1.5798" />
-      <parent link="kitchen_walls"/>
-      <child link="hsr_lab_wall_8"/>
-    </joint>
     <joint name="wall_9_joint" type="fixed">
         <origin xyz="-2.35 1.5 0" rpy="0 -0 1.5798" />

Commit message: size  and position changes

File: packages/suturo_urdf_publisher/urdf/robocup_sim_walls.urdf.xacro (robot description, xacro)
@@ -8,5 +8,5 @@
         <origin xyz="0 0 0.35" rpy="0 0 0" />
         <geometry>
-            <box size="2 0.15 0.7" />
+            <box size="2.5 0.15 0.7" />
         </geometry>
       </visual>
@@ -14,5 +14,5 @@
         <origin xyz="0 0 0.35" rpy="0 0 0" />
         <geometry>
-            <box size="2 0.15 0.7" />
+            <box size="2.5 0.15 0.7" />
         </geometry>
       </collision>
@@ -23,5 +23,5 @@
         <origin xyz="0 0 0.35" rpy="0 0 0" />
         <geometry>
-            <box size="2.25 0.15 0.7" />
+            <box size="2.5 0.15 0.7" />
         </geometry>
      </visual>
@@ -29,5 +29,5 @@
         <origin xyz="0 0 0.35" rpy="0 0 0" />
         <geometry>
-            <box size="2.25 0.15 0.7" />
+            <box size="2.5 0.15 0.7" />
         </geometry>
       </collision>
@@ -54,5 +54,5 @@
         <origin xyz="0 0 0.35" rpy="0 0 0" />
         <geometry>
-            <box size="2.24 0.15 0.7" />
+            <box size="2.5 0.15 0.7" />
         </geometry>
      </visual>
@@ -60,5 +60,5 @@
         <origin xyz="0 0 0.35" rpy="0 0 0" />
         <geometry>
-            <box size="2.24 0.15 0.7" />
+            <box size="2.5 0.15 0.7" />
         </geometry>
       </collision>
@@ -122,5 +122,5 @@
     </joint>
     <joint name="wall_2_joint" type="fixed">
-        <origin xyz="-2.25 -0.94 0" rpy="0 -0 0" />
+        <origin xyz="-1.25 -0.94 0" rpy="0 -0 0" />
       <parent link="kitchen_walls"/>
       <child link="hsr_lab_wall_2"/>
@@ -132,5 +132,5 @@
     </joint>
     <joint name="wall_4_joint" type="fixed">
-        <origin xyz="-2.25 -0.5 0" rpy="0 -0 1.5798" />
+        <origin xyz="-2.25 0.5 0" rpy="0 -0 1.5798" />
       <parent link="kitchen_walls"/>
       <child link="hsr_lab_wall_4"/>

Commit message: fixes for the rest of the walls?

File: packages/suturo_urdf_publisher/urdf/robocup_sim_walls.urdf.xacro (robot description, xacro)
@@ -127,5 +127,5 @@
     </joint>
     <joint name="wall_3_joint" type="fixed">
-        <origin xyz="2.5 -0.94 0" rpy="0 -0 1.5798" />
+        <origin xyz="2.5 2.25 0" rpy="0 -0 1.5798" />
       <parent link="kitchen_walls"/>
       <child link="hsr_lab_wall_3"/>
@@ -137,10 +137,10 @@
     </joint>
     <joint name="wall_5_joint" type="fixed">
-        <origin xyz="-2.35 4.55 0" rpy="0 -0 3.14159" />
+        <origin xyz="-2.35 3 0" rpy="0 -0 1.5798" />
       <parent link="kitchen_walls"/>
       <child link="hsr_lab_wall_5"/>
     </joint>
     <joint name="wall_6_joint" type="fixed">
-        <origin xyz="-2.35 5.15 0" rpy="0 -0 1.5798" />
+        <origin xyz="0 5.15 0" rpy="0 -0 0" />
       <parent link="kitchen_walls"/>
       <child link="hsr_lab_wall_6"/>

Commit message: finishing the walls

File: packages/suturo_urdf_publisher/urdf/robocup_sim_walls.urdf.xacro (robot description, xacro)
@@ -39,5 +39,5 @@
         <origin xyz="0 0 0.35" rpy="0 0 0" />
         <geometry>
-            <box size="6 0.15 0.7" />
+            <box size="6.2 0.15 0.7" />
         </geometry>
      </visual>
@@ -45,5 +45,5 @@
         <origin xyz="0 0 0.35" rpy="0 0 0" />
         <geometry>
-            <box size="6 0.15 0.7" />
+            <box size="6.2 0.15 0.7" />
         </geometry>
       </collision>
@@ -84,5 +84,5 @@
         <origin xyz="0 0 0.35" rpy="0 0 0" />
         <geometry>
-            <box size="4.7 0.15 0.7" />
+            <box size="4.8 0.15 0.7" />
         </geometry>
      </visual>
@@ -90,5 +90,5 @@
         <origin xyz="0 0 0.35" rpy="0 0 0" />
         <geometry>
-            <box size="4.7 0.15 0.7" />
+            <box size="4.8 0.15 0.7" />
         </geometry>
       </collision>
@@ -127,10 +127,10 @@
     </joint>
     <joint name="wall_3_joint" type="fixed">
-        <origin xyz="2.5 2.25 0" rpy="0 -0 1.5798" />
+        <origin xyz="2.5 2 0" rpy="0 -0 1.5798" />
       <parent link="kitchen_walls"/>
       <child link="hsr_lab_wall_3"/>
     </joint>
     <joint name="wall_4_joint" type="fixed">
-        <origin xyz="-2.25 0.5 0" rpy="0 -0 1.5798" />
+        <origin xyz="-2.25 0.3 0" rpy="0 -0 1.5798" />
       <parent link="kitchen_walls"/>
       <child link="hsr_lab_wall_4"/>

Commit message: wall fix

File: packages/suturo_urdf_publisher/urdf/robocup_sim_walls.urdf.xacro (robot description, xacro)
@@ -8,5 +8,5 @@
         <origin xyz="0 0 0.35" rpy="0 0 0" />
         <geometry>
-            <box size="2.5 0.15 0.7" />
+            <box size="3 0.15 0.7" />
         </geometry>
       </visual>
@@ -14,5 +14,5 @@
         <origin xyz="0 0 0.35" rpy="0 0 0" />
         <geometry>
-            <box size="2.5 0.15 0.7" />
+            <box size="3 0.15 0.7" />
         </geometry>
       </collision>
