Commit message: Fixed bug, where the HSR cant grab the shelf door correctly

File: packages/suturo_urdf_publisher/urdf/hsrb_sim_v1_openable_door.urdf.xacro (robot description, xacro)
@@ -184,5 +184,5 @@
     <suturo_movable_door name="door_1" parent="room_link" height="2" width="0.83" depth="0.055" x="-1.4694" y="4.9966" z="1.045" r="0" p="0" yr="${pi}" door_lower="${-half_pi}" door_max="${half_pi}" >
     </suturo_movable_door>
-    <suturo_shelf name="openable_shelf_1" parent="room_link" size_x="0.5" size_y="1" size_z="0.7" floors_height="[0.2, 0.2, 0.2]" number_of_floors="3" door="no" >
+    <suturo_shelf name="openable_shelf_1" parent="room_link" size_x="0.5" size_y="1" size_z="0.7" floors_height="[0.055, 0.45]" number_of_floors="2" door="none" >
 	<origin xyz="1 1 0" rpy="0 0 ${pi}" />
     </suturo_shelf>

File: packages/suturo_urdf_publisher/urdf/suturo_shelf_openable.urdf.xacro (robot description, xacro)
@@ -43,14 +43,4 @@
       <origin xyz="${size_x/2} ${size_y} ${size_z/2}" rpy="0 0 0"/>
     </xacro:suturo_shelf_piece>
-    <xacro:macro name="shelf_floor_loop" params="floor_number">
-        <xacro:suturo_shelf_piece name="${name}_floor_${floor_number}" parent="${name}_base_center"
-          size_x="${size_x}" size_y="${size_y}" size_z="0.04" box_z_offset="-0.02">
-        <origin xyz="0.0 0.0 0.2" rpy="0 0 0"/>
-      </xacro:suturo_shelf_piece>
-      <xacro:if value="${(number_of_floors - 1) > floor_number}">
-            <xacro:shelf_floor_loop floor_number="${floor_number + 1}" />
-      </xacro:if>
-    </xacro:macro>
-    <xacro:shelf_floor_loop floor_number="0" />
     <!-- door -->
     <xacro:if value="${door == 'left'}">
@@ -103,5 +93,5 @@
       </visual>
       <collision>
-        <origin xyz="0 ${size_y} 0" rpy="0 0 0" />
+        <origin xyz="0 ${size_y/2} 0" rpy="0 0 0" />
         <geometry>
           <box size="${size_x} ${size_y} ${size_z}" />
@@ -125,5 +115,5 @@
     </link>
     <joint name="${name}_link_handle_joint" type="fixed">
-      <origin xyz="-0.01 ${size_y + 0.03} ${size_z/3}" rpy="0 0 0"/>
+      <origin xyz="-0.01 ${size_y - 0.02} ${size_z/3}" rpy="0 0 0"/>
       <axis xyz="0 0 1" />
       <parent link="${name}_link"/>
