Commit message: Adjusted small offset errors at the suturo_shelves

File: packages/suturo_urdf_publisher/urdf/suturo_shelf_openable.urdf.xacro (robot description, xacro)
@@ -87,5 +87,5 @@
       <visual>
         <material name="shelf_door_green"/>
-        <origin xyz="0 ${size_y/2} 0" rpy="0 0 0" />
+        <origin xyz="0 ${size_y/2.15} 0" rpy="0 0 0" />
         <geometry>
           <box size="${size_x} ${size_y} ${size_z}" />
@@ -93,5 +93,5 @@
       </visual>
       <collision>
-        <origin xyz="0 ${size_y/2} 0" rpy="0 0 0" />
+        <origin xyz="0 ${size_y/2.15} 0" rpy="0 0 0" />
         <geometry>
           <box size="${size_x} ${size_y} ${size_z}" />
@@ -104,5 +104,5 @@
         <origin xyz="0 0 0" rpy="0 0 0" />
         <geometry>
-          <box size="0.04 0.01 0.07" />
+          <box size="0.025 0.01 0.07" />
         </geometry>
       </visual>
@@ -115,5 +115,5 @@
     </link>
     <joint name="${name}_link_handle_joint" type="fixed">
-      <origin xyz="-0.01 ${size_y - 0.02} ${size_z/3}" rpy="0 0 0"/>
+      <origin xyz="-0.01 ${size_y - 0.04} ${size_z/3}" rpy="0 0 0"/>
       <axis xyz="0 0 1" />
       <parent link="${name}_link"/>

File: suturo_resources/urdf/hsrb_sim_v1_openable_door.urdf.xacro (robot description, xacro)
@@ -185,5 +185,5 @@
     </suturo_movable_door>
     <suturo_shelf name="openable_shelf_1" parent="room_link" size_x="0.44" size_y="0.75" size_z="0.585" floors_height="[0.2,0.2]" number_of_floors="2" door="left" >
-	<origin xyz="0.75 3 0" rpy="0 0 ${half_pi}" />
+	<origin xyz="0.75 3.01 0" rpy="0 0 ${half_pi}" />
     </suturo_shelf>
 </robot>
