Commit message: Added handles

File: packages/suturo_urdf_publisher/urdf/hsr_movable_door.urdf.xacro (robot description, xacro)
@@ -7,4 +7,9 @@
     <color rgba="0.74 0.25 0.25 1"/>
   </material>
+  <material name="handle_blue">
+    <color rgba="0.3 0.5 0.78 1"/>
+  </material>
+  <xacro:property name="pi" value="3.1415926535897931" />
+  <xacro:property name="half_pi" value="1.570796327" />
   <macro name="suturo_movable_door" params="name parent height width depth x y z r p yr door_lower door_max">
     <!-- LINKS -->
@@ -34,6 +39,38 @@
       <collision>
         <origin xyz="0 ${depth/2} 0" rpy="0 0 0" />
+        <geometry>-
+          <box size="0.05 0.05 ${height}" />
+        </geometry>
+      </collision>
+    </link>
+    <link name="${name}_handle_outside">
+      <sphere_inertia radius="0" mass="0"/>
+      <visual>
+	<material name="handle_blue"/>
+        <origin xyz="0 ${-0.5 * depth} 0" rpy="${half_pi} 0 ${pi}" />
+        <geometry>-
+          <box size="0.05 0.015 0.015" />
+        </geometry>
+      </visual>
+      <collision>
+        <origin xyz="0 ${-0.5 * depth} 0" rpy="${half_pi} 0 ${pi}" />
         <geometry>
-          <box size="0.05 0.05 ${height}" />
+          <box size="0.05 0.015 0.015" />
+        </geometry>
+      </collision>
+    </link>
+    <link name="${name}_handle_inside">
+      <sphere_inertia radius="0" mass="0"/>
+      <visual>
+	<material name="handle_blue"/>
+        <origin xyz="0 ${1.5 * depth} 0" rpy="${half_pi} 0 ${pi}" />
+        <geometry>-
+          <box size="0.05 0.015 0.015" />
+        </geometry>
+      </visual>
+      <collision>
+        <origin xyz="0 ${1.5 * depth} 0" rpy="${half_pi} 0 ${pi}" />
+        <geometry>
+          <box size="0.05 0.015 0.015" />
         </geometry>
       </collision>
@@ -42,5 +79,5 @@
     <joint name="${name}_origin_revolute_joint" type="revolute">
       <axis xyz="0 0 1"/>
-      <limit effort="1" lower="${door_lower}" upper="${door_max}" velocity="1"/>
+      <limit effort="100" lower="${door_lower}" upper="${door_max}" velocity="10"/>
       <origin xyz="${depth/2} 0 0" rpy="0 0 ${yr}" />
       <parent link="${name}_hinge"/>
@@ -54,4 +91,18 @@
       <child link="${name}_hinge"/>
     </joint>
+    <joint name="${name}_handle_inside_joint" type="fixed">
+      <axis xyz="0 0 1"/>
+      <limit effort="1" lower="0" upper="1.5708" velocity="1"/>
+      <origin xyz="${0.9 * width} 0 -0.08" rpy="0 0 0" />
+      <parent link="${name}_center"/>
+      <child link="${name}_handle_inside"/>
+    </joint>
+    <joint name="${name}_handle_outside_joint" type="fixed">
+      <axis xyz="0 0 1"/>
+      <limit effort="1" lower="0" upper="1.5708" velocity="1"/>
+      <origin xyz="${0.9 * width} 0 -0.08" rpy="0 0 0" />
+      <parent link="${name}_center"/>
+      <child link="${name}_handle_outside"/>
+    </joint>
   </macro>
 </robot>

Commit message: Adjusted handle Joints

File: packages/suturo_urdf_publisher/urdf/hsr_movable_door.urdf.xacro (robot description, xacro)
@@ -48,13 +48,13 @@
       <visual>
 	<material name="handle_blue"/>
-        <origin xyz="0 ${-0.5 * depth} 0" rpy="${half_pi} 0 ${pi}" />
+        <origin xyz="0 0 0" rpy="${half_pi} 0 ${pi}" />
         <geometry>-
-          <box size="0.05 0.015 0.015" />
+          <box size="0.15 0.1 0.03" />
         </geometry>
       </visual>
       <collision>
-        <origin xyz="0 ${-0.5 * depth} 0" rpy="${half_pi} 0 ${pi}" />
+        <origin xyz="0 0 0" rpy="${half_pi} 0 ${pi}" />
         <geometry>
-          <box size="0.05 0.015 0.015" />
+          <box size="0.15 0.1 0.03" />
         </geometry>
       </collision>
@@ -64,13 +64,13 @@
       <visual>
 	<material name="handle_blue"/>
-        <origin xyz="0 ${1.5 * depth} 0" rpy="${half_pi} 0 ${pi}" />
+        <origin xyz="0 0 0" rpy="${half_pi} 0 ${pi}" />
         <geometry>-
-          <box size="0.05 0.015 0.015" />
+          <box size="0.15 0.1 0.03" />
         </geometry>
       </visual>
       <collision>
-        <origin xyz="0 ${1.5 * depth} 0" rpy="${half_pi} 0 ${pi}" />
+        <origin xyz="0 0 0" rpy="${half_pi} 0 ${pi}" />
         <geometry>
-          <box size="0.05 0.015 0.015" />
+          <box size="0.15 0.1 0.03" />
         </geometry>
       </collision>
@@ -85,5 +85,5 @@
     </joint>
     <joint name="${name}_hinge_joint" type="fixed">
-      <axis xyz="0 0 1"/>
+      <axis xyz="0 0 0"/>
       <limit effort="1" lower="0" upper="1.5708" velocity="1"/>
       <origin xyz="${x} ${y - 0.415} ${z}" rpy="0 0 0" />
@@ -92,14 +92,14 @@
     </joint>
     <joint name="${name}_handle_inside_joint" type="fixed">
-      <axis xyz="0 0 1"/>
+      <axis xyz="0 0 0"/>
       <limit effort="1" lower="0" upper="1.5708" velocity="1"/>
-      <origin xyz="${0.9 * width} 0 -0.08" rpy="0 0 0" />
+      <origin xyz="${0.9 * width} ${-0.5 * depth} -0.1" rpy="0 0 0" />
       <parent link="${name}_center"/>
       <child link="${name}_handle_inside"/>
     </joint>
     <joint name="${name}_handle_outside_joint" type="fixed">
-      <axis xyz="0 0 1"/>
+      <axis xyz="0 0 0"/>
       <limit effort="1" lower="0" upper="1.5708" velocity="1"/>
-      <origin xyz="${0.9 * width} 0 -0.08" rpy="0 0 0" />
+      <origin xyz="${0.9 * width} ${1.5 * depth} -0.1" rpy="0 0 0" />
       <parent link="${name}_center"/>
       <child link="${name}_handle_outside"/>

Commit message: Adjusted Handle height

File: packages/suturo_urdf_publisher/urdf/hsr_movable_door.urdf.xacro (robot description, xacro)
@@ -50,5 +50,5 @@
         <origin xyz="0 0 0" rpy="${half_pi} 0 ${pi}" />
         <geometry>-
-          <box size="0.15 0.1 0.03" />
+          <box size="0.15 0.03 0.03" />
         </geometry>
       </visual>
@@ -56,5 +56,5 @@
         <origin xyz="0 0 0" rpy="${half_pi} 0 ${pi}" />
         <geometry>
-          <box size="0.15 0.1 0.03" />
+          <box size="0.15 0.03 0.03" />
         </geometry>
       </collision>
@@ -66,5 +66,5 @@
         <origin xyz="0 0 0" rpy="${half_pi} 0 ${pi}" />
         <geometry>-
-          <box size="0.15 0.1 0.03" />
+          <box size="0.15 0.03 0.03" />
         </geometry>
       </visual>
@@ -72,5 +72,5 @@
         <origin xyz="0 0 0" rpy="${half_pi} 0 ${pi}" />
         <geometry>
-          <box size="0.15 0.1 0.03" />
+          <box size="0.15 0.03 0.03" />
         </geometry>
       </collision>

File: suturo_resources/urdf/sim_doors_test.urdf.xacro (robot description, xacro)
@@ -28,8 +28,8 @@
     </xacro:if>
     <link name="room_link" />
-    <suturo_movable_door name="door_1" parent="room_link" height="2" width="0.83" depth="0.055" x="1.995590" y="-0.099165" z="1.045" r="0" p="0" yr="${half_pi}" door_lower="0" door_max="${half_pi}" >
+    <suturo_movable_door name="door_1" parent="room_link" height="2" width="0.83" depth="0.055" x="1.995590" y="-0.099165" z="1.045" r="0" p="0" yr="${half_pi}" door_lower="${-half_pi}" door_max="${half_pi}" >
     </suturo_movable_door>
     <suturo_movable_door name="door_2" parent="room_link" height="2" width="0.83" depth="0.055"
-x="1.983010" y="1.43728" z="1.045" r="0" p="0" yr="${half_pi}" door_lower="${-half_pi}" door_max="0">
+x="1.983010" y="1.43728" z="1.045" r="0" p="0" yr="${half_pi}" door_lower="${-half_pi}" door_max="${half_pi}">
     </suturo_movable_door>
 </robot>

Commit message: Added urdf with rooms and cloned the cleanup world with openable doors

File: packages/suturo_urdf_publisher/urdf/hsr_movable_door.urdf.xacro (robot description, xacro)
@@ -17,5 +17,5 @@
       <visual>
         <material name="door_green"/>
-        <origin xyz="${width/2} ${depth/2} 0" rpy="0 0 0" />
+        <origin xyz="${width/2} 0 0" rpy="0 0 0" />
         <geometry>
           <box size="${width} ${depth} ${height}" />
@@ -23,5 +23,5 @@
       </visual>
       <collision>
-        <origin xyz="${width/2} ${depth/2} 0" rpy="0 0 0" />
+        <origin xyz="${width/2} 0 0" rpy="0 0 0" />
         <geometry>
           <box size="${width} ${depth} ${height}" />
@@ -32,5 +32,5 @@
       <visual>
         <material name="hinge_red"/>
-        <origin xyz="0 ${depth/2} 0" rpy="0 0 0" />
+        <origin xyz="0 0 0" rpy="0 0 0" />
         <geometry>
           <box size="0.05 0.05 ${height}" />
@@ -38,5 +38,5 @@
       </visual>
       <collision>
-        <origin xyz="0 ${depth/2} 0" rpy="0 0 0" />
+        <origin xyz="0 0 0" rpy="0 0 0" />
         <geometry>-
           <box size="0.05 0.05 ${height}" />
@@ -80,5 +80,5 @@
       <axis xyz="0 0 1"/>
       <limit effort="100" lower="${door_lower}" upper="${door_max}" velocity="10"/>
-      <origin xyz="${depth/2} 0 0" rpy="0 0 ${yr}" />
+      <origin xyz="0 0 0" rpy="0 0 ${yr}" />
       <parent link="${name}_hinge"/>
       <child link="${name}_center"/>
@@ -87,5 +87,5 @@
       <axis xyz="0 0 0"/>
       <limit effort="1" lower="0" upper="1.5708" velocity="1"/>
-      <origin xyz="${x} ${y - 0.415} ${z}" rpy="0 0 0" />
+      <origin xyz="${x} ${y} ${z}" rpy="0 0 0" />
       <parent link="${parent}"/>
       <child link="${name}_hinge"/>
@@ -94,5 +94,5 @@
       <axis xyz="0 0 0"/>
       <limit effort="1" lower="0" upper="1.5708" velocity="1"/>
-      <origin xyz="${0.9 * width} ${-0.5 * depth} -0.1" rpy="0 0 0" />
+      <origin xyz="${0.9 * width} ${-depth} -0.1" rpy="0 0 0" />
       <parent link="${name}_center"/>
       <child link="${name}_handle_inside"/>
@@ -101,5 +101,5 @@
       <axis xyz="0 0 0"/>
       <limit effort="1" lower="0" upper="1.5708" velocity="1"/>
-      <origin xyz="${0.9 * width} ${1.5 * depth} -0.1" rpy="0 0 0" />
+      <origin xyz="${0.9 * width} ${depth} -0.1" rpy="0 0 0" />
       <parent link="${name}_center"/>
       <child link="${name}_handle_outside"/>

File: suturo_resources/urdf/sim_door_room.xacro (robot description, xacro)
@@ -2,4 +2,5 @@
 <robot name="hsrb_lab" xmlns:xacro="http://ros.org/wiki/xacro">
     <xacro:include filename="$(find suturo_urdf_publisher)/urdf/hsr_movable_door.urdf.xacro"/>
+    <xacro:include filename="$(find suturo_urdf_publisher)/urdf/robocup_sim_walls.urdf.xacro"/>
     <xacro:property name="pi" value="3.1415926535897931" />
     <xacro:property name="half_pi" value="1.570796327" />
@@ -28,8 +29,8 @@
     </xacro:if>
     <link name="room_link" />
-    <suturo_movable_door name="door_1" parent="room_link" height="2" width="0.83" depth="0.055" x="1.995590" y="-0.5" z="1.045" r="0" p="0" yr="${half_pi}" door_lower="${-half_pi}" door_max="${half_pi}" >
+    <suturo_movable_door name="door_1" parent="room_link" height="2" width="0.83" depth="0.055" x="1.995590" y="-0.099165" z="1.045" r="0" p="0" yr="${half_pi}" door_lower="${-half_pi}" door_max="${half_pi}" >
     </suturo_movable_door>
-    <suturo_movable_door name="door_2" parent="room_link" height="2" width="0.83" depth="0.055"
-x="1.983010" y="1.02228" z="1.045" r="0" p="0" yr="${half_pi}" door_lower="${-half_pi}" door_max="${half_pi}">
-    </suturo_movable_door>
+    <hsr_lab_walls parent="room_link" >
+	<origin xyz="0 0 0" rpy="0 0 ${half_pi}" />
+    </hsr_lab_walls>
 </robot>

Commit message: Added movable doors

File: packages/suturo_urdf_publisher/urdf/hsr_movable_door.urdf.xacro (robot description, xacro)
@@ -46,9 +46,9 @@
     <link name="${name}_handle_outside">
       <sphere_inertia radius="0" mass="0"/>
-      <visual>
+      <visual>--
 	<material name="handle_blue"/>
         <origin xyz="0 0 0" rpy="${half_pi} 0 ${pi}" />
         <geometry>-
-          <box size="0.15 0.03 0.03" />
+          <box size="0.15 0.025 0.015" />
         </geometry>
       </visual>
@@ -56,5 +56,5 @@
         <origin xyz="0 0 0" rpy="${half_pi} 0 ${pi}" />
         <geometry>
-          <box size="0.15 0.03 0.03" />
+          <box size="0.15 0.025 0.015" />
         </geometry>
       </collision>
@@ -66,5 +66,5 @@
         <origin xyz="0 0 0" rpy="${half_pi} 0 ${pi}" />
         <geometry>-
-          <box size="0.15 0.03 0.03" />
+          <box size="0.15 0.025 0.015" />
         </geometry>
       </visual>
@@ -72,5 +72,5 @@
         <origin xyz="0 0 0" rpy="${half_pi} 0 ${pi}" />
         <geometry>
-          <box size="0.15 0.03 0.03" />
+          <box size="0.15 0.025 0.015" />
         </geometry>
       </collision>
@@ -94,5 +94,5 @@
       <axis xyz="0 0 0"/>
       <limit effort="1" lower="0" upper="1.5708" velocity="1"/>
-      <origin xyz="${0.9 * width} ${-depth} -0.1" rpy="0 0 0" />
+      <origin xyz="${0.9 * width} ${-1.25 * depth} -0.13" rpy="0 0 0" />
       <parent link="${name}_center"/>
       <child link="${name}_handle_inside"/>
@@ -101,5 +101,5 @@
       <axis xyz="0 0 0"/>
       <limit effort="1" lower="0" upper="1.5708" velocity="1"/>
-      <origin xyz="${0.9 * width} ${depth} -0.1" rpy="0 0 0" />
+      <origin xyz="${0.9 * width} ${1.25 * depth} -0.13" rpy="0 0 0" />
       <parent link="${name}_center"/>
       <child link="${name}_handle_outside"/>

File: packages/suturo_urdf_publisher/urdf/hsrb_sim_v1_openable_door.urdf.xacro (robot description, xacro)
@@ -184,5 +184,6 @@
     <suturo_movable_door name="door_1" parent="room_link" height="2" width="0.83" depth="0.055" x="-1.4694" y="4.9966" z="1.045" r="0" p="0" yr="${pi}" door_lower="${-half_pi}" door_max="${half_pi}" >
     </suturo_movable_door>
-    <suturo_shelf name="openable_shelf_1" parent="room_link" x="2" y="2" z="1" xr="0" yr="0" zr="0" size_x="0.5" size_y="1" size_z="0.7" floors_height="[0.4]" number_of_floors="1" door="right" >
+    <suturo_shelf name="openable_shelf_1" parent="room_link" size_x="0.5" size_y="1" size_z="0.7" floors_height="[0.2, 0.2, 0.2]" number_of_floors="3" door="no" >
+	<origin xyz="1 1 0" rpy="0 0 ${pi}" />
     </suturo_shelf>
 </robot>

File: packages/suturo_urdf_publisher/urdf/suturo_shelf_openable.urdf.xacro (robot description, xacro)
@@ -6,4 +6,7 @@
   <material name="shelf_door_green">
     <color rgba="0.64 0.87 0.82 1"/>
+  </material>
+  <material name="handle_red">
+    <color rgba="0.74 0.25 0.25 1"/>
   </material>
   <xacro:macro name="suturo_shelf" params="name parent *origin size_x size_y size_z floors_height number_of_floors door">
@@ -94,5 +97,5 @@
       <visual>
         <material name="shelf_door_green"/>
-        <origin xyz="0 0 0" rpy="0 0 0" />
+        <origin xyz="0 ${size_y/2} 0" rpy="0 0 0" />
         <geometry>
           <box size="${size_x} ${size_y} ${size_z}" />
@@ -100,5 +103,5 @@
       </visual>
       <collision>
-        <origin xyz="0 0 0" rpy="0 0 0" />
+        <origin xyz="0 ${size_y} 0" rpy="0 0 0" />
         <geometry>
           <box size="${size_x} ${size_y} ${size_z}" />
@@ -106,6 +109,27 @@
       </collision>
     </link>
+    <link name="${name}_link_handle">
+      <visual>
+        <material name="handle_red"/>
+        <origin xyz="0 0 0" rpy="0 0 0" />
+        <geometry>
+          <box size="0.04 0.01 0.07" />
+        </geometry>
+      </visual>
+      <collision>
+        <origin xyz="0 0 0" rpy="0 0 0" />
+        <geometry>
+          <box size="0.04 0.01 0.07" />
+        </geometry>
+      </collision>
+    </link>
+    <joint name="${name}_link_handle_joint" type="fixed">
+      <origin xyz="-0.01 ${size_y + 0.03} ${size_z/3}" rpy="0 0 0"/>
+      <axis xyz="0 0 1" />
+      <parent link="${name}_link"/>
+      <child link="${name}_link_handle"/>
+    </joint>
     <joint name="${name}_joint" type="revolute">
-      <origin xyz="${shelf_x_size/-2} ${size_y/-2} 0" rpy="0 0 3.1416"/>
+      <origin xyz="${shelf_x_size/-2} 0 0" rpy="0 0 3.1416"/>
       <axis xyz="0 0 1" />
       <parent link="${parent}_piece"/>

File: suturo_resources/urdf/hsrb_sim_v1_openable_door.urdf.xacro (robot description, xacro)
@@ -184,5 +184,6 @@
     <suturo_movable_door name="door_1" parent="room_link" height="2" width="0.83" depth="0.055" x="-1.48708" y="4.9803" z="1.045" r="0" p="0" yr="${pi}" door_lower="${-half_pi}" door_max="${half_pi}" >
     </suturo_movable_door>
-    <suturo_shelf name="openable_shelf_1" parent="room_link" x="1" y="1" z="1" xr="0" yr="0" zr="0" size_x="0.5" size_y="1" size_z="0.7" floors_height="[0.4]" number_of_floors="0" door="no" >
+    <suturo_shelf name="openable_shelf_1" parent="room_link" size_x="0.44" size_y="0.75" size_z="0.585" floors_height="[0.2,0.2]" number_of_floors="2" door="left" >
+	<origin xyz="0.75 3 0" rpy="0 0 ${half_pi}" />
     </suturo_shelf>
 </robot>

Commit message: Removed unwanted dashes

File: packages/suturo_urdf_publisher/urdf/hsr_movable_door.urdf.xacro (robot description, xacro)
@@ -46,8 +46,8 @@
     <link name="${name}_handle_outside">
       <sphere_inertia radius="0" mass="0"/>
-      <visual>--
+      <visual>
 	<material name="handle_blue"/>
         <origin xyz="0 0 0" rpy="${half_pi} 0 ${pi}" />
-        <geometry>-
+        <geometry>
           <box size="0.15 0.025 0.015" />
         </geometry>

Commit message: Changed grasp depth of the door handle

File: packages/suturo_urdf_publisher/urdf/hsr_movable_door.urdf.xacro (robot description, xacro)
@@ -101,5 +101,5 @@
       <axis xyz="0 0 0"/>
       <limit effort="1" lower="0" upper="1.5708" velocity="1"/>
-      <origin xyz="${0.9 * width} ${1.25 * depth} -0.13" rpy="0 0 0" />
+      <origin xyz="${0.9 * width} ${depth} -0.13" rpy="0 0 0" />
       <parent link="${name}_center"/>
       <child link="${name}_handle_outside"/>
