Commit message: add doors to rework

File: packages/suturo_urdf_publisher_rework/urdf/suturo_enviorment.urdf.xacro (robot description, xacro)
@@ -33,5 +33,6 @@
                           size_z="${data['shelves'][shelf_number]['height']}"
                           floors_height="${data['shelves'][shelf_number]['floors_height']}"
-                          number_of_floors="${data['shelves'][shelf_number]['number_of_floors']}">
+                          number_of_floors="${data['shelves'][shelf_number]['number_of_floors']}"
+                          door="${data['shelves'][shelf_number]['door']}">
             <origin xyz="${data['shelves'][shelf_number]['x_pos']} ${data['shelves'][shelf_number]['y_pos']} 0"
                             rpy="0 0 ${data['shelves'][shelf_number]['z_rot']}" />

File: packages/suturo_urdf_publisher_rework/urdf/suturo_shelf.urdf.xacro (robot description, xacro)
@@ -4,5 +4,8 @@
     <color rgba="0.59 0.88 0.9 1"/>
   </material>
-  <xacro:macro name="suturo_shelf" params="name parent *origin size_x size_y size_z floors_height number_of_floors">
+  <material name="shelf_door_green">
+    <color rgba="0.64 0.87 0.82 1"/>
+  </material>
+  <xacro:macro name="suturo_shelf" params="name parent *origin size_x size_y size_z floors_height number_of_floors door">
     <!-- General conveinience links -->
     <link name="${name}_origin"/>
@@ -47,4 +50,17 @@
     </xacro:macro>
     <xacro:shelf_floor_loop floor_number="0" />
+    <!-- door -->
+    <xacro:if value="${door == 'left'}">
+      <xacro:suturo_shelf_door name="${name}_door_left" parent="${name}_left_side"
+        size_x="0.01" size_y="${size_y/2}" size_z="${size_z}" offset_x="${size_x}">
+        <origin xyz="0 ${size_y*0.75} ${size_z/2}" rpy="0 0 0"/>
+      </xacro:suturo_shelf_door>
+    </xacro:if>
+    <xacro:if value="${door == 'right'}">
+      <xacro:suturo_shelf_door name="${name}right" parent="${name}_right_side"
+        size_x="0.01" size_y="${size_y/2}" size_z="${size_z}" offset_x="${size_x}">
+        <origin xyz="0 ${size_y*0.75} ${size_z/2}" rpy="0 0 0"/>
+      </xacro:suturo_shelf_door>
+    </xacro:if>
   </xacro:macro>
   <!-- Creates a link with collision and visual box of given dimensions,
@@ -74,3 +90,27 @@
     </joint>
   </xacro:macro>
+  <xacro:macro name="suturo_shelf_door" params="name parent *origin box_z_offset=0.0 size_x size_y size_z offset_x">
+    <link name="${name}_door">
+      <visual>
+        <material name="shelf_door_green"/>
+        <origin xyz="0 0 ${box_z_offset}" rpy="0 0 0" />
+        <geometry>
+          <box size="${size_x} ${size_y} ${size_z}" />
+        </geometry>
+      </visual>
+      <collision>
+        <origin xyz="0 0 ${box_z_offset}" rpy="0 0 0" />
+        <geometry>
+          <box size="${size_x} ${size_y} ${size_z}" />
+        </geometry>
+      </collision>
+    </link>
+    <joint name="${name}_door_joint" type="revolute">
+      <origin xyz="${offset_x/-2} ${size_y/-2} 0" rpy="0 0 3.1416"/>
+      <axis xyz="0 0 1" />
+      <parent link="${parent}_piece"/>
+      <child link="${name}_door"/>
+      <limit effort="30" velocity="1.0" lower="0.0" upper="1.91986" />
+    </joint>
+  </xacro:macro>
 </robot>

Commit message: make the urdf-map-offset a yaml parameter

File: packages/suturo_urdf_publisher_rework/urdf/suturo_enviorment.urdf.xacro (robot description, xacro)
@@ -67,5 +67,5 @@
     <link name="world"/>
     <joint name="world_room_joint" type="fixed">
-        <origin xyz="0.0 0.12 0 " rpy="0 0 0" />
+        <origin xyz="${data['world_offset']['X']} ${data['world_offset']['Y']} 0 " rpy="0 0 0" />
         <parent link="world"/>
         <child link="room_link"/>
