Commit message: add table front edge center

File: packages/suturo_urdf_publisher_rework/urdf/suturo_table.urdf.xacro (robot description, xacro)
@@ -22,4 +22,5 @@
     </link>
     <link name="${name}_origin"/>
+     <link name="${name}_front_edge_center"/>
     <!-- JOINTS -->
     <joint name="${name}_origin_joint" type="fixed">
@@ -33,4 +34,9 @@
       <child link="${name}_center"/>
     </joint>
+    <joint name="${name}_front_edge_center_joint" type="fixed">
+      <origin xyz="0 ${size_y/2} ${size_z}" rpy="0 0 0" />
+      <parent link="${name}_origin"/>
+      <child link="${name}_front_edge_center"/>
+    </joint>
   </xacro:macro>
 </robot>
