Commit message: added openable_doors

File: suturo_resources/urdf/suturo_environment.urdf.xacro (robot description, xacro)
@@ -7,4 +7,5 @@
     <xacro:include filename="$(find suturo_resources)/urdf/urdf_components/suturo_wall.urdf.xacro"/>
     <xacro:include filename="$(find suturo_resources)/urdf/urdf_components/suturo_shelf.urdf.xacro"/>
+    <xacro:include filename="$(find suturo_resources)/urdf/urdf_components/suturo_shelf_openable.urdf.xacro"/>
     <xacro:include filename="$(find suturo_resources)/urdf/urdf_components/suturo_door.urdf.xacro"/>
     <xacro:include filename="$(find suturo_resources)/urdf/urdf_components/suturo_room.urdf.xacro"/>
@@ -14,4 +15,5 @@
     <xacro:property name="number_of_buckets" value="${data['buckets']['amount']}" />
     <xacro:property name="number_of_shelves" value="${data['shelves']['amount']}" />
+    <xacro:property name="number_of_shelves_openable" value="${data['shelves_openable']['amount']}" />
     <xacro:property name="number_of_walls" value="${data['walls']['amount']}" />
     <xacro:property name="number_of_doors" value="${data['doors']['amount']}" />
@@ -60,4 +62,21 @@
         <xacro:if value="${(number_of_shelves - 1) > shelf_number}">
             <xacro:shelf_loop shelf_number="${shelf_number + 1}" />
+        </xacro:if>
+    </xacro:macro>
+    <!--  ~~Openable_Shelves~~  -->
+    <xacro:macro name="shelf_openable_loop" params="shelf_openable_number">
+        <xacro:suturo_shelf name="${data['shelves_openable'][shelf_openable_number]['name']}"
+                          parent="${data['shelves_openable'][shelf_openable_number]['parent']}"
+                          size_x="${data['shelves_openable'][shelf_openable_number]['depth']}"
+                          size_y="${data['shelves_openable'][shelf_openable_number]['width']}"
+                          size_z="${data['shelves_openable'][shelf_openable_number]['height']}"
+                          floors_height="${data['shelves_openable'][shelf_openable_number]['floors_height']}"
+                          number_of_floors="${data['shelves_openable'][shelf_openable_number]['number_of_floors']}"
+                          door="${data['shelves_openable'][shelf_openable_number]['door']}">
+            <origin xyz="${data['shelves_openable'][shelf_openable_number]['x_pos']} ${data['shelves_openable'][shelf_openable_number]['y_pos']} 0"
+                            rpy="0 0 ${data['shelves_openable'][shelf_openable_number]['z_rot']}" />
+        </xacro:suturo_shelf>
+        <xacro:if value="${(number_of_shelves_openable - 1) > shelf_openable_number}">
+            <xacro:shelf_openable_loop shelf_number="${shelf_openable_number + 1}" />
         </xacro:if>
     </xacro:macro>
@@ -118,4 +137,7 @@
         <xacro:shelf_loop shelf_number="0" />
     </xacro:if>
+    <xacro:if value="${number_of_shelves_openable > 0}">
+        <xacro:shelf_openable_loop shelf_openable_number="0" />
+    </xacro:if>
     <xacro:if value="${number_of_walls > 0}">
         <xacro:wall_loop wall_number="0" />

Commit message: Fixed shelf_door bug

File: suturo_resources/urdf/suturo_environment.urdf.xacro (robot description, xacro)
@@ -66,5 +66,5 @@
     <!--  ~~Openable_Shelves~~  -->
     <xacro:macro name="shelf_openable_loop" params="shelf_openable_number">
-        <xacro:suturo_shelf name="${data['shelves_openable'][shelf_openable_number]['name']}"
+        <xacro:suturo_shelf_openable name="${data['shelves_openable'][shelf_openable_number]['name']}"
                           parent="${data['shelves_openable'][shelf_openable_number]['parent']}"
                           size_x="${data['shelves_openable'][shelf_openable_number]['depth']}"
@@ -76,5 +76,5 @@
             <origin xyz="${data['shelves_openable'][shelf_openable_number]['x_pos']} ${data['shelves_openable'][shelf_openable_number]['y_pos']} 0"
                             rpy="0 0 ${data['shelves_openable'][shelf_openable_number]['z_rot']}" />
-        </xacro:suturo_shelf>
+        </xacro:suturo_shelf_openable>
         <xacro:if value="${(number_of_shelves_openable - 1) > shelf_openable_number}">
             <xacro:shelf_openable_loop shelf_number="${shelf_openable_number + 1}" />

File: suturo_resources/urdf/urdf_components/suturo_shelf_openable.urdf.xacro (robot description, xacro)
@@ -4,9 +4,9 @@
     <color rgba="0.74 0.25 0.25 1"/>
   </material>
-  <xacro:macro name="suturo_shelf" params="name parent *origin size_x size_y size_z floors_height number_of_floors door">
+  <xacro:macro name="suturo_shelf_openable" params="name parent *origin size_x size_y size_z floors_height number_of_floors door">
     <!-- General conveinience links -->
     <link name="${name}_origin"/>
     <link name="${name}_center"/>
-    <link name="${name}_base_center"/>
+    <link name="${name}_shelf_base_center"/>
     <joint name="${name}_origin_joint" type="fixed">
       <xacro:insert_block name="origin" />
@@ -22,5 +22,5 @@
       <origin xyz="${size_x/2} ${size_y/2} 0.0" rpy="0 0 0" />
       <parent link="${name}_origin"/>
-      <child link="${name}_base_center"/>
+      <child link="${name}_shelf_base_center"/>
     </joint>
     <!-- WALLS -->
@@ -37,4 +37,14 @@
       <origin xyz="${size_x/2} ${size_y} ${size_z/2}" rpy="0 0 0"/>
     </xacro:suturo_shelf_piece>
+    <xacro:macro name="shelf_floor_loop" params="floor_number">
+        <xacro:suturo_shelf_piece name="${name}_shelf_floor_${floor_number}" parent="${name}_shelf_base_center"
+          size_x="${size_x}" size_y="${size_y}" size_z="0.04" box_z_offset="-0.02">
+        <origin xyz="0.0 0.0 ${floors_height[floor_number]}" rpy="0 0 0"/>
+      </xacro:suturo_shelf_piece>
+      <xacro:if value="${(number_of_floors - 1) > floor_number}">
+            <xacro:shelf_floor_loop floor_number="${floor_number + 1}" />
+      </xacro:if>
+    </xacro:macro>
+    <xacro:shelf_floor_loop floor_number="0" />
     <!-- door -->
     <xacro:if value="${door == 'left'}">

Commit message: add knowledgerole to urdf

File: suturo_resources/urdf/suturo_environment.urdf.xacro (robot description, xacro)
@@ -11,4 +11,5 @@
     <xacro:include filename="$(find suturo_resources)/urdf/urdf_components/suturo_room.urdf.xacro"/>
     <xacro:include filename="$(find suturo_resources)/urdf/urdf_components/suturo_bucket.urdf.xacro"/>
+    <xacro:include filename="$(find suturo_resources)/urdf/urdf_components/suturo_path.urdf.xacro"/>
     <!-- general data -->
     <xacro:property name="number_of_tables" value="${data['tables']['amount']}" />
@@ -21,5 +22,5 @@
     <!--  ~~Tables~~  -->
     <xacro:macro name="table_loop" params="table_number">
-        <xacro:suturo_table name="${data['tables'][table_number]['name']}"
+        <xacro:suturo_table name="${data['tables'][table_number]['name']}#${data['tables'][table_number]['knowledge_role']}"
                           parent="${data['tables'][table_number]['parent']}"
                           size_x="${data['tables'][table_number]['depth']}"
@@ -49,5 +50,5 @@
     <!--  ~~Shelves~~  -->
     <xacro:macro name="shelf_loop" params="shelf_number">
-        <xacro:suturo_shelf name="${data['shelves'][shelf_number]['name']}"
+        <xacro:suturo_shelf name="${data['shelves'][shelf_number]['name']}#${data['shelves'][shelf_number]['knowledge_role']}"
                           parent="${data['shelves'][shelf_number]['parent']}"
                           size_x="${data['shelves'][shelf_number]['depth']}"
@@ -66,5 +67,5 @@
     <!--  ~~Openable_Shelves~~  -->
     <xacro:macro name="shelf_openable_loop" params="shelf_openable_number">
-        <xacro:suturo_shelf_openable name="${data['shelves_openable'][shelf_openable_number]['name']}"
+        <xacro:suturo_shelf_openable name="${data['shelves_openable'][shelf_openable_number]['name']}#${data['shelves_openable'][shelf_openable_number]['knowledge_role']}"
                           parent="${data['shelves_openable'][shelf_openable_number]['parent']}"
                           size_x="${data['shelves_openable'][shelf_openable_number]['depth']}"
@@ -111,5 +112,5 @@
     <!--  ~~Doors~~  -->
     <xacro:macro name="door_loop" params="door_number">
-      <xacro:suturo_door name="${data['doors'][door_number]['name']}"
+      <xacro:suturo_door name="${data['doors'][door_number]['room1']}#${data['doors'][door_number]['room2']}"
                          parent="${data['doors'][door_number]['parent']}"
                          height="${data['doors'][door_number]['height']}"
@@ -125,4 +126,16 @@
       <xacro:if value="${(number_of_doors - 1) > door_number}">
         <xacro:door_loop door_number="${door_number + 1}" />
+      </xacro:if>
+    </xacro:macro>
+    <!--  ~~Paths~~  -->
+    <xacro:macro name="path_loop" params="path_number">
+      <xacro:suturo_path name="${data['paths'][path_number]['room1']}#${data['paths'][path_number]['room2']}"
+                         parent="${data['paths'][path_number]['parent']}"
+                         x_pos="${data['paths'][path_number]['x']}"
+                         y_pos="${data['paths'][path_number]['y']}"
+                         >
+      </xacro:suturo_path>
+      <xacro:if value="${(number_of_paths - 1) > path_number}">
+        <xacro:path_loop path_number="${path_number + 1}" />
       </xacro:if>
     </xacro:macro>

File: suturo_resources/urdf/urdf_components/suturo_bucket.urdf.xacro (robot description, xacro)
@@ -6,5 +6,5 @@
   <xacro:macro name="suturo_bucket" params="name parent *origin size_x size_y size_z">
     <!-- LINKS -->
-    <link name="${name}_bucket_center">
+    <link name="${name}#bucket_center">
       <visual>
         <material name="bucket_grey"/>
@@ -21,28 +21,28 @@
       </collision>
     </link>
-    <link name="${name}_bucket_origin"/>
+    <link name="${name}#bucket_origin"/>
     <!-- Additional tf-frames -->
-    <link name="${name}_bucket_surface_center"/>
-    <link name="${name}_bucket_front_edge_center"/>
+    <link name="${name}#bucket_surface_center"/>
+    <link name="${name}#bucket_front_edge_center"/>
     <!-- JOINTS -->
-    <joint name="${name}_bucket_origin_joint" type="fixed">
+    <joint name="${name}#bucket_origin_joint" type="fixed">
       <xacro:insert_block name="origin" />
       <parent link="${parent}"/>
-      <child link="${name}_bucket_origin"/>
+      <child link="${name}#bucket_origin"/>
     </joint>
-    <joint name="${name}_bucket_center_joint" type="fixed">
+    <joint name="${name}#bucket_center_joint" type="fixed">
       <origin xyz="${size_x/2} ${size_y/2} ${size_z/2}" rpy="0 0 0" />
-      <parent link="${name}_bucket_origin"/>
-      <child link="${name}_bucket_center"/>
+      <parent link="${name}#bucket_origin"/>
+      <child link="${name}#bucket_center"/>
     </joint>
-    <joint name="${name}_bucket_surface_center_joint" type="fixed">
+    <joint name="${name}#bucket_surface_center_joint" type="fixed">
       <origin xyz="${size_x/2} ${size_y/2} ${size_z}" rpy="0 0 0" />
-      <parent link="${name}_bucket_origin"/>
-      <child link="${name}_bucket_surface_center"/>
+      <parent link="${name}#bucket_origin"/>
+      <child link="${name}#bucket_surface_center"/>
     </joint>
-    <joint name="${name}_bucket_front_edge_center_joint" type="fixed">
+    <joint name="${name}#bucket_front_edge_center_joint" type="fixed">
       <origin xyz="0 ${size_y/2} ${size_z}" rpy="0 0 0" />
-      <parent link="${name}_bucket_origin"/>
-      <child link="${name}_bucket_front_edge_center"/>
+      <parent link="${name}#bucket_origin"/>
+      <child link="${name}#bucket_front_edge_center"/>
     </joint>
   </xacro:macro>

File: suturo_resources/urdf/urdf_components/suturo_door.urdf.xacro (robot description, xacro)
@@ -13,5 +13,5 @@
   <xacro:macro name="suturo_door" params="name parent height width depth x y z zrot door_turn_limit_lower door_turn_limit_max">
     <!-- LINKS -->
-    <link name="${name}_door_center">
+    <link name="${name}#door_center">
       <visual>
         <material name="door_green"/>
@@ -28,5 +28,5 @@
       </collision>
     </link>
-    <link name="${name}_door_hinge">
+    <link name="${name}#door_hinge">
       <visual>
         <material name="hinge_red"/>
@@ -43,5 +43,5 @@
       </collision>
     </link>
-    <link name="${name}_door_handle_outside">
+    <link name="${name}#door_handle_outside">
       <sphere_inertia radius="0" mass="0"/>
       <visual>
@@ -59,5 +59,5 @@
       </collision>
     </link>
-    <link name="${name}_door_handle_inside">
+    <link name="${name}#door_handle_inside">
       <sphere_inertia radius="0" mass="0"/>
       <visual>
@@ -76,31 +76,31 @@
     </link>
     <!-- JOINTS -->
-    <joint name="${name}_door_origin_revolute_joint" type="revolute">
+    <joint name="${name}#door_origin_revolute_joint" type="revolute">
       <axis xyz="0 0 1"/>
       <limit effort="100" lower="${door_turn_limit_lower}" upper="${door_turn_limit_max}" velocity="10"/>
       <origin xyz="0 0 0" rpy="0 0 ${zrot}" />
-      <parent link="${name}_door_hinge"/>
-      <child link="${name}_door_center"/>
+      <parent link="${name}#door_hinge"/>
+      <child link="${name}#door_center"/>
     </joint>
-    <joint name="${name}_door_hinge_joint" type="fixed">
+    <joint name="${name}#door_hinge_joint" type="fixed">
       <axis xyz="0 0 0"/>
       <limit effort="1" lower="0" upper="1.5708" velocity="1"/>
       <origin xyz="${x} ${y} ${z}" rpy="0 0 0" />
       <parent link="${parent}"/>
-      <child link="${name}_door_hinge"/>
+      <child link="${name}#door_hinge"/>
     </joint>
-    <joint name="${name}_door_handle_inside_joint" type="fixed">
+    <joint name="${name}#door_handle_inside_joint" type="fixed">
       <axis xyz="0 0 0"/>
       <limit effort="1" lower="0" upper="1.5708" velocity="1"/>
       <origin xyz="${0.9 * width} ${-1.25 * depth} -0.13" rpy="0 0 0" />
-      <parent link="${name}_door_center"/>
-      <child link="${name}_door_handle_inside"/>
+      <parent link="${name}#door_center"/>
+      <child link="${name}#door_handle_inside"/>
     </joint>
-    <joint name="${name}_door_handle_outside_joint" type="fixed">
+    <joint name="${name}#door_handle_outside_joint" type="fixed">
       <axis xyz="0 0 0"/>
       <limit effort="1" lower="0" upper="1.5708" velocity="1"/>
       <origin xyz="${0.9 * width} ${depth} -0.13" rpy="0 0 0" />
-      <parent link="${name}_door_center"/>
-      <child link="${name}_door_handle_outside"/>
+      <parent link="${name}#door_center"/>
+      <child link="${name}#door_handle_outside"/>
     </joint>
   </xacro:macro>

File: suturo_resources/urdf/urdf_components/suturo_room.urdf.xacro (robot description, xacro)
@@ -4,10 +4,10 @@
   <xacro:macro name="suturo_room" params="name parent num_of_corners corners_x_pos corners_y_pos center_x center_y color">
     <!-- define a central joint to wich every corner is connected -->
-    <joint name="world_${name}-room_joint" type="fixed">
+    <joint name="world_${name}#room_joint" type="fixed">
         <origin xyz="${center_x} ${center_y} 0 " rpy="0 0 0" />
         <parent link="${parent}"/>
-        <child link="${name}-room_center_link"/>
+        <child link="${name}#room_center_link"/>
     </joint>
-    <link name="${name}-room_center_link">
+    <link name="${name}#room_center_link">
       <visual>
         <geometry>
@@ -21,10 +21,10 @@
     <!-- room loop to create every corner -->
     <xacro:macro name="corner_loop" params="loop_number">
-      <joint name="${name}-room_joint_${loop_number}" type="fixed">
+      <joint name="${name}#room_joint_${loop_number}" type="fixed">
           <origin xyz="${corners_x_pos[loop_number] - center_x} ${corners_y_pos[loop_number] - center_y} 0 " rpy="0 0 0" />
-          <parent link="${name}-room_center_link"/>
-          <child link="${name}-room_corner_${loop_number}_link"/>
+          <parent link="${name}#room_center_link"/>
+          <child link="${name}#room_corner_${loop_number}_link"/>
       </joint>
-      <link name="${name}-room_corner_${loop_number}_link" />
+      <link name="${name}#room_corner_${loop_number}_link" />
       <xacro:if value="${(num_of_corners - 1) > loop_number}">
         <xacro:corner_loop loop_number="${loop_number + 1}" />

File: suturo_resources/urdf/urdf_components/suturo_shelf.urdf.xacro (robot description, xacro)
@@ -9,37 +9,37 @@
   <xacro:macro name="suturo_shelf" params="name parent *origin size_x size_y size_z floors_height number_of_floors door">
     <!-- General conveinience links -->
-    <link name="${name}_shelf_origin"/>
-    <link name="${name}_shelf_center"/>
-    <link name="${name}_shelf_base_center"/>
-    <joint name="${name}_shelf_origin_joint" type="fixed">
+    <link name="${name}#shelf_origin"/>
+    <link name="${name}#shelf_center"/>
+    <link name="${name}#shelf_base_center"/>
+    <joint name="${name}#shelf_origin_joint" type="fixed">
       <xacro:insert_block name="origin" />
       <parent link="${parent}"/>
-      <child link="${name}_shelf_origin"/>
+      <child link="${name}#shelf_origin"/>
     </joint>
-    <joint name="${name}_shelf_center_joint" type="fixed">
+    <joint name="${name}#shelf_center_joint" type="fixed">
       <origin xyz="${size_x/2} ${size_y/2} ${size_z/2}" rpy="0 0 0" />
-      <parent link="${name}_shelf_origin"/>
-      <child link="${name}_shelf_center"/>
+      <parent link="${name}#shelf_origin"/>
+      <child link="${name}#shelf_center"/>
     </joint>
-    <joint name="${name}_shelf_base_center_joint" type="fixed">
+    <joint name="${name}#shelf_base_center_joint" type="fixed">
       <origin xyz="${size_x/2} ${size_y/2} 0.0" rpy="0 0 0" />
-      <parent link="${name}_shelf_origin"/>
-      <child link="${name}_shelf_base_center"/>
+      <parent link="${name}#shelf_origin"/>
+      <child link="${name}#shelf_base_center"/>
     </joint>
     <!-- WALLS -->
-    <xacro:suturo_shelf_piece name="${name}_shelf_back" parent="${name}_shelf_origin"
+    <xacro:suturo_shelf_piece name="${name}#shelf_back" parent="${name}#shelf_origin"
       size_x="0.01" size_y="${size_y}" size_z="${size_z}">
       <origin xyz="${size_x} ${size_y/2} ${size_z/2}" rpy="0 0 0"/>
     </xacro:suturo_shelf_piece>
-    <xacro:suturo_shelf_piece name="${name}_shelf_right_side" parent="${name}_shelf_origin"
+    <xacro:suturo_shelf_piece name="${name}#shelf_right_side" parent="${name}#shelf_origin"
       size_x="${size_x}" size_y="0.01" size_z="${size_z}">
       <origin xyz="${size_x/2} 0.0 ${size_z/2}" rpy="0 0 0"/>
     </xacro:suturo_shelf_piece>
-    <xacro:suturo_shelf_piece name="${name}_shelf_left_side" parent="${name}_shelf_origin"
+    <xacro:suturo_shelf_piece name="${name}#shelf_left_side" parent="${name}#shelf_origin"
       size_x="${size_x}" size_y="0.01" size_z="${size_z}">
       <origin xyz="${size_x/2} ${size_y} ${size_z/2}" rpy="0 0 0"/>
     </xacro:suturo_shelf_piece>
     <xacro:macro name="shelf_floor_loop" params="floor_number">
-        <xacro:suturo_shelf_piece name="${name}_shelf_floor_${floor_number}" parent="${name}_shelf_base_center"
+        <xacro:suturo_shelf_piece name="${name}#shelf_floor_${floor_number}" parent="${name}#shelf_base_center"
           size_x="${size_x}" size_y="${size_y}" size_z="0.04" box_z_offset="-0.02">
         <origin xyz="0.0 0.0 ${floors_height[floor_number]}" rpy="0 0 0"/>
@@ -53,5 +53,5 @@
     <!-- left -->
     <xacro:if value="${door == 'left'}">
-      <xacro:suturo_shelf_left_door name="${name}_shelf_door_left" parent="${name}_left_side"
+      <xacro:suturo_shelf_left_door name="${name}#shelf_door_left" parent="${name}#left_side"
         size_x="0.01" size_y="${size_y/2}" size_z="${size_z}" shelf_x_size="${size_x}">
         <origin xyz="0 ${size_y*0.75} ${size_z/2}" rpy="0 0 0"/>
@@ -60,5 +60,5 @@
     <!-- right -->
     <xacro:if value="${door == 'right'}">
-      <xacro:suturo_shelf_right_door name="${name}_shelf_door_right" parent="${name}_right_side"
+      <xacro:suturo_shelf_right_door name="${name}#shelf_door_right" parent="${name}#right_side"
         size_x="0.01" size_y="${size_y/2}" size_z="${size_z}" shelf_x_size="${size_x}">
         <origin xyz="0 ${size_y*0.75} ${size_z/2}" rpy="0 0 0"/>
@@ -67,9 +67,9 @@
     <!-- both -->
     <xacro:if value="${door == 'both'}">
-      <xacro:suturo_shelf_left_door name="${name}_shelf_door_left" parent="${name}_left_side"
+      <xacro:suturo_shelf_left_door name="${name}#shelf_door_left" parent="${name}#left_side"
         size_x="0.01" size_y="${size_y/2}" size_z="${size_z}" shelf_x_size="${size_x}">
         <origin xyz="0 ${size_y*0.75} ${size_z/2}" rpy="0 0 0"/>
       </xacro:suturo_shelf_left_door>
-      <xacro:suturo_shelf_right_door name="${name}_shelf_door_right" parent="${name}_shelf_right_side"
+      <xacro:suturo_shelf_right_door name="${name}#shelf_door_right" parent="${name}#shelf_right_side"
         size_x="0.01" size_y="${size_y/2}" size_z="${size_z}" shelf_x_size="${size_x}">
         <origin xyz="0 ${size_y*0.75} ${size_z/2}" rpy="0 0 0"/>
@@ -97,5 +97,5 @@
     </link>
     <!-- JOINT -->
-    <joint name="${name}_joint" type="fixed">
+    <joint name="${name}#joint" type="fixed">
       <xacro:insert_block name="origin" />
       <parent link="${parent}"/>
@@ -104,5 +104,5 @@
   </xacro:macro>
   <xacro:macro name="suturo_shelf_left_door" params="name parent *origin size_x size_y size_z shelf_x_size">
-    <link name="${name}_link">
+    <link name="${name}#link">
       <visual>
         <material name="shelf_door_green"/>
@@ -119,14 +119,14 @@
       </collision>
     </link>
-    <joint name="${name}_shelf_joint" type="revolute">
+    <joint name="${name}#shelf_joint" type="revolute">
       <origin xyz="${shelf_x_size/-2} ${size_y/-2} 0" rpy="0 0 3.1416"/>
       <axis xyz="0 0 1" />
-      <parent link="${parent}_piece"/>
-      <child link="${name}_link"/>
+      <parent link="${parent}#piece"/>
+      <child link="${name}#link"/>
       <limit effort="30" velocity="1.0" lower="0.0" upper="1.91986" />
     </joint>
   </xacro:macro>
   <xacro:macro name="suturo_shelf_right_door" params="name parent *origin size_x size_y size_z shelf_x_size">
-    <link name="${name}_shelf_link">
+    <link name="${name}#shelf_link">
       <visual>
         <material name="shelf_door_green"/>
@@ -143,9 +143,9 @@
       </collision>
     </link>
-    <joint name="${name}_shelf_joint" type="revolute">
+    <joint name="${name}#shelf_joint" type="revolute">
       <origin xyz="${shelf_x_size/-2} ${size_y/2} 0" rpy="0 0 -3.1416"/>
       <axis xyz="0 0 1" />
-      <parent link="${parent}_shelf_piece"/>
-      <child link="${name}_shelf_link"/>
+      <parent link="${parent}#shelf_piece"/>
+      <child link="${name}#shelf_link"/>
       <limit effort="30" velocity="1.0" lower="0.0" upper="1.91986" />
     </joint>
