Commit message: add knowledgerole to urdf

File: suturo_resources/urdf/urdf_components/suturo_shelf_openable.urdf.xacro (robot description, xacro)
@@ -6,37 +6,37 @@
   <xacro:macro name="suturo_shelf_openable" params="name parent *origin size_x size_y size_z floors_height number_of_floors door">
     <!-- General conveinience links -->
-    <link name="${name}_shelf_origin"/>
-    <link name="${name}_shelf_center"/>
-    <link name="${name}_shelf_base_center"/>
-    <joint name="${name}_shelf_origin_joint" type="fixed">
+    <link name="${name}#shelf_origin"/>
+    <link name="${name}#shelf_center"/>
+    <link name="${name}#shelf_base_center"/>
+    <joint name="${name}#shelf_origin_joint" type="fixed">
       <xacro:insert_block name="origin" />
       <parent link="${parent}"/>
-      <child link="${name}_shelf_origin"/>
+      <child link="${name}#shelf_origin"/>
     </joint>
-    <joint name="${name}_shelf_center_joint" type="fixed">
+    <joint name="${name}#shelf_center_joint" type="fixed">
       <origin xyz="${size_x/2} ${size_y/2} ${size_z/2}" rpy="0 0 0" />
-      <parent link="${name}_shelf_origin"/>
-      <child link="${name}_shelf_center"/>
+      <parent link="${name}#shelf_origin"/>
+      <child link="${name}#shelf_center"/>
     </joint>
-    <joint name="${name}_shelf_base_center_joint" type="fixed">
+    <joint name="${name}#shelf_base_center_joint" type="fixed">
       <origin xyz="${size_x/2} ${size_y/2} 0.0" rpy="0 0 0" />
-      <parent link="${name}_shelf_origin"/>
-      <child link="${name}_shelf_base_center"/>
+      <parent link="${name}#shelf_origin"/>
+      <child link="${name}#shelf_base_center"/>
     </joint>
     <!-- WALLS -->
-    <xacro:suturo_shelf_piece_openable name="${name}_shelf_back" parent="${name}_shelf_origin"
+    <xacro:suturo_shelf_piece_openable name="${name}#shelf_back" parent="${name}#shelf_origin"
       size_x="0.01" size_y="${size_y}" size_z="${size_z}">
       <origin xyz="${size_x} ${size_y/2} ${size_z/2}" rpy="0 0 0"/>
     </xacro:suturo_shelf_piece_openable>
-    <xacro:suturo_shelf_piece_openable name="${name}_shelf_right_side" parent="${name}_shelf_origin"
+    <xacro:suturo_shelf_piece_openable name="${name}#shelf_right_side" parent="${name}#shelf_origin"
       size_x="${size_x}" size_y="0.01" size_z="${size_z}">
       <origin xyz="${size_x/2} 0.0 ${size_z/2}" rpy="0 0 0"/>
     </xacro:suturo_shelf_piece_openable>
-    <xacro:suturo_shelf_piece_openable name="${name}_shelf_left_side" parent="${name}_shelf_origin"
+    <xacro:suturo_shelf_piece_openable name="${name}#shelf_left_side" parent="${name}#shelf_origin"
       size_x="${size_x}" size_y="0.01" size_z="${size_z}">
       <origin xyz="${size_x/2} ${size_y} ${size_z/2}" rpy="0 0 0"/>
     </xacro:suturo_shelf_piece_openable>
     <xacro:macro name="shelf_floor_loop_openable" params="floor_number">
-        <xacro:suturo_shelf_piece_openable name="${name}_shelf_floor_${floor_number}" parent="${name}_shelf_base_center"
+        <xacro:suturo_shelf_piece_openable name="${name}#shelf_floor_${floor_number}" parent="${name}#shelf_base_center"
           size_x="${size_x}" size_y="${size_y}" size_z="0.04" box_z_offset="-0.02">
         <origin xyz="0.0 0.0 ${floors_height[floor_number]}" rpy="0 0 0"/>
@@ -49,5 +49,5 @@
     <!-- door -->
     <xacro:if value="${door == 'left'}">
-      <xacro:suturo_shelf_left_door_openable name="${name}_shelf_door_left" parent="${name}_shelf_left_side"
+      <xacro:suturo_shelf_left_door_openable name="${name}#shelf_door_left" parent="${name}#shelf_left_side"
         size_x="0.01" size_y="${size_y/2}" size_z="${size_z}" shelf_x_size="${size_x}">
         <origin xyz="0 ${size_y*0.75} ${size_z/2}" rpy="0 0 0"/>
@@ -55,5 +55,5 @@
     </xacro:if>
     <xacro:if value="${door == 'right'}">
-      <xacro:suturo_shelf_right_door_openable name="${name}_shelf_door_right" parent="${name}_shelf_right_side"
+      <xacro:suturo_shelf_right_door_openable name="${name}#shelf_door_right" parent="${name}#shelf_right_side"
         size_x="0.01" size_y="${size_y/2}" size_z="${size_z}" shelf_x_size="${size_x}">
         <origin xyz="0 ${size_y*0.75} ${size_z/2}" rpy="0 0 0"/>
@@ -65,5 +65,5 @@
   <xacro:macro name="suturo_shelf_piece_openable" params="name parent *origin box_z_offset=0.0 size_x size_y size_z">
     <!-- LINK -->
-    <link name="${name}_shelf_piece">
+    <link name="${name}#shelf_piece">
       <visual>
         <material name="shelf_blue"/>
@@ -81,12 +81,12 @@
     </link>
     <!-- JOINT -->
-    <joint name="${name}_shelf_piece_joint" type="fixed">
+    <joint name="${name}#shelf_piece_joint" type="fixed">
       <xacro:insert_block name="origin" />
       <parent link="${parent}"/>
-      <child link="${name}_shelf_piece"/>
+      <child link="${name}#shelf_piece"/>
     </joint>
   </xacro:macro>
   <xacro:macro name="suturo_shelf_left_door_openable" params="name parent *origin size_x size_y size_z shelf_x_size">
-    <link name="${name}_shelf_link">
+    <link name="${name}#shelf_link">
       <visual>
         <material name="shelf_door_green"/>
@@ -103,5 +103,5 @@
       </collision>
     </link>
-    <link name="${name}_shelf_link_handle">
+    <link name="${name}#shelf_link_handle">
       <visual>
         <material name="handle_red"/>
@@ -118,20 +118,20 @@
       </collision>
     </link>
-    <joint name="${name}_shelf_link_handle_joint" type="fixed">
+    <joint name="${name}#shelf_link_handle_joint" type="fixed">
       <origin xyz="-0.01 ${size_y - 0.04} ${size_z/3}" rpy="0 0 0"/>
       <axis xyz="0 0 1" />
-      <parent link="${name}_shelf_link"/>
-      <child link="${name}_shelf_link_handle"/>
+      <parent link="${name}#shelf_link"/>
+      <child link="${name}#shelf_link_handle"/>
     </joint>
-    <joint name="${name}_shelf_joint" type="revolute">
+    <joint name="${name}#shelf_joint" type="revolute">
       <origin xyz="${shelf_x_size/-2} 0 0" rpy="0 0 3.1416"/>
       <axis xyz="0 0 1" />
-      <parent link="${parent}_shelf_piece"/>
-      <child link="${name}_shelf_link"/>
+      <parent link="${parent}#shelf_piece"/>
+      <child link="${name}#shelf_link"/>
       <limit effort="30" velocity="1.0" lower="0.0" upper="1.91986" />
     </joint>
   </xacro:macro>
   <xacro:macro name="suturo_shelf_right_door_openable" params="name parent *origin size_x size_y size_z shelf_x_size">
-    <link name="${name}_shelf_link">
+    <link name="${name}#shelf_link">
       <visual>
         <material name="shelf_door_green"/>
@@ -148,9 +148,9 @@
       </collision>
     </link>
-    <joint name="${name}_shelf_joint" type="revolute">
+    <joint name="${name}#shelf_joint" type="revolute">
       <origin xyz="${shelf_x_size/-2} ${size_y/2} 0" rpy="0 0 -3.1416"/>
       <axis xyz="0 0 1" />
-      <parent link="${parent}_shelf_piece"/>
-      <child link="${name}_shelf_link"/>
+      <parent link="${parent}#shelf_piece"/>
+      <child link="${name}#shelf_link"/>
       <limit effort="30" velocity="1.0" lower="0.0" upper="1.91986" />
     </joint>

File: suturo_resources/urdf/urdf_components/suturo_table.urdf.xacro (robot description, xacro)
@@ -6,5 +6,5 @@
   <xacro:macro name="suturo_table" params="name parent *origin size_x size_y size_z">
     <!-- LINKS -->
-    <link name="${name}_table_center">
+    <link name="${name}#table_center">
       <visual>
         <material name="table_grey"/>
@@ -21,21 +21,21 @@
       </collision>
     </link>
-    <link name="${name}_table_origin"/>
-     <link name="${name}_table_front_edge_center"/>
+    <link name="${name}#table_origin"/>
+     <link name="${name}#table_front_edge_center"/>
     <!-- JOINTS -->
-    <joint name="${name}_table_origin_joint" type="fixed">
+    <joint name="${name}#table_origin_joint" type="fixed">
       <xacro:insert_block name="origin" />
       <parent link="${parent}"/>
-      <child link="${name}_table_origin"/>
+      <child link="${name}#table_origin"/>
     </joint>
-    <joint name="${name}_center_joint" type="fixed">
+    <joint name="${name}#center_joint" type="fixed">
       <origin xyz="${size_x/2} ${size_y/2} ${size_z}" rpy="0 0 0" />
-      <parent link="${name}_table_origin"/>
-      <child link="${name}_table_center"/>
+      <parent link="${name}#table_origin"/>
+      <child link="${name}#table_center"/>
     </joint>
-    <joint name="${name}_table_front_edge_center_joint" type="fixed">
+    <joint name="${name}#table_front_edge_center_joint" type="fixed">
       <origin xyz="0 ${size_y/2} ${size_z}" rpy="0 0 0" />
-      <parent link="${name}_table_origin"/>
-      <child link="${name}_table_front_edge_center"/>
+      <parent link="${name}#table_origin"/>
+      <child link="${name}#table_front_edge_center"/>
     </joint>
   </xacro:macro>
