Commit message: change # to : because knowrob cant handle it right

File: suturo_resources/urdf/suturo_environment.urdf.xacro (robot description, xacro)
@@ -22,5 +22,5 @@
     <!--  ~~Tables~~  -->
     <xacro:macro name="table_loop" params="table_number">
-        <xacro:suturo_table name="${data['tables'][table_number]['name']}#${data['tables'][table_number]['knowledge_role']}"
+        <xacro:suturo_table name="${data['tables'][table_number]['name']}:${data['tables'][table_number]['knowledge_role']}"
                           parent="${data['tables'][table_number]['parent']}"
                           size_x="${data['tables'][table_number]['depth']}"
@@ -50,5 +50,5 @@
     <!--  ~~Shelves~~  -->
     <xacro:macro name="shelf_loop" params="shelf_number">
-        <xacro:suturo_shelf name="${data['shelves'][shelf_number]['name']}#${data['shelves'][shelf_number]['knowledge_role']}"
+        <xacro:suturo_shelf name="${data['shelves'][shelf_number]['name']}:${data['shelves'][shelf_number]['knowledge_role']}"
                           parent="${data['shelves'][shelf_number]['parent']}"
                           size_x="${data['shelves'][shelf_number]['depth']}"
@@ -67,5 +67,5 @@
     <!--  ~~Openable_Shelves~~  -->
     <xacro:macro name="shelf_openable_loop" params="shelf_openable_number">
-        <xacro:suturo_shelf_openable name="${data['shelves_openable'][shelf_openable_number]['name']}#${data['shelves_openable'][shelf_openable_number]['knowledge_role']}"
+        <xacro:suturo_shelf_openable name="${data['shelves_openable'][shelf_openable_number]['name']}:${data['shelves_openable'][shelf_openable_number]['knowledge_role']}"
                           parent="${data['shelves_openable'][shelf_openable_number]['parent']}"
                           size_x="${data['shelves_openable'][shelf_openable_number]['depth']}"
@@ -112,5 +112,5 @@
     <!--  ~~Doors~~  -->
     <xacro:macro name="door_loop" params="door_number">
-      <xacro:suturo_door name="${data['doors'][door_number]['room1']}#${data['doors'][door_number]['room2']}"
+      <xacro:suturo_door name="${data['doors'][door_number]['room1']}:${data['doors'][door_number]['room2']}"
                          parent="${data['doors'][door_number]['parent']}"
                          height="${data['doors'][door_number]['height']}"
@@ -130,5 +130,5 @@
     <!--  ~~Paths~~  -->
     <xacro:macro name="path_loop" params="path_number">
-      <xacro:suturo_path name="${data['paths'][path_number]['room1']}#${data['paths'][path_number]['room2']}"
+      <xacro:suturo_path name="${data['paths'][path_number]['room1']}:${data['paths'][path_number]['room2']}"
                          parent="${data['paths'][path_number]['parent']}"
                          x_pos="${data['paths'][path_number]['x']}"

File: suturo_resources/urdf/urdf_components/suturo_bucket.urdf.xacro (robot description, xacro)
@@ -6,5 +6,5 @@
   <xacro:macro name="suturo_bucket" params="name parent *origin size_x size_y size_z">
     <!-- LINKS -->
-    <link name="${name}#bucket_center">
+    <link name="${name}:bucket_center">
       <visual>
         <material name="bucket_grey"/>
@@ -21,28 +21,28 @@
       </collision>
     </link>
-    <link name="${name}#bucket_origin"/>
+    <link name="${name}:bucket_origin"/>
     <!-- Additional tf-frames -->
-    <link name="${name}#bucket_surface_center"/>
-    <link name="${name}#bucket_front_edge_center"/>
+    <link name="${name}:bucket_surface_center"/>
+    <link name="${name}:bucket_front_edge_center"/>
     <!-- JOINTS -->
-    <joint name="${name}#bucket_origin_joint" type="fixed">
+    <joint name="${name}:bucket_origin_joint" type="fixed">
       <xacro:insert_block name="origin" />
       <parent link="${parent}"/>
-      <child link="${name}#bucket_origin"/>
+      <child link="${name}:bucket_origin"/>
     </joint>
-    <joint name="${name}#bucket_center_joint" type="fixed">
+    <joint name="${name}:bucket_center_joint" type="fixed">
       <origin xyz="${size_x/2} ${size_y/2} ${size_z/2}" rpy="0 0 0" />
-      <parent link="${name}#bucket_origin"/>
-      <child link="${name}#bucket_center"/>
+      <parent link="${name}:bucket_origin"/>
+      <child link="${name}:bucket_center"/>
     </joint>
-    <joint name="${name}#bucket_surface_center_joint" type="fixed">
+    <joint name="${name}:bucket_surface_center_joint" type="fixed">
       <origin xyz="${size_x/2} ${size_y/2} ${size_z}" rpy="0 0 0" />
-      <parent link="${name}#bucket_origin"/>
-      <child link="${name}#bucket_surface_center"/>
+      <parent link="${name}:bucket_origin"/>
+      <child link="${name}:bucket_surface_center"/>
     </joint>
-    <joint name="${name}#bucket_front_edge_center_joint" type="fixed">
+    <joint name="${name}:bucket_front_edge_center_joint" type="fixed">
       <origin xyz="0 ${size_y/2} ${size_z}" rpy="0 0 0" />
-      <parent link="${name}#bucket_origin"/>
-      <child link="${name}#bucket_front_edge_center"/>
+      <parent link="${name}:bucket_origin"/>
+      <child link="${name}:bucket_front_edge_center"/>
     </joint>
   </xacro:macro>

File: suturo_resources/urdf/urdf_components/suturo_door.urdf.xacro (robot description, xacro)
@@ -13,5 +13,5 @@
   <xacro:macro name="suturo_door" params="name parent height width depth x y z zrot door_turn_limit_lower door_turn_limit_max">
     <!-- LINKS -->
-    <link name="${name}#door_center">
+    <link name="${name}:door_center">
       <visual>
         <material name="door_green"/>
@@ -28,5 +28,5 @@
       </collision>
     </link>
-    <link name="${name}#door_hinge">
+    <link name="${name}:door_hinge">
       <visual>
         <material name="hinge_red"/>
@@ -43,5 +43,5 @@
       </collision>
     </link>
-    <link name="${name}#door_handle_outside">
+    <link name="${name}:door_handle_outside">
       <sphere_inertia radius="0" mass="0"/>
       <visual>
@@ -59,5 +59,5 @@
       </collision>
     </link>
-    <link name="${name}#door_handle_inside">
+    <link name="${name}:door_handle_inside">
       <sphere_inertia radius="0" mass="0"/>
       <visual>
@@ -76,31 +76,31 @@
     </link>
     <!-- JOINTS -->
-    <joint name="${name}#door_origin_revolute_joint" type="revolute">
+    <joint name="${name}:door_origin_revolute_joint" type="revolute">
       <axis xyz="0 0 1"/>
       <limit effort="100" lower="${door_turn_limit_lower}" upper="${door_turn_limit_max}" velocity="10"/>
       <origin xyz="0 0 0" rpy="0 0 ${zrot}" />
-      <parent link="${name}#door_hinge"/>
-      <child link="${name}#door_center"/>
+      <parent link="${name}:door_hinge"/>
+      <child link="${name}:door_center"/>
     </joint>
-    <joint name="${name}#door_hinge_joint" type="fixed">
+    <joint name="${name}:door_hinge_joint" type="fixed">
       <axis xyz="0 0 0"/>
       <limit effort="1" lower="0" upper="1.5708" velocity="1"/>
       <origin xyz="${x} ${y} ${z}" rpy="0 0 0" />
       <parent link="${parent}"/>
-      <child link="${name}#door_hinge"/>
+      <child link="${name}:door_hinge"/>
     </joint>
-    <joint name="${name}#door_handle_inside_joint" type="fixed">
+    <joint name="${name}:door_handle_inside_joint" type="fixed">
       <axis xyz="0 0 0"/>
       <limit effort="1" lower="0" upper="1.5708" velocity="1"/>
       <origin xyz="${0.9 * width} ${-1.25 * depth} -0.13" rpy="0 0 0" />
-      <parent link="${name}#door_center"/>
-      <child link="${name}#door_handle_inside"/>
+      <parent link="${name}:door_center"/>
+      <child link="${name}:door_handle_inside"/>
     </joint>
-    <joint name="${name}#door_handle_outside_joint" type="fixed">
+    <joint name="${name}:door_handle_outside_joint" type="fixed">
       <axis xyz="0 0 0"/>
       <limit effort="1" lower="0" upper="1.5708" velocity="1"/>
       <origin xyz="${0.9 * width} ${depth} -0.13" rpy="0 0 0" />
-      <parent link="${name}#door_center"/>
-      <child link="${name}#door_handle_outside"/>
+      <parent link="${name}:door_center"/>
+      <child link="${name}:door_handle_outside"/>
     </joint>
   </xacro:macro>

File: suturo_resources/urdf/urdf_components/suturo_path.urdf.xacro (robot description, xacro)
@@ -3,10 +3,10 @@
 <robot name="suturo_path" xmlns:xacro="http://ros.org/wiki/xacro">
   <xacro:macro name="suturo_path" params="name parent x_pos y_pos">
-    <joint name="${name}#path_joint" type="fixed">
+    <joint name="${name}:path_joint" type="fixed">
         <origin xyz="${x_pos} ${y_pos} 0 " rpy="0 0 0" />
         <parent link="${parent}"/>
-        <child link="${name}#path_link"/>
+        <child link="${name}:path_link"/>
     </joint>
-    <link name="${name}#path_link">
+    <link name="${name}:path_link">
     </link>
   </xacro:macro>

File: suturo_resources/urdf/urdf_components/suturo_room.urdf.xacro (robot description, xacro)
@@ -4,10 +4,10 @@
   <xacro:macro name="suturo_room" params="name parent num_of_corners corners_x_pos corners_y_pos center_x center_y color">
     <!-- define a central joint to wich every corner is connected -->
-    <joint name="world_${name}#room_joint" type="fixed">
+    <joint name="world_${name}:room_joint" type="fixed">
         <origin xyz="${center_x} ${center_y} 0 " rpy="0 0 0" />
         <parent link="${parent}"/>
-        <child link="${name}#room_center_link"/>
+        <child link="${name}:room_center_link"/>
     </joint>
-    <link name="${name}#room_center_link">
+    <link name="${name}:room_center_link">
       <visual>
         <geometry>
@@ -21,10 +21,10 @@
     <!-- room loop to create every corner -->
     <xacro:macro name="corner_loop" params="loop_number">
-      <joint name="${name}#room_joint_${loop_number}" type="fixed">
+      <joint name="${name}:room_joint_${loop_number}" type="fixed">
           <origin xyz="${corners_x_pos[loop_number] - center_x} ${corners_y_pos[loop_number] - center_y} 0 " rpy="0 0 0" />
-          <parent link="${name}#room_center_link"/>
-          <child link="${name}#room_corner_${loop_number}_link"/>
+          <parent link="${name}:room_center_link"/>
+          <child link="${name}:room_corner_${loop_number}_link"/>
       </joint>
-      <link name="${name}#room_corner_${loop_number}_link" />
+      <link name="${name}:room_corner_${loop_number}_link" />
       <xacro:if value="${(num_of_corners - 1) > loop_number}">
         <xacro:corner_loop loop_number="${loop_number + 1}" />

File: suturo_resources/urdf/urdf_components/suturo_shelf.urdf.xacro (robot description, xacro)
@@ -9,37 +9,37 @@
   <xacro:macro name="suturo_shelf" params="name parent *origin size_x size_y size_z floors_height number_of_floors door">
     <!-- General conveinience links -->
-    <link name="${name}#shelf_origin"/>
-    <link name="${name}#shelf_center"/>
-    <link name="${name}#shelf_base_center"/>
-    <joint name="${name}#shelf_origin_joint" type="fixed">
+    <link name="${name}:shelf_origin"/>
+    <link name="${name}:shelf_center"/>
+    <link name="${name}:shelf_base_center"/>
+    <joint name="${name}:shelf_origin_joint" type="fixed">
       <xacro:insert_block name="origin" />
       <parent link="${parent}"/>
-      <child link="${name}#shelf_origin"/>
+      <child link="${name}:shelf_origin"/>
     </joint>
-    <joint name="${name}#shelf_center_joint" type="fixed">
+    <joint name="${name}:shelf_center_joint" type="fixed">
       <origin xyz="${size_x/2} ${size_y/2} ${size_z/2}" rpy="0 0 0" />
-      <parent link="${name}#shelf_origin"/>
-      <child link="${name}#shelf_center"/>
+      <parent link="${name}:shelf_origin"/>
+      <child link="${name}:shelf_center"/>
     </joint>
-    <joint name="${name}#shelf_base_center_joint" type="fixed">
+    <joint name="${name}:shelf_base_center_joint" type="fixed">
       <origin xyz="${size_x/2} ${size_y/2} 0.0" rpy="0 0 0" />
-      <parent link="${name}#shelf_origin"/>
-      <child link="${name}#shelf_base_center"/>
+      <parent link="${name}:shelf_origin"/>
+      <child link="${name}:shelf_base_center"/>
     </joint>
     <!-- WALLS -->
-    <xacro:suturo_shelf_piece name="${name}#shelf_back" parent="${name}#shelf_origin"
+    <xacro:suturo_shelf_piece name="${name}:shelf_back" parent="${name}:shelf_origin"
       size_x="0.01" size_y="${size_y}" size_z="${size_z}">
       <origin xyz="${size_x} ${size_y/2} ${size_z/2}" rpy="0 0 0"/>
     </xacro:suturo_shelf_piece>
-    <xacro:suturo_shelf_piece name="${name}#shelf_right_side" parent="${name}#shelf_origin"
+    <xacro:suturo_shelf_piece name="${name}:shelf_right_side" parent="${name}:shelf_origin"
       size_x="${size_x}" size_y="0.01" size_z="${size_z}">
       <origin xyz="${size_x/2} 0.0 ${size_z/2}" rpy="0 0 0"/>
     </xacro:suturo_shelf_piece>
-    <xacro:suturo_shelf_piece name="${name}#shelf_left_side" parent="${name}#shelf_origin"
+    <xacro:suturo_shelf_piece name="${name}:shelf_left_side" parent="${name}:shelf_origin"
       size_x="${size_x}" size_y="0.01" size_z="${size_z}">
       <origin xyz="${size_x/2} ${size_y} ${size_z/2}" rpy="0 0 0"/>
     </xacro:suturo_shelf_piece>
     <xacro:macro name="shelf_floor_loop" params="floor_number">
-        <xacro:suturo_shelf_piece name="${name}#shelf_floor_${floor_number}" parent="${name}#shelf_base_center"
+        <xacro:suturo_shelf_piece name="${name}:shelf_floor_${floor_number}" parent="${name}:shelf_base_center"
           size_x="${size_x}" size_y="${size_y}" size_z="0.04" box_z_offset="-0.02">
         <origin xyz="0.0 0.0 ${floors_height[floor_number]}" rpy="0 0 0"/>
@@ -53,5 +53,5 @@
     <!-- left -->
     <xacro:if value="${door == 'left'}">
-      <xacro:suturo_shelf_left_door name="${name}#shelf_door_left" parent="${name}#left_side"
+      <xacro:suturo_shelf_left_door name="${name}:shelf_door_left" parent="${name}:left_side"
         size_x="0.01" size_y="${size_y/2}" size_z="${size_z}" shelf_x_size="${size_x}">
         <origin xyz="0 ${size_y*0.75} ${size_z/2}" rpy="0 0 0"/>
@@ -60,5 +60,5 @@
     <!-- right -->
     <xacro:if value="${door == 'right'}">
-      <xacro:suturo_shelf_right_door name="${name}#shelf_door_right" parent="${name}#right_side"
+      <xacro:suturo_shelf_right_door name="${name}:shelf_door_right" parent="${name}:right_side"
         size_x="0.01" size_y="${size_y/2}" size_z="${size_z}" shelf_x_size="${size_x}">
         <origin xyz="0 ${size_y*0.75} ${size_z/2}" rpy="0 0 0"/>
@@ -67,9 +67,9 @@
     <!-- both -->
     <xacro:if value="${door == 'both'}">
-      <xacro:suturo_shelf_left_door name="${name}#shelf_door_left" parent="${name}#left_side"
+      <xacro:suturo_shelf_left_door name="${name}:shelf_door_left" parent="${name}:left_side"
         size_x="0.01" size_y="${size_y/2}" size_z="${size_z}" shelf_x_size="${size_x}">
         <origin xyz="0 ${size_y*0.75} ${size_z/2}" rpy="0 0 0"/>
       </xacro:suturo_shelf_left_door>
-      <xacro:suturo_shelf_right_door name="${name}#shelf_door_right" parent="${name}#shelf_right_side"
+      <xacro:suturo_shelf_right_door name="${name}:shelf_door_right" parent="${name}#shelf_right_side"
         size_x="0.01" size_y="${size_y/2}" size_z="${size_z}" shelf_x_size="${size_x}">
         <origin xyz="0 ${size_y*0.75} ${size_z/2}" rpy="0 0 0"/>
@@ -97,5 +97,5 @@
     </link>
     <!-- JOINT -->
-    <joint name="${name}#joint" type="fixed">
+    <joint name="${name}:joint" type="fixed">
       <xacro:insert_block name="origin" />
       <parent link="${parent}"/>
@@ -104,5 +104,5 @@
   </xacro:macro>
   <xacro:macro name="suturo_shelf_left_door" params="name parent *origin size_x size_y size_z shelf_x_size">
-    <link name="${name}#link">
+    <link name="${name}:link">
       <visual>
         <material name="shelf_door_green"/>
@@ -119,14 +119,14 @@
       </collision>
     </link>
-    <joint name="${name}#shelf_joint" type="revolute">
+    <joint name="${name}:shelf_joint" type="revolute">
       <origin xyz="${shelf_x_size/-2} ${size_y/-2} 0" rpy="0 0 3.1416"/>
       <axis xyz="0 0 1" />
-      <parent link="${parent}#piece"/>
-      <child link="${name}#link"/>
+      <parent link="${parent}:piece"/>
+      <child link="${name}:link"/>
       <limit effort="30" velocity="1.0" lower="0.0" upper="1.91986" />
     </joint>
   </xacro:macro>
   <xacro:macro name="suturo_shelf_right_door" params="name parent *origin size_x size_y size_z shelf_x_size">
-    <link name="${name}#shelf_link">
+    <link name="${name}:shelf_link">
       <visual>
         <material name="shelf_door_green"/>
@@ -143,9 +143,9 @@
       </collision>
     </link>
-    <joint name="${name}#shelf_joint" type="revolute">
+    <joint name="${name}:shelf_joint" type="revolute">
       <origin xyz="${shelf_x_size/-2} ${size_y/2} 0" rpy="0 0 -3.1416"/>
       <axis xyz="0 0 1" />
-      <parent link="${parent}#shelf_piece"/>
-      <child link="${name}#shelf_link"/>
+      <parent link="${parent}:shelf_piece"/>
+      <child link="${name}:shelf_link"/>
       <limit effort="30" velocity="1.0" lower="0.0" upper="1.91986" />
     </joint>
