Commit message: change # to : because knowrob cant handle it right

File: suturo_resources/urdf/urdf_components/suturo_shelf_openable.urdf.xacro (robot description, xacro)
@@ -6,37 +6,37 @@
   <xacro:macro name="suturo_shelf_openable" params="name parent *origin size_x size_y size_z floors_height number_of_floors door">
     <!-- General conveinience links -->
-    <link name="${name}#shelf_origin"/>
-    <link name="${name}#shelf_center"/>
-    <link name="${name}#shelf_base_center"/>
-    <joint name="${name}#shelf_origin_joint" type="fixed">
+    <link name="${name}:shelf_origin"/>
+    <link name="${name}:shelf_center"/>
+    <link name="${name}:shelf_base_center"/>
+    <joint name="${name}:shelf_origin_joint" type="fixed">
       <xacro:insert_block name="origin" />
       <parent link="${parent}"/>
-      <child link="${name}#shelf_origin"/>
+      <child link="${name}:shelf_origin"/>
     </joint>
-    <joint name="${name}#shelf_center_joint" type="fixed">
+    <joint name="${name}:shelf_center_joint" type="fixed">
       <origin xyz="${size_x/2} ${size_y/2} ${size_z/2}" rpy="0 0 0" />
-      <parent link="${name}#shelf_origin"/>
-      <child link="${name}#shelf_center"/>
+      <parent link="${name}:shelf_origin"/>
+      <child link="${name}:shelf_center"/>
     </joint>
-    <joint name="${name}#shelf_base_center_joint" type="fixed">
+    <joint name="${name}:shelf_base_center_joint" type="fixed">
       <origin xyz="${size_x/2} ${size_y/2} 0.0" rpy="0 0 0" />
-      <parent link="${name}#shelf_origin"/>
-      <child link="${name}#shelf_base_center"/>
+      <parent link="${name}:shelf_origin"/>
+      <child link="${name}:shelf_base_center"/>
     </joint>
     <!-- WALLS -->
-    <xacro:suturo_shelf_piece_openable name="${name}#shelf_back" parent="${name}#shelf_origin"
+    <xacro:suturo_shelf_piece_openable name="${name}:shelf_back" parent="${name}:shelf_origin"
       size_x="0.01" size_y="${size_y}" size_z="${size_z}">
       <origin xyz="${size_x} ${size_y/2} ${size_z/2}" rpy="0 0 0"/>
     </xacro:suturo_shelf_piece_openable>
-    <xacro:suturo_shelf_piece_openable name="${name}#shelf_right_side" parent="${name}#shelf_origin"
+    <xacro:suturo_shelf_piece_openable name="${name}:shelf_right_side" parent="${name}:shelf_origin"
       size_x="${size_x}" size_y="0.01" size_z="${size_z}">
       <origin xyz="${size_x/2} 0.0 ${size_z/2}" rpy="0 0 0"/>
     </xacro:suturo_shelf_piece_openable>
-    <xacro:suturo_shelf_piece_openable name="${name}#shelf_left_side" parent="${name}#shelf_origin"
+    <xacro:suturo_shelf_piece_openable name="${name}:shelf_left_side" parent="${name}:shelf_origin"
       size_x="${size_x}" size_y="0.01" size_z="${size_z}">
       <origin xyz="${size_x/2} ${size_y} ${size_z/2}" rpy="0 0 0"/>
     </xacro:suturo_shelf_piece_openable>
     <xacro:macro name="shelf_floor_loop_openable" params="floor_number">
-        <xacro:suturo_shelf_piece_openable name="${name}#shelf_floor_${floor_number}" parent="${name}#shelf_base_center"
+        <xacro:suturo_shelf_piece_openable name="${name}:shelf_floor_${floor_number}" parent="${name}:shelf_base_center"
           size_x="${size_x}" size_y="${size_y}" size_z="0.04" box_z_offset="-0.02">
         <origin xyz="0.0 0.0 ${floors_height[floor_number]}" rpy="0 0 0"/>
@@ -49,5 +49,5 @@
     <!-- door -->
     <xacro:if value="${door == 'left'}">
-      <xacro:suturo_shelf_left_door_openable name="${name}#shelf_door_left" parent="${name}#shelf_left_side"
+      <xacro:suturo_shelf_left_door_openable name="${name}:shelf_door_left" parent="${name}:shelf_left_side"
         size_x="0.01" size_y="${size_y/2}" size_z="${size_z}" shelf_x_size="${size_x}">
         <origin xyz="0 ${size_y*0.75} ${size_z/2}" rpy="0 0 0"/>
@@ -55,5 +55,5 @@
     </xacro:if>
     <xacro:if value="${door == 'right'}">
-      <xacro:suturo_shelf_right_door_openable name="${name}#shelf_door_right" parent="${name}#shelf_right_side"
+      <xacro:suturo_shelf_right_door_openable name="${name}:shelf_door_right" parent="${name}:shelf_right_side"
         size_x="0.01" size_y="${size_y/2}" size_z="${size_z}" shelf_x_size="${size_x}">
         <origin xyz="0 ${size_y*0.75} ${size_z/2}" rpy="0 0 0"/>
@@ -81,12 +81,12 @@
     </link>
     <!-- JOINT -->
-    <joint name="${name}#shelf_piece_joint" type="fixed">
+    <joint name="${name}:shelf_piece_joint" type="fixed">
       <xacro:insert_block name="origin" />
       <parent link="${parent}"/>
-      <child link="${name}#shelf_piece"/>
+      <child link="${name}:shelf_piece"/>
     </joint>
   </xacro:macro>
   <xacro:macro name="suturo_shelf_left_door_openable" params="name parent *origin size_x size_y size_z shelf_x_size">
-    <link name="${name}#shelf_link">
+    <link name="${name}:shelf_link">
       <visual>
         <material name="shelf_door_green"/>
@@ -103,5 +103,5 @@
       </collision>
     </link>
-    <link name="${name}#shelf_link_handle">
+    <link name="${name}:shelf_link_handle">
       <visual>
         <material name="handle_red"/>
@@ -118,20 +118,20 @@
       </collision>
     </link>
-    <joint name="${name}#shelf_link_handle_joint" type="fixed">
+    <joint name="${name}:shelf_link_handle_joint" type="fixed">
       <origin xyz="-0.01 ${size_y - 0.04} ${size_z/3}" rpy="0 0 0"/>
       <axis xyz="0 0 1" />
-      <parent link="${name}#shelf_link"/>
-      <child link="${name}#shelf_link_handle"/>
+      <parent link="${name}:shelf_link"/>
+      <child link="${name}:shelf_link_handle"/>
     </joint>
-    <joint name="${name}#shelf_joint" type="revolute">
+    <joint name="${name}:shelf_joint" type="revolute">
       <origin xyz="${shelf_x_size/-2} 0 0" rpy="0 0 3.1416"/>
       <axis xyz="0 0 1" />
-      <parent link="${parent}#shelf_piece"/>
-      <child link="${name}#shelf_link"/>
+      <parent link="${parent}:shelf_piece"/>
+      <child link="${name}:shelf_link"/>
       <limit effort="30" velocity="1.0" lower="0.0" upper="1.91986" />
     </joint>
   </xacro:macro>
   <xacro:macro name="suturo_shelf_right_door_openable" params="name parent *origin size_x size_y size_z shelf_x_size">
-    <link name="${name}#shelf_link">
+    <link name="${name}:shelf_link">
       <visual>
         <material name="shelf_door_green"/>
@@ -148,9 +148,9 @@
       </collision>
     </link>
-    <joint name="${name}#shelf_joint" type="revolute">
+    <joint name="${name}:shelf_joint" type="revolute">
       <origin xyz="${shelf_x_size/-2} ${size_y/2} 0" rpy="0 0 -3.1416"/>
       <axis xyz="0 0 1" />
-      <parent link="${parent}#shelf_piece"/>
-      <child link="${name}#shelf_link"/>
+      <parent link="${parent}:shelf_piece"/>
+      <child link="${name}:shelf_link"/>
       <limit effort="30" velocity="1.0" lower="0.0" upper="1.91986" />
     </joint>

File: suturo_resources/urdf/urdf_components/suturo_table.urdf.xacro (robot description, xacro)
@@ -6,5 +6,5 @@
   <xacro:macro name="suturo_table" params="name parent *origin size_x size_y size_z">
     <!-- LINKS -->
-    <link name="${name}#table_center">
+    <link name="${name}:table_center">
       <visual>
         <material name="table_grey"/>
@@ -21,21 +21,21 @@
       </collision>
     </link>
-    <link name="${name}#table_origin"/>
-     <link name="${name}#table_front_edge_center"/>
+    <link name="${name}:table_origin"/>
+     <link name="${name}:table_front_edge_center"/>
     <!-- JOINTS -->
-    <joint name="${name}#table_origin_joint" type="fixed">
+    <joint name="${name}:table_origin_joint" type="fixed">
       <xacro:insert_block name="origin" />
       <parent link="${parent}"/>
-      <child link="${name}#table_origin"/>
+      <child link="${name}:table_origin"/>
     </joint>
-    <joint name="${name}#center_joint" type="fixed">
+    <joint name="${name}:center_joint" type="fixed">
       <origin xyz="${size_x/2} ${size_y/2} ${size_z}" rpy="0 0 0" />
-      <parent link="${name}#table_origin"/>
-      <child link="${name}#table_center"/>
+      <parent link="${name}:table_origin"/>
+      <child link="${name}:table_center"/>
     </joint>
-    <joint name="${name}#table_front_edge_center_joint" type="fixed">
+    <joint name="${name}:table_front_edge_center_joint" type="fixed">
       <origin xyz="0 ${size_y/2} ${size_z}" rpy="0 0 0" />
-      <parent link="${name}#table_origin"/>
-      <child link="${name}#table_front_edge_center"/>
+      <parent link="${name}:table_origin"/>
+      <child link="${name}:table_front_edge_center"/>
     </joint>
   </xacro:macro>

Commit message: added call path loop in urdf creation

File: suturo_resources/urdf/suturo_environment.urdf.xacro (robot description, xacro)
@@ -20,4 +20,5 @@
     <xacro:property name="number_of_doors" value="${data['doors']['amount']}" />
     <xacro:property name="number_of_rooms" value="${data['rooms']['amount']}" />
+    <xacro:property name="number_of_paths" value="${data['paths']['amount']}" />
     <!--  ~~Tables~~  -->
     <xacro:macro name="table_loop" params="table_number">
@@ -132,6 +133,6 @@
       <xacro:suturo_path name="${data['paths'][path_number]['room1']}:${data['paths'][path_number]['room2']}"
                          parent="${data['paths'][path_number]['parent']}"
-                         x_pos="${data['paths'][path_number]['x']}"
-                         y_pos="${data['paths'][path_number]['y']}"
+                         x_pos="${data['paths'][path_number]['x_pos']}"
+                         y_pos="${data['paths'][path_number]['y_pos']}"
                          >
       </xacro:suturo_path>
@@ -162,4 +163,7 @@
         <xacro:door_loop door_number="0" />
     </xacro:if>
+    <xacro:if value="${number_of_paths > 0}">
+	<xacro:path_loop path_number="0" />
+    </xacro:if>
     <link name="urdf_main" />
     <joint name="map_urdf_joint" type="fixed">

Commit message: Drawer urdf and sponge

File: suturo_resources/urdf/suturo_environment.urdf.xacro (robot description, xacro)
@@ -12,5 +12,7 @@
     <xacro:include filename="$(find suturo_resources)/urdf/urdf_components/suturo_bucket.urdf.xacro"/>
     <xacro:include filename="$(find suturo_resources)/urdf/urdf_components/suturo_path.urdf.xacro"/>
+    <xacro:include filename="$(find suturo_resources)/urdf/urdf_components/suturo_drawer.urdf.xacro"/>
     <!-- general data -->
+    <xacro:property name="number_of_drawers" value="${data['drawers']['amount']}" />
     <xacro:property name="number_of_tables" value="${data['tables']['amount']}" />
     <xacro:property name="number_of_buckets" value="${data['buckets']['amount']}" />
@@ -83,4 +85,18 @@
         </xacro:if>
     </xacro:macro>
+     <!--  ~~Drawers~~  -->
+    <xacro:macro name="drawer_loop" params="drawer_number">
+        <xacro:suturo_drawer name="${data['drawers'][drawer_number]['name']}:${data['drawers'][drawer_number]['knowledge_role']}"
+                          parent="${data['drawers'][drawer_number]['parent']}"
+                          size_x="${data['drawers'][drawer_number]['depth']}"
+                          size_y="${data['drawers'][drawer_number]['width']}"
+                          size_z="${data['drawers'][drawer_number]['height']}">
+            <origin xyz="${data['drawers'][drawer_number]['x_pos']} ${data['drawers'][drawer_number]['y_pos']} 0"
+                            rpy="0 0 ${data['drawers'][drawer_number]['z_rot']}" />
+        </xacro:suturo_drawer>
+        <!--<xacro:if value="${(number_of_drawers - 1) > drawer_number}">
+            <xacro:drawer_loop drawer_number="${drawer_number + 1}" />
+        </xacro:if>-->
+    </xacro:macro>
     <!--  ~~Walls~~  -->
     <xacro:macro name="wall_loop" params="wall_number">
@@ -142,4 +158,7 @@
     </xacro:macro>
     <!--Calling the loops-->
+    <xacro:if value="${number_of_drawers > 0}">
+        <xacro:drawer_loop drawer_number="0" />
+    </xacro:if>
     <xacro:if value="${number_of_tables > 0}">
         <xacro:table_loop table_number="0" />

Commit message: Semantic Map

File: suturo_resources/urdf/suturo_environment.urdf.xacro (robot description, xacro)
@@ -1,4 +1,4 @@
 <?xml version="1.0"?>
-<robot name="hsrb_lab" xmlns:xacro="http://ros.org/wiki/xacro">
+<robot name="iai-kitchen" xmlns:xacro="http://ros.org/wiki/xacro">
     <xacro:property name="data"
     value="${load_yaml('$(arg yaml_file)')}" />

File: suturo_resources/urdf/urdf_components/suturo_shelf.urdf.xacro (robot description, xacro)
@@ -27,4 +27,10 @@
       <child link="${name}:shelf_base_center"/>
     </joint>
+    <!-- <joint name="${name}:shelf_left_side" type="fixed" -->
+    <!--        size_x="${size_x}" size_y="0.01" size_z="${size_z}"> -->
+    <!--   <origin xyz="${size_x/2} ${size_y} ${size_z/2}" rpy="0 0 0"/> -->
+    <!--   <parent link="${name}:shelf_origin"/> -->
+    <!--   <child link="${name}:shelf_door_left"/> -->
+    <!-- </joint>  -->
     <!-- WALLS -->
     <xacro:suturo_shelf_piece name="${name}:shelf_back" parent="${name}:shelf_origin"

File: suturo_resources/urdf/urdf_components/suturo_shelf_openable.urdf.xacro (robot description, xacro)
@@ -43,8 +43,8 @@
       </xacro:suturo_shelf_piece_openable>
       <xacro:if value="${(number_of_floors - 1) > floor_number}">
-            <xacro:shelf_floor_loop floor_number="${floor_number + 1}" />
+            <xacro:shelf_floor_loop_openable floor_number="${floor_number + 1}" />
       </xacro:if>
     </xacro:macro>
-    <xacro:shelf_floor_loop floor_number="0" />
+    <xacro:shelf_floor_loop_openable floor_number="0" />
     <!-- door -->
     <xacro:if value="${door == 'left'}">
@@ -60,4 +60,14 @@
       </xacro:suturo_shelf_right_door_openable>
     </xacro:if>
+    <xacro:if value="${door == 'both'}">
+       <xacro:suturo_shelf_right_door_openable name="${name}:shelf_door_right" parent="${name}:shelf_right_side"
+        size_x="0.01" size_y="${size_y/2}" size_z="${size_z}" shelf_x_size="${size_x}">
+        <origin xyz="0 ${size_y*0.75} ${size_z/2}" rpy="0 0 0"/>
+       </xacro:suturo_shelf_right_door_openable>
+         <xacro:suturo_shelf_left_door_openable name="${name}:shelf_door_left" parent="${name}:shelf_left_side"
+        size_x="0.01" size_y="${size_y/2}" size_z="${size_z}" shelf_x_size="${size_x}">
+        <origin xyz="0 ${size_y} ${size_z/2}" rpy="0 0 0"/>
+      </xacro:suturo_shelf_left_door_openable>
+    </xacro:if>
   </xacro:macro>
   <!-- Creates a link with collision and visual box of given dimensions,
@@ -91,11 +101,56 @@
       <visual>
         <material name="shelf_door_green"/>
-        <origin xyz="0 ${size_y/2.15} 0" rpy="0 0 0" />
-        <geometry>
-          <box size="${size_x} ${size_y} ${size_z}" />
-        </geometry>
-      </visual>
-      <collision>
-        <origin xyz="0 ${size_y/2.15} 0" rpy="0 0 0" />
+        <origin xyz="0 ${size_y/2.02} 0" rpy="0 0 0" />
+        <geometry>
+          <box size="${size_x} ${size_y} ${size_z}" />
+        </geometry>
+      </visual>
+      <collision>
+        <origin xyz="0 ${size_y/2.02} 0" rpy="0 0 0" />
+        <geometry>
+          <box size="${size_x} ${size_y} ${size_z}" />
+        </geometry>
+      </collision>
+    </link>
+    <link name="${name}:shelf_link_handle">
+      <visual>
+        <material name="shelf_openable_handle_red"/>
+        <origin xyz="0 0 0" rpy="0 0 0" />
+        <geometry>
+          <box size="0.025 0.01 0.07" />
+        </geometry>
+      </visual>
+      <collision>
+        <origin xyz="0 0 0" rpy="0 0 0" />
+        <geometry>
+          <box size="0.04 0.01 0.07" />
+        </geometry>
+      </collision>
+    </link>
+    <joint name="${name}:shelf_link_handle_joint" type="fixed">
+      <origin xyz="0.01 ${size_y - 0.04} ${size_z/3}" rpy="0 0 0"/>
+      <axis xyz="0 0 1" />
+      <parent link="${name}:shelf_link"/>
+      <child link="${name}:shelf_link_handle"/>
+    </joint>
+    <joint name="${name}:shelf_joint" type="revolute">
+      <origin xyz="${shelf_x_size/-2} 0 0" rpy="0 0 3.1416"/>
+      <axis xyz="0 0 1" />
+      <parent link="${parent}:shelf_piece"/>
+      <child link="${name}:shelf_link"/>
+      <limit effort="30" velocity="1.0" lower="-1.7" upper="0.0" />
+    </joint>
+  </xacro:macro>
+  <xacro:macro name="suturo_shelf_right_door_openable" params="name parent *origin size_x size_y size_z shelf_x_size">
+    <link name="${name}:shelf_link">
+      <visual>
+        <material name="shelf_door_green"/>
+        <origin xyz="0 ${size_y/2.02} 0" rpy="0 0 0" />
+        <geometry>
+          <box size="${size_x} ${size_y} ${size_z}" />
+        </geometry>
+      </visual>
+      <collision>
+        <origin xyz="0 ${size_y/2.02} 0" rpy="0 0 0" />
         <geometry>
           <box size="${size_x} ${size_y} ${size_z}" />
@@ -125,34 +180,34 @@
     </joint>
     <joint name="${name}:shelf_joint" type="revolute">
-      <origin xyz="${shelf_x_size/-2} 0 0" rpy="0 0 3.1416"/>
+      <origin xyz="${shelf_x_size/-2} 0 0" rpy="0 0 0"/>
       <axis xyz="0 0 1" />
       <parent link="${parent}:shelf_piece"/>
       <child link="${name}:shelf_link"/>
-      <limit effort="30" velocity="1.0" lower="0.0" upper="1.91986" />
-    </joint>
-  </xacro:macro>
-  <xacro:macro name="suturo_shelf_right_door_openable" params="name parent *origin size_x size_y size_z shelf_x_size">
-    <link name="${name}:shelf_link">
-      <visual>
-        <material name="shelf_door_green"/>
-        <origin xyz="0 0 0" rpy="0 0 0" />
-        <geometry>
-          <box size="${size_x} ${size_y} ${size_z}" />
-        </geometry>
-      </visual>
-      <collision>
-        <origin xyz="0 0 0" rpy="0 0 0" />
-        <geometry>
-          <box size="${size_x} ${size_y} ${size_z}" />
-        </geometry>
-      </collision>
-    </link>
-    <joint name="${name}:shelf_joint" type="revolute">
-      <origin xyz="${shelf_x_size/-2} ${size_y/2} 0" rpy="0 0 -3.1416"/>
-      <axis xyz="0 0 1" />
-      <parent link="${parent}:shelf_piece"/>
-      <child link="${name}:shelf_link"/>
-      <limit effort="30" velocity="1.0" lower="0.0" upper="1.91986" />
-    </joint>
-  </xacro:macro>
+      <limit effort="30" velocity="1.0" lower="0.0" upper="1.7" />
+    </joint>
+  </xacro:macro>
+  <!-- <xacro:macro name="suturo_shelf_right_door_openable" params="name parent *origin size_x size_y size_z shelf_x_size"> -->
+  <!--   <link name="${name}:shelf_link"> -->
+  <!--     <visual> -->
+  <!--       <material name="shelf_door_green"/> -->
+  <!--       <origin xyz="0 0 0" rpy="0 0 0" /> -->
+  <!--       <geometry> -->
+  <!--         <box size="${size_x} ${size_y} ${size_z}" /> -->
+  <!--       </geometry> -->
+  <!--     </visual> -->
+  <!--     <collision> -->
+  <!--       <origin xyz="0 0 0" rpy="0 0 0" /> -->
+  <!--       <geometry> -->
+  <!--         <box size="${size_x} ${size_y} ${size_z}" /> -->
+  <!--       </geometry> -->
+  <!--     </collision> -->
+  <!--   </link> -->
+  <!--   <joint name="${name}:shelf_joint" type="revolute"> -->
+  <!--     <origin xyz="${shelf_x_size/-2} ${size_y/2} 0" rpy="0 0 -3.1416"/> -->
+  <!--     <axis xyz="0 0 1" /> -->
+  <!--     <parent link="${parent}:shelf_piece"/> -->
+  <!--     <child link="${name}:shelf_link"/> -->
+  <!--     <limit effort="30" velocity="1.0" lower="0.0" upper="1.91986" /> -->
+  <!--   </joint> -->
+  <!-- </xacro:macro> -->
 </robot>

File: suturo_resources/urdf/urdf_components/suturo_table.urdf.xacro (robot description, xacro)
@@ -22,5 +22,5 @@
     </link>
     <link name="${name}:table_origin"/>
-     <link name="${name}:table_front_edge_center"/>
+    <link name="${name}:table_front_edge_center"/>
     <!-- JOINTS -->
     <joint name="${name}:table_origin_joint" type="fixed">
