Commit message: Alpha: improve doors of openable shelves

File: suturo_resources/urdf/suturo_environment.urdf.xacro (robot description, xacro)
@@ -77,5 +77,11 @@
                           floors_height="${data['shelves_openable'][shelf_openable_number]['floors_height']}"
                           number_of_floors="${data['shelves_openable'][shelf_openable_number]['number_of_floors']}"
-                          door="${data['shelves_openable'][shelf_openable_number]['door']}">
+                          door="${data['shelves_openable'][shelf_openable_number]['door']}"
+			  wall_thickness="${data['shelves_openable'][shelf_openable_number]['wall_thickness']}"
+			  handle_from_bottom="${data['shelves_openable'][shelf_openable_number]['handle_from_bottom']}"
+			  handle_from_side="${data['shelves_openable'][shelf_openable_number]['handle_from_side']}"
+			  handle_height="${data['shelves_openable'][shelf_openable_number]['handle_height']}"
+			  handle_width="${data['shelves_openable'][shelf_openable_number]['handle_width']}"
+			  handle_depth="${data['shelves_openable'][shelf_openable_number]['handle_depth']}">
             <origin xyz="${data['shelves_openable'][shelf_openable_number]['x_pos']} ${data['shelves_openable'][shelf_openable_number]['y_pos']} 0"
                             rpy="0 0 ${data['shelves_openable'][shelf_openable_number]['z_rot']}" />

File: suturo_resources/urdf/urdf_components/suturo_shelf_openable.urdf.xacro (robot description, xacro)
@@ -4,5 +4,5 @@
     <color rgba="0.74 0.25 0.25 1"/>
   </material>
-  <xacro:macro name="suturo_shelf_openable" params="name parent *origin size_x size_y size_z floors_height number_of_floors door">
+  <xacro:macro name="suturo_shelf_openable" params="name parent *origin size_x size_y size_z floors_height number_of_floors door wall_thickness handle_from_bottom handle_from_side handle_height handle_width handle_depth">
     <!-- General conveinience links -->
     <link name="${name}:shelf_origin"/>
@@ -26,14 +26,14 @@
     <!-- WALLS -->
     <xacro:suturo_shelf_piece_openable name="${name}:shelf_back" parent="${name}:shelf_origin"
-      size_x="0.01" size_y="${size_y}" size_z="${size_z}">
+      size_x="${wall_thickness}" size_y="${size_y}" size_z="${size_z}">
       <origin xyz="${size_x} ${size_y/2} ${size_z/2}" rpy="0 0 0"/>
     </xacro:suturo_shelf_piece_openable>
     <xacro:suturo_shelf_piece_openable name="${name}:shelf_right_side" parent="${name}:shelf_origin"
-      size_x="${size_x}" size_y="0.01" size_z="${size_z}">
-      <origin xyz="${size_x/2} 0.0 ${size_z/2}" rpy="0 0 0"/>
+      size_x="${size_x}" size_y="${wall_thickness}" size_z="${size_z}">
+      <origin xyz="${size_x/2} ${+wall_thickness/2} ${size_z/2}" rpy="0 0 0"/>
     </xacro:suturo_shelf_piece_openable>
     <xacro:suturo_shelf_piece_openable name="${name}:shelf_left_side" parent="${name}:shelf_origin"
-      size_x="${size_x}" size_y="0.01" size_z="${size_z}">
-      <origin xyz="${size_x/2} ${size_y} ${size_z/2}" rpy="0 0 0"/>
+      size_x="${size_x}" size_y="${wall_thickness}" size_z="${size_z}">
+      <origin xyz="${size_x/2} ${size_y-wall_thickness/2} ${size_z/2}" rpy="0 0 0"/>
     </xacro:suturo_shelf_piece_openable>
     <xacro:macro name="shelf_floor_loop_openable" params="floor_number">
@@ -47,8 +47,10 @@
     </xacro:macro>
     <xacro:shelf_floor_loop_openable floor_number="0" />
+    <xacro:property name="door_width" value="${(size_y-2*wall_thickness)/2}"/>
     <!-- door -->
     <xacro:if value="${door == 'left'}">
       <xacro:suturo_shelf_left_door_openable name="${name}:shelf_door_left" parent="${name}:shelf_left_side"
-        size_x="0.01" size_y="${size_y/2}" size_z="${size_z}" shelf_x_size="${size_x}">
+       wall_thickness="${wall_thickness}" size_y="${door_width}" size_z="${size_z}" shelf_x_size="${size_x}"
+       handle_from_bottom="${handle_from_bottom}" handle_from_side="${handle_from_side}" handle_height="${handle_height}" handle_width="${handle_width}" handle_depth="${handle_depth}">
         <origin xyz="0 ${size_y*0.75} ${size_z/2}" rpy="0 0 0"/>
       </xacro:suturo_shelf_left_door_openable>
@@ -56,5 +58,6 @@
     <xacro:if value="${door == 'right'}">
       <xacro:suturo_shelf_right_door_openable name="${name}:shelf_door_right" parent="${name}:shelf_right_side"
-        size_x="0.01" size_y="${size_y/2}" size_z="${size_z}" shelf_x_size="${size_x}">
+        wall_thickness="${wall_thickness}" size_y="${door_width}" size_z="${size_z}" shelf_x_size="${size_x}"
+       handle_from_bottom="${handle_from_bottom}" handle_from_side="${handle_from_side}" handle_height="${handle_height}" handle_width="${handle_width}" handle_depth="${handle_depth}">
         <origin xyz="0 ${size_y*0.75} ${size_z/2}" rpy="0 0 0"/>
       </xacro:suturo_shelf_right_door_openable>
@@ -62,9 +65,11 @@
     <xacro:if value="${door == 'both'}">
        <xacro:suturo_shelf_right_door_openable name="${name}:shelf_door_right" parent="${name}:shelf_right_side"
-        size_x="0.01" size_y="${size_y/2}" size_z="${size_z}" shelf_x_size="${size_x}">
-        <origin xyz="0 ${size_y*0.75} ${size_z/2}" rpy="0 0 0"/>
+        wall_thickness="${wall_thickness}" size_y="${door_width}" size_z="${size_z}" shelf_x_size="${size_x}"
+       handle_from_bottom="${handle_from_bottom}" handle_from_side="${handle_from_side}" handle_height="${handle_height}" handle_width="${handle_width}" handle_depth="${handle_depth}">
+        <origin xyz="0 ${size_y} ${size_z/2}" rpy="0 0 0"/>
        </xacro:suturo_shelf_right_door_openable>
          <xacro:suturo_shelf_left_door_openable name="${name}:shelf_door_left" parent="${name}:shelf_left_side"
-        size_x="0.01" size_y="${size_y/2}" size_z="${size_z}" shelf_x_size="${size_x}">
+          wall_thickness="${wall_thickness}" size_y="${door_width}" size_z="${size_z}" shelf_x_size="${size_x}"
+	  handle_from_bottom="${handle_from_bottom}" handle_from_side="${handle_from_side}" handle_height="${handle_height}" handle_width="${handle_width}" handle_depth="${handle_depth}">
         <origin xyz="0 ${size_y} ${size_z/2}" rpy="0 0 0"/>
       </xacro:suturo_shelf_left_door_openable>
@@ -97,15 +102,16 @@
     </joint>
   </xacro:macro>
-  <xacro:macro name="suturo_shelf_left_door_openable" params="name parent *origin size_x size_y size_z shelf_x_size">
+  <xacro:macro name="suturo_shelf_left_door_openable" params="name parent *origin wall_thickness size_y size_z shelf_x_size handle_from_bottom handle_from_side handle_height handle_width handle_depth">
+    <xacro:property name="size_x" value="${wall_thickness}"/>
     <link name="${name}">
       <visual>
         <material name="shelf_door_green"/>
-        <origin xyz="0 ${size_y/2.02} 0" rpy="0 0 0" />
-        <geometry>
-          <box size="${size_x} ${size_y} ${size_z}" />
-        </geometry>
-      </visual>
-      <collision>
-        <origin xyz="0 ${size_y/2.02} 0" rpy="0 0 0" />
+        <origin xyz="0 ${-size_y/2+wall_thickness/2} 0" rpy="0 0 0" />
+        <geometry>
+          <box size="${size_x} ${size_y} ${size_z}" />
+        </geometry>
+      </visual>
+      <collision>
+        <origin xyz="0 ${-size_y/2+wall_thickness/2} 0" rpy="0 0 0" />
         <geometry>
           <box size="${size_x} ${size_y} ${size_z}" />
@@ -118,16 +124,16 @@
         <origin xyz="0 0 0" rpy="0 0 0" />
         <geometry>
-          <box size="0.025 0.01 0.07" />
-        </geometry>
-      </visual>
-      <collision>
-        <origin xyz="0 0 0" rpy="0 0 0" />
-        <geometry>
-          <box size="0.04 0.01 0.07" />
+          <box size="${handle_depth} ${handle_width} ${handle_height}" />
+        </geometry>
+      </visual>
+      <collision>
+        <origin xyz="0 0 0" rpy="0 0 0" />
+        <geometry>
+          <box size="${handle_depth} ${handle_width} ${handle_height}" />
         </geometry>
       </collision>
     </link>
     <joint name="${name}:handle_joint" type="fixed">
-      <origin xyz="0.01 ${size_y - 0.04} ${size_z/3}" rpy="0 0 0"/>
+      <origin xyz="${-wall_thickness-handle_depth/2} ${-handle_from_side} ${handle_from_bottom-size_z/2}" rpy="0 0 0"/>
       <axis xyz="0 0 1" />
       <parent link="${name}"/>
@@ -135,5 +141,5 @@
     </joint>
     <joint name="${name}:joint" type="revolute">
-      <origin xyz="${shelf_x_size/-2} 0 0" rpy="0 0 3.1416"/>
+      <origin xyz="${shelf_x_size/-2} ${-wall_thickness} 0" rpy="0 0 0"/>
       <axis xyz="0 0 1" />
       <parent link="${parent}"/>
@@ -142,15 +148,16 @@
     </joint>
   </xacro:macro>
-  <xacro:macro name="suturo_shelf_right_door_openable" params="name parent *origin size_x size_y size_z shelf_x_size">
+  <xacro:macro name="suturo_shelf_right_door_openable" params="name parent *origin wall_thickness size_y size_z shelf_x_size handle_from_bottom handle_from_side handle_height handle_width handle_depth">
+    <xacro:property name="size_x" value="${wall_thickness}"/>
     <link name="${name}">
       <visual>
         <material name="shelf_door_green"/>
-        <origin xyz="0 ${size_y/2.02} 0" rpy="0 0 0" />
-        <geometry>
-          <box size="${size_x} ${size_y} ${size_z}" />
-        </geometry>
-      </visual>
-      <collision>
-        <origin xyz="0 ${size_y/2.02} 0" rpy="0 0 0" />
+        <origin xyz="0 ${size_y/2-wall_thickness/2} 0" rpy="0 0 0" />
+        <geometry>
+          <box size="${size_x} ${size_y} ${size_z}" />
+        </geometry>
+      </visual>
+      <collision>
+        <origin xyz="0 ${size_y/2-wall_thickness/2} 0" rpy="0 0 0" />
         <geometry>
           <box size="${size_x} ${size_y} ${size_z}" />
@@ -163,16 +170,16 @@
         <origin xyz="0 0 0" rpy="0 0 0" />
         <geometry>
-          <box size="0.025 0.01 0.07" />
-        </geometry>
-      </visual>
-      <collision>
-        <origin xyz="0 0 0" rpy="0 0 0" />
-        <geometry>
-          <box size="0.04 0.01 0.07" />
+          <box size="${handle_depth} ${handle_width} ${handle_height}" />
+        </geometry>
+      </visual>
+      <collision>
+        <origin xyz="0 0 0" rpy="0 0 0" />
+        <geometry>
+          <box size="${handle_depth} ${handle_width} ${handle_height}" />
         </geometry>
       </collision>
     </link>
     <joint name="${name}:handle_joint" type="fixed">
-      <origin xyz="-0.01 ${size_y - 0.04} ${size_z/3}" rpy="0 0 0"/>
+      <origin xyz="${-wall_thickness-handle_depth/2} ${+handle_from_side} ${handle_from_bottom-size_z/2}" rpy="0 0 0"/>
       <axis xyz="0 0 1" />
       <parent link="${name}"/>
@@ -180,5 +187,5 @@
     </joint>
     <joint name="${name}:joint" type="revolute">
-      <origin xyz="${shelf_x_size/-2} 0 0" rpy="0 0 0"/>
+      <origin xyz="${shelf_x_size/-2} ${wall_thickness} 0" rpy="0 0 0"/>
       <axis xyz="0 0 1" />
       <parent link="${parent}"/>

Commit message: Added dishwasher to map.

File: suturo_resources/urdf/suturo_environment.urdf.xacro (robot description, xacro)
@@ -2,5 +2,16 @@
 <robot name="iai-kitchen" xmlns:xacro="http://ros.org/wiki/xacro">
     <xacro:property name="data"
-    value="${load_yaml('$(arg yaml_file)')}" />
+                    value="${load_yaml('$(arg yaml_file)')}" />
+    <xacro:property name="simulated" value="true" />
+  <xacro:macro name="sphere_inertia" params="radius mass">
+        <inertial>
+          <origin xyz="0.0 0.0 0.0" rpy="0 0 0"/>
+          <mass value="1"/>
+          <inertia
+              ixx="1" ixy="0.0" ixz="0.0"
+              iyy="1" iyz="0.0"
+              izz="1"/>
+        </inertial>
+  </xacro:macro>
     <!--  Include the files containing the macros -->
     <xacro:include filename="$(find suturo_resources)/urdf/urdf_components/suturo_table.urdf.xacro"/>
@@ -13,4 +24,5 @@
     <xacro:include filename="$(find suturo_resources)/urdf/urdf_components/suturo_path.urdf.xacro"/>
     <xacro:include filename="$(find suturo_resources)/urdf/urdf_components/suturo_drawer.urdf.xacro"/>
+    <xacro:include filename="$(find suturo_resources)/urdf/urdf_components/suturo_dishwasher.urdf.xacro"/>
     <!-- general data -->
     <xacro:property name="number_of_drawers" value="${data['drawers']['amount']}" />
@@ -23,4 +35,5 @@
     <xacro:property name="number_of_rooms" value="${data['rooms']['amount']}" />
     <xacro:property name="number_of_paths" value="${data['paths']['amount']}" />
+    <xacro:property name="number_of_dishwashers" value="${data['dishwashers']['amount']}" />
     <!--  ~~Tables~~  -->
     <xacro:macro name="table_loop" params="table_number">
@@ -35,4 +48,15 @@
         <xacro:if value="${(number_of_tables - 1) > table_number}">
             <xacro:table_loop table_number="${table_number + 1}" />
+        </xacro:if>
+    </xacro:macro>
+     <!--  ~~Dishwashers~~  -->
+    <xacro:macro name="dishwasher_loop" params="dishwasher_number">
+        <xacro:suturo_dishwasher name="${data['dishwashers'][dishwasher_number]['name']}:${data['dishwashers'][dishwasher_number]['knowledge_role']}"
+                          parent="${data['dishwashers'][dishwasher_number]['parent']}">
+            <origin xyz="${data['dishwashers'][dishwasher_number]['x_pos']} ${data['dishwashers'][dishwasher_number]['y_pos']} 0.33475"
+                            rpy="0 0 ${data['dishwashers'][dishwasher_number]['z_rot']}" />
+        </xacro:suturo_dishwasher>
+        <xacro:if value="${(number_of_dishwashers - 1) > dishwasher_number}">
+            <xacro:table_loop table_number="${dishwasher_number + 1}" />
         </xacro:if>
     </xacro:macro>
@@ -191,4 +215,7 @@
 	<xacro:path_loop path_number="0" />
     </xacro:if>
+     <xacro:if value="${number_of_dishwashers > 0}">
+	<xacro:dishwasher_loop dishwasher_number="0" />
+    </xacro:if>
     <link name="urdf_main" />
     <joint name="map_urdf_joint" type="fixed">

Commit message: add simple drawer to semantic map

File: suturo_resources/urdf/suturo_environment.urdf.xacro (robot description, xacro)
@@ -24,7 +24,9 @@
     <xacro:include filename="$(find suturo_resources)/urdf/urdf_components/suturo_path.urdf.xacro"/>
     <xacro:include filename="$(find suturo_resources)/urdf/urdf_components/suturo_drawer.urdf.xacro"/>
+    <xacro:include filename="$(find suturo_resources)/urdf/urdf_components/suturo_simple_drawer.urdf.xacro"/>
     <xacro:include filename="$(find suturo_resources)/urdf/urdf_components/suturo_dishwasher.urdf.xacro"/>
     <!-- general data -->
     <xacro:property name="number_of_drawers" value="${data['drawers']['amount']}" />
+    <xacro:property name="number_of_simple_drawers" value="${data['simple_drawers']['amount']}" />
     <xacro:property name="number_of_tables" value="${data['tables']['amount']}" />
     <xacro:property name="number_of_buckets" value="${data['buckets']['amount']}" />
@@ -129,4 +131,23 @@
         </xacro:if>-->
     </xacro:macro>
+     <!--  ~~Simple Drawers~~  -->
+    <xacro:macro name="simple_drawer_loop" params="drawer_number">
+        <xacro:suturo_simple_drawer name="${data['simple_drawers'][drawer_number]['name']}:${data['simple_drawers'][drawer_number]['knowledge_role']}"
+                          parent="${data['simple_drawers'][drawer_number]['parent']}"
+                          size_x="${data['simple_drawers'][drawer_number]['depth']}"
+                          size_y="${data['simple_drawers'][drawer_number]['width']}"
+                          size_z="${data['simple_drawers'][drawer_number]['height']}"
+                          handle_x="${data['simple_drawers'][drawer_number]['handle_x']}"
+                          handle_z="${data['simple_drawers'][drawer_number]['handle_z']}"
+                          handle_size_x="${data['simple_drawers'][drawer_number]['handle_size_x']}"
+                          handle_size_y="${data['simple_drawers'][drawer_number]['handle_size_y']}"
+                          handle_size_z="${data['simple_drawers'][drawer_number]['handle_size_z']}">
+            <origin xyz="${data['simple_drawers'][drawer_number]['x_pos']} ${data['simple_drawers'][drawer_number]['y_pos']} ${data['simple_drawers'][drawer_number]['z_pos']}"
+                            rpy="0 0 ${data['simple_drawers'][drawer_number]['z_rot']}" />
+        </xacro:suturo_simple_drawer>
+        <xacro:if value="${(number_of_drawers - 1) > drawer_number}">
+            <xacro:simple_drawer_loop drawer_number="${drawer_number + 1}" />
+        </xacro:if>
+    </xacro:macro>
     <!--  ~~Walls~~  -->
     <xacro:macro name="wall_loop" params="wall_number">
@@ -191,4 +212,7 @@
         <xacro:drawer_loop drawer_number="0" />
     </xacro:if>
+    <xacro:if value="${number_of_simple_drawers > 0}">
+        <xacro:simple_drawer_loop drawer_number="0" />
+    </xacro:if>
     <xacro:if value="${number_of_tables > 0}">
         <xacro:table_loop table_number="0" />

Commit message: add new rooms to urdf

File: suturo_resources/urdf/suturo_environment.urdf.xacro (robot description, xacro)
@@ -165,11 +165,10 @@
     <!--  ~~Rooms~~  -->
     <xacro:macro name="room_loop" params="room_number">
-      <xacro:suturo_room name="${data['rooms'][room_number]['name']}"
+      <xacro:suturo_room name="${data['rooms'][room_number]['name']}:${data['rooms'][room_number]['knowledge_role']}"
                          parent="urdf_offset"
-                         num_of_corners="${data['rooms'][room_number]['num_of_corners']}"
-                         corners_x_pos="${data['rooms'][room_number]['corners_x_pos']}"
-                         corners_y_pos="${data['rooms'][room_number]['corners_y_pos']}"
                          center_x="${data['rooms'][room_number]['center_x']}"
                          center_y="${data['rooms'][room_number]['center_y']}"
+                         size_x="${data['rooms'][room_number]['size_x']}"
+                         size_y="${data['rooms'][room_number]['size_y']}"
                          color="${data['rooms'][room_number]['color']}">
       </xacro:suturo_room>

File: suturo_resources/urdf/urdf_components/suturo_room.urdf.xacro (robot description, xacro)
@@ -2,8 +2,7 @@
 <!-- Rooms are for Knowledge Information only-->
 <robot name="suturo_room" xmlns:xacro="http://ros.org/wiki/xacro">
-  <xacro:macro name="suturo_room" params="name parent num_of_corners corners_x_pos corners_y_pos center_x center_y color">
-    <!-- define a central joint to wich every corner is connected -->
+  <xacro:macro name="suturo_room" params="name parent center_x center_y color size_x size_y">
     <joint name="world_${name}:room_joint" type="fixed">
-        <origin xyz="${center_x} ${center_y} 0 " rpy="0 0 0" />
+        <origin xyz="${center_x} ${center_y} -0.01 " rpy="0 0 0" />
         <parent link="${parent}"/>
         <child link="${name}:room_center_link"/>
@@ -12,5 +11,5 @@
       <visual>
         <geometry>
-          <cylinder length="0" radius="0"/>
+          <box size="${size_x} ${size_y} 0.01" />
         </geometry>
         <material name="color">
@@ -18,19 +17,10 @@
         </material>
       </visual>
+      <collision>
+        <geometry>
+          <box size="${size_x} ${size_y} 0.01" />
+        </geometry>
+      </collision>
     </link>
-    <!-- room loop to create every corner -->
-    <xacro:macro name="corner_loop" params="loop_number">
-      <joint name="${name}:room_joint_${loop_number}" type="fixed">
-          <origin xyz="${corners_x_pos[loop_number] - center_x} ${corners_y_pos[loop_number] - center_y} 0 " rpy="0 0 0" />
-          <parent link="${name}:room_center_link"/>
-          <child link="${name}:room_corner_${loop_number}_link"/>
-      </joint>
-      <link name="${name}:room_corner_${loop_number}_link" />
-      <xacro:if value="${(num_of_corners - 1) > loop_number}">
-        <xacro:corner_loop loop_number="${loop_number + 1}" />
-      </xacro:if>
-    </xacro:macro>
-    <!-- room call loop to create every corner -->
-    <xacro:corner_loop loop_number="0" />
   </xacro:macro>
 </robot>

Commit message: add room connections

File: suturo_resources/urdf/suturo_environment.urdf.xacro (robot description, xacro)
@@ -171,5 +171,6 @@
                          size_x="${data['rooms'][room_number]['size_x']}"
                          size_y="${data['rooms'][room_number]['size_y']}"
-                         color="${data['rooms'][room_number]['color']}">
+                         color="${data['rooms'][room_number]['color']}"
+						 connections="${data['rooms'][room_number]['connections']}">
       </xacro:suturo_room>
       <xacro:if value="${(number_of_rooms - 1) > room_number}">

File: suturo_resources/urdf/urdf_components/suturo_room.urdf.xacro (robot description, xacro)
@@ -2,5 +2,14 @@
 <!-- Rooms are for Knowledge Information only-->
 <robot name="suturo_room" xmlns:xacro="http://ros.org/wiki/xacro">
-  <xacro:macro name="suturo_room" params="name parent center_x center_y color size_x size_y">
+  <!-- The parent needs to be the room this belongs to, otherwise knowledge won't find it. -->
+  <xacro:macro name="suturo_room_connection" params="name parent center_x center_y">
+    <joint name="room_${name}:connection_joint" type="fixed">
+      <origin xyz="${center_x} ${center_y} 0 " rpy="0 0 0" />
+      <parent link="${parent}"/>
+      <child link="${name}:link"/>
+    </joint>
+    <link name="${name}:link"/>
+  </xacro:macro>
+  <xacro:macro name="suturo_room" params="name parent center_x center_y color size_x size_y connections">
     <joint name="world_${name}:room_joint" type="fixed">
         <origin xyz="${center_x} ${center_y} -0.01 " rpy="0 0 0" />
@@ -23,4 +32,19 @@
       </collision>
     </link>
+    <xacro:property name="number_of_connections" value="${connections['amount']}" />
+    <!--  ~~Rooms~~  -->
+    <xacro:macro name="room_connection_loop" params="room_connection_number">
+      <xacro:suturo_room_connection name="${connections[room_connection_number]['name']}:${connections[room_connection_number]['knowledge_role']}"
+									parent="${name}:room_center_link"
+									center_x="${connections[room_connection_number]['center_x']-center_x}"
+									center_y="${connections[room_connection_number]['center_y']-center_y}">
+      </xacro:suturo_room_connection>
+      <xacro:if value="${(number_of_connections - 1) > room_connection_number}">
+        <xacro:room_connection_loop room_connection_number="${room_connection_number + 1}" />
+      </xacro:if>
+    </xacro:macro>
+	<xacro:if value="${number_of_connections > 0}">
+      <xacro:room_connection_loop room_connection_number="0" />
+    </xacro:if>
   </xacro:macro>
 </robot>
