Commit message: add round_table in robocup semantic map

File: suturo_resources/urdf/suturo_environment.urdf.xacro (robot description, xacro)
@@ -16,4 +16,5 @@
     <!--  Include the files containing the macros -->
     <xacro:include filename="$(find suturo_resources)/urdf/urdf_components/suturo_table.urdf.xacro"/>
+    <xacro:include filename="$(find suturo_resources)/urdf/urdf_components/suturo_round_table.urdf.xacro"/>
     <xacro:include filename="$(find suturo_resources)/urdf/urdf_components/suturo_wall.urdf.xacro"/>
     <xacro:include filename="$(find suturo_resources)/urdf/urdf_components/suturo_shelf.urdf.xacro"/>
@@ -30,4 +31,5 @@
     <xacro:property name="number_of_simple_drawers" value="${data['simple_drawers']['amount']}" />
     <xacro:property name="number_of_tables" value="${data['tables']['amount']}" />
+    <xacro:property name="number_of_round_tables" value="${data['round_tables']['amount']}" />
     <xacro:property name="number_of_buckets" value="${data['buckets']['amount']}" />
     <xacro:property name="number_of_shelves" value="${data['shelves']['amount']}" />
@@ -50,4 +52,17 @@
         <xacro:if value="${(number_of_tables - 1) > table_number}">
             <xacro:table_loop table_number="${table_number + 1}" />
+        </xacro:if>
+    </xacro:macro>
+    <!--  ~~Round_tables~~  -->
+    <xacro:macro name="round_table_loop" params="round_table_number">
+        <xacro:suturo_round_table name="${data['round_tables'][round_table_number]['name']}:${data['tables'][round_table_number]['knowledge_role']}"
+                          parent="${data['round_tables'][round_table_number]['parent']}"
+                          radius="${data['round_tables'][round_table_number]['radius']}"
+                          length="${data['round_tables'][round_table_number]['length']}">
+            <origin xyz="${data['round_tables'][round_table_number]['x_pos']} ${data['round_tables'][round_table_number]['y_pos']} 0"
+                            rpy="0 0 ${data['round_tables'][round_table_number]['z_rot']}" />
+        </xacro:suturo_round_table>
+        <xacro:if value="${(number_of_round_tables - 1) > round_table_number}">
+            <xacro:round_table_loop round_table_number="${round_table_number + 1}" />
         </xacro:if>
     </xacro:macro>
@@ -218,4 +233,7 @@
         <xacro:table_loop table_number="0" />
     </xacro:if>
+    <xacro:if value="${number_of_round_tables > 0}">
+        <xacro:round_table_loop round_table_number="0" />
+    </xacro:if>
     <xacro:if value="${number_of_buckets > 0}">
         <xacro:bucket_loop bucket_number="0" />

Commit message: Fix: Dishwasher knowledge role link names and position

File: suturo_resources/urdf/suturo_environment.urdf.xacro (robot description, xacro)
@@ -75,5 +75,5 @@
         </xacro:suturo_dishwasher>
         <xacro:if value="${(number_of_dishwashers - 1) > dishwasher_number}">
-            <xacro:table_loop table_number="${dishwasher_number + 1}" />
+            <xacro:dishwasher_loop dishwasher_number="${dishwasher_number + 1}" />
         </xacro:if>
     </xacro:macro>

File: suturo_resources/urdf/urdf_components/suturo_dishwasher.urdf.xacro (robot description, xacro)
@@ -3,5 +3,5 @@
   <xacro:property name="pi" value="3.1415926535897931" />
   <xacro:macro name="suturo_dishwasher" params="name parent *origin">
-     <link name="${name}_main">
+     <link name="${name}:dishwasher_main">
       <xacro:sphere_inertia radius="0" mass="0"/>
       <visual>
@@ -18,5 +18,5 @@
       </collision>
     </link>
-    <link name="${name}_door">
+    <link name="${name}:dishwasher_door">
       <xacro:sphere_inertia radius="0" mass="0"/>
       <visual>
@@ -33,5 +33,5 @@
       </collision>
     </link>
-    <link name="${name}_door_handle">
+    <link name="${name}:dishwasher_door_handle">
       <xacro:sphere_inertia radius="0" mass="0"/>
       <visual>
@@ -51,15 +51,15 @@
     <xacro:if value="simulated"/>
     -->
-    <joint name="${name}_main_joint" type="fixed">
+    <joint name="${name}:dishwasher_main_joint" type="fixed">
       <xacro:insert_block name="origin" />
       <parent link="${parent}"/>
-      <child link="${name}_main"/>
+      <child link="${name}:dishwasher_main"/>
     </joint>
     <!--
     <xacro:if value="${simulated}">
-    <joint name="${name}_door_joint" type="revolute">
+    <joint name="${name}:dishwasher_door_joint" type="revolute">
       <origin xyz="0.27 0. -0.325" rpy="${-0.5*pi} 0 0" />
-      <parent link="${name}_main"/>
-      <child link="${name}_door"/>
+      <parent link="${name}:dishwasher_main"/>
+      <child link="${name}:dishwasher_door"/>
       <axis xyz="0 0 1"/>
        FIXME make closed position stable instead of forbidding opening...
@@ -71,8 +71,8 @@
     <xacro:unless value="${simulated}">
     -->
-    <joint name="${name}_door_joint" type="revolute">
+    <joint name="${name}:dishwasher_door_joint" type="revolute">
       <origin xyz="-0.27 0. -0.285" rpy="${-0.5*pi} 0 0" />
-      <parent link="${name}_main"/>
-      <child link="${name}_door"/>
+      <parent link="${name}:dishwasher_main"/>
+      <child link="${name}:dishwasher_door"/>
       <axis xyz="0 0 1"/>
       <!--
@@ -84,13 +84,13 @@
     </xacro:unless>
   -->
-    <joint name="${name}_door_handle_joint" type="fixed">
+    <joint name="${name}:dishwasher_door_handle_joint" type="fixed">
       <origin xyz="-0.065 -0.575 0.0" rpy="${pi/2} 0 0" />
-      <parent link="${name}_door"/>
-      <child link="${name}_door_handle"/>
-    </joint>
-    <xacro:dishwasher_tray name="${name}_tray" parent="${name}_main">
+      <parent link="${name}:dishwasher_door"/>
+      <child link="${name}:dishwasher_door_handle"/>
+    </joint>
+    <xacro:dishwasher_tray name="${name}:dishwasher_tray" parent="${name}:dishwasher_main">
       <origin xyz="-0.08 0 0.15"/>
     </xacro:dishwasher_tray>
-    <xacro:dishwasher_tray name="${name}_tray_2" parent="${name}_main">
+    <xacro:dishwasher_tray name="${name}:dishwasher_tray_2" parent="${name}:dishwasher_main">
       <origin xyz="-0.08 0 -0.15"/>
     </xacro:dishwasher_tray>
