Commit message: added both tables and changed orientation of shelf

File: suturo_resources/urdf/suturo_environment.urdf.xacro (robot description, xacro)
@@ -16,4 +16,5 @@
     <!--  Include the files containing the macros -->
     <xacro:include filename="$(find suturo_resources)/urdf/urdf_components/suturo_table.urdf.xacro" />
+    <xacro:include filename="$(find suturo_resources)/urdf/urdf_components/suturo_popcorn_table.urdf.xacro" />
     <xacro:include filename="$(find suturo_resources)/urdf/urdf_components/suturo_couch.urdf.xacro" />
     <xacro:include
@@ -39,4 +40,6 @@
     <xacro:property name="number_of_tables"
         value="${data.get('tables', dict(amount=0)).get('amount', 0)}" />
+    <xacro:property name="number_of_popcorn_tables"
+        value="${data.get('popcorn_tables', dict(amount=0)).get('amount', 0)}" />
     <xacro:property name="number_of_couches"
         value="${data.get('couch', dict(amount=0)).get('amount', 0)}" />
@@ -75,4 +78,20 @@
         </xacro:if>
     </xacro:macro>
+    <!--  ~~Popcorn_tables~~  -->
+    <xacro:macro name="popcorn_table_loop" params="popcorn_table_number">
+        <xacro:suturo_popcorn_table
+            name="${data['popcorn_tables'][popcorn_table_number]['name']}:${data['popcorn_tables'][popcorn_table_number]['knowledge_role']}"
+            parent="${data['popcorn_tables'][popcorn_table_number]['parent']}"
+            size_x="${data['popcorn_tables'][popcorn_table_number]['depth']}"
+            size_y="${data['popcorn_tables'][popcorn_table_number]['width']}"
+            size_z="${data['popcorn_tables'][popcorn_table_number]['height']}">
+            <origin
+                xyz="${data['popcorn_tables'][popcorn_table_number]['x_pos']} ${data['popcorn_tables'][popcorn_table_number]['y_pos']} 0"
+                rpy="0 0 ${data['popcorn_tables'][popcorn_table_number]['z_rot']}" />
+        </xacro:suturo_popcorn_table>
+        <xacro:if value="${(number_of_popcorn_tables - 1) > popcorn_table_number}">
+            <xacro:popcorn_table_loop popcorn_table_number="${popcorn_table_number + 1}" />
+        </xacro:if>
+    </xacro:macro>
       <!--  ~~Couches~~  -->
     <xacro:macro name="couch_loop" params="couch_number">
@@ -288,4 +307,7 @@
         <xacro:table_loop table_number="0" />
     </xacro:if>
+    <xacro:if value="${number_of_popcorn_tables > 0}">
+        <xacro:popcorn_table_loop popcorn_table_number="0" />
+    </xacro:if>
     <xacro:if value="${number_of_couches > 0}">
         <xacro:couch_loop couch_number="0" />

Commit message: changed dishwasher handle and added open door state to shelf

File: suturo_resources/urdf/suturo_environment.urdf.xacro (robot description, xacro)
@@ -125,4 +125,19 @@
         </xacro:if>
     </xacro:macro>
+         <!--<xacro:macro name="dishwasher_loop" params="dishwasher_number">
+        <xacro:suturo_dishwasher
+            name="${data['dishwashers'][dishwasher_number]['name']}:${data['dishwashers'][dishwasher_number]['knowledge_role']}"
+            parent="${data['dishwashers'][dishwasher_number]['parent']}"
+             size_x="${data['dishwashers'][dishwasher_number]['depth']}"
+            size_y="${data['dishwashers'][dishwasher_number]['width']}"
+            size_z="${data['dishwashers'][dishwasher_number]['height']}">
+            <origin
+                xyz="${data['dishwashers'][dishwasher_number]['x_pos']} ${data['dishwashers'][dishwasher_number]['y_pos']} 0.33475"
+                rpy="0 0 ${data['dishwashers'][dishwasher_number]['z_rot']}" />
+        </xacro:suturo_dishwasher>
+        <xacro:if value="${(number_of_dishwashers - 1) > dishwasher_number}">
+            <xacro:dishwasher_loop couch_number="${dishwasher_number + 1}" />
+        </xacro:if>
+    </xacro:macro> -->
     <!--  ~~Dishwashers~~  -->
     <xacro:macro name="dishwasher_loop" params="dishwasher_number">

File: suturo_resources/urdf/urdf_components/suturo_dishwasher.urdf.xacro (robot description, xacro)
@@ -6,13 +6,13 @@
       <xacro:sphere_inertia radius="0" mass="0"/>
       <visual>
-        <origin xyz="0 0 0" rpy="0 0 ${pi}" />
-        <geometry>
-          <mesh filename="package://iai_kitchen/meshes/misc/DishWasher.dae" scale="1.1 1.2 1"/>
-        </geometry>
-      </visual>
-      <collision>
-        <origin xyz="0 0 0" rpy="0 0 0" />
-        <geometry>
-          <mesh filename="package://iai_kitchen/meshes/misc/DishWasher.obj"  scale="1.1 1.2 1"/>
+        <origin xyz="0 0 0.148" rpy="0 0 ${pi}" />
+        <geometry>
+          <mesh filename="package://iai_kitchen/meshes/misc/DishWasher.dae" scale="1.1 1.2 1.1"/>
+        </geometry>
+      </visual>
+      <collision>
+        <origin xyz="0 0 0.148" rpy="0 0 0" />
+        <geometry>
+          <mesh filename="package://iai_kitchen/meshes/misc/DishWasher.obj"  scale="1.1 1.2 1.1"/>
         </geometry>
       </collision>
@@ -21,5 +21,5 @@
       <xacro:sphere_inertia radius="0" mass="0"/>
       <visual>
-        <origin xyz="0 0.055 0" rpy="${0.5*pi} 0 0" />
+        <origin xyz="0 -0.108 0" rpy="${0.5*pi} 0 0" />
         <geometry>
           <mesh filename="package://iai_kitchen/meshes/misc/DishWasherDoor.dae"/>
@@ -27,5 +27,5 @@
       </visual>
       <collision>
-        <origin xyz="0 0.055 0" rpy="${0.5*pi} 0 0" />
+        <origin xyz="0 -0.108 0" rpy="${0.5*pi} 0 0" />
         <geometry>
           <mesh filename="package://iai_kitchen/meshes/misc/DishWasherDoor.obj"/>
@@ -78,5 +78,5 @@
     -->
     <joint name="${name}:dishwasher_door_joint" type="revolute">
-      <origin xyz="-0.27 0. -0.285" rpy="${-0.5*pi} 0 0" />
+      <origin xyz="-0.27 0. -0.285" rpy="${-0.5*pi} 0 0" />   <!-- <origin xyz="-0.085 0. -0.13" rpy="${-0.5*pi} -1.57 0" /> -->
       <parent link="${name}:dishwasher_main"/>
       <child link="${name}:dishwasher_door"/>
@@ -91,5 +91,5 @@
   -->
     <joint name="${name}:dishwasher_door_handle_joint" type="fixed">
-      <origin xyz="-0.065 -0.575 0.0" rpy="${pi/2} 0 0" />
+      <origin xyz="-0.08 -0.728 0.0" rpy="${pi/2} 0 0" />
       <parent link="${name}:dishwasher_door"/>
       <child link="${name}:dishwasher_door_handle"/>

File: suturo_resources/urdf/urdf_components/suturo_shelf_openable.urdf.xacro (robot description, xacro)
@@ -75,4 +75,16 @@
       </xacro:suturo_shelf_left_door_openable>
     </xacro:if>
+    <xacro:if value="${door == 'both_open'}">
+       <xacro:suturo_shelf_right_door_openable name="${name}:shelf_door_right" parent="${name}:shelf_right_side"
+        wall_thickness="${wall_thickness}" size_y="${door_width}" size_z="${size_z}" shelf_x_size="${size_x}"
+       handle_from_bottom="${handle_from_bottom}" handle_from_side="${handle_from_side}" handle_height="${handle_height}" handle_width="${handle_width}" handle_depth="${handle_depth}">
+        <origin xyz="0 ${size_y} ${size_z/2}" rpy="0 0 0"/>
+       </xacro:suturo_shelf_right_door_openable>
+         <xacro:suturo_shelf_left_door_openable name="${name}:shelf_door_left" parent="${name}:shelf_left_side"
+          wall_thickness="${wall_thickness}" size_y="${door_width}" size_z="${size_z}" shelf_x_size="${size_x}"
+	  handle_from_bottom="${handle_from_bottom}" handle_from_side="${handle_from_side}" handle_height="${handle_height}" handle_width="${handle_width}" handle_depth="${handle_depth}">
+        <origin xyz="0 ${size_y} ${size_z/2}" rpy="0 0 0"/>
+      </xacro:suturo_shelf_left_door_openable>
+    </xacro:if>
   </xacro:macro>
   <!-- Creates a link with collision and visual box of given dimensions,
@@ -140,11 +152,22 @@
       <child link="${name}:handle"/>
     </joint>
-    <joint name="${name}:joint" type="revolute">
-      <origin xyz="${-shelf_x_size/2+wall_thickness/2} ${-wall_thickness} 0" rpy="0 0 0"/>
-      <axis xyz="0 0 1" />
-      <parent link="${parent}"/>
-      <child link="${name}"/>
-      <limit effort="30" velocity="1.0" lower="-1.7" upper="0.0" />
-    </joint>
+    <xacro:if value="${door == 'both_open'}">
+      <joint name="${name}:joint" type="revolute">
+        <origin xyz="${-shelf_x_size/2+wall_thickness/2} ${-wall_thickness} 0" rpy="0 0 -1.77"/>
+        <axis xyz="0 0 1" />
+        <parent link="${parent}"/>
+        <child link="${name}"/>
+        <limit effort="30" velocity="1.0" lower="-1.7" upper="0.0" />
+      </joint>
+    </xacro:if>
+    <xacro:if value="${door == 'both'}">
+      <joint name="${name}:joint" type="revolute">
+        <origin xyz="${-shelf_x_size/2+wall_thickness/2} ${-wall_thickness} 0" rpy="0 0 0"/>
+        <axis xyz="0 0 1" />
+        <parent link="${parent}"/>
+        <child link="${name}"/>
+        <limit effort="30" velocity="1.0" lower="-1.7" upper="0.0" />
+      </joint>
+    </xacro:if>
   </xacro:macro>
   <xacro:macro name="suturo_shelf_right_door_openable" params="name parent *origin wall_thickness size_y size_z shelf_x_size handle_from_bottom handle_from_side handle_height handle_width handle_depth">
@@ -186,11 +209,22 @@
       <child link="${name}:handle"/>
     </joint>
-    <joint name="${name}:joint" type="revolute">
-      <origin xyz="${-shelf_x_size/2+wall_thickness/2} ${wall_thickness} 0" rpy="0 0 0"/>
-      <axis xyz="0 0 1" />
-      <parent link="${parent}"/>
-      <child link="${name}"/>
-      <limit effort="30" velocity="1.0" lower="0.0" upper="1.7" />
-    </joint>
+    <xacro:if value="${door == 'both_open'}">
+      <joint name="${name}:joint" type="revolute">
+        <origin xyz="${-shelf_x_size/2+wall_thickness/2} ${wall_thickness} 0" rpy="0 0 1.77"/>
+        <axis xyz="0 0 1" />
+        <parent link="${parent}"/>
+        <child link="${name}"/>
+        <limit effort="30" velocity="1.0" lower="0.0" upper="1.7" />
+      </joint>
+    </xacro:if>
+    <xacro:if value="${door == 'both'}">
+      <joint name="${name}:joint" type="revolute">
+        <origin xyz="${-shelf_x_size/2+wall_thickness/2} ${wall_thickness} 0" rpy="0 0 0"/>
+        <axis xyz="0 0 1" />
+        <parent link="${parent}"/>
+        <child link="${name}"/>
+        <limit effort="30" velocity="1.0" lower="0.0" upper="1.7" />
+      </joint>
+    </xacro:if>
   </xacro:macro>
   <!-- <xacro:macro name="suturo_shelf_right_door_openable" params="name parent *origin size_x size_y size_z shelf_x_size"> -->

Commit message: kitchen added

File: suturo_resources/urdf/suturo_environment.urdf.xacro (robot description, xacro)
@@ -25,5 +25,5 @@
         filename="$(find suturo_resources)/urdf/urdf_components/suturo_shelf_openable.urdf.xacro" />
     <xacro:include filename="$(find suturo_resources)/urdf/urdf_components/suturo_door.urdf.xacro" />
-    <xacro:include filename="$(find suturo_resources)/urdf/urdf_components/suturo_room.urdf.xacro" />
+    <!-- <xacro:include filename="$(find suturo_resources)/urdf/urdf_components/suturo_room.urdf.xacro" />-->
     <xacro:include filename="$(find suturo_resources)/urdf/urdf_components/suturo_bucket.urdf.xacro" />
     <xacro:include filename="$(find suturo_resources)/urdf/urdf_components/suturo_path.urdf.xacro" />
@@ -32,5 +32,5 @@
         filename="$(find suturo_resources)/urdf/urdf_components/suturo_simple_drawer.urdf.xacro" />
     <xacro:include
-        filename="$(find suturo_resources)/urdf/urdf_components/suturo_dishwasher.urdf.xacro" />
+        filename="$(find suturo_resources)/urdf/urdf_components/suturo_kitchen.urdf.xacro" />
     <!-- general data -->
     <xacro:property name="number_of_drawers"
@@ -56,10 +56,10 @@
     <xacro:property name="number_of_doors"
         value="${data.get('doors', dict(amount=0)).get('amount', 0)}" />
-    <xacro:property name="number_of_rooms"
-        value="${data.get('rooms', dict(amount=0)).get('amount', 0)}" />
+    <!-- <xacro:property name="number_of_rooms"
+        value="${data.get('rooms', dict(amount=0)).get('amount', 0)}" /> -->
     <xacro:property name="number_of_paths"
         value="${data.get('paths', dict(amount=0)).get('amount', 0)}" />
-    <xacro:property name="number_of_dishwashers"
-        value="${data.get('dishwashers', dict(amount=0)).get('amount', 0)}" />
+    <xacro:property name="number_of_kitchens"
+        value="${data.get('kitchens', dict(amount=0)).get('amount', 0)}" />
     <!--  ~~Tables~~  -->
     <xacro:macro name="table_loop" params="table_number">
@@ -140,5 +140,5 @@
         </xacro:if>
     </xacro:macro> -->
-    <!--  ~~Dishwashers~~  -->
+    <!--  ~~Dishwashers~~
     <xacro:macro name="dishwasher_loop" params="dishwasher_number">
         <xacro:suturo_dishwasher
@@ -152,5 +152,5 @@
             <xacro:dishwasher_loop dishwasher_number="${dishwasher_number + 1}" />
         </xacro:if>
-    </xacro:macro>
+    </xacro:macro> -->
     <!--  ~~Bucket~~  -->
     <xacro:macro name="bucket_loop" params="bucket_number">
@@ -263,19 +263,13 @@
         </xacro:if>
     </xacro:macro>
-    <!--  ~~Rooms~~  -->
-    <xacro:macro name="room_loop" params="room_number">
-        <xacro:suturo_room
-            name="${data['rooms'][room_number]['name']}:${data['rooms'][room_number]['knowledge_role']}"
-            parent="urdf_offset"
-            center_x="${data['rooms'][room_number]['center_x']}"
-            center_y="${data['rooms'][room_number]['center_y']}"
-            size_x="${data['rooms'][room_number]['size_x']}"
-            size_y="${data['rooms'][room_number]['size_y']}"
-            color="${data['rooms'][room_number]['color']}"
-            connections="${data['rooms'][room_number]['connections']}">
-        </xacro:suturo_room>
-        <xacro:if value="${(number_of_rooms - 1) > room_number}">
-            <xacro:room_loop room_number="${room_number + 1}" />
-        </xacro:if>
+    <!--  ~~Kitchen~~  -->
+     <xacro:macro name="kitchen_loop" params="kitchen_number">
+        <xacro:suturo_kitchen
+            name="${data['kitchens'][kitchen_number]['name']}:${data['kitchens'][kitchen_number]['knowledge_role']}"
+            parent="${data['kitchens'][kitchen_number]['parent']}">
+            <origin
+                xyz="${data['kitchens'][kitchen_number]['x_pos']} ${data['kitchens'][kitchen_number]['y_pos']} 0"
+                rpy="0 0 ${data['kitchens'][kitchen_number]['z_rot']}" />
+        </xacro:suturo_kitchen>
     </xacro:macro>
     <!--  ~~Doors~~  -->
@@ -343,6 +337,9 @@
         <xacro:wall_loop wall_number="0" />
     </xacro:if>
-    <xacro:if value="${number_of_rooms > 0}">
+    <!--<xacro:if value="${number_of_rooms > 0}">
         <xacro:room_loop room_number="0" />
+    </xacro:if> -->
+    <xacro:if value="${number_of_kitchens > 0}">
+        <xacro:kitchen_loop kitchen_number="0" />
     </xacro:if>
     <xacro:if value="${number_of_doors > 0}">
@@ -352,7 +349,7 @@
         <xacro:path_loop path_number="0" />
     </xacro:if>
-    <xacro:if value="${number_of_dishwashers > 0}">
+    <!--<xacro:if value="${number_of_dishwashers > 0}">
         <xacro:dishwasher_loop dishwasher_number="0" />
-    </xacro:if>
+    </xacro:if> -->
     <link name="urdf_main" />
     <joint name="map_urdf_joint" type="fixed">

Commit message: added rooms for knowledge

File: suturo_resources/urdf/suturo_environment.urdf.xacro (robot description, xacro)
@@ -25,5 +25,5 @@
         filename="$(find suturo_resources)/urdf/urdf_components/suturo_shelf_openable.urdf.xacro" />
     <xacro:include filename="$(find suturo_resources)/urdf/urdf_components/suturo_door.urdf.xacro" />
-    <!-- <xacro:include filename="$(find suturo_resources)/urdf/urdf_components/suturo_room.urdf.xacro" />-->
+    <xacro:include filename="$(find suturo_resources)/urdf/urdf_components/suturo_room.urdf.xacro" />
     <xacro:include filename="$(find suturo_resources)/urdf/urdf_components/suturo_bucket.urdf.xacro" />
     <xacro:include filename="$(find suturo_resources)/urdf/urdf_components/suturo_path.urdf.xacro" />
@@ -56,6 +56,6 @@
     <xacro:property name="number_of_doors"
         value="${data.get('doors', dict(amount=0)).get('amount', 0)}" />
-    <!-- <xacro:property name="number_of_rooms"
-        value="${data.get('rooms', dict(amount=0)).get('amount', 0)}" /> -->
+    <xacro:property name="number_of_rooms"
+        value="${data.get('rooms', dict(amount=0)).get('amount', 0)}" />
     <xacro:property name="number_of_paths"
         value="${data.get('paths', dict(amount=0)).get('amount', 0)}" />
@@ -212,4 +212,20 @@
         </xacro:if>
     </xacro:macro>
+  <!--  ~~Rooms~~  -->
+    <xacro:macro name="room_loop" params="room_number">
+        <xacro:suturo_room
+            name="${data['rooms'][room_number]['name']}:${data['rooms'][room_number]['knowledge_role']}"
+            parent="urdf_offset"
+            center_x="${data['rooms'][room_number]['center_x']}"
+            center_y="${data['rooms'][room_number]['center_y']}"
+            size_x="${data['rooms'][room_number]['size_x']}"
+            size_y="${data['rooms'][room_number]['size_y']}"
+            color="${data['rooms'][room_number]['color']}"
+            connections="${data['rooms'][room_number]['connections']}">
+        </xacro:suturo_room>
+        <xacro:if value="${(number_of_rooms - 1) > room_number}">
+            <xacro:room_loop room_number="${room_number + 1}" />
+        </xacro:if>
+    </xacro:macro>
     <!--  ~~Drawers~~  -->
     <xacro:macro name="drawer_loop" params="drawer_number">
@@ -337,7 +353,7 @@
         <xacro:wall_loop wall_number="0" />
     </xacro:if>
-    <!--<xacro:if value="${number_of_rooms > 0}">
+    <xacro:if value="${number_of_rooms > 0}">
         <xacro:room_loop room_number="0" />
-    </xacro:if> -->
+    </xacro:if>
     <xacro:if value="${number_of_kitchens > 0}">
         <xacro:kitchen_loop kitchen_number="0" />

Commit message: - suturo.rviz Änderungen

File: suturo_resources/urdf/suturo_environment.urdf.xacro (robot description, xacro)
@@ -125,5 +125,5 @@
         </xacro:if>
     </xacro:macro>
-         <!--<xacro:macro name="dishwasher_loop" params="dishwasher_number">
+<!--<xacro:macro name="dishwasher_loop" params="dishwasher_number">
         <xacro:suturo_dishwasher
             name="${data['dishwashers'][dishwasher_number]['name']}:${data['dishwashers'][dishwasher_number]['knowledge_role']}"
@@ -263,6 +263,6 @@
         </xacro:if>
     </xacro:macro>
-    <!--  ~~Kitchen~~  -->
-     <xacro:macro name="kitchen_loop" params="kitchen_number">
+<!--  ~~Kitchen~~  -->
+    <xacro:macro name="kitchen_loop" params="kitchen_number">
         <xacro:suturo_kitchen
             name="${data['kitchens'][kitchen_number]['name']}:${data['kitchens'][kitchen_number]['knowledge_role']}"
@@ -339,5 +339,5 @@
     <!--<xacro:if value="${number_of_rooms > 0}">
         <xacro:room_loop room_number="0" />
-    </xacro:if> -->
+</xacro:if> -->
     <xacro:if value="${number_of_kitchens > 0}">
         <xacro:kitchen_loop kitchen_number="0" />
