Commit message: pushing all changes from backpack laptop

File: suturo_resources/urdf/suturo_environment.urdf.xacro (robot description, xacro)
@@ -302,5 +302,7 @@
             zrot="${data['doors'][door_number]['zrot']}"
             door_turn_limit_lower="${data['doors'][door_number]['door_turn_limit_lower']}"
-            door_turn_limit_max="${data['doors'][door_number]['door_turn_limit_max']}">
+            door_turn_limit_max="${data['doors'][door_number]['door_turn_limit_max']}"
+            handle_x="${data['doors'][door_number]['handle_x']}"
+            handle_z="${data['doors'][door_number]['handle_z']}">
         </xacro:suturo_door>
         <xacro:if value="${(number_of_doors - 1) > door_number}">

File: suturo_resources/urdf/urdf_components/suturo_dishwasher.urdf.xacro (robot description, xacro)
@@ -21,5 +21,5 @@
       <xacro:sphere_inertia radius="0" mass="0"/>
       <visual>
-        <origin xyz="0 -0.108 0" rpy="${0.5*pi} 0 0" />
+        <origin xyz="0 0.055 0" rpy="${0.5*pi} 0 0" />
         <geometry>
           <mesh filename="package://iai_kitchen/meshes/misc/DishWasherDoor.dae"/>
@@ -27,5 +27,5 @@
       </visual>
       <collision>
-        <origin xyz="0 -0.108 0" rpy="${0.5*pi} 0 0" />
+        <origin xyz="0 0.055 0" rpy="${0.5*pi} 0 0" />
         <geometry>
           <mesh filename="package://iai_kitchen/meshes/misc/DishWasherDoor.obj"/>
@@ -91,5 +91,5 @@
   -->
     <joint name="${name}:dishwasher_door_handle_joint" type="fixed">
-      <origin xyz="-0.08 -0.728 0.0" rpy="${pi/2} 0 0" />
+      <origin xyz="-0.065 -0.575 0.0" rpy="${pi/2} 0 0" />
       <parent link="${name}:dishwasher_door"/>
       <child link="${name}:dishwasher_door_handle"/>

File: suturo_resources/urdf/urdf_components/suturo_door.urdf.xacro (robot description, xacro)
@@ -11,5 +11,5 @@
   </material>
   <xacro:property name="half_pi" value="1.570796327" />
-  <xacro:macro name="suturo_door" params="name parent height width depth x y z zrot door_turn_limit_lower door_turn_limit_max">
+  <xacro:macro name="suturo_door" params="name parent height width depth x y z zrot door_turn_limit_lower door_turn_limit_max handle_x handle_z">
     <!-- LINKS -->
     <link name="${name}:door_center">
@@ -47,5 +47,5 @@
         <origin xyz="0.0 0.0 0.0" rpy="0 0 0" />
         <geometry name="handle_blue">
-          <cylinder radius="0.013" length="0.15" />
+          <cylinder radius="0.013" length="0.10" />
         </geometry>
       </visual>
@@ -53,5 +53,5 @@
         <origin xyz="0.0 0.0 0.0" rpy="0 0 0" />
         <geometry name="handle_collision_geom">
-          <cylinder radius="0.013" length="0.15" />
+          <cylinder radius="0.013" length="0.10" />
         </geometry>
       </collision>
@@ -107,15 +107,15 @@
       <axis xyz="0 0 1"/>
       <limit effort="1" lower="0" upper="${pi/5}" velocity="1"/>
-      <origin xyz="${0.92 * width} 0 0.05" rpy="${pi/2} 0 0" />
+      <origin xyz="${handle_x} 0 ${handle_z}" rpy="${pi/2} 0 0" />
       <parent link="${name}:door_center"/>
 	  <child link="${name}:door_handle_link"/>
     </joint>
     <joint name="${name}:door_handle_inside_joint" type="fixed">
-      <origin xyz="-0.075 0 0.075" rpy="0 0 ${pi/2}" />
+      <origin xyz="-0.06 0 0.035" rpy="0 0 ${pi/2}" />
       <parent link="${name}:door_handle_link"/>
       <child link="${name}:door_handle_inside"/>
     </joint>
     <joint name="${name}:door_handle_outside_joint" type="fixed">
-      <origin xyz="-0.075 0 -0.075" rpy="0 0 ${-pi/2}" />
+      <origin xyz="-0.075 0 -0.05" rpy="0 0 ${-pi/2}" />
       <parent link="${name}:door_handle_link"/>
       <child link="${name}:door_handle_outside"/>

File: suturo_resources/urdf/urdf_components/suturo_kitchen.urdf.xacro (robot description, xacro)
@@ -396,7 +396,7 @@
     <xacro:if value="simulated"/>
     -->
-  <joint name="sink_area_dish_washer_main_joint" type="revolute">
+  <joint name="sink_area_dish_washer_main_joint" type="fixed"> <!-- was revolute before, changed to fixed -->
     <axis xyz="1 0 0" />
-    <limit effort="300" lower="0" upper="0" velocity="10"/>
+    <!-- <limit effort="300" lower="0" upper="0" velocity="10"/> -->
     <origin rpy="0 0 0" xyz="0.01 0.1 0.044 "/>
     <parent link="sink_area"/>
@@ -404,10 +404,11 @@
   </joint>
   <joint name="sink_area_dish_washer_door_joint" type="revolute">
-    <origin rpy="-1.57079632679 0 0" xyz="0.27 0. -0.325"/>
+    <origin rpy="-1.57079632679 0.03 0" xyz="0.27 0. -0.325"/>
     <parent link="sink_area_dish_washer_main"/>
     <child link="sink_area_dish_washer_door"/>
     <axis xyz="0 0 1"/>
     <!-- FIXME make closed position stable instead of forbidding opening... -->
-    <limit effort="300" lower="0" upper="0" velocity="10"/>
+    <!-- TODO Fix Limits to be able to open dishwasher-->
+    <limit effort="300" lower="0.0" upper="1.57079632679" velocity="10"/>
   </joint>
   <joint name="sink_area_dish_washer_door_handle_joint" type="fixed">

Commit message: new dishwasher with table ontop

File: suturo_resources/urdf/suturo_environment.urdf.xacro (robot description, xacro)
@@ -31,4 +31,6 @@
     <xacro:include
         filename="$(find suturo_resources)/urdf/urdf_components/suturo_simple_drawer.urdf.xacro" />
+    <xacro:include
+        filename="$(find suturo_resources)/urdf/urdf_components/suturo_dishwasher.urdf.xacro" />
     <xacro:include
         filename="$(find suturo_resources)/urdf/urdf_components/suturo_kitchen.urdf.xacro" />
@@ -62,4 +64,6 @@
     <xacro:property name="number_of_kitchens"
         value="${data.get('kitchens', dict(amount=0)).get('amount', 0)}" />
+    <xacro:property name="number_of_dishwashers"
+        value="${data.get('dishwashers', dict(amount=0)).get('amount', 0)}" />
     <!--  ~~Tables~~  -->
     <xacro:macro name="table_loop" params="table_number">
@@ -140,5 +144,5 @@
         </xacro:if>
     </xacro:macro> -->
-    <!--  ~~Dishwashers~~
+    <!--  ~~Dishwashers~~ -->
     <xacro:macro name="dishwasher_loop" params="dishwasher_number">
         <xacro:suturo_dishwasher
@@ -146,5 +150,5 @@
             parent="${data['dishwashers'][dishwasher_number]['parent']}">
             <origin
-                xyz="${data['dishwashers'][dishwasher_number]['x_pos']} ${data['dishwashers'][dishwasher_number]['y_pos']} 0.33475"
+                xyz="${data['dishwashers'][dishwasher_number]['x_pos']} ${data['dishwashers'][dishwasher_number]['y_pos']} 0.0"
                 rpy="0 0 ${data['dishwashers'][dishwasher_number]['z_rot']}" />
         </xacro:suturo_dishwasher>
@@ -152,5 +156,5 @@
             <xacro:dishwasher_loop dishwasher_number="${dishwasher_number + 1}" />
         </xacro:if>
-    </xacro:macro> -->
+    </xacro:macro>
     <!--  ~~Bucket~~  -->
     <xacro:macro name="bucket_loop" params="bucket_number">
@@ -280,5 +284,5 @@
     </xacro:macro>
 <!--  ~~Kitchen~~  -->
-    <xacro:macro name="kitchen_loop" params="kitchen_number">
+     <xacro:macro name="kitchen_loop" params="kitchen_number">
         <xacro:suturo_kitchen
             name="${data['kitchens'][kitchen_number]['name']}:${data['kitchens'][kitchen_number]['knowledge_role']}"
@@ -367,7 +371,7 @@
         <xacro:path_loop path_number="0" />
     </xacro:if>
-    <!--<xacro:if value="${number_of_dishwashers > 0}">
+    <xacro:if value="${number_of_dishwashers > 0}">
         <xacro:dishwasher_loop dishwasher_number="0" />
-    </xacro:if> -->
+    </xacro:if>
     <link name="urdf_main" />
     <joint name="map_urdf_joint" type="fixed">

File: suturo_resources/urdf/urdf_components/suturo_dishwasher.urdf.xacro (robot description, xacro)
@@ -1,341 +1,145 @@
 <?xml version="1.0"?>
 <robot name="suturo_dishwasher" xmlns:xacro="http://ros.org/wiki/xacro">
-  <xacro:property name="pi" value="3.1415926535897931" />
+  <material name="dishwasher_table_color">
+	<color rgba="0.255 0.62 0.223 1"/>
+  </material>
   <xacro:macro name="suturo_dishwasher" params="name parent *origin">
-     <link name="${name}:dishwasher_main">
-      <xacro:sphere_inertia radius="0" mass="0"/>
+     <link name="dishwasher_main">
+       <inertial>
+         <origin rpy="0 0 0" xyz="0.0 0.0 0.0"/>
+         <mass value="1"/>
+         <inertia ixx="1" ixy="0.0" ixz="0.0" iyy="1" iyz="0.0" izz="1"/>
+       </inertial>
+    </link>
+    <joint name="dishwasher_main" type="fixed">
+	  <xacro:insert_block name="origin" />
+	  <parent link="${parent}"/>
+	  <child link="dishwasher_main"/>
+    </joint>
+    <joint name="dishwasher_main_joint" type="fixed">
+	  <xacro:insert_block name="origin" />
+	  <parent link="dishwasher_main"/>
+	  <child link="sink_area_dish_washer_main"/>
+    </joint>
+  <link name="sink_area_dish_washer_main">
+    <inertial>
+      <origin rpy="0 0 0" xyz="0.0 0.0 0.0"/>
+      <mass value="1"/>
+      <inertia ixx="1" ixy="0.0" ixz="0.0" iyy="1" iyz="0.0" izz="1"/>
+    </inertial>
+    <visual>
+      <origin rpy="0 0 0" xyz="0 0 0"/>
+      <geometry>
+        <mesh filename="package://iai_kitchen/meshes/misc/DishWasher.obj"/>
+      </geometry>
+    </visual>
+    <collision>
+      <origin rpy="0 0 0" xyz="0 0 0"/>
+      <geometry>
+        <mesh filename="package://iai_kitchen/meshes/misc/DishWasher.obj"/>
+      </geometry>
+    </collision>
+  </link>
+  <link name="sink_area_dish_washer_door">
+    <inertial>
+      <origin rpy="0 0 0" xyz="0.0 0.0 0.0"/>
+      <mass value="1"/>
+      <inertia ixx="1" ixy="0.0" ixz="0.0" iyy="1" iyz="0.0" izz="1"/>
+    </inertial>
+    <visual>
+      <origin rpy="1.57079632679 0 0" xyz="0 0 0"/>
+      <geometry>
+        <mesh filename="package://iai_kitchen/meshes/misc/DishWasherDoor.obj"/>
+      </geometry>
+    </visual>
+    <collision>
+      <origin rpy="1.57079632679 0 0" xyz="0 0 0"/>
+      <geometry>
+        <mesh filename="package://iai_kitchen/meshes/misc/DishWasherDoor.obj"/>
+      </geometry>
+    </collision>
+  </link>
+  <link name="sink_area_dish_washer_door_handle">
+    <inertial>
+      <origin rpy="0 0 0" xyz="0.0 0.0 0.0"/>
+      <mass value="1"/>
+      <inertia ixx="1" ixy="0.0" ixz="0.0" iyy="1" iyz="0.0" izz="1"/>
+    </inertial>
+    <visual>
+      <origin rpy="0 0 0" xyz="0 0 0"/>
+      <geometry>
+        <mesh filename="package://iai_kitchen/meshes/handles/Handle60.obj"/>
+      </geometry>
+    </visual>
+    <collision>
+      <origin rpy="0 0 0" xyz="0 0 0"/>
+      <geometry>
+        <mesh filename="package://iai_kitchen/meshes/handles/Handle60.obj"/>
+      </geometry>
+    </collision>
+  </link>
+  <link name="dishwasher_tab"/>
+  <link name="dishwasher_table:d_table:table_origin"/>
+  <link name="dishwasher_table:d_table:table_front_edge_center"/>
+  <link name="dishwasher_table:d_table:table_center">
       <visual>
-        <origin xyz="0 0 0.148" rpy="0 0 ${pi}" />
+        <material name="dishwasher_table_color"/>
+        <origin xyz="0 0 0" rpy="0 0 0" />
         <geometry>
-          <mesh filename="package://iai_kitchen/meshes/misc/DishWasher.dae" scale="1.1 1.2 1.1"/>
+          <box size="0.6 0.6 0.02" />
         </geometry>
       </visual>
       <collision>
-        <origin xyz="0 0 0.148" rpy="0 0 0" />
+        <origin xyz="0 0 0" rpy="0 0 0" />
         <geometry>
-          <mesh filename="package://iai_kitchen/meshes/misc/DishWasher.obj"  scale="1.1 1.2 1.1"/>
+          <box size="0.6 0.6 0.02" />
         </geometry>
       </collision>
-    </link>
-    <link name="${name}:dishwasher_door">
-      <xacro:sphere_inertia radius="0" mass="0"/>
-      <visual>
-        <origin xyz="0 0.055 0" rpy="${0.5*pi} 0 0" />
-        <geometry>
-          <mesh filename="package://iai_kitchen/meshes/misc/DishWasherDoor.dae"/>
-        </geometry>
-      </visual>
-      <collision>
-        <origin xyz="0 0.055 0" rpy="${0.5*pi} 0 0" />
-        <geometry>
-          <mesh filename="package://iai_kitchen/meshes/misc/DishWasherDoor.obj"/>
-        </geometry>
-      </collision>
-    </link>
-    <link name="${name}:dishwasher_door_handle">
-      <xacro:sphere_inertia radius="0" mass="0"/>
-      <visual>
-        <origin xyz="0 0 0" rpy="0 ${pi} 0" />
-        <geometry>
-          <mesh filename="package://iai_kitchen/meshes/handles/Handle60.dae"/>
-        </geometry>
-      </visual>
-      <collision>
-        <origin xyz="0 0 0" rpy="0 ${pi} 0" />
-        <geometry>
-          <mesh filename="package://iai_kitchen/meshes/handles/Handle60.obj"/>
-        </geometry>
-      </collision>
-    </link>
-	<link name="${name}:dishwasher_tab"/>
+  </link>
 	<!--
     <xacro:if value="simulated"/>
     -->
-	<joint name="${name}:dishwasher_tab_joint" type="fixed">
-	  <origin xyz="0.18 -0.33 0.1775" rpy="0 0 0" />
-	  <parent link="${name}:dishwasher_door"/>
-      <child link="${name}:dishwasher_tab"/>
+	<joint name="dishwasher_tab_joint" type="fixed">
+	  <origin xyz="-0.1 0.1 0.15" rpy="0 0 0" />
+	  <parent link="sink_area_dish_washer_door_handle"/>
+      <child link="dishwasher_tab"/>
 	</joint>
-    <joint name="${name}:dishwasher_main_joint" type="fixed">
-      <xacro:insert_block name="origin" />
-      <parent link="${parent}"/>
-      <child link="${name}:dishwasher_main"/>
-    </joint>
-    <!--
-    <xacro:if value="${simulated}">
-    <joint name="${name}:dishwasher_door_joint" type="revolute">
-      <origin xyz="0.27 0. -0.325" rpy="${-0.5*pi} 0 0" />
-      <parent link="${name}:dishwasher_main"/>
-      <child link="${name}:dishwasher_door"/>
-      <axis xyz="0 0 1"/>
-       FIXME make closed position stable instead of forbidding opening...
-      <limit lower="0" upper="0" effort="300" velocity="10"/>
-    </joint>
-    </xacro:if>
-    -->
-    <!--
-    <xacro:unless value="${simulated}">
-    -->
-    <joint name="${name}:dishwasher_door_joint" type="revolute">
-      <origin xyz="-0.27 0. -0.285" rpy="${-0.5*pi} 0 0" />   <!-- <origin xyz="-0.085 0. -0.13" rpy="${-0.5*pi} -1.57 0" /> -->
-      <parent link="${name}:dishwasher_main"/>
-      <child link="${name}:dishwasher_door"/>
-      <axis xyz="0 0 1"/>
-      <!--
-      <limit lower="0" upper="${0.5*pi}" effort="300" velocity="10"/>
-      -->
-      <limit lower="${-0.5*pi}" upper="0" effort="300" velocity="10"/>
-    </joint>
-    <!--
-    </xacro:unless>
-  -->
-    <joint name="${name}:dishwasher_door_handle_joint" type="fixed">
-      <origin xyz="-0.065 -0.575 0.0" rpy="${pi/2} 0 0" />
-      <parent link="${name}:dishwasher_door"/>
-      <child link="${name}:dishwasher_door_handle"/>
-    </joint>
-    <xacro:dishwasher_tray name="${name}:dishwasher_tray" parent="${name}:dishwasher_main">
-      <origin xyz="-0.08 0 0.26"/>
-    </xacro:dishwasher_tray>
-    <xacro:dishwasher_tray name="${name}:dishwasher_tray_2" parent="${name}:dishwasher_main">
-      <origin xyz="-0.08 0 -0.07"/>
-    </xacro:dishwasher_tray>
-  </xacro:macro>
-  <xacro:macro name="dishwasher_tray" params="name parent *origin">
-    <joint name="${name}_main" type="prismatic">
-      <xacro:insert_block name="origin"/>
-      <parent link="${parent}"/>
-      <child link="${name}_bottom"/>
-      <axis xyz="1 0 0"/>
-      <limit lower="-0.33" upper="0" effort="300" velocity="10"/>
-    </joint>
-    <link name="${name}_bottom">
-      <visual>
-        <geometry>
-          <box size="0.32 0.5 0.05"/>
-        </geometry>
-      </visual>
-      <collision>
-        <geometry>
-          <box size="0.32 0.5 0.05"/>
-        </geometry>
-      </collision>
-    </link>
-    <link name="${name}_left_side">
-      <visual>
-        <geometry>
-          <box size="0.32 0.005 0.17"/>
-        </geometry>
-      </visual>
-      <collision>
-        <geometry>
-          <box size="0.32 0.005 0.17"/>
-        </geometry>
-      </collision>
-    </link>
-    <link name="${name}_right_side">
-      <visual>
-        <geometry>
-          <box size="0.32 0.005 0.17"/>
-        </geometry>
-      </visual>
-      <collision>
-        <geometry>
-          <box size="0.32 0.005 0.17"/>
-        </geometry>
-      </collision>
-    </link>
-    <link name="${name}_back_side">
-      <visual>
-        <geometry>
-          <box size="0.005 0.5 0.17"/>
-        </geometry>
-      </visual>
-      <collision>
-        <geometry>
-          <box size="0.005 0.5 0.17"/>
-        </geometry>
-      </collision>
-    </link>
-    <link name="${name}_front_side">
-      <visual>
-        <geometry>
-          <box size="0.005 0.5 0.17"/>
-        </geometry>
-      </visual>
-      <collision>
-        <geometry>
-          <box size="0.005 0.5 0.17"/>
-        </geometry>
-      </collision>
-    </link>
-    <joint name="${name}_bottom_left" type="fixed">
-      <origin xyz="-0.0 -0.25 0.075"/>
-      <child link="${name}_left_side" />
-      <parent link="${name}_bottom"/>
-    </joint>
-    <joint name="${name}_bottom_right" type="fixed">
-      <origin xyz="-0.0 0.25 0.075"/>
-      <child link="${name}_right_side" />
-      <parent link="${name}_bottom"/>
-    </joint>
-    <joint name="${name}_bottom_back" type="fixed">
-      <origin xyz="0.16 0 0.075"/>
-      <child link="${name}_back_side" />
-      <parent link="${name}_bottom"/>
-    </joint>
-    <joint name="${name}_bottom_front" type="fixed">
-      <origin xyz="-0.16 0 0.075" rpy="0 0 0"/>
-      <child link="${name}_front_side" />
-      <parent link="${name}_bottom"/>
-    </joint>
-    <xacro:tray_handle name="${name}_handle" parent="${name}_front_side">
-      <origin xyz="-0.03 -0.1 -0.02"/>
-    </xacro:tray_handle>
-  </xacro:macro>
-    <xacro:macro name="dishwasher_tray_2" params="name parent *origin">
-    <joint name="${name}_main_2" type="prismatic">
-      <xacro:insert_block name="origin"/>
-      <parent link="${parent}"/>
-      <child link="${name}_bottom_2"/>
-      <axis xyz="1 0 0"/>
-      <limit lower="-0.33" upper="0" effort="300" velocity="10"/>
-    </joint>
-    <link name="${name}_bottom_2">
-      <visual>
-        <geometry>
-          <box size="0.32 0.5 0.05"/>
-        </geometry>
-      </visual>
-      <collision>
-        <geometry>
-          <box size="0.32 0.5 0.05"/>
-        </geometry>
-      </collision>
-    </link>
-    <link name="${name}_left_side_2">
-      <visual>
-        <geometry>
-          <box size="0.32 0.005 0.17"/>
-        </geometry>
-      </visual>
-      <collision>
-        <geometry>
-          <box size="0.32 0.005 0.17"/>
-        </geometry>
-      </collision>
-    </link>
-    <link name="${name}_right_side_2">
-      <visual>
-        <geometry>
-          <box size="0.32 0.005 0.17"/>
-        </geometry>
-      </visual>
-      <collision>
-        <geometry>
-          <box size="0.32 0.005 0.17"/>
-        </geometry>
-      </collision>
-    </link>
-    <link name="${name}_back_side_2">
-      <visual>
-        <geometry>
-          <box size="0.005 0.5 0.17"/>
-        </geometry>
-      </visual>
-      <collision>
-        <geometry>
-          <box size="0.005 0.5 0.17"/>
-        </geometry>
-      </collision>
-    </link>
-    <link name="${name}_front_side_2">
-      <visual>
-        <geometry>
-          <box size="0.005 0.5 0.17"/>
-        </geometry>
-      </visual>
-      <collision>
-        <geometry>
-          <box size="0.005 0.5 0.17"/>
-        </geometry>
-      </collision>
-    </link>
-    <joint name="${name}_bottom_left_2" type="fixed">
-      <origin xyz="-0.0 -0.25 -0.075"/>
-      <child link="${name}_left_side_2" />
-      <parent link="${name}_bottom_2"/>
-    </joint>
-    <joint name="${name}_bottom_right_2" type="fixed">
-      <origin xyz="-0.0 0.25 -0.075"/>
-      <child link="${name}_right_side_2" />
-      <parent link="${name}_bottom_2"/>
-    </joint>
-    <joint name="${name}_bottom_back" type="fixed">
-      <origin xyz="0.16 0 -0.075"/>
-      <child link="${name}_back_side_2" />
-      <parent link="${name}_bottom_2"/>
-    </joint>
-    <joint name="${name}_bottom_front" type="fixed">
-      <origin xyz="-0.16 0 -0.075" rpy="0 0 0"/>
-      <child link="${name}_front_side_2" />
-      <parent link="${name}_bottom_2"/>
-    </joint>
-    <xacro:tray_handle name="${name}_handle_2" parent="${name}_front_side_2">
-      <origin xyz="-0.03 -0.1 -0.02"/>
-    </xacro:tray_handle>
-  </xacro:macro>
-  <xacro:macro name="tray_handle" params="name parent *origin">
-    <joint name="${name}_joint" type="fixed">
-      <xacro:insert_block name="origin"/>
-      <child link="${name}_front_side" />
-      <parent link="${parent}"/>
-    </joint>
-    <link name="${name}_left_side">
-      <visual>
-        <geometry>
-          <box size="0.03 0.01 0.01"/>
-        </geometry>
-      </visual>
-      <collision>
-        <geometry>
-          <box size="0.03 0.01 0.01"/>
-        </geometry>
-      </collision>
-    </link>
-    <link name="${name}_right_side">
-      <visual>
-        <geometry>
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