Commit message: added new chair and first step of an new shelve

File: suturo_resources/urdf/suturo_environment.urdf.xacro (robot description, xacro)
@@ -35,4 +35,8 @@
     <xacro:include
         filename="$(find suturo_resources)/urdf/urdf_components/suturo_kitchen.urdf.xacro" />
+    <xacro:include
+        filename="$(find suturo_resources)/urdf/urdf_components/suturo_chair.urdf.xacro" />
+    <xacro:include
+        filename="$(find suturo_resources)/urdf/urdf_components/suturo_shelf_hohc.urdf.xacro" />
     <!-- general data -->
     <xacro:property name="number_of_drawers"
@@ -66,4 +70,8 @@
     <xacro:property name="number_of_dishwashers"
         value="${data.get('dishwashers', dict(amount=0)).get('amount', 0)}" />
+    <xacro:property name="number_of_chairs"
+        value="${data.get('chairs', dict(amount=0)).get('amount', 0)}" />
+    <xacro:property name="number_of_shelves_hohc"
+        value="${data.get('shelves_hohc', dict(amount=0)).get('amount', 0)}" />
     <!--  ~~Tables~~  -->
     <xacro:macro name="table_loop" params="table_number">
@@ -214,4 +222,29 @@
         <xacro:if value="${(number_of_shelves_openable - 1) > shelf_openable_number}">
             <xacro:shelf_openable_loop shelf_openable_number="${shelf_openable_number + 1}" />
+        </xacro:if>
+    </xacro:macro>
+    <!--  ~~Shelves_hohc~~  -->
+    <xacro:macro name="shelf_hohc_loop" params="shelf_hohc_number">
+        <xacro:suturo_shelf_hohc
+            name="${data['shelves_hohc'][shelf_hohc_number]['name']}:${data['shelves_hohc'][shelf_hohc_number]['knowledge_role']}"
+            parent="${data['shelves_hohc'][shelf_hohc_number]['parent']}"
+            size_x="${data['shelves_hohc'][shelf_hohc_number]['depth']}"
+            size_y="${data['shelves_hohc'][shelf_hohc_number]['width']}"
+            size_z="${data['shelves_hohc'][shelf_hohc_number]['height']}"
+            floors_height="${data['shelves_hohc'][shelf_hohc_number]['floors_height']}"
+            number_of_floors="${data['shelves_hohc'][shelf_hohc_number]['number_of_floors']}"
+            door="${data['shelves_hohc'][shelf_hohc_number]['door']}"
+            wall_thickness="${data['shelves_hohc'][shelf_hohc_number]['wall_thickness']}"
+            handle_from_bottom="${data['shelves_hohc'][shelf_hohc_number]['handle_from_bottom']}"
+            handle_from_side="${data['shelves_hohc'][shelf_hohc_number]['handle_from_side']}"
+            handle_height="${data['shelves_hohc'][shelf_hohc_number]['handle_height']}"
+            handle_width="${data['shelves_hohc'][shelf_hohc_number]['handle_width']}"
+            handle_depth="${data['shelves_hohc'][shelf_hohc_number]['handle_depth']}">
+            <origin
+                xyz="${data['shelves_hohc'][shelf_hohc_number]['x_pos']} ${data['shelves_hohc'][shelf_hohc_number]['y_pos']} 0"
+                rpy="0 0 ${data['shelves_hohc'][shelf_hohc_number]['z_rot']}" />
+        </xacro:suturo_shelf_hohc>
+        <xacro:if value="${(number_of_shelves_hohc - 1) > shelf_hohc_number}">
+            <xacro:shelf_hohc_loop shelf_hohc_number="${shelf_hohc_number + 1}" />
         </xacro:if>
     </xacro:macro>
@@ -314,4 +347,20 @@
         </xacro:if>
     </xacro:macro>
+        <!--  ~~Chairs~~  -->
+    <xacro:macro name="chair_loop" params="chair_number">
+        <xacro:suturo_chair
+            name="${data['chairs'][chair_number]['name']}:${data['chairs'][chair_number]['knowledge_role']}"
+            parent="${data['chairs'][chair_number]['parent']}"
+            size_x="${data['chairs'][chair_number]['depth']}"
+            size_y="${data['chairs'][chair_number]['width']}"
+            size_z="${data['chairs'][chair_number]['height']}">
+            <origin
+                xyz="${data['chairs'][chair_number]['x_pos']} ${data['chairs'][chair_number]['y_pos']} 0"
+                rpy="0 0 ${data['chairs'][chair_number]['z_rot']}" />
+        </xacro:suturo_chair>
+        <xacro:if value="${(number_of_chairs - 1) > chair_number}">
+            <xacro:chair_loop chair_number="${chair_number + 1}" />
+        </xacro:if>
+    </xacro:macro>
     <!--  ~~Paths~~  -->
     <xacro:macro name="path_loop" params="path_number">
@@ -374,4 +423,10 @@
         <xacro:dishwasher_loop dishwasher_number="0" />
     </xacro:if>
+        <xacro:if value="${number_of_chairs > 0}">
+        <xacro:chair_loop chair_number="0" />
+    </xacro:if>
+    <xacro:if value="${number_of_shelves_hohc > 0}">
+        <xacro:shelf_hohc_loop shelf_hohc_number="0" />
+    </xacro:if>
     <link name="urdf_main" />
     <joint name="map_urdf_joint" type="fixed">

Commit message: new shelf

File: suturo_resources/urdf/suturo_environment.urdf.xacro (robot description, xacro)
@@ -235,4 +235,6 @@
             number_of_floors="${data['shelves_hohc'][shelf_hohc_number]['number_of_floors']}"
             door="${data['shelves_hohc'][shelf_hohc_number]['door']}"
+            door_height="${data['shelves_hohc'][shelf_hohc_number]['door_height']}"
+            door_length="${data['shelves_hohc'][shelf_hohc_number]['door_length']}"
             wall_thickness="${data['shelves_hohc'][shelf_hohc_number]['wall_thickness']}"
             handle_from_bottom="${data['shelves_hohc'][shelf_hohc_number]['handle_from_bottom']}"

File: suturo_resources/urdf/urdf_components/suturo_shelf_hohc.urdf.xacro (robot description, xacro)
@@ -4,5 +4,5 @@
     <color rgba="0.74 0.25 0.25 1"/>
   </material>
-  <xacro:macro name="suturo_shelf_hohc" params="name parent *origin size_x size_y size_z floors_height number_of_floors door wall_thickness handle_from_bottom handle_from_side handle_height handle_width handle_depth">
+  <xacro:macro name="suturo_shelf_hohc" params="name parent *origin size_x size_y size_z floors_height number_of_floors door door_height door_length wall_thickness handle_from_bottom handle_from_side handle_height handle_width handle_depth">
     <!-- General conveinience links -->
     <link name="${name}:shelf_origin"/>
@@ -51,5 +51,5 @@
     <xacro:if value="${door == 'left'}">
       <xacro:suturo_shelf_left_door_openable name="${name}:shelf_door_left" parent="${name}:shelf_left_side"
-       wall_thickness="${wall_thickness}" size_y="${door_width}" size_z="${size_z}" shelf_x_size="${size_x}"
+       wall_thickness="${wall_thickness}" size_y="${door_width}" size_z="${door_length}" shelf_x_size="${size_x}"
        handle_from_bottom="${handle_from_bottom}" handle_from_side="${handle_from_side}" handle_height="${handle_height}" handle_width="${handle_width}" handle_depth="${handle_depth}">
         <origin xyz="0 ${size_y*0.75} ${size_z/2}" rpy="0 0 0"/>
@@ -58,31 +58,31 @@
     <xacro:if value="${door == 'right'}">
       <xacro:suturo_shelf_right_door_openable name="${name}:shelf_door_right" parent="${name}:shelf_right_side"
-        wall_thickness="${wall_thickness}" size_y="${door_width}" size_z="${size_z}" shelf_x_size="${size_x}"
-       handle_from_bottom="${handle_from_bottom}" handle_from_side="${handle_from_side}" handle_height="${handle_height}" handle_width="${handle_width}" handle_depth="${handle_depth}">
-        <origin xyz="0 ${size_y*0.75} ${size_z/2}" rpy="0 0 0"/>
+        wall_thickness="${wall_thickness}" size_y="${door_width}" size_z="${door_length}" shelf_x_size="${size_x}"
+       handle_from_bottom="${handle_from_bottom}" handle_from_side="${handle_from_side}" handle_height="${handle_height}" handle_width="${handle_width}" handle_depth="${handle_depth}">
+        <origin xyz="0 ${size_y*0.75} ${door_length/2}" rpy="0 0 0"/>
       </xacro:suturo_shelf_right_door_openable>
     </xacro:if>
     <xacro:if value="${door == 'both'}">
        <xacro:suturo_shelf_right_door_openable name="${name}:shelf_door_right" parent="${name}:shelf_right_side"
-        wall_thickness="${wall_thickness}" size_y="${door_width}" size_z="${size_z}" shelf_x_size="${size_x}"
-       handle_from_bottom="${handle_from_bottom}" handle_from_side="${handle_from_side}" handle_height="${handle_height}" handle_width="${handle_width}" handle_depth="${handle_depth}">
-        <origin xyz="0 ${size_y} ${size_z/2}" rpy="0 0 0"/>
+        wall_thickness="${wall_thickness}" size_y="${door_width}" size_z="${door_length}" shelf_x_size="${size_x}"
+       handle_from_bottom="${handle_from_bottom}" handle_from_side="${handle_from_side}" handle_height="${handle_height}" handle_width="${handle_width}" handle_depth="${handle_depth}">
+        <origin xyz="0 ${size_y} ${door_length/2}" rpy="0 0 0"/>
        </xacro:suturo_shelf_right_door_openable>
          <xacro:suturo_shelf_left_door_openable name="${name}:shelf_door_left" parent="${name}:shelf_left_side"
-          wall_thickness="${wall_thickness}" size_y="${door_width}" size_z="${size_z}" shelf_x_size="${size_x}"
+          wall_thickness="${wall_thickness}" door_height="${door_height}" size_y="${door_width}" size_z="${door_length}" shelf_x_size="${size_x}"
 	  handle_from_bottom="${handle_from_bottom}" handle_from_side="${handle_from_side}" handle_height="${handle_height}" handle_width="${handle_width}" handle_depth="${handle_depth}">
-        <origin xyz="0 ${size_y} ${size_z/2}" rpy="0 0 0"/>
+        <origin xyz="0 ${size_y} ${door_length/2}" rpy="0 0 0"/>
       </xacro:suturo_shelf_left_door_openable>
     </xacro:if>
     <xacro:if value="${door == 'both_open'}">
        <xacro:suturo_shelf_right_door_openable name="${name}:shelf_door_right" parent="${name}:shelf_right_side"
-        wall_thickness="${wall_thickness}" size_y="${door_width}" size_z="${size_z}" shelf_x_size="${size_x}"
-       handle_from_bottom="${handle_from_bottom}" handle_from_side="${handle_from_side}" handle_height="${handle_height}" handle_width="${handle_width}" handle_depth="${handle_depth}">
-        <origin xyz="0 ${size_y} ${size_z/2}" rpy="0 0 0"/>
+        wall_thickness="${wall_thickness}" door_height="${door_height}" size_y="${door_width}" size_z="${door_length}" shelf_x_size="${size_x}"
+       handle_from_bottom="${handle_from_bottom}" handle_from_side="${handle_from_side}" handle_height="${handle_height}" handle_width="${handle_width}" handle_depth="${handle_depth}">
+        <origin xyz="0 ${size_y} ${door_length/2}" rpy="0 0 0"/>
        </xacro:suturo_shelf_right_door_openable>
          <xacro:suturo_shelf_left_door_openable name="${name}:shelf_door_left" parent="${name}:shelf_left_side"
-          wall_thickness="${wall_thickness}" size_y="${door_width}" size_z="${size_z}" shelf_x_size="${size_x}"
+          wall_thickness="${wall_thickness}" door_height="${door_height}" size_y="${door_width}" size_z="${door_length}" shelf_x_size="${size_x}"
 	  handle_from_bottom="${handle_from_bottom}" handle_from_side="${handle_from_side}" handle_height="${handle_height}" handle_width="${handle_width}" handle_depth="${handle_depth}">
-        <origin xyz="0 ${size_y} ${size_z/2}" rpy="0 0 0"/>
+        <origin xyz="0 ${size_y} ${door_length/2}" rpy="0 0 0"/>
       </xacro:suturo_shelf_left_door_openable>
     </xacro:if>
@@ -114,5 +114,5 @@
     </joint>
   </xacro:macro>
-  <xacro:macro name="suturo_shelf_left_door_openable" params="name parent *origin wall_thickness size_y size_z shelf_x_size handle_from_bottom handle_from_side handle_height handle_width handle_depth">
+  <xacro:macro name="suturo_shelf_left_door_openable" params="name parent *origin wall_thickness door_height size_y size_z shelf_x_size handle_from_bottom handle_from_side handle_height handle_width handle_depth">
     <xacro:property name="size_x" value="${wall_thickness}"/>
     <link name="${name}">
@@ -154,5 +154,5 @@
     <xacro:if value="${door == 'both_open'}">
       <joint name="${name}:joint" type="revolute">
-        <origin xyz="${-shelf_x_size/2+wall_thickness/2} ${-wall_thickness} 0" rpy="0 0 -1.77"/>
+        <origin xyz="${-shelf_x_size/2+wall_thickness/2} ${-wall_thickness} ${door_height}" rpy="0 0 -1.77"/>
         <axis xyz="0 0 1" />
         <parent link="${parent}"/>
@@ -163,5 +163,5 @@
     <xacro:if value="${door == 'both'}">
       <joint name="${name}:joint" type="revolute">
-        <origin xyz="${-shelf_x_size/2+wall_thickness/2} ${-wall_thickness} 0" rpy="0 0 0"/>
+        <origin xyz="${-shelf_x_size/2+wall_thickness/2} ${-wall_thickness} ${door_height}" rpy="0 0 0"/>
         <axis xyz="0 0 1" />
         <parent link="${parent}"/>
@@ -171,5 +171,5 @@
     </xacro:if>
   </xacro:macro>
-  <xacro:macro name="suturo_shelf_right_door_openable" params="name parent *origin wall_thickness size_y size_z shelf_x_size handle_from_bottom handle_from_side handle_height handle_width handle_depth">
+  <xacro:macro name="suturo_shelf_right_door_openable" params="name parent *origin wall_thickness door_height size_y size_z shelf_x_size handle_from_bottom handle_from_side handle_height handle_width handle_depth">
     <xacro:property name="size_x" value="${wall_thickness}"/>
     <link name="${name}">
@@ -211,5 +211,5 @@
     <xacro:if value="${door == 'both_open'}">
       <joint name="${name}:joint" type="revolute">
-        <origin xyz="${-shelf_x_size/2+wall_thickness/2} ${wall_thickness} 0" rpy="0 0 1.77"/>
+        <origin xyz="${-shelf_x_size/2+wall_thickness/2} ${wall_thickness} ${door_height}" rpy="0 0 1.77"/>
         <axis xyz="0 0 1" />
         <parent link="${parent}"/>
@@ -220,5 +220,5 @@
     <xacro:if value="${door == 'both'}">
       <joint name="${name}:joint" type="revolute">
-        <origin xyz="${-shelf_x_size/2+wall_thickness/2} ${wall_thickness} 0" rpy="0 0 0"/>
+        <origin xyz="${-shelf_x_size/2+wall_thickness/2} ${wall_thickness} ${door_height}" rpy="0 0 0"/>
         <axis xyz="0 0 1" />
         <parent link="${parent}"/>

Commit message: - added simple_couch furniture - door_height param

File: suturo_resources/urdf/suturo_environment.urdf.xacro (robot description, xacro)
@@ -17,11 +17,9 @@
     <xacro:include filename="$(find suturo_resources)/urdf/urdf_components/suturo_table.urdf.xacro" />
     <xacro:include filename="$(find suturo_resources)/urdf/urdf_components/suturo_popcorn_table.urdf.xacro" />
-    <xacro:include filename="$(find suturo_resources)/urdf/urdf_components/suturo_couch.urdf.xacro" />
-    <xacro:include
-        filename="$(find suturo_resources)/urdf/urdf_components/suturo_round_table.urdf.xacro" />
+    <xacro:include filename="$(find suturo_resources)/urdf/urdf_components/suturo_round_table.urdf.xacro" />
     <xacro:include filename="$(find suturo_resources)/urdf/urdf_components/suturo_wall.urdf.xacro" />
     <xacro:include filename="$(find suturo_resources)/urdf/urdf_components/suturo_shelf.urdf.xacro" />
-    <xacro:include
-        filename="$(find suturo_resources)/urdf/urdf_components/suturo_shelf_openable.urdf.xacro" />
+    <xacro:include filename="$(find suturo_resources)/urdf/urdf_components/suturo_shelf_openable.urdf.xacro" />
+    <xacro:include filename="$(find suturo_resources)/urdf/urdf_components/suturo_shelf_hohc.urdf.xacro" />
     <xacro:include filename="$(find suturo_resources)/urdf/urdf_components/suturo_door.urdf.xacro" />
     <xacro:include filename="$(find suturo_resources)/urdf/urdf_components/suturo_room.urdf.xacro" />
@@ -29,14 +27,10 @@
     <xacro:include filename="$(find suturo_resources)/urdf/urdf_components/suturo_path.urdf.xacro" />
     <xacro:include filename="$(find suturo_resources)/urdf/urdf_components/suturo_drawer.urdf.xacro" />
-    <xacro:include
-        filename="$(find suturo_resources)/urdf/urdf_components/suturo_simple_drawer.urdf.xacro" />
-    <xacro:include
-        filename="$(find suturo_resources)/urdf/urdf_components/suturo_dishwasher.urdf.xacro" />
-    <xacro:include
-        filename="$(find suturo_resources)/urdf/urdf_components/suturo_kitchen.urdf.xacro" />
-    <xacro:include
-        filename="$(find suturo_resources)/urdf/urdf_components/suturo_chair.urdf.xacro" />
-    <xacro:include
-        filename="$(find suturo_resources)/urdf/urdf_components/suturo_shelf_hohc.urdf.xacro" />
+    <xacro:include filename="$(find suturo_resources)/urdf/urdf_components/suturo_simple_drawer.urdf.xacro" />
+    <xacro:include filename="$(find suturo_resources)/urdf/urdf_components/suturo_dishwasher.urdf.xacro" />
+    <xacro:include filename="$(find suturo_resources)/urdf/urdf_components/suturo_kitchen.urdf.xacro" />
+    <xacro:include filename="$(find suturo_resources)/urdf/urdf_components/suturo_couch.urdf.xacro" />
+    <xacro:include filename="$(find suturo_resources)/urdf/urdf_components/suturo_simple_couch.urdf.xacro" />
+    <xacro:include filename="$(find suturo_resources)/urdf/urdf_components/suturo_chair.urdf.xacro" />
     <!-- general data -->
     <xacro:property name="number_of_drawers"
@@ -50,4 +44,6 @@
     <xacro:property name="number_of_couches"
         value="${data.get('couch', dict(amount=0)).get('amount', 0)}" />
+    <xacro:property name="number_of_simple_couches"
+        value="${data.get('simple_couch', dict(amount=0)).get('amount', 0)}" />
     <xacro:property name="number_of_round_tables"
         value="${data.get('round_tables', dict(amount=0)).get('amount', 0)}" />
@@ -122,4 +118,20 @@
         </xacro:if>
     </xacro:macro>
+      <!--  ~~Simple Couches~~  -->
+    <xacro:macro name="simple_couch_loop" params="simple_couch_number">
+        <xacro:suturo_simple_couch
+            name="${data['simple_couch'][simple_couch_number]['name']}:${data['simple_couch'][simple_couch_number]['knowledge_role']}"
+            parent="${data['simple_couch'][simple_couch_number]['parent']}"
+            size_x="${data['simple_couch'][simple_couch_number]['depth']}"
+            size_y="${data['simple_couch'][simple_couch_number]['width']}"
+            size_z="${data['simple_couch'][simple_couch_number]['height']}">
+            <origin
+                xyz="${data['simple_couch'][simple_couch_number]['x_pos']} ${data['simple_couch'][simple_couch_number]['y_pos']} 0"
+                rpy="0 0 ${data['simple_couch'][simple_couch_number]['z_rot']}" />
+        </xacro:suturo_simple_couch>
+        <xacro:if value="${(number_of_simple_couches - 1) > simple_couch_number}">
+            <xacro:simple_couch_loop simple_couch_number="${simple_couch_number + 1}" />
+        </xacro:if>
+    </xacro:macro>
     <!--  ~~Round_tables~~  -->
     <xacro:macro name="round_table_loop" params="round_table_number">
@@ -431,4 +443,7 @@
         <xacro:shelf_hohc_loop shelf_hohc_number="0" />
     </xacro:if>
+    <xacro:if value="${number_of_simple_couches > 0}">
+        <xacro:simple_couch_loop simple_couch_number="0" />
+    </xacro:if>
     <link name="urdf_main" />
     <joint name="map_urdf_joint" type="fixed">

File: suturo_resources/urdf/urdf_components/suturo_shelf_hohc.urdf.xacro (robot description, xacro)
@@ -51,5 +51,5 @@
     <xacro:if value="${door == 'left'}">
       <xacro:suturo_shelf_left_door_openable name="${name}:shelf_door_left" parent="${name}:shelf_left_side"
-       wall_thickness="${wall_thickness}" size_y="${door_width}" size_z="${door_length}" shelf_x_size="${size_x}"
+       wall_thickness="${wall_thickness}" door_height="${door_height}" size_y="${door_width}" size_z="${door_length}" shelf_x_size="${size_x}"
        handle_from_bottom="${handle_from_bottom}" handle_from_side="${handle_from_side}" handle_height="${handle_height}" handle_width="${handle_width}" handle_depth="${handle_depth}">
         <origin xyz="0 ${size_y*0.75} ${size_z/2}" rpy="0 0 0"/>
@@ -58,5 +58,5 @@
     <xacro:if value="${door == 'right'}">
       <xacro:suturo_shelf_right_door_openable name="${name}:shelf_door_right" parent="${name}:shelf_right_side"
-        wall_thickness="${wall_thickness}" size_y="${door_width}" size_z="${door_length}" shelf_x_size="${size_x}"
+        wall_thickness="${wall_thickness}" door_height="${door_height}" size_y="${door_width}" size_z="${door_length}" shelf_x_size="${size_x}"
        handle_from_bottom="${handle_from_bottom}" handle_from_side="${handle_from_side}" handle_height="${handle_height}" handle_width="${handle_width}" handle_depth="${handle_depth}">
         <origin xyz="0 ${size_y*0.75} ${door_length/2}" rpy="0 0 0"/>
@@ -65,5 +65,5 @@
     <xacro:if value="${door == 'both'}">
        <xacro:suturo_shelf_right_door_openable name="${name}:shelf_door_right" parent="${name}:shelf_right_side"
-        wall_thickness="${wall_thickness}" size_y="${door_width}" size_z="${door_length}" shelf_x_size="${size_x}"
+        wall_thickness="${wall_thickness}" door_height="${door_height}" size_y="${door_width}" size_z="${door_length}" shelf_x_size="${size_x}"
        handle_from_bottom="${handle_from_bottom}" handle_from_side="${handle_from_side}" handle_height="${handle_height}" handle_width="${handle_width}" handle_depth="${handle_depth}">
         <origin xyz="0 ${size_y} ${door_length/2}" rpy="0 0 0"/>
