Commit message: new trashbin and dishwasher

File: suturo_resources/urdf/suturo_environment.urdf.xacro (robot description, xacro)
@@ -29,7 +29,9 @@
     <xacro:include filename="$(find suturo_resources)/urdf/urdf_components/suturo_simple_drawer.urdf.xacro" />
     <xacro:include filename="$(find suturo_resources)/urdf/urdf_components/suturo_dishwasher.urdf.xacro" />
+    <xacro:include filename="$(find suturo_resources)/urdf/urdf_components/suturo_dishwasher_robocup.urdf.xacro" />
     <xacro:include filename="$(find suturo_resources)/urdf/urdf_components/suturo_kitchen.urdf.xacro" />
     <xacro:include filename="$(find suturo_resources)/urdf/urdf_components/suturo_couch.urdf.xacro" />
     <xacro:include filename="$(find suturo_resources)/urdf/urdf_components/suturo_simple_couch.urdf.xacro" />
+    <xacro:include filename="$(find suturo_resources)/urdf/urdf_components/suturo_trashbin.urdf.xacro" />
     <xacro:include filename="$(find suturo_resources)/urdf/urdf_components/suturo_chair.urdf.xacro" />
     <!-- general data -->
@@ -66,8 +68,12 @@
     <xacro:property name="number_of_dishwashers"
         value="${data.get('dishwashers', dict(amount=0)).get('amount', 0)}" />
+    <xacro:property name="number_of_dishwashers_robocup"
+        value="${data.get('dishwashers_robocup', dict(amount=0)).get('amount', 0)}" />
     <xacro:property name="number_of_chairs"
         value="${data.get('chairs', dict(amount=0)).get('amount', 0)}" />
     <xacro:property name="number_of_shelves_hohc"
         value="${data.get('shelves_hohc', dict(amount=0)).get('amount', 0)}" />
+    <xacro:property name="number_of_trashbins"
+        value="${data.get('trashbins', dict(amount=0)).get('amount', 0)}" />
     <!--  ~~Tables~~  -->
     <xacro:macro name="table_loop" params="table_number">
@@ -149,4 +155,19 @@
         </xacro:if>
     </xacro:macro>
+    <!--  ~~Trashbins~~  -->
+    <xacro:macro name="trashbin_loop" params="trashbin_number">
+        <xacro:suturo_trashbin
+            name="${data['trashbins'][trashbin_number]['name']}:${data['trashbins'][trashbin_number]['knowledge_role']}"
+            parent="${data['trashbins'][trashbin_number]['parent']}"
+            radius="${data['trashbins'][trashbin_number]['radius']}"
+            length="${data['trashbins'][trashbin_number]['length']}">
+            <origin
+                xyz="${data['trashbins'][trashbin_number]['x_pos']} ${data['trashbins'][trashbin_number]['y_pos']} 0"
+                rpy="0 0 ${data['trashbins'][trashbin_number]['z_rot']}" />
+        </xacro:suturo_trashbin>
+        <xacro:if value="${(number_of_round_tables - 1) > trashbin_number}">
+            <xacro:trashbin_loop trashbin_number="${trashbin_number + 1}" />
+        </xacro:if>
+    </xacro:macro>
 <!--<xacro:macro name="dishwasher_loop" params="dishwasher_number">
         <xacro:suturo_dishwasher
@@ -175,4 +196,17 @@
         <xacro:if value="${(number_of_dishwashers - 1) > dishwasher_number}">
             <xacro:dishwasher_loop dishwasher_number="${dishwasher_number + 1}" />
+        </xacro:if>
+    </xacro:macro>
+    <!--  ~~Dishwashers Robocup~~ -->
+    <xacro:macro name="dishwasher_robocup_loop" params="dishwasher_robocup_number">
+        <xacro:suturo_dishwasher_robocup
+            name="${data['dishwashers_robocup'][dishwasher_robocup_number]['name']}:${data['dishwashers_robocup'][dishwasher_robocup_number]['knowledge_role']}"
+            parent="${data['dishwashers_robocup'][dishwasher_robocup_number]['parent']}">
+            <origin
+                xyz="${data['dishwashers_robocup'][dishwasher_robocup_number]['x_pos']} ${data['dishwashers_robocup'][dishwasher_robocup_number]['y_pos']} 0.0"
+                rpy="0 0 ${data['dishwashers_robocup'][dishwasher_robocup_number]['z_rot']}" />
+        </xacro:suturo_dishwasher_robocup>
+        <xacro:if value="${(number_of_dishwashers_robocup - 1) > dishwasher_robocup_number}">
+            <xacro:dishwasher_robocup_loop dishwasher_robocup_number="${dishwasher_robocup_number + 1}" />
         </xacro:if>
     </xacro:macro>
@@ -437,4 +471,7 @@
         <xacro:dishwasher_loop dishwasher_number="0" />
     </xacro:if>
+    <xacro:if value="${number_of_dishwashers_robocup > 0}">
+        <xacro:dishwasher_robocup_loop dishwasher_robocup_number="0" />
+    </xacro:if>
         <xacro:if value="${number_of_chairs > 0}">
         <xacro:chair_loop chair_number="0" />
@@ -445,4 +482,7 @@
     <xacro:if value="${number_of_simple_couches > 0}">
         <xacro:simple_couch_loop simple_couch_number="0" />
+    </xacro:if>
+    <xacro:if value="${number_of_trashbins > 0}">
+        <xacro:trashbin_loop trashbin_number="0" />
     </xacro:if>
     <link name="urdf_main" />

Commit message: new coathanger

File: suturo_resources/urdf/suturo_environment.urdf.xacro (robot description, xacro)
@@ -35,4 +35,5 @@
     <xacro:include filename="$(find suturo_resources)/urdf/urdf_components/suturo_trashbin.urdf.xacro" />
     <xacro:include filename="$(find suturo_resources)/urdf/urdf_components/suturo_chair.urdf.xacro" />
+    <xacro:include filename="$(find suturo_resources)/urdf/urdf_components/suturo_coathanger.urdf.xacro" />
     <!-- general data -->
     <xacro:property name="number_of_drawers"
@@ -76,4 +77,6 @@
     <xacro:property name="number_of_trashbins"
         value="${data.get('trashbins', dict(amount=0)).get('amount', 0)}" />
+    <xacro:property name="number_of_coathangers"
+        value="${data.get('coathangers', dict(amount=0)).get('amount', 0)}" />
     <!--  ~~Tables~~  -->
     <xacro:macro name="table_loop" params="table_number">
@@ -374,4 +377,20 @@
         </xacro:suturo_kitchen>
     </xacro:macro>
+<!--  ~~Coathangers~~  -->
+    <xacro:macro name="coathanger_loop" params="coathanger_number">
+        <xacro:suturo_coathanger
+            name="${data['coathangers'][coathanger_number]['name']}:${data['coathangers'][coathanger_number]['knowledge_role']}"
+            parent="${data['coathangers'][coathanger_number]['parent']}"
+            size_x="${data['coathangers'][coathanger_number]['depth']}"
+            size_y="${data['coathangers'][coathanger_number]['width']}"
+            size_z="${data['coathangers'][coathanger_number]['height']}">
+            <origin
+                xyz="${data['coathangers'][coathanger_number]['x_pos']} ${data['coathangers'][coathanger_number]['y_pos']} 0"
+                rpy="0 0 ${data['coathangers'][coathanger_number]['z_rot']}" />
+        </xacro:suturo_coathanger>
+        <xacro:if value="${(number_of_coathangers - 1) > coathanger_number}">
+            <xacro:coathanger_loop coathanger_number="${coathanger_number + 1}" />
+        </xacro:if>
+    </xacro:macro>
     <!--  ~~Doors~~  -->
     <xacro:macro name="door_loop" params="door_number">
@@ -486,4 +505,7 @@
         <xacro:trashbin_loop trashbin_number="0" />
     </xacro:if>
+    <xacro:if value="${number_of_coathangers > 0}">
+        <xacro:coathanger_loop coathanger_number="0" />
+    </xacro:if>
     <link name="urdf_main" />
     <joint name="map_urdf_joint" type="fixed">

Commit message: - changes in TrashCan

File: suturo_resources/urdf/suturo_environment.urdf.xacro (robot description, xacro)
@@ -33,5 +33,5 @@
     <xacro:include filename="$(find suturo_resources)/urdf/urdf_components/suturo_couch.urdf.xacro" />
     <xacro:include filename="$(find suturo_resources)/urdf/urdf_components/suturo_simple_couch.urdf.xacro" />
-    <xacro:include filename="$(find suturo_resources)/urdf/urdf_components/suturo_trashbin.urdf.xacro" />
+    <xacro:include filename="$(find suturo_resources)/urdf/urdf_components/suturo_trashcan.urdf.xacro" />
     <xacro:include filename="$(find suturo_resources)/urdf/urdf_components/suturo_chair.urdf.xacro" />
     <xacro:include filename="$(find suturo_resources)/urdf/urdf_components/suturo_coathanger.urdf.xacro" />
@@ -75,6 +75,6 @@
     <xacro:property name="number_of_shelves_hohc"
         value="${data.get('shelves_hohc', dict(amount=0)).get('amount', 0)}" />
-    <xacro:property name="number_of_trashbins"
-        value="${data.get('trashbins', dict(amount=0)).get('amount', 0)}" />
+    <xacro:property name="number_of_trashcans"
+        value="${data.get('trashcans', dict(amount=0)).get('amount', 0)}" />
     <xacro:property name="number_of_coathangers"
         value="${data.get('coathangers', dict(amount=0)).get('amount', 0)}" />
@@ -159,16 +159,16 @@
     </xacro:macro>
     <!--  ~~Trashbins~~  -->
-    <xacro:macro name="trashbin_loop" params="trashbin_number">
-        <xacro:suturo_trashbin
-            name="${data['trashbins'][trashbin_number]['name']}:${data['trashbins'][trashbin_number]['knowledge_role']}"
-            parent="${data['trashbins'][trashbin_number]['parent']}"
-            radius="${data['trashbins'][trashbin_number]['radius']}"
-            length="${data['trashbins'][trashbin_number]['length']}">
-            <origin
-                xyz="${data['trashbins'][trashbin_number]['x_pos']} ${data['trashbins'][trashbin_number]['y_pos']} 0"
-                rpy="0 0 ${data['trashbins'][trashbin_number]['z_rot']}" />
-        </xacro:suturo_trashbin>
-        <xacro:if value="${(number_of_round_tables - 1) > trashbin_number}">
-            <xacro:trashbin_loop trashbin_number="${trashbin_number + 1}" />
+    <xacro:macro name="trashcan_loop" params="trashcan_number">
+        <xacro:suturo_trashcan
+            name="${data['trashcans'][trashcan_number]['name']}:${data['trashcans'][trashcan_number]['knowledge_role']}"
+            parent="${data['trashcans'][trashcan_number]['parent']}"
+            radius="${data['trashcans'][trashcan_number]['radius']}"
+            length="${data['trashcans'][trashcan_number]['length']}">
+            <origin
+                xyz="${data['trashcans'][trashcan_number]['x_pos']} ${data['trashcans'][trashcan_number]['y_pos']} 0"
+                rpy="0 0 ${data['trashcans'][trashcan_number]['z_rot']}" />
+        </xacro:suturo_trashcan>
+        <xacro:if value="${(number_of_round_tables - 1) > trashcan_number}">
+            <xacro:trashcan_loop trashcan_number="${trashcan_number + 1}" />
         </xacro:if>
     </xacro:macro>
@@ -502,6 +502,6 @@
         <xacro:simple_couch_loop simple_couch_number="0" />
     </xacro:if>
-    <xacro:if value="${number_of_trashbins > 0}">
-        <xacro:trashbin_loop trashbin_number="0" />
+    <xacro:if value="${number_of_trashcans > 0}">
+        <xacro:trashcan_loop trashcan_number="0" />
     </xacro:if>
     <xacro:if value="${number_of_coathangers > 0}">

File: suturo_resources/urdf/urdf_components/suturo_trashcan.urdf.xacro (robot description, xacro)
@@ -1,12 +1,12 @@
 <?xml version="1.0"?>
-<robot name="suturo_trashbin" xmlns:xacro="http://ros.org/wiki/xacro">
-  <material name="trashbin_color">
+<robot name="suturo_trashcan" xmlns:xacro="http://ros.org/wiki/xacro">
+  <material name="trashcan_color">
     <color rgba="0.8 0.8 0.8 1"/>
   </material>
-  <xacro:macro name="suturo_trashbin" params="name parent *origin radius length">
+  <xacro:macro name="suturo_trashcan" params="name parent *origin radius length">
     <!-- LINKS -->
-    <link name="${name}:trashbin_center">
+    <link name="${name}:trashcan_center">
       <visual>
-        <material name="trashbin_color"/>
+        <material name="trashcan_color"/>
         <origin xyz="0 0 ${-(length)/2}" rpy="0 0 0" />
         <geometry>
@@ -26,21 +26,21 @@
       </inertial>
     </link>
-    <link name="${name}:trashbin_origin"/>
-    <link name="${name}:trashbin_front_edge_center"/>
+    <link name="${name}:trashcan_origin"/>
+    <link name="${name}:trashcan_front_edge_center"/>
     <!-- JOINTS -->
-    <joint name="${name}:trashbin_origin_joint" type="fixed">
+    <joint name="${name}:trashcan_origin_joint" type="fixed">
       <xacro:insert_block name="origin" />
       <parent link="${parent}"/>
-      <child link="${name}:trashbin_origin"/>
+      <child link="${name}:trashcan_origin"/>
     </joint>
     <joint name="${name}:center_joint" type="fixed">
       <origin xyz="${radius} 0 ${length}" rpy="0 0 0" />
-      <parent link="${name}:trashbin_origin"/>
-      <child link="${name}:trashbin_center"/>
+      <parent link="${name}:trashcan_origin"/>
+      <child link="${name}:trashcan_center"/>
     </joint>
-    <joint name="${name}:trashbin_front_edge_center_joint" type="fixed">
+    <joint name="${name}:trashcan_front_edge_center_joint" type="fixed">
       <origin xyz="0 0 ${length}" rpy="0 0 0" />
-      <parent link="${name}:trashbin_origin"/>
-      <child link="${name}:trashbin_front_edge_center"/>
+      <parent link="${name}:trashcan_origin"/>
+      <child link="${name}:trashcan_front_edge_center"/>
     </joint>
   </xacro:macro>

Commit message: - added a lamp

File: suturo_resources/urdf/suturo_environment.urdf.xacro (robot description, xacro)
@@ -36,4 +36,5 @@
     <xacro:include filename="$(find suturo_resources)/urdf/urdf_components/suturo_chair.urdf.xacro" />
     <xacro:include filename="$(find suturo_resources)/urdf/urdf_components/suturo_coathanger.urdf.xacro" />
+    <xacro:include filename="$(find suturo_resources)/urdf/urdf_components/suturo_lamp.urdf.xacro" />
     <!-- general data -->
     <xacro:property name="number_of_drawers"
@@ -79,4 +80,6 @@
     <xacro:property name="number_of_coathangers"
         value="${data.get('coathangers', dict(amount=0)).get('amount', 0)}" />
+    <xacro:property name="number_of_lamps"
+        value="${data.get('lamps', dict(amount=0)).get('amount', 0)}" />
     <!--  ~~Tables~~  -->
     <xacro:macro name="table_loop" params="table_number">
@@ -156,4 +159,19 @@
         <xacro:if value="${(number_of_round_tables - 1) > round_table_number}">
             <xacro:round_table_loop round_table_number="${round_table_number + 1}" />
+        </xacro:if>
+    </xacro:macro>
+    <!--  ~~Lamps~~  -->
+    <xacro:macro name="lamp_loop" params="lamp_number">
+        <xacro:suturo_lamp
+            name="${data['lamps'][lamp_number]['name']}:${data['lamps'][lamp_number]['knowledge_role']}"
+            parent="${data['lamps'][lamp_number]['parent']}"
+            radius="${data['lamps'][lamp_number]['radius']}"
+            length="${data['lamps'][lamp_number]['length']}">
+            <origin
+                xyz="${data['lamps'][lamp_number]['x_pos']} ${data['lamps'][lamp_number]['y_pos']} 0"
+                rpy="0 0 ${data['lamps'][lamp_number]['z_rot']}" />
+        </xacro:suturo_lamp>
+        <xacro:if value="${(number_of_lamps - 1) > lamp_number}">
+            <xacro:lamp_loop lamp_number="${lamp_number + 1}" />
         </xacro:if>
     </xacro:macro>
@@ -508,4 +526,7 @@
         <xacro:coathanger_loop coathanger_number="0" />
     </xacro:if>
+    <xacro:if value="${number_of_lamps > 0}">
+        <xacro:lamp_loop lamp_number="0" />
+    </xacro:if>
     <link name="urdf_main" />
     <joint name="map_urdf_joint" type="fixed">

Commit message: fix billy shelf

File: suturo_resources/urdf/suturo_environment.urdf.xacro (robot description, xacro)
@@ -22,4 +22,5 @@
     <xacro:include filename="$(find suturo_resources)/urdf/urdf_components/suturo_shelf_openable.urdf.xacro" />
     <xacro:include filename="$(find suturo_resources)/urdf/urdf_components/suturo_shelf_hohc.urdf.xacro" />
+	<xacro:include filename="$(find suturo_resources)/urdf/urdf_components/suturo_shelf_billy.urdf.xacro" />
     <xacro:include filename="$(find suturo_resources)/urdf/urdf_components/suturo_door.urdf.xacro" />
     <xacro:include filename="$(find suturo_resources)/urdf/urdf_components/suturo_room.urdf.xacro" />
@@ -76,4 +77,6 @@
     <xacro:property name="number_of_shelves_hohc"
         value="${data.get('shelves_hohc', dict(amount=0)).get('amount', 0)}" />
+    <xacro:property name="number_of_shelves_billy"
+        value="${data.get('shelves_billy', dict(amount=0)).get('amount', 0)}" />
     <xacro:property name="number_of_trashcans"
         value="${data.get('trashcans', dict(amount=0)).get('amount', 0)}" />
@@ -318,4 +321,30 @@
         </xacro:if>
     </xacro:macro>
+    <!--  ~~Shelves_billy~~  -->
+    <xacro:macro name="shelf_billy_loop" params="shelf_billy_number">
+        <xacro:suturo_shelf_billy
+            name="${data['shelves_billy'][shelf_billy_number]['name']}:${data['shelves_billy'][shelf_billy_number]['knowledge_role']}"
+            parent="${data['shelves_billy'][shelf_billy_number]['parent']}"
+            size_x="${data['shelves_billy'][shelf_billy_number]['depth']}"
+            size_y="${data['shelves_billy'][shelf_billy_number]['width']}"
+            size_z="${data['shelves_billy'][shelf_billy_number]['height']}"
+            floors_height="${data['shelves_billy'][shelf_billy_number]['floors_height']}"
+            number_of_floors="${data['shelves_billy'][shelf_billy_number]['number_of_floors']}"
+            door="${data['shelves_billy'][shelf_billy_number]['door']}"
+            door_height="${data['shelves_billy'][shelf_billy_number]['door_height']}"
+            door_length="${data['shelves_billy'][shelf_billy_number]['door_length']}"
+            wall_thickness="${data['shelves_billy'][shelf_billy_number]['wall_thickness']}"
+            handle_from_bottom="${data['shelves_billy'][shelf_billy_number]['handle_from_bottom']}"
+            handle_from_side="${data['shelves_billy'][shelf_billy_number]['handle_from_side']}"
+            handle_diameter="${data['shelves_billy'][shelf_billy_number]['handle_diameter']}"
+            handle_depth="${data['shelves_billy'][shelf_billy_number]['handle_depth']}">
+            <origin
+                xyz="${data['shelves_billy'][shelf_billy_number]['x_pos']} ${data['shelves_billy'][shelf_billy_number]['y_pos']} 0"
+                rpy="0 0 ${data['shelves_billy'][shelf_billy_number]['z_rot']}" />
+        </xacro:suturo_shelf_billy>
+        <xacro:if value="${(number_of_shelves_billy - 1) > shelf_billy_number}">
+            <xacro:shelf_billy_loop shelf_billy_number="${shelf_billy_number + 1}" />
+        </xacro:if>
+    </xacro:macro>
   <!--  ~~Rooms~~  -->
     <xacro:macro name="room_loop" params="room_number">
@@ -517,4 +546,7 @@
         <xacro:shelf_hohc_loop shelf_hohc_number="0" />
     </xacro:if>
+    <xacro:if value="${number_of_shelves_billy > 0}">
+        <xacro:shelf_billy_loop shelf_billy_number="0" />
+    </xacro:if>
     <xacro:if value="${number_of_simple_couches > 0}">
         <xacro:simple_couch_loop simple_couch_number="0" />

Commit message: added armchair

File: suturo_resources/urdf/suturo_environment.urdf.xacro (robot description, xacro)
@@ -18,4 +18,5 @@
     <xacro:include filename="$(find suturo_resources)/urdf/urdf_components/suturo_popcorn_table.urdf.xacro" />
     <xacro:include filename="$(find suturo_resources)/urdf/urdf_components/suturo_round_table.urdf.xacro" />
+    <xacro:include filename="$(find suturo_resources)/urdf/urdf_components/suturo_round_armchair.urdf.xacro" />
     <xacro:include filename="$(find suturo_resources)/urdf/urdf_components/suturo_wall.urdf.xacro" />
     <xacro:include filename="$(find suturo_resources)/urdf/urdf_components/suturo_shelf.urdf.xacro" />
@@ -53,4 +54,6 @@
     <xacro:property name="number_of_round_tables"
         value="${data.get('round_tables', dict(amount=0)).get('amount', 0)}" />
+    <xacro:property name="number_of_round_armchairs"
+        value="${data.get('round_armchairs', dict(amount=0)).get('amount', 0)}" />
     <xacro:property name="number_of_buckets"
         value="${data.get('buckets', dict(amount=0)).get('amount', 0)}" />
@@ -164,4 +167,19 @@
         </xacro:if>
     </xacro:macro>
+    <!--  ~~Round_armchairs~~  -->
+    <xacro:macro name="round_armchair_loop" params="round_armchair_number">
+        <xacro:suturo_round_armchair
+            name="${data['round_armchairs'][round_armchair_number]['name']}:${data['round_armchairs'][round_armchair_number]['knowledge_role']}"
+            parent="${data['round_armchairs'][round_armchair_number]['parent']}"
+            radius="${data['round_armchairs'][round_armchair_number]['radius']}"
+            length="${data['round_armchairs'][round_armchair_number]['length']}">
+            <origin
+                xyz="${data['round_armchairs'][round_armchair_number]['x_pos']} ${data['round_armchairs'][round_armchair_number]['y_pos']} 0"
+                rpy="0 0 ${data['round_armchairs'][round_armchair_number]['z_rot']}" />
+        </xacro:suturo_round_armchair>
+        <xacro:if value="${(number_of_round_armchairs - 1) > round_armchair_number}">
+            <xacro:round_armchair_loop round_armchair_number="${round_armchair_number + 1}" />
+        </xacro:if>
+    </xacro:macro>
     <!--  ~~Lamps~~  -->
     <xacro:macro name="lamp_loop" params="lamp_number">
@@ -510,4 +528,7 @@
         <xacro:round_table_loop round_table_number="0" />
     </xacro:if>
+    <xacro:if value="${number_of_round_armchairs > 0}">
+        <xacro:round_armchair_loop round_armchair_number="0" />
+    </xacro:if>
     <xacro:if value="${number_of_buckets > 0}">
         <xacro:bucket_loop bucket_number="0" />
