Commit message: added parameters for handle from left side and right side instead of general

File: suturo_resources/urdf/ms3_room_04.urdf.xacro (robot description, xacro)
@@ -281,5 +281,6 @@
             wall_thickness="${data['shelves_billy'][shelf_billy_number]['wall_thickness']}"
             handle_from_bottom="${data['shelves_billy'][shelf_billy_number]['handle_from_bottom']}"
-            handle_from_side="${data['shelves_billy'][shelf_billy_number]['handle_from_side']}"
+            handle_from_side_left="${data['shelves_billy'][shelf_billy_number]['handle_from_side_left']}"
+            handle_from_side_right="${data['shelves_billy'][shelf_billy_number]['handle_from_side_right']}"
             handle_diameter="${data['shelves_billy'][shelf_billy_number]['handle_diameter']}"
             handle_depth="${data['shelves_billy'][shelf_billy_number]['handle_depth']}">

File: suturo_resources/urdf/urdf_components/suturo_shelf_billy.urdf.xacro (robot description, xacro)
@@ -4,5 +4,5 @@
     <color rgba="0.74 0.25 0.25 1"/>
   </material>
-  <xacro:macro name="suturo_shelf_billy" params="name parent *origin size_x size_y size_z floors_height number_of_floors door door_height door_length wall_thickness handle_from_bottom handle_from_side handle_diameter handle_depth">
+  <xacro:macro name="suturo_shelf_billy" params="name parent *origin size_x size_y size_z floors_height number_of_floors door door_height door_length wall_thickness handle_from_bottom handle_from_side_left handle_from_side_right handle_diameter handle_depth">
     <!-- General conveinience links -->
     <link name="${name}:shelf_origin"/>
@@ -52,5 +52,5 @@
       <xacro:suturo_shelf_billy_left_door name="${name}:shelf_door_left" parent="${name}:shelf_left_side"
        wall_thickness="${wall_thickness}" door_height="${door_height}" size_y="${door_width}" size_z="${door_length}" shelf_x_size="${size_x}"
-       handle_from_bottom="${handle_from_bottom}" handle_from_side="${handle_from_side}" handle_diameter="${handle_diameter}" handle_depth="${handle_depth}">
+       handle_from_bottom="${handle_from_bottom}" handle_from_side="${handle_from_side_left}" handle_diameter="${handle_diameter}" handle_depth="${handle_depth}">
         <origin xyz="0 ${size_y} ${size_z/2}" rpy="0 0 0"/>
       </xacro:suturo_shelf_billy_left_door>
@@ -59,5 +59,5 @@
       <xacro:suturo_shelf_billy_right_door name="${name}:shelf_door_right" parent="${name}:shelf_right_side"
         wall_thickness="${wall_thickness}" door_height="${door_height}" size_y="${door_width}" size_z="${door_length}" shelf_x_size="${size_x}"
-       handle_from_bottom="${handle_from_bottom}" handle_from_side="${handle_from_side}" handle_diameter="${handle_diameter}" handle_depth="${handle_depth}">
+       handle_from_bottom="${handle_from_bottom}" handle_from_side="${handle_from_side_right}" handle_diameter="${handle_diameter}" handle_depth="${handle_depth}">
         <origin xyz="0 ${size_y} ${size_z/2}" rpy="0 0 0"/>
       </xacro:suturo_shelf_billy_right_door>
@@ -66,10 +66,10 @@
        <xacro:suturo_shelf_billy_right_door name="${name}:shelf_door_right" parent="${name}:shelf_right_side"
         wall_thickness="${wall_thickness}" door_height="${door_height}" size_y="${door_width}" size_z="${door_length}" shelf_x_size="${size_x}"
-       handle_from_bottom="${handle_from_bottom}" handle_from_side="${handle_from_side}" handle_diameter="${handle_diameter}" handle_depth="${handle_depth}">
+       handle_from_bottom="${handle_from_bottom}" handle_from_side="${handle_from_side_right}" handle_diameter="${handle_diameter}" handle_depth="${handle_depth}">
         <origin xyz="0 ${size_y} ${size_z/2}" rpy="0 0 0"/>
        </xacro:suturo_shelf_billy_right_door>
          <xacro:suturo_shelf_billy_left_door name="${name}:shelf_door_left" parent="${name}:shelf_left_side"
           wall_thickness="${wall_thickness}" door_height="${door_height}" size_y="${door_width}" size_z="${door_length}" shelf_x_size="${size_x}"
-	  handle_from_bottom="${handle_from_bottom}" handle_from_side="${handle_from_side}" handle_diameter="${handle_diameter}" handle_depth="${handle_depth}">
+	  handle_from_bottom="${handle_from_bottom}" handle_from_side="${handle_from_side_left}" handle_diameter="${handle_diameter}" handle_depth="${handle_depth}">
         <origin xyz="0 ${size_y} ${size_z/2}" rpy="0 0 0"/>
       </xacro:suturo_shelf_billy_left_door>
@@ -206,5 +206,5 @@
     </link>
     <joint name="${name}:handle_joint" type="fixed">
-      <origin xyz="${-wall_thickness-handle_depth/2} ${+handle_from_side+handle_depth/2} ${handle_from_bottom-size_z/2+handle_depth/2}" rpy="0 ${pi/2} 0"/>
+      <origin xyz="${-wall_thickness-handle_depth/2} ${+handle_from_side+handle_diameter/2} ${handle_from_bottom-size_z/2+handle_diameter/2}" rpy="0 ${pi/2} 0"/>
       <axis xyz="0 0 1" />
       <parent link="${name}"/>

Commit message: dishwasher changes

File: suturo_resources/urdf/ms3_room_04.urdf.xacro (robot description, xacro)
@@ -171,5 +171,14 @@
         <xacro:suturo_dishwasher
             name="${data['dishwashers'][dishwasher_number]['name']}:${data['dishwashers'][dishwasher_number]['knowledge_role']}"
-            parent="${data['dishwashers'][dishwasher_number]['parent']}">
+            parent="${data['dishwashers'][dishwasher_number]['parent']}"
+            table_size_x="${data['dishwashers'][dishwasher_number]['table_size_x']}"
+            table_size_y="${data['dishwashers'][dishwasher_number]['table_size_y']}"
+            table_size_z="${data['dishwashers'][dishwasher_number]['table_size_z']}"
+            height="${data['dishwashers'][dishwasher_number]['height']}"
+            table_height="${data['dishwashers'][dishwasher_number]['table_height']}"
+            handle_x="${data['dishwashers'][dishwasher_number]['handle_x']}"
+            handle_y="${data['dishwashers'][dishwasher_number]['handle_y']}"
+            handle_z="${data['dishwashers'][dishwasher_number]['handle_z']}"
+            >
             <origin
                 xyz="${data['dishwashers'][dishwasher_number]['x_pos']} ${data['dishwashers'][dishwasher_number]['y_pos']} 0.0"

File: suturo_resources/urdf/suturo_environment.urdf.xacro (robot description, xacro)
@@ -231,5 +231,14 @@
         <xacro:suturo_dishwasher
             name="${data['dishwashers'][dishwasher_number]['name']}:${data['dishwashers'][dishwasher_number]['knowledge_role']}"
-            parent="${data['dishwashers'][dishwasher_number]['parent']}">
+            parent="${data['dishwashers'][dishwasher_number]['parent']}"
+            table_size_x="${data['dishwashers'][dishwasher_number]['table_size_x']}"
+            table_size_y="${data['dishwashers'][dishwasher_number]['table_size_y']}"
+            table_size_z="${data['dishwashers'][dishwasher_number]['table_size_z']}"
+            height="${data['dishwashers'][dishwasher_number]['height']}"
+            table_height="${data['dishwashers'][dishwasher_number]['table_height']}"
+            handle_x="${data['dishwashers'][dishwasher_number]['handle_x']}"
+            handle_y="${data['dishwashers'][dishwasher_number]['handle_y']}"
+            handle_z="${data['dishwashers'][dishwasher_number]['handle_z']}"
+            >
             <origin
                 xyz="${data['dishwashers'][dishwasher_number]['x_pos']} ${data['dishwashers'][dishwasher_number]['y_pos']} 0.0"
@@ -354,5 +363,6 @@
             wall_thickness="${data['shelves_billy'][shelf_billy_number]['wall_thickness']}"
             handle_from_bottom="${data['shelves_billy'][shelf_billy_number]['handle_from_bottom']}"
-            handle_from_side="${data['shelves_billy'][shelf_billy_number]['handle_from_side']}"
+            handle_from_side_left="${data['shelves_billy'][shelf_billy_number]['handle_from_side_left']}"
+            handle_from_side_right="${data['shelves_billy'][shelf_billy_number]['handle_from_side_right']}"
             handle_diameter="${data['shelves_billy'][shelf_billy_number]['handle_diameter']}"
             handle_depth="${data['shelves_billy'][shelf_billy_number]['handle_depth']}">

File: suturo_resources/urdf/urdf_components/suturo_dishwasher.urdf.xacro (robot description, xacro)
@@ -4,5 +4,5 @@
 	<color rgba="0.255 0.62 0.223 1"/>
   </material>
-  <xacro:macro name="suturo_dishwasher" params="name parent *origin">
+  <xacro:macro name="suturo_dishwasher" params="name parent *origin table_size_x table_size_y table_size_z height table_height handle_x handle_y handle_z">
      <link name="dishwasher_main">
        <inertial>
@@ -95,5 +95,5 @@
         <origin xyz="0 0 0" rpy="0 0 0" />
         <geometry>
-          <box size="0.6 0.6 0.02" />
+          <box size="${table_size_x} ${table_size_y} ${table_size_z}" />
         </geometry>
       </visual>
@@ -101,5 +101,5 @@
         <origin xyz="0 0 0" rpy="0 0 0" />
         <geometry>
-          <box size="0.6 0.6 0.02" />
+          <box size="${table_size_x} ${table_size_y} ${table_size_z}" />
         </geometry>
       </collision>
@@ -116,5 +116,5 @@
     <axis xyz="1 0 0" />
     <!-- <limit effort="300" lower="0" upper="0" velocity="10"/> -->
-    <origin rpy="0 0 0" xyz="0.08 -0.78 0.455 "/>
+    <origin rpy="0 0 0" xyz="0 0 ${height} "/>
     <parent link="dishwasher_main"/>
     <child link="sink_area_dish_washer_main"/>
@@ -131,5 +131,5 @@
   <!--x,y,z Handle position change-->
   <joint name="sink_area_dish_washer_door_handle_joint" type="fixed">
-    <origin rpy="-1.57079632679 0 0" xyz="0.0625 -0.6325 0."/>
+    <origin rpy="-1.57079632679 0 0" xyz="${handle_x} ${handle_y} ${handle_z}"/>
     <parent link="sink_area_dish_washer_door"/>
     <child link="sink_area_dish_washer_door_handle"/>
@@ -137,5 +137,5 @@
   <!-- from here for dishwasher_table -->
   <joint name="dish_washer_table_main_joint" type="fixed">
-    <origin rpy="0 0 ${pi}" xyz="0.0 0.0 0.39"/>
+    <origin rpy="0 0 ${pi}" xyz="0.0 0.0 ${table_height}"/>
     <parent link="sink_area_dish_washer_main"/>
     <child link="dishwasher_table:d_table:table_origin"/>

Commit message: new bed added

File: suturo_resources/urdf/ms3_room_04.urdf.xacro (robot description, xacro)
@@ -16,4 +16,5 @@
     <!--  Include the files containing the macros -->
     <xacro:include filename="$(find suturo_resources)/urdf/urdf_components/suturo_table.urdf.xacro" />
+    <xacro:include filename="$(find suturo_resources)/urdf/urdf_components/suturo_bed.urdf.xacro" />
     <xacro:include filename="$(find suturo_resources)/urdf/urdf_components/suturo_popcorn_table.urdf.xacro" />
     <xacro:include filename="$(find suturo_resources)/urdf/urdf_components/suturo_round_table.urdf.xacro" />
@@ -41,4 +42,6 @@
     <xacro:property name="number_of_tables"
         value="${data.get('tables', dict(amount=0)).get('amount', 0)}" />
+    <xacro:property name="number_of_beds"
+        value="${data.get('beds', dict(amount=0)).get('amount', 0)}" />
     <xacro:property name="number_of_popcorn_tables"
         value="${data.get('popcorn_tables', dict(amount=0)).get('amount', 0)}" />
@@ -89,4 +92,20 @@
         </xacro:if>
     </xacro:macro>
+    <!--  ~~Beds~~  -->
+    <xacro:macro name="bed_loop" params="bed_number">
+        <xacro:suturo_bed
+            name="${data['beds'][bed_number]['name']}:${data['beds'][bed_number]['knowledge_role']}"
+            parent="${data['beds'][bed_number]['parent']}"
+            size_x="${data['beds'][bed_number]['depth']}"
+            size_y="${data['beds'][bed_number]['width']}"
+            size_z="${data['beds'][bed_number]['height']}">
+            <origin
+                xyz="${data['beds'][bed_number]['x_pos']} ${data['beds'][bed_number]['y_pos']} 0"
+                rpy="0 0 ${data['beds'][bed_number]['z_rot']}" />
+        </xacro:suturo_bed>
+        <xacro:if value="${(number_of_beds - 1) > bed_number}">
+            <xacro:bed_loop bed_number="${bed_number + 1}" />
+        </xacro:if>
+    </xacro:macro>
     <!--  ~~Popcorn_tables~~  -->
     <xacro:macro name="popcorn_table_loop" params="popcorn_table_number">
@@ -440,4 +459,7 @@
         <xacro:table_loop table_number="0" />
     </xacro:if>
+    <xacro:if value="${number_of_beds > 0}">
+        <xacro:bed_loop bed_number="0" />
+    </xacro:if>
     <xacro:if value="${number_of_popcorn_tables > 0}">
         <xacro:popcorn_table_loop popcorn_table_number="0" />

File: suturo_resources/urdf/suturo_environment.urdf.xacro (robot description, xacro)
@@ -16,4 +16,5 @@
     <!--  Include the files containing the macros -->
     <xacro:include filename="$(find suturo_resources)/urdf/urdf_components/suturo_table.urdf.xacro" />
+    <xacro:include filename="$(find suturo_resources)/urdf/urdf_components/suturo_bed.urdf.xacro" />
     <xacro:include filename="$(find suturo_resources)/urdf/urdf_components/suturo_popcorn_table.urdf.xacro" />
     <xacro:include filename="$(find suturo_resources)/urdf/urdf_components/suturo_round_table.urdf.xacro" />
@@ -46,4 +47,6 @@
     <xacro:property name="number_of_tables"
         value="${data.get('tables', dict(amount=0)).get('amount', 0)}" />
+    <xacro:property name="number_of_beds"
+        value="${data.get('beds', dict(amount=0)).get('amount', 0)}" />
     <xacro:property name="number_of_popcorn_tables"
         value="${data.get('popcorn_tables', dict(amount=0)).get('amount', 0)}" />
@@ -104,4 +107,20 @@
         </xacro:if>
     </xacro:macro>
+    <!--  ~~Beds~~  -->
+    <xacro:macro name="bed_loop" params="bed_number">
+        <xacro:suturo_bed
+            name="${data['beds'][bed_number]['name']}:${data['beds'][bed_number]['knowledge_role']}"
+            parent="${data['beds'][bed_number]['parent']}"
+            size_x="${data['beds'][bed_number]['depth']}"
+            size_y="${data['beds'][bed_number]['width']}"
+            size_z="${data['beds'][bed_number]['height']}">
+            <origin
+                xyz="${data['beds'][bed_number]['x_pos']} ${data['beds'][bed_number]['y_pos']} 0"
+                rpy="0 0 ${data['beds'][bed_number]['z_rot']}" />
+        </xacro:suturo_bed>
+        <xacro:if value="${(number_of_beds - 1) > bed_number}">
+            <xacro:bed_loop bed_number="${bed_number + 1}" />
+        </xacro:if>
+    </xacro:macro>
     <!--  ~~Popcorn_tables~~  -->
     <xacro:macro name="popcorn_table_loop" params="popcorn_table_number">
@@ -529,4 +548,7 @@
         <xacro:table_loop table_number="0" />
     </xacro:if>
+    <xacro:if value="${number_of_beds > 0}">
+        <xacro:bed_loop bed_number="0" />
+    </xacro:if>
     <xacro:if value="${number_of_popcorn_tables > 0}">
         <xacro:popcorn_table_loop popcorn_table_number="0" />

Commit message: fixed trashcan urdf.xacro

File: suturo_resources/urdf/ms3_room_04.urdf.xacro (robot description, xacro)
@@ -34,4 +34,5 @@
     <xacro:include filename="$(find suturo_resources)/urdf/urdf_components/suturo_couch.urdf.xacro" />
     <xacro:include filename="$(find suturo_resources)/urdf/urdf_components/suturo_simple_couch.urdf.xacro" />
+    <xacro:include filename="$(find suturo_resources)/urdf/urdf_components/suturo_trashcan.urdf.xacro" />
     <xacro:include filename="$(find suturo_resources)/urdf/urdf_components/suturo_chair.urdf.xacro" />
     <!-- general data -->
@@ -76,4 +77,6 @@
     <xacro:property name="number_of_shelves_billy"
         value="${data.get('shelves_billy', dict(amount=0)).get('amount', 0)}" />
+    <xacro:property name="number_of_trashcans"
+        value="${data.get('trashcans', dict(amount=0)).get('amount', 0)}" />
     <!--  ~~Tables~~  -->
     <xacro:macro name="table_loop" params="table_number">
@@ -375,4 +378,19 @@
         </xacro:if>
     </xacro:macro>
+    <!--  ~~Trashcans~~  -->
+    <xacro:macro name="trashcan_loop" params="trashcan_number">
+        <xacro:suturo_trashcan
+            name="${data['trashcans'][trashcan_number]['name']}:${data['trashcans'][trashcan_number]['knowledge_role']}"
+            parent="${data['trashcans'][trashcan_number]['parent']}"
+            radius="${data['trashcans'][trashcan_number]['radius']}"
+            length="${data['trashcans'][trashcan_number]['length']}">
+            <origin
+                xyz="${data['trashcans'][trashcan_number]['x_pos']} ${data['trashcans'][trashcan_number]['y_pos']} 0"
+                rpy="0 0 ${data['trashcans'][trashcan_number]['z_rot']}" />
+        </xacro:suturo_trashcan>
+        <xacro:if value="${(number_of_trashcans - 1) > trashcan_number}">
+            <xacro:trashcan_loop trashcan_number="${trashcan_number + 1}" />
+        </xacro:if>
+    </xacro:macro>
     <!--  ~~Walls~~  -->
     <xacro:macro name="wall_loop" params="wall_number">
@@ -506,4 +524,6 @@
     <xacro:if value="${number_of_shelves_billy > 0}">
         <xacro:shelf_billy_loop shelf_billy_number="0" />
+    <xacro:if value="${number_of_trashcans > 0}">
+        <xacro:trashcan_loop trashcan_number="0" />
     </xacro:if>
     <xacro:if value="${number_of_simple_couches > 0}">

File: suturo_resources/urdf/suturo_environment.urdf.xacro (robot description, xacro)
@@ -227,5 +227,5 @@
                 rpy="0 0 ${data['trashcans'][trashcan_number]['z_rot']}" />
         </xacro:suturo_trashcan>
-        <xacro:if value="${(number_of_round_tables - 1) > trashcan_number}">
+        <xacro:if value="${(number_of_trashcans - 1) > trashcan_number}">
             <xacro:trashcan_loop trashcan_number="${trashcan_number + 1}" />
         </xacro:if>

Commit message: added coathanger

File: suturo_resources/urdf/ms3_room_04.urdf.xacro (robot description, xacro)
@@ -36,4 +36,5 @@
     <xacro:include filename="$(find suturo_resources)/urdf/urdf_components/suturo_trashcan.urdf.xacro" />
     <xacro:include filename="$(find suturo_resources)/urdf/urdf_components/suturo_chair.urdf.xacro" />
+    <xacro:include filename="$(find suturo_resources)/urdf/urdf_components/suturo_coathanger.urdf.xacro" />
     <!-- general data -->
     <xacro:property name="number_of_drawers"
@@ -79,4 +80,6 @@
     <xacro:property name="number_of_trashcans"
         value="${data.get('trashcans', dict(amount=0)).get('amount', 0)}" />
+    <xacro:property name="number_of_coathangers"
+        value="${data.get('coathangers', dict(amount=0)).get('amount', 0)}" />
     <!--  ~~Tables~~  -->
     <xacro:macro name="table_loop" params="table_number">
@@ -453,4 +456,20 @@
         </xacro:if>
     </xacro:macro>
+<!--  ~~Coathangers~~  -->
+    <xacro:macro name="coathanger_loop" params="coathanger_number">
+        <xacro:suturo_coathanger
+            name="${data['coathangers'][coathanger_number]['name']}:${data['coathangers'][coathanger_number]['knowledge_role']}"
+            parent="${data['coathangers'][coathanger_number]['parent']}"
+            size_x="${data['coathangers'][coathanger_number]['depth']}"
+            size_y="${data['coathangers'][coathanger_number]['width']}"
+            size_z="${data['coathangers'][coathanger_number]['height']}">
+            <origin
+                xyz="${data['coathangers'][coathanger_number]['x_pos']} ${data['coathangers'][coathanger_number]['y_pos']} 0"
+                rpy="0 0 ${data['coathangers'][coathanger_number]['z_rot']}" />
+        </xacro:suturo_coathanger>
+        <xacro:if value="${(number_of_coathangers - 1) > coathanger_number}">
+            <xacro:coathanger_loop coathanger_number="${coathanger_number + 1}" />
+        </xacro:if>
+    </xacro:macro>
     <!--  ~~Paths~~  -->
     <xacro:macro name="path_loop" params="path_number">
@@ -528,4 +547,7 @@
         <xacro:trashcan_loop trashcan_number="0" />
     </xacro:if>
+    <xacro:if value="${number_of_coathangers > 0}">
+        <xacro:coathanger_loop coathanger_number="0" />
+    </xacro:if>
     <xacro:if value="${number_of_simple_couches > 0}">
         <xacro:simple_couch_loop simple_couch_number="0" />

Commit message: - added round armchair - updated arena exit and entry

File: suturo_resources/urdf/ms3_room_04.urdf.xacro (robot description, xacro)
@@ -36,4 +36,5 @@
     <xacro:include filename="$(find suturo_resources)/urdf/urdf_components/suturo_trashcan.urdf.xacro" />
     <xacro:include filename="$(find suturo_resources)/urdf/urdf_components/suturo_chair.urdf.xacro" />
+    <xacro:include filename="$(find suturo_resources)/urdf/urdf_components/suturo_round_armchair.urdf.xacro" />
     <xacro:include filename="$(find suturo_resources)/urdf/urdf_components/suturo_coathanger.urdf.xacro" />
     <!-- general data -->
@@ -74,4 +75,6 @@
     <xacro:property name="number_of_chairs"
         value="${data.get('chairs', dict(amount=0)).get('amount', 0)}" />
+    <xacro:property name="number_of_round_armchairs"
+        value="${data.get('round_armchairs', dict(amount=0)).get('amount', 0)}" />
     <xacro:property name="number_of_shelves_hohc"
         value="${data.get('shelves_hohc', dict(amount=0)).get('amount', 0)}" />
@@ -175,4 +178,19 @@
         <xacro:if value="${(number_of_round_tables - 1) > round_table_number}">
             <xacro:round_table_loop round_table_number="${round_table_number + 1}" />
+        </xacro:if>
+    </xacro:macro>
+     <!--  ~~Round_armchairs~~  -->
+    <xacro:macro name="round_armchair_loop" params="round_armchair_number">
+        <xacro:suturo_round_armchair
+            name="${data['round_armchairs'][round_armchair_number]['name']}:${data['round_armchairs'][round_armchair_number]['knowledge_role']}"
+            parent="${data['round_armchairs'][round_armchair_number]['parent']}"
+            radius="${data['round_armchairs'][round_armchair_number]['radius']}"
+            length="${data['round_armchairs'][round_armchair_number]['length']}">
+            <origin
+                xyz="${data['round_armchairs'][round_armchair_number]['x_pos']} ${data['round_armchairs'][round_armchair_number]['y_pos']} 0"
+                rpy="0 0 ${data['round_armchairs'][round_armchair_number]['z_rot']}" />
+        </xacro:suturo_round_armchair>
+        <xacro:if value="${(number_of_round_armchairs - 1) > round_armchair_number}">
+            <xacro:round_armchair_loop round_armchair_number="${round_armchair_number + 1}" />
         </xacro:if>
     </xacro:macro>
@@ -538,4 +556,7 @@
         <xacro:chair_loop chair_number="0" />
     </xacro:if>
+     <xacro:if value="${number_of_round_armchairs > 0}">
+        <xacro:round_armchair_loop round_armchair_number="0" />
+    </xacro:if>
     <xacro:if value="${number_of_shelves_hohc > 0}">
         <xacro:shelf_hohc_loop shelf_hohc_number="0" />
