Commit message: bad commit message

File: suturo_resources/urdf/urdf_components/suturo_bucket.urdf.xacro (robot description, xacro)
@@ -1,10 +1,10 @@
 <?xml version="1.0"?>
-<robot name="robocup_bucket" xmlns:xacro="http://ros.org/wiki/xacro">
+<robot name="suturo_bucket" xmlns:xacro="http://ros.org/wiki/xacro">
   <material name="bucket_grey">
     <color rgba="0.8 0.8 0.8 1"/>
   </material>
-  <macro name="robocup_bucket" params="name parent *origin size_x size_y size_z">
+  <xacro:macro name="suturo_bucket" params="name parent *origin size_x size_y size_z">
     <!-- LINKS -->
-    <link name="${name}_center">
+    <link name="${name}_bucket_center">
       <visual>
         <material name="bucket_grey"/>
@@ -21,29 +21,29 @@
       </collision>
     </link>
-    <link name="${name}_origin"/>
+    <link name="${name}_bucket_origin"/>
     <!-- Additional tf-frames -->
-    <link name="${name}_surface_center"/>
-    <link name="${name}_front_edge_center"/>
+    <link name="${name}_bucket_surface_center"/>
+    <link name="${name}_bucket_front_edge_center"/>
     <!-- JOINTS -->
-    <joint name="${name}_origin_joint" type="fixed">
+    <joint name="${name}_bucket_origin_joint" type="fixed">
       <xacro:insert_block name="origin" />
       <parent link="${parent}"/>
-      <child link="${name}_origin"/>
+      <child link="${name}_bucket_origin"/>
     </joint>
-    <joint name="${name}_center_joint" type="fixed">
+    <joint name="${name}_bucket_center_joint" type="fixed">
       <origin xyz="${size_x/2} ${size_y/2} ${size_z/2}" rpy="0 0 0" />
-      <parent link="${name}_origin"/>
-      <child link="${name}_center"/>
+      <parent link="${name}_bucket_origin"/>
+      <child link="${name}_bucket_center"/>
     </joint>
-    <joint name="${name}_surface_center_joint" type="fixed">
+    <joint name="${name}_bucket_surface_center_joint" type="fixed">
       <origin xyz="${size_x/2} ${size_y/2} ${size_z}" rpy="0 0 0" />
-      <parent link="${name}_origin"/>
-      <child link="${name}_surface_center"/>
+      <parent link="${name}_bucket_origin"/>
+      <child link="${name}_bucket_surface_center"/>
     </joint>
-    <joint name="${name}_front_edge_center_joint" type="fixed">
+    <joint name="${name}_bucket_front_edge_center_joint" type="fixed">
       <origin xyz="0 ${size_y/2} ${size_z}" rpy="0 0 0" />
-      <parent link="${name}_origin"/>
-      <child link="${name}_front_edge_center"/>
+      <parent link="${name}_bucket_origin"/>
+      <child link="${name}_bucket_front_edge_center"/>
     </joint>
-  </macro>
+  </xacro:macro>
 </robot>

File: suturo_resources/urdf/urdf_components/suturo_door.urdf.xacro (robot description, xacro)
@@ -1,4 +1,4 @@
 <?xml version="1.0"?>
-<robot name="suturo_movable_door" xmlns:xacro="http://ros.org/wiki/xacro">
+<robot name="suturo_door" xmlns:xacro="http://ros.org/wiki/xacro">
   <material name="door_green">
     <color rgba="0 0.31 0.22 1"/>
@@ -10,9 +10,8 @@
     <color rgba="0.3 0.5 0.78 1"/>
   </material>
-  <xacro:property name="pi" value="3.1415926535897931" />
   <xacro:property name="half_pi" value="1.570796327" />
-  <macro name="suturo_movable_door" params="name parent height width depth x y z r p yr door_lower door_max">
+  <xacro:macro name="suturo_door" params="name parent height width depth x y z zrot door_turn_limit_lower door_turn_limit_max">
     <!-- LINKS -->
-    <link name="${name}_center">
+    <link name="${name}_door_center">
       <visual>
         <material name="door_green"/>
@@ -29,5 +28,5 @@
       </collision>
     </link>
-    <link name="${name}_hinge">
+    <link name="${name}_door_hinge">
       <visual>
         <material name="hinge_red"/>
@@ -44,5 +43,5 @@
       </collision>
     </link>
-    <link name="${name}_handle_outside">
+    <link name="${name}_door_handle_outside">
       <sphere_inertia radius="0" mass="0"/>
       <visual>
@@ -60,5 +59,5 @@
       </collision>
     </link>
-    <link name="${name}_handle_inside">
+    <link name="${name}_door_handle_inside">
       <sphere_inertia radius="0" mass="0"/>
       <visual>
@@ -77,32 +76,32 @@
     </link>
     <!-- JOINTS -->
-    <joint name="${name}_origin_revolute_joint" type="revolute">
+    <joint name="${name}_door_origin_revolute_joint" type="revolute">
       <axis xyz="0 0 1"/>
-      <limit effort="100" lower="${door_lower}" upper="${door_max}" velocity="10"/>
-      <origin xyz="0 0 0" rpy="0 0 ${yr}" />
-      <parent link="${name}_hinge"/>
-      <child link="${name}_center"/>
+      <limit effort="100" lower="${door_turn_limit_lower}" upper="${door_turn_limit_max}" velocity="10"/>
+      <origin xyz="0 0 0" rpy="0 0 ${zrot}" />
+      <parent link="${name}_door_hinge"/>
+      <child link="${name}_door_center"/>
     </joint>
-    <joint name="${name}_hinge_joint" type="fixed">
+    <joint name="${name}_door_hinge_joint" type="fixed">
       <axis xyz="0 0 0"/>
       <limit effort="1" lower="0" upper="1.5708" velocity="1"/>
       <origin xyz="${x} ${y} ${z}" rpy="0 0 0" />
       <parent link="${parent}"/>
-      <child link="${name}_hinge"/>
+      <child link="${name}_door_hinge"/>
     </joint>
-    <joint name="${name}_handle_inside_joint" type="fixed">
+    <joint name="${name}_door_handle_inside_joint" type="fixed">
       <axis xyz="0 0 0"/>
       <limit effort="1" lower="0" upper="1.5708" velocity="1"/>
       <origin xyz="${0.9 * width} ${-depth} -0.1" rpy="0 0 0" />
-      <parent link="${name}_center"/>
-      <child link="${name}_handle_inside"/>
+      <parent link="${name}_door_center"/>
+      <child link="${name}_door_handle_inside"/>
     </joint>
-    <joint name="${name}_handle_outside_joint" type="fixed">
+    <joint name="${name}_door_handle_outside_joint" type="fixed">
       <axis xyz="0 0 0"/>
       <limit effort="1" lower="0" upper="1.5708" velocity="1"/>
       <origin xyz="${0.9 * width} ${depth} -0.1" rpy="0 0 0" />
-      <parent link="${name}_center"/>
-      <child link="${name}_handle_outside"/>
+      <parent link="${name}_door_center"/>
+      <child link="${name}_door_handle_outside"/>
     </joint>
-  </macro>
+  </xacro:macro>
 </robot>

File: suturo_resources/urdf/urdf_components/suturo_room.urdf.xacro (robot description, xacro)
@@ -2,16 +2,25 @@
 <!-- Rooms are for Knowledge Information only-->
 <robot name="suturo_room" xmlns:xacro="http://ros.org/wiki/xacro">
-  <xacro:macro name="suturo_room" params="name parent num_of_corners corners_x_pos corners_y_pos center_x center_y">
+  <xacro:macro name="suturo_room" params="name parent num_of_corners corners_x_pos corners_y_pos center_x center_y color">
     <!-- define a central joint to wich every corner is connected -->
     <joint name="world_${name}_room_joint" type="fixed">
         <origin xyz="${center_x} ${center_y} 0 " rpy="0 0 0" />
-        <parent link="world"/>
+        <parent link="${parent}"/>
         <child link="${name}_room_center_link"/>
     </joint>
-    <link name="${name}_room_center_link" />
+    <link name="${name}_room_center_link">
+      <visual>
+        <geometry>
+          <cylinder length="0" radius="0"/>
+        </geometry>
+        <material name="color">
+          <color rgba="${color}"/>
+        </material>
+      </visual>
+    </link>
     <!-- room loop to create every corner -->
     <xacro:macro name="corner_loop" params="loop_number">
       <joint name="${name}_room_joint_${loop_number}" type="fixed">
-          <origin xyz="${corners_x_pos[loop_number]} ${corners_y_pos[loop_number]} 0 " rpy="0 0 0" />
+          <origin xyz="${corners_x_pos[loop_number] - center_x} ${corners_y_pos[loop_number] - center_y} 0 " rpy="0 0 0" />
           <parent link="${name}_room_center_link"/>
           <child link="${name}_room_corner_${loop_number}_link"/>
