Commit message: Positionsanpassung

File: suturo_resources/urdf/urdf_components/suturo_drawer.urdf.xacro (robot description, xacro)
@@ -26,5 +26,5 @@
           <visual name="trofast">
             <material name="orange"/>
-            <origin xyz="0 0 0.1" rpy="0 0 0" />
+            <origin xyz="0.01 0 0.11" rpy="0 0 0" />
             <geometry>
               <mesh filename="package://suturo_resources/gazebo_models/trofast/meshes/trofast.stl" scale="1 1 1"/>

Commit message: Rotate drawer frames so taht knowledge calculates the correct pose to percieve

File: suturo_resources/urdf/urdf_components/suturo_drawer.urdf.xacro (robot description, xacro)
@@ -10,5 +10,5 @@
         <color rgba="1 1 1 1"/>
     </material>
-    <xacro:property name="half_pi" value="1.570796327" />
+    <xacro:property name="half_pi" value="${pi/2}" />
     <xacro:macro name="suturo_drawer" params="name parent *origin size_x size_y size_z ">
         <!-- LINKS-->
@@ -26,5 +26,5 @@
           <visual name="trofast">
             <material name="orange"/>
-            <origin xyz="0.01 0 0.11" rpy="0 0 0" />
+            <origin xyz="0.01 0 0.01" rpy="0 0 0" />
             <geometry>
               <mesh filename="package://suturo_resources/gazebo_models/trofast/meshes/trofast.stl" scale="1 1 1"/>
@@ -32,5 +32,5 @@
           </visual>
           <visual name="knob_base">
-            <origin xyz="0.205 0 0.28" rpy="0 1.56 0" />
+            <origin xyz="-0.205 0 0.18" rpy="0 1.56 ${pi}" />
             <geometry>
                 <cylinder radius="0.034" length="0.02"/>
@@ -39,5 +39,5 @@
           </visual>
           <visual name="knob_pole">
-            <origin xyz="0.22 0 0.28" rpy="0 1.56 0" />
+            <origin xyz="-0.22 0 0.18" rpy="0 1.56 ${pi}" />
             <geometry>
                 <cylinder radius="0.015" length="0.05"/>
@@ -46,5 +46,5 @@
           </visual>
           <visual name="knob_handle">
-            <origin xyz="0.24 0 0.28" rpy="0 0 0" />
+            <origin xyz="-0.24 0 0.18" rpy="0 0 ${pi}" />
             <geometry>
                 <box size= "0.01 0.066 0.03"/>
@@ -68,5 +68,5 @@
           </collision>
           <collision name="collision_knob_base">
-            <origin xyz="0.205 0 0.28" rpy="0 1.56 0" />
+            <origin xyz="-0.205 0 0.18" rpy="0 1.56 ${pi}" />
             <geometry>
                 <cylinder radius="0.034" length="0.02"/>
@@ -74,5 +74,5 @@
           </collision>
           <collision name="collision_knob_pole">
-            <origin xyz="0.22 0 0.28" rpy="0 1.56 0" />
+            <origin xyz="-0.22 0 0.18" rpy="0 1.56 ${pi}" />
             <geometry>
                 <cylinder radius="0.015" length="0.05"/>
@@ -80,5 +80,5 @@
           </collision>
           <collision name="collision_knob_handle">
-            <origin xyz="0.24 0 0.28" rpy="0 0 0" />
+            <origin xyz="-0.24 0 0.18" rpy="0 0 ${pi}" />
             <geometry>
                 <box size= "0.01 0.066 0.03"/>
@@ -387,6 +387,6 @@
           </visual>
         </link>
-        <link name="${name}:drawer_front_top"/>
         <link name="${name}:drawer_knob"/>
+	<link name="${name}:drawer_front_top"/>
         <!-- JOINTS-->
         <!--<joint name="${name}:drawer_center_joint" type="fixed">
@@ -396,15 +396,15 @@
         </joint>-->
         <joint name="${name}:drawer_center_joint" type="fixed">
-          <xacro:insert_block name="origin" />
-          <parent link="${parent}"/>
+          <origin xyz="0 0 0.1" rpy="0 0 ${pi}"/>
+          <parent link="${name}:wrc_stair_like_drawer"/>
           <child link="${name}:drawer_center"/>
         </joint>
         <joint name="${name}:drawer_front_joint" type="fixed">
-          <origin xyz="${size_x/2} 0 ${size_z/2+0.1}" rpy="0 0 0" />
+          <origin xyz="${-size_x/2} 0 ${size_z}" rpy="0 0 0" />
           <parent link="${name}:drawer_center"/>
           <child link="${name}:drawer_front_top"/>
         </joint>
         <joint name="${name}:knob_joint" type="fixed">
-          <origin xyz="${size_x/2} 0 ${size_z/2+0.05}" rpy="0 0 0" />
+          <origin xyz="${-size_x/2} 0 ${size_z*0.7}" rpy="0 0 0" />
           <parent link="${name}:drawer_center"/>
           <child link="${name}:drawer_knob"/>

Commit message: prismatic joint und x umgedreht um pi

File: suturo_resources/urdf/urdf_components/suturo_drawer.urdf.xacro (robot description, xacro)
@@ -32,5 +32,5 @@
           </visual>
           <visual name="knob_base">
-            <origin xyz="-0.205 0 0.18" rpy="0 1.56 ${pi}" />
+            <origin xyz="0.205 0 0.18" rpy="0 1.56 ${pi}" />
             <geometry>
                 <cylinder radius="0.034" length="0.02"/>
@@ -39,5 +39,5 @@
           </visual>
           <visual name="knob_pole">
-            <origin xyz="-0.22 0 0.18" rpy="0 1.56 ${pi}" />
+            <origin xyz="0.22 0 0.18" rpy="0 1.56 ${pi}" />
             <geometry>
                 <cylinder radius="0.015" length="0.05"/>
@@ -46,5 +46,5 @@
           </visual>
           <visual name="knob_handle">
-            <origin xyz="-0.24 0 0.18" rpy="0 0 ${pi}" />
+            <origin xyz="0.24 0 0.18" rpy="0 0 ${pi}" />
             <geometry>
                 <box size= "0.01 0.066 0.03"/>
@@ -68,5 +68,5 @@
           </collision>
           <collision name="collision_knob_base">
-            <origin xyz="-0.205 0 0.18" rpy="0 1.56 ${pi}" />
+            <origin xyz="0.205 0 0.18" rpy="0 1.56 ${pi}" />
             <geometry>
                 <cylinder radius="0.034" length="0.02"/>
@@ -74,5 +74,5 @@
           </collision>
           <collision name="collision_knob_pole">
-            <origin xyz="-0.22 0 0.18" rpy="0 1.56 ${pi}" />
+            <origin xyz="0.22 0 0.18" rpy="0 1.56 ${pi}" />
             <geometry>
                 <cylinder radius="0.015" length="0.05"/>
@@ -80,5 +80,5 @@
           </collision>
           <collision name="collision_knob_handle">
-            <origin xyz="-0.24 0 0.18" rpy="0 0 ${pi}" />
+            <origin xyz="0.24 0 0.18" rpy="0 0 ${pi}" />
             <geometry>
                 <box size= "0.01 0.066 0.03"/>
@@ -401,10 +401,10 @@
         </joint>
         <joint name="${name}:drawer_front_joint" type="fixed">
-          <origin xyz="${-size_x/2} 0 ${size_z}" rpy="0 0 0" />
+          <origin xyz="${size_x/2} 0 ${size_z}" rpy="0 0 0" />
           <parent link="${name}:drawer_center"/>
           <child link="${name}:drawer_front_top"/>
         </joint>
         <joint name="${name}:knob_joint" type="fixed">
-          <origin xyz="${-size_x/2} 0 ${size_z*0.7}" rpy="0 0 0" />
+          <origin xyz="${size_x/2} 0 ${size_z*0.7}" rpy="0 0 0" />
           <parent link="${name}:drawer_center"/>
           <child link="${name}:drawer_knob"/>
@@ -415,4 +415,10 @@
           <child link="${name}:wrc_stair_like_drawer"/>
         </joint>
+        <joint name="drawer_move" type="prismatic">
+          <parent link="${name}:wrc_stair_like_drawer"/>
+          <child link="${name}:drawer_center"/>
+          <limit effort="1000.0" lower="-0.38" upper="0" velocity="0.5"/>
+          <origin xyz="0 0 0.1" rpy="0 0 0" />
+        </joint>
   </xacro:macro>
 </robot>

Commit message: joint fixed entfernt

File: suturo_resources/urdf/urdf_components/suturo_drawer.urdf.xacro (robot description, xacro)
@@ -395,9 +395,4 @@
           <child link="${name}:drawer_center"/>
         </joint>-->
-        <joint name="${name}:drawer_center_joint" type="fixed">
-          <origin xyz="0 0 0.1" rpy="0 0 ${pi}"/>
-          <parent link="${name}:wrc_stair_like_drawer"/>
-          <child link="${name}:drawer_center"/>
-        </joint>
         <joint name="${name}:drawer_front_joint" type="fixed">
           <origin xyz="${size_x/2} 0 ${size_z}" rpy="0 0 0" />

Commit message: frames an der richtigen Stelle und richtige rotation

File: suturo_resources/urdf/urdf_components/suturo_drawer.urdf.xacro (robot description, xacro)
@@ -32,5 +32,5 @@
           </visual>
           <visual name="knob_base">
-            <origin xyz="0.205 0 0.18" rpy="0 1.56 ${pi}" />
+            <origin xyz="-0.205 0 0.18" rpy="0 1.56 ${pi}" />
             <geometry>
                 <cylinder radius="0.034" length="0.02"/>
@@ -39,5 +39,5 @@
           </visual>
           <visual name="knob_pole">
-            <origin xyz="0.22 0 0.18" rpy="0 1.56 ${pi}" />
+            <origin xyz="-0.22 0 0.18" rpy="0 1.56 ${pi}" />
             <geometry>
                 <cylinder radius="0.015" length="0.05"/>
@@ -46,5 +46,5 @@
           </visual>
           <visual name="knob_handle">
-            <origin xyz="0.24 0 0.18" rpy="0 0 ${pi}" />
+            <origin xyz="-0.24 0 0.18" rpy="0 0 ${pi}" />
             <geometry>
                 <box size= "0.01 0.066 0.03"/>
@@ -68,5 +68,5 @@
           </collision>
           <collision name="collision_knob_base">
-            <origin xyz="0.205 0 0.18" rpy="0 1.56 ${pi}" />
+            <origin xyz="-0.205 0 0.18" rpy="0 1.56 ${pi}" />
             <geometry>
                 <cylinder radius="0.034" length="0.02"/>
@@ -74,5 +74,5 @@
           </collision>
           <collision name="collision_knob_pole">
-            <origin xyz="0.22 0 0.18" rpy="0 1.56 ${pi}" />
+            <origin xyz="-0.22 0 0.18" rpy="0 1.56 ${pi}" />
             <geometry>
                 <cylinder radius="0.015" length="0.05"/>
@@ -80,5 +80,5 @@
           </collision>
           <collision name="collision_knob_handle">
-            <origin xyz="0.24 0 0.18" rpy="0 0 ${pi}" />
+            <origin xyz="-0.24 0 0.18" rpy="0 0 ${pi}" />
             <geometry>
                 <box size= "0.01 0.066 0.03"/>
@@ -396,10 +396,10 @@
         </joint>-->
         <joint name="${name}:drawer_front_joint" type="fixed">
-          <origin xyz="${size_x/2} 0 ${size_z}" rpy="0 0 0" />
+          <origin xyz="${-size_x/2} 0 ${size_z}" rpy="0 0 0" />
           <parent link="${name}:drawer_center"/>
           <child link="${name}:drawer_front_top"/>
         </joint>
         <joint name="${name}:knob_joint" type="fixed">
-          <origin xyz="${size_x/2} 0 ${size_z*0.7}" rpy="0 0 0" />
+          <origin xyz="${-size_x/2} 0 ${size_z*0.7}" rpy="0 0 0" />
           <parent link="${name}:drawer_center"/>
           <child link="${name}:drawer_knob"/>
@@ -414,5 +414,5 @@
           <child link="${name}:drawer_center"/>
           <limit effort="1000.0" lower="-0.38" upper="0" velocity="0.5"/>
-          <origin xyz="0 0 0.1" rpy="0 0 0" />
+          <origin xyz="0 0 0.1" rpy="0 0 ${pi}" />
         </joint>
   </xacro:macro>

Commit message: change upper lower velocity prismatic

File: suturo_resources/urdf/urdf_components/suturo_drawer.urdf.xacro (robot description, xacro)
@@ -413,5 +413,5 @@
           <parent link="${name}:wrc_stair_like_drawer"/>
           <child link="${name}:drawer_center"/>
-          <limit effort="1000.0" lower="-0.38" upper="0" velocity="0.5"/>
+          <limit effort="100.0" lower="-1" upper="1" velocity="1"/>
           <origin xyz="0 0 0.1" rpy="0 0 ${pi}" />
         </joint>

Commit message: axis joint prismatic

File: suturo_resources/urdf/urdf_components/suturo_drawer.urdf.xacro (robot description, xacro)
@@ -414,4 +414,5 @@
           <child link="${name}:drawer_center"/>
           <limit effort="100.0" lower="-1" upper="1" velocity="1"/>
+          <axis xyz="1 0 0"/>
           <origin xyz="0 0 0.1" rpy="0 0 ${pi}" />
         </joint>

Commit message: Frame verschoben etc

File: suturo_resources/urdf/urdf_components/suturo_drawer.urdf.xacro (robot description, xacro)
@@ -401,5 +401,5 @@
         </joint>
         <joint name="${name}:knob_joint" type="fixed">
-          <origin xyz="${-size_x/2} 0 ${size_z*0.7}" rpy="0 0 0" />
+          <origin xyz="${-size_x/2-0.03} 0 ${size_z*0.7}" rpy="0 0 0" />
           <parent link="${name}:drawer_center"/>
           <child link="${name}:drawer_knob"/>
@@ -413,5 +413,5 @@
           <parent link="${name}:wrc_stair_like_drawer"/>
           <child link="${name}:drawer_center"/>
-          <limit effort="100.0" lower="-1" upper="1" velocity="1"/>
+          <limit effort="100.0" lower="-0.36" upper="0.0" velocity="1"/>
           <axis xyz="1 0 0"/>
           <origin xyz="0 0 0.1" rpy="0 0 ${pi}" />
