Commit message: make naming standard

File: suturo_resources/urdf/urdf_components/suturo_shelf.urdf.xacro (robot description, xacro)
@@ -7,5 +7,5 @@
     <color rgba="0.64 0.87 0.82 1"/>
   </material>
-  <xacro:macro name="suturo_shelf" params="name parent x y z xr yr zr size_x size_y size_z floors_height number_of_floors door">
+  <xacro:macro name="suturo_shelf" params="name parent *origin size_x size_y size_z floors_height number_of_floors door">
     <!-- General conveinience links -->
     <link name="${name}_origin"/>
@@ -13,5 +13,5 @@
     <link name="${name}_base_center"/>
     <joint name="${name}_origin_joint" type="fixed">
-     <origin xyz="${x} ${y} ${z}" rpy="${xr} ${yr} ${zr}"/>
+      <xacro:insert_block name="origin" />
       <parent link="${parent}"/>
       <child link="${name}_origin"/>
@@ -50,5 +50,6 @@
     </xacro:macro>
     <xacro:shelf_floor_loop floor_number="0" />
-    <!-- door -->
+    <!-- ****************SHELF DOOR**************** -->
+    <!-- left -->
     <xacro:if value="${door == 'left'}">
       <xacro:suturo_shelf_left_door name="${name}_door_left" parent="${name}_left_side"
@@ -57,5 +58,17 @@
       </xacro:suturo_shelf_left_door>
     </xacro:if>
+    <!-- right -->
     <xacro:if value="${door == 'right'}">
+      <xacro:suturo_shelf_right_door name="${name}_door_right" parent="${name}_right_side"
+        size_x="0.01" size_y="${size_y/2}" size_z="${size_z}" shelf_x_size="${size_x}">
+        <origin xyz="0 ${size_y*0.75} ${size_z/2}" rpy="0 0 0"/>
+      </xacro:suturo_shelf_right_door>
+    </xacro:if>
+    <!-- both -->
+    <xacro:if value="${door == 'both'}">
+      <xacro:suturo_shelf_left_door name="${name}_door_left" parent="${name}_left_side"
+        size_x="0.01" size_y="${size_y/2}" size_z="${size_z}" shelf_x_size="${size_x}">
+        <origin xyz="0 ${size_y*0.75} ${size_z/2}" rpy="0 0 0"/>
+      </xacro:suturo_shelf_left_door>
       <xacro:suturo_shelf_right_door name="${name}_door_right" parent="${name}_right_side"
         size_x="0.01" size_y="${size_y/2}" size_z="${size_z}" shelf_x_size="${size_x}">
@@ -85,5 +98,5 @@
     <!-- JOINT -->
     <joint name="${name}_piece_joint" type="fixed">
-      <origin xyz="${x} ${y} ${z}" rpy="${xr} ${yr} ${zr}"/>
+      <xacro:insert_block name="origin" />
       <parent link="${parent}"/>
       <child link="${name}_piece"/>

Commit message: name stuff

File: suturo_resources/urdf/urdf_components/suturo_shelf.urdf.xacro (robot description, xacro)
@@ -9,37 +9,37 @@
   <xacro:macro name="suturo_shelf" params="name parent *origin size_x size_y size_z floors_height number_of_floors door">
     <!-- General conveinience links -->
-    <link name="${name}_origin"/>
-    <link name="${name}_center"/>
-    <link name="${name}_base_center"/>
-    <joint name="${name}_origin_joint" type="fixed">
+    <link name="${name}_shelf_origin"/>
+    <link name="${name}_shelf_center"/>
+    <link name="${name}_shelf_base_center"/>
+    <joint name="${name}_shelf_origin_joint" type="fixed">
       <xacro:insert_block name="origin" />
       <parent link="${parent}"/>
-      <child link="${name}_origin"/>
+      <child link="${name}_shelf_origin"/>
     </joint>
-    <joint name="${name}_center_joint" type="fixed">
+    <joint name="${name}_shelf_center_joint" type="fixed">
       <origin xyz="${size_x/2} ${size_y/2} ${size_z/2}" rpy="0 0 0" />
-      <parent link="${name}_origin"/>
-      <child link="${name}_center"/>
+      <parent link="${name}_shelf_origin"/>
+      <child link="${name}_shelf_center"/>
     </joint>
-    <joint name="${name}_base_center_joint" type="fixed">
+    <joint name="${name}_shelf_base_center_joint" type="fixed">
       <origin xyz="${size_x/2} ${size_y/2} 0.0" rpy="0 0 0" />
-      <parent link="${name}_origin"/>
-      <child link="${name}_base_center"/>
+      <parent link="${name}_shelf_origin"/>
+      <child link="${name}_shelf_base_center"/>
     </joint>
     <!-- WALLS -->
-    <xacro:suturo_shelf_piece name="${name}_back" parent="${name}_origin"
+    <xacro:suturo_shelf_piece name="${name}_shelf_back" parent="${name}_shelf_origin"
       size_x="0.01" size_y="${size_y}" size_z="${size_z}">
       <origin xyz="${size_x} ${size_y/2} ${size_z/2}" rpy="0 0 0"/>
     </xacro:suturo_shelf_piece>
-    <xacro:suturo_shelf_piece name="${name}_right_side" parent="${name}_origin"
+    <xacro:suturo_shelf_piece name="${name}_shelf_right_side" parent="${name}_shelf_origin"
       size_x="${size_x}" size_y="0.01" size_z="${size_z}">
       <origin xyz="${size_x/2} 0.0 ${size_z/2}" rpy="0 0 0"/>
     </xacro:suturo_shelf_piece>
-    <xacro:suturo_shelf_piece name="${name}_left_side" parent="${name}_origin"
+    <xacro:suturo_shelf_piece name="${name}_shelf_left_side" parent="${name}_shelf_origin"
       size_x="${size_x}" size_y="0.01" size_z="${size_z}">
       <origin xyz="${size_x/2} ${size_y} ${size_z/2}" rpy="0 0 0"/>
     </xacro:suturo_shelf_piece>
     <xacro:macro name="shelf_floor_loop" params="floor_number">
-        <xacro:suturo_shelf_piece name="${name}_floor_${floor_number}" parent="${name}_base_center"
+        <xacro:suturo_shelf_piece name="${name}_shelf_floor_${floor_number}" parent="${name}_shelf_base_center"
           size_x="${size_x}" size_y="${size_y}" size_z="0.04" box_z_offset="-0.02">
         <origin xyz="0.0 0.0 ${floors_height[floor_number]}" rpy="0 0 0"/>
@@ -53,5 +53,5 @@
     <!-- left -->
     <xacro:if value="${door == 'left'}">
-      <xacro:suturo_shelf_left_door name="${name}_door_left" parent="${name}_left_side"
+      <xacro:suturo_shelf_left_door name="${name}_shelf_door_left" parent="${name}_left_side"
         size_x="0.01" size_y="${size_y/2}" size_z="${size_z}" shelf_x_size="${size_x}">
         <origin xyz="0 ${size_y*0.75} ${size_z/2}" rpy="0 0 0"/>
@@ -60,5 +60,5 @@
     <!-- right -->
     <xacro:if value="${door == 'right'}">
-      <xacro:suturo_shelf_right_door name="${name}_door_right" parent="${name}_right_side"
+      <xacro:suturo_shelf_right_door name="${name}_shelf_door_right" parent="${name}_right_side"
         size_x="0.01" size_y="${size_y/2}" size_z="${size_z}" shelf_x_size="${size_x}">
         <origin xyz="0 ${size_y*0.75} ${size_z/2}" rpy="0 0 0"/>
@@ -67,9 +67,9 @@
     <!-- both -->
     <xacro:if value="${door == 'both'}">
-      <xacro:suturo_shelf_left_door name="${name}_door_left" parent="${name}_left_side"
+      <xacro:suturo_shelf_left_door name="${name}_shelf_door_left" parent="${name}_left_side"
         size_x="0.01" size_y="${size_y/2}" size_z="${size_z}" shelf_x_size="${size_x}">
         <origin xyz="0 ${size_y*0.75} ${size_z/2}" rpy="0 0 0"/>
       </xacro:suturo_shelf_left_door>
-      <xacro:suturo_shelf_right_door name="${name}_door_right" parent="${name}_right_side"
+      <xacro:suturo_shelf_right_door name="${name}_shelf_door_right" parent="${name}_shelf_right_side"
         size_x="0.01" size_y="${size_y/2}" size_z="${size_z}" shelf_x_size="${size_x}">
         <origin xyz="0 ${size_y*0.75} ${size_z/2}" rpy="0 0 0"/>
@@ -81,5 +81,5 @@
   <xacro:macro name="suturo_shelf_piece" params="name parent *origin box_z_offset=0.0 size_x size_y size_z">
     <!-- LINK -->
-    <link name="${name}_piece">
+    <link name="${name}_shelf_piece">
       <visual>
         <material name="shelf_blue"/>
@@ -97,8 +97,8 @@
     </link>
     <!-- JOINT -->
-    <joint name="${name}_piece_joint" type="fixed">
+    <joint name="${name}_shelf_piece_joint" type="fixed">
       <xacro:insert_block name="origin" />
       <parent link="${parent}"/>
-      <child link="${name}_piece"/>
+      <child link="${name}_shelf_piece"/>
     </joint>
   </xacro:macro>
@@ -119,5 +119,5 @@
       </collision>
     </link>
-    <joint name="${name}_joint" type="revolute">
+    <joint name="${name}_shelf_joint" type="revolute">
       <origin xyz="${shelf_x_size/-2} ${size_y/-2} 0" rpy="0 0 3.1416"/>
       <axis xyz="0 0 1" />
@@ -128,5 +128,5 @@
   </xacro:macro>
   <xacro:macro name="suturo_shelf_right_door" params="name parent *origin size_x size_y size_z shelf_x_size">
-    <link name="${name}_link">
+    <link name="${name}_shelf_link">
       <visual>
         <material name="shelf_door_green"/>
@@ -143,9 +143,9 @@
       </collision>
     </link>
-    <joint name="${name}_joint" type="revolute">
+    <joint name="${name}_shelf_joint" type="revolute">
       <origin xyz="${shelf_x_size/-2} ${size_y/2} 0" rpy="0 0 -3.1416"/>
       <axis xyz="0 0 1" />
-      <parent link="${parent}_piece"/>
-      <child link="${name}_link"/>
+      <parent link="${parent}_shelf_piece"/>
+      <child link="${name}_shelf_link"/>
       <limit effort="30" velocity="1.0" lower="0.0" upper="1.91986" />
     </joint>

File: suturo_resources/urdf/urdf_components/suturo_table.urdf.xacro (robot description, xacro)
@@ -6,5 +6,5 @@
   <xacro:macro name="suturo_table" params="name parent *origin size_x size_y size_z">
     <!-- LINKS -->
-    <link name="${name}_center">
+    <link name="${name}_table_center">
       <visual>
         <material name="table_grey"/>
@@ -21,21 +21,21 @@
       </collision>
     </link>
-    <link name="${name}_origin"/>
-     <link name="${name}_front_edge_center"/>
+    <link name="${name}_table_origin"/>
+     <link name="${name}_table_front_edge_center"/>
     <!-- JOINTS -->
-    <joint name="${name}_origin_joint" type="fixed">
+    <joint name="${name}_table_origin_joint" type="fixed">
       <xacro:insert_block name="origin" />
       <parent link="${parent}"/>
-      <child link="${name}_origin"/>
+      <child link="${name}_table_origin"/>
     </joint>
     <joint name="${name}_center_joint" type="fixed">
       <origin xyz="${size_x/2} ${size_y/2} ${size_z}" rpy="0 0 0" />
-      <parent link="${name}_origin"/>
-      <child link="${name}_center"/>
+      <parent link="${name}_table_origin"/>
+      <child link="${name}_table_center"/>
     </joint>
-    <joint name="${name}_front_edge_center_joint" type="fixed">
+    <joint name="${name}_table_front_edge_center_joint" type="fixed">
       <origin xyz="0 ${size_y/2} ${size_z}" rpy="0 0 0" />
-      <parent link="${name}_origin"/>
-      <child link="${name}_front_edge_center"/>
+      <parent link="${name}_table_origin"/>
+      <child link="${name}_table_front_edge_center"/>
     </joint>
   </xacro:macro>

Commit message: simplify shelf names

File: suturo_resources/urdf/urdf_components/suturo_shelf.urdf.xacro (robot description, xacro)
@@ -81,5 +81,5 @@
   <xacro:macro name="suturo_shelf_piece" params="name parent *origin box_z_offset=0.0 size_x size_y size_z">
     <!-- LINK -->
-    <link name="${name}_shelf_piece">
+    <link name="${name}">
       <visual>
         <material name="shelf_blue"/>
@@ -97,8 +97,8 @@
     </link>
     <!-- JOINT -->
-    <joint name="${name}_shelf_piece_joint" type="fixed">
+    <joint name="${name}_joint" type="fixed">
       <xacro:insert_block name="origin" />
       <parent link="${parent}"/>
-      <child link="${name}_shelf_piece"/>
+      <child link="${name}"/>
     </joint>
   </xacro:macro>

Commit message: adjusted shelf urdfs to have similarlz named joints and links

File: suturo_resources/urdf/urdf_components/suturo_shelf.urdf.xacro (robot description, xacro)
@@ -110,5 +110,5 @@
   </xacro:macro>
   <xacro:macro name="suturo_shelf_left_door" params="name parent *origin size_x size_y size_z shelf_x_size">
-    <link name="${name}:link">
+    <link name="${name}">
       <visual>
         <material name="shelf_door_green"/>
@@ -125,14 +125,14 @@
       </collision>
     </link>
-    <joint name="${name}:shelf_joint" type="revolute">
+    <joint name="${name}:joint" type="revolute">
       <origin xyz="${shelf_x_size/-2} ${size_y/-2} 0" rpy="0 0 3.1416"/>
       <axis xyz="0 0 1" />
-      <parent link="${parent}:piece"/>
-      <child link="${name}:link"/>
+      <parent link="${parent}"/>
+      <child link="${name}"/>
       <limit effort="30" velocity="1.0" lower="0.0" upper="1.91986" />
     </joint>
   </xacro:macro>
   <xacro:macro name="suturo_shelf_right_door" params="name parent *origin size_x size_y size_z shelf_x_size">
-    <link name="${name}:shelf_link">
+    <link name="${name}">
       <visual>
         <material name="shelf_door_green"/>
@@ -149,9 +149,9 @@
       </collision>
     </link>
-    <joint name="${name}:shelf_joint" type="revolute">
+    <joint name="${name}:joint" type="revolute">
       <origin xyz="${shelf_x_size/-2} ${size_y/2} 0" rpy="0 0 -3.1416"/>
       <axis xyz="0 0 1" />
-      <parent link="${parent}:shelf_piece"/>
-      <child link="${name}:shelf_link"/>
+      <parent link="${parent}"/>
+      <child link="${name}"/>
       <limit effort="30" velocity="1.0" lower="0.0" upper="1.91986" />
     </joint>

File: suturo_resources/urdf/urdf_components/suturo_shelf_openable.urdf.xacro (robot description, xacro)
@@ -75,5 +75,5 @@
   <xacro:macro name="suturo_shelf_piece_openable" params="name parent *origin box_z_offset=0.0 size_x size_y size_z">
     <!-- LINK -->
-    <link name="${name}:shelf_piece">
+    <link name="${name}">
       <visual>
         <material name="shelf_blue"/>
@@ -91,12 +91,12 @@
     </link>
     <!-- JOINT -->
-    <joint name="${name}:shelf_piece_joint" type="fixed">
+    <joint name="${name}:joint" type="fixed">
       <xacro:insert_block name="origin" />
       <parent link="${parent}"/>
-      <child link="${name}:shelf_piece"/>
+      <child link="${name}"/>
     </joint>
   </xacro:macro>
   <xacro:macro name="suturo_shelf_left_door_openable" params="name parent *origin size_x size_y size_z shelf_x_size">
-    <link name="${name}:shelf_link">
+    <link name="${name}">
       <visual>
         <material name="shelf_door_green"/>
@@ -113,5 +113,5 @@
       </collision>
     </link>
-    <link name="${name}:shelf_link_handle">
+    <link name="${name}:handle">
       <visual>
         <material name="shelf_openable_handle_red"/>
@@ -128,20 +128,20 @@
       </collision>
     </link>
-    <joint name="${name}:shelf_link_handle_joint" type="fixed">
+    <joint name="${name}:handle_joint" type="fixed">
       <origin xyz="0.01 ${size_y - 0.04} ${size_z/3}" rpy="0 0 0"/>
       <axis xyz="0 0 1" />
-      <parent link="${name}:shelf_link"/>
-      <child link="${name}:shelf_link_handle"/>
-    </joint>
-    <joint name="${name}:shelf_joint" type="revolute">
+      <parent link="${name}"/>
+      <child link="${name}:handle"/>
+    </joint>
+    <joint name="${name}:joint" type="revolute">
       <origin xyz="${shelf_x_size/-2} 0 0" rpy="0 0 3.1416"/>
       <axis xyz="0 0 1" />
-      <parent link="${parent}:shelf_piece"/>
-      <child link="${name}:shelf_link"/>
+      <parent link="${parent}"/>
+      <child link="${name}"/>
       <limit effort="30" velocity="1.0" lower="-1.7" upper="0.0" />
     </joint>
   </xacro:macro>
   <xacro:macro name="suturo_shelf_right_door_openable" params="name parent *origin size_x size_y size_z shelf_x_size">
-    <link name="${name}:shelf_link">
+    <link name="${name}">
       <visual>
         <material name="shelf_door_green"/>
@@ -158,5 +158,5 @@
       </collision>
     </link>
-    <link name="${name}:shelf_link_handle">
+    <link name="${name}:handle">
       <visual>
         <material name="shelf_openable_handle_red"/>
@@ -173,15 +173,15 @@
       </collision>
     </link>
-    <joint name="${name}:shelf_link_handle_joint" type="fixed">
+    <joint name="${name}:handle_joint" type="fixed">
       <origin xyz="-0.01 ${size_y - 0.04} ${size_z/3}" rpy="0 0 0"/>
       <axis xyz="0 0 1" />
-      <parent link="${name}:shelf_link"/>
-      <child link="${name}:shelf_link_handle"/>
-    </joint>
-    <joint name="${name}:shelf_joint" type="revolute">
+      <parent link="${name}"/>
+      <child link="${name}:handle"/>
+    </joint>
+    <joint name="${name}:joint" type="revolute">
       <origin xyz="${shelf_x_size/-2} 0 0" rpy="0 0 0"/>
       <axis xyz="0 0 1" />
-      <parent link="${parent}:shelf_piece"/>
-      <child link="${name}:shelf_link"/>
+      <parent link="${parent}"/>
+      <child link="${name}"/>
       <limit effort="30" velocity="1.0" lower="0.0" upper="1.7" />
     </joint>
