Commit message: finish urdf door fic

File: suturo_resources/urdf/urdf_components/suturo_shelf_openable.urdf.xacro (robot description, xacro)
@@ -6,40 +6,40 @@
   <xacro:macro name="suturo_shelf_openable" params="name parent *origin size_x size_y size_z floors_height number_of_floors door">
     <!-- General conveinience links -->
-    <link name="${name}_origin"/>
-    <link name="${name}_center"/>
+    <link name="${name}_shelf_origin"/>
+    <link name="${name}_shelf_center"/>
     <link name="${name}_shelf_base_center"/>
-    <joint name="${name}_origin_joint" type="fixed">
+    <joint name="${name}_shelf_origin_joint" type="fixed">
       <xacro:insert_block name="origin" />
       <parent link="${parent}"/>
-      <child link="${name}_origin"/>
+      <child link="${name}_shelf_origin"/>
     </joint>
-    <joint name="${name}_center_joint" type="fixed">
+    <joint name="${name}_shelf_center_joint" type="fixed">
       <origin xyz="${size_x/2} ${size_y/2} ${size_z/2}" rpy="0 0 0" />
-      <parent link="${name}_origin"/>
-      <child link="${name}_center"/>
+      <parent link="${name}_shelf_origin"/>
+      <child link="${name}_shelf_center"/>
     </joint>
-    <joint name="${name}_base_center_joint" type="fixed">
+    <joint name="${name}_shelf_base_center_joint" type="fixed">
       <origin xyz="${size_x/2} ${size_y/2} 0.0" rpy="0 0 0" />
-      <parent link="${name}_origin"/>
+      <parent link="${name}_shelf_origin"/>
       <child link="${name}_shelf_base_center"/>
     </joint>
     <!-- WALLS -->
-    <xacro:suturo_shelf_piece name="${name}_back" parent="${name}_origin"
+    <xacro:suturo_shelf_piece_openable name="${name}_shelf_back" parent="${name}_shelf_origin"
       size_x="0.01" size_y="${size_y}" size_z="${size_z}">
       <origin xyz="${size_x} ${size_y/2} ${size_z/2}" rpy="0 0 0"/>
-    </xacro:suturo_shelf_piece>
-    <xacro:suturo_shelf_piece name="${name}_right_side" parent="${name}_origin"
+    </xacro:suturo_shelf_piece_openable>
+    <xacro:suturo_shelf_piece_openable name="${name}_shelf_right_side" parent="${name}_shelf_origin"
       size_x="${size_x}" size_y="0.01" size_z="${size_z}">
       <origin xyz="${size_x/2} 0.0 ${size_z/2}" rpy="0 0 0"/>
-    </xacro:suturo_shelf_piece>
-    <xacro:suturo_shelf_piece name="${name}_left_side" parent="${name}_origin"
+    </xacro:suturo_shelf_piece_openable>
+    <xacro:suturo_shelf_piece_openable name="${name}_shelf_left_side" parent="${name}_shelf_origin"
       size_x="${size_x}" size_y="0.01" size_z="${size_z}">
       <origin xyz="${size_x/2} ${size_y} ${size_z/2}" rpy="0 0 0"/>
-    </xacro:suturo_shelf_piece>
-    <xacro:macro name="shelf_floor_loop" params="floor_number">
-        <xacro:suturo_shelf_piece name="${name}_shelf_floor_${floor_number}" parent="${name}_shelf_base_center"
+    </xacro:suturo_shelf_piece_openable>
+    <xacro:macro name="shelf_floor_loop_openable" params="floor_number">
+        <xacro:suturo_shelf_piece_openable name="${name}_shelf_floor_${floor_number}" parent="${name}_shelf_base_center"
           size_x="${size_x}" size_y="${size_y}" size_z="0.04" box_z_offset="-0.02">
         <origin xyz="0.0 0.0 ${floors_height[floor_number]}" rpy="0 0 0"/>
-      </xacro:suturo_shelf_piece>
+      </xacro:suturo_shelf_piece_openable>
       <xacro:if value="${(number_of_floors - 1) > floor_number}">
             <xacro:shelf_floor_loop floor_number="${floor_number + 1}" />
@@ -49,21 +49,21 @@
     <!-- door -->
     <xacro:if value="${door == 'left'}">
-      <xacro:suturo_shelf_left_door name="${name}_door_left" parent="${name}_left_side"
+      <xacro:suturo_shelf_left_door_openable name="${name}_shelf_door_left" parent="${name}_shelf_left_side"
         size_x="0.01" size_y="${size_y/2}" size_z="${size_z}" shelf_x_size="${size_x}">
         <origin xyz="0 ${size_y*0.75} ${size_z/2}" rpy="0 0 0"/>
-      </xacro:suturo_shelf_left_door>
+      </xacro:suturo_shelf_left_door_openable>
     </xacro:if>
     <xacro:if value="${door == 'right'}">
-      <xacro:suturo_shelf_right_door name="${name}_door_right" parent="${name}_right_side"
+      <xacro:suturo_shelf_right_door_openable name="${name}_shelf_door_right" parent="${name}_shelf_right_side"
         size_x="0.01" size_y="${size_y/2}" size_z="${size_z}" shelf_x_size="${size_x}">
         <origin xyz="0 ${size_y*0.75} ${size_z/2}" rpy="0 0 0"/>
-      </xacro:suturo_shelf_right_door>
+      </xacro:suturo_shelf_right_door_openable>
     </xacro:if>
   </xacro:macro>
   <!-- Creates a link with collision and visual box of given dimensions,
   and a respective joint to append it to the parent with given origin.  -->
-  <xacro:macro name="suturo_shelf_piece" params="name parent *origin box_z_offset=0.0 size_x size_y size_z">
+  <xacro:macro name="suturo_shelf_piece_openable" params="name parent *origin box_z_offset=0.0 size_x size_y size_z">
     <!-- LINK -->
-    <link name="${name}_piece">
+    <link name="${name}_shelf_piece">
       <visual>
         <material name="shelf_blue"/>
@@ -81,12 +81,12 @@
     </link>
     <!-- JOINT -->
-    <joint name="${name}_piece_joint" type="fixed">
+    <joint name="${name}_shelf_piece_joint" type="fixed">
       <xacro:insert_block name="origin" />
       <parent link="${parent}"/>
-      <child link="${name}_piece"/>
+      <child link="${name}_shelf_piece"/>
     </joint>
   </xacro:macro>
-  <xacro:macro name="suturo_shelf_left_door" params="name parent *origin size_x size_y size_z shelf_x_size">
-    <link name="${name}_link">
+  <xacro:macro name="suturo_shelf_left_door_openable" params="name parent *origin size_x size_y size_z shelf_x_size">
+    <link name="${name}_shelf_link">
       <visual>
         <material name="shelf_door_green"/>
@@ -103,5 +103,5 @@
       </collision>
     </link>
-    <link name="${name}_link_handle">
+    <link name="${name}_shelf_link_handle">
       <visual>
         <material name="handle_red"/>
@@ -118,20 +118,20 @@
       </collision>
     </link>
-    <joint name="${name}_link_handle_joint" type="fixed">
+    <joint name="${name}_shelf_link_handle_joint" type="fixed">
       <origin xyz="-0.01 ${size_y - 0.04} ${size_z/3}" rpy="0 0 0"/>
       <axis xyz="0 0 1" />
-      <parent link="${name}_link"/>
-      <child link="${name}_link_handle"/>
+      <parent link="${name}_shelf_link"/>
+      <child link="${name}_shelf_link_handle"/>
     </joint>
-    <joint name="${name}_joint" type="revolute">
+    <joint name="${name}_shelf_joint" type="revolute">
       <origin xyz="${shelf_x_size/-2} 0 0" rpy="0 0 3.1416"/>
       <axis xyz="0 0 1" />
-      <parent link="${parent}_piece"/>
-      <child link="${name}_link"/>
+      <parent link="${parent}_shelf_piece"/>
+      <child link="${name}_shelf_link"/>
       <limit effort="30" velocity="1.0" lower="0.0" upper="1.91986" />
     </joint>
   </xacro:macro>
-  <xacro:macro name="suturo_shelf_right_door" params="name parent *origin size_x size_y size_z shelf_x_size">
-    <link name="${name}_link">
+  <xacro:macro name="suturo_shelf_right_door_openable" params="name parent *origin size_x size_y size_z shelf_x_size">
+    <link name="${name}_shelf_link">
       <visual>
         <material name="shelf_door_green"/>
@@ -148,9 +148,9 @@
       </collision>
     </link>
-    <joint name="${name}_joint" type="revolute">
+    <joint name="${name}_shelf_joint" type="revolute">
       <origin xyz="${shelf_x_size/-2} ${size_y/2} 0" rpy="0 0 -3.1416"/>
       <axis xyz="0 0 1" />
-      <parent link="${parent}_piece"/>
-      <child link="${name}_link"/>
+      <parent link="${parent}_shelf_piece"/>
+      <child link="${name}_shelf_link"/>
       <limit effort="30" velocity="1.0" lower="0.0" upper="1.91986" />
     </joint>

Commit message: adjusted materialname and remapped base_scan

File: suturo_resources/urdf/urdf_components/suturo_shelf_openable.urdf.xacro (robot description, xacro)
@@ -1,5 +1,5 @@
 <?xml version="1.0"?>
 <robot name="suturo_shelf" xmlns:xacro="http://ros.org/wiki/xacro">
-  <material name="handle_red">
+  <material name="shelf_openable_handle_red">
     <color rgba="0.74 0.25 0.25 1"/>
   </material>
@@ -105,5 +105,5 @@
     <link name="${name}_shelf_link_handle">
       <visual>
-        <material name="handle_red"/>
+        <material name="shelf_openable_handle_red"/>
         <origin xyz="0 0 0" rpy="0 0 0" />
         <geometry>

Commit message: fixed naming bug

File: suturo_resources/urdf/urdf_components/suturo_shelf_openable.urdf.xacro (robot description, xacro)
@@ -65,5 +65,5 @@
   <xacro:macro name="suturo_shelf_piece_openable" params="name parent *origin box_z_offset=0.0 size_x size_y size_z">
     <!-- LINK -->
-    <link name="${name}#shelf_piece">
+    <link name="${name}:shelf_piece">
       <visual>
         <material name="shelf_blue"/>

Commit message: fix handle position

File: suturo_resources/urdf/urdf_components/suturo_shelf_openable.urdf.xacro (robot description, xacro)
@@ -135,5 +135,5 @@
     </link>
     <joint name="${name}:handle_joint" type="fixed">
-      <origin xyz="${-wall_thickness-handle_depth/2} ${-handle_from_side} ${handle_from_bottom-size_z/2}" rpy="0 0 0"/>
+      <origin xyz="${-wall_thickness-handle_depth/2} ${-handle_from_side-handle_width/2} ${handle_from_bottom-size_z/2+handle_height/2}" rpy="0 0 0"/>
       <axis xyz="0 0 1" />
       <parent link="${name}"/>
@@ -181,5 +181,5 @@
     </link>
     <joint name="${name}:handle_joint" type="fixed">
-      <origin xyz="${-wall_thickness-handle_depth/2} ${+handle_from_side} ${handle_from_bottom-size_z/2}" rpy="0 0 0"/>
+      <origin xyz="${-wall_thickness-handle_depth/2} ${+handle_from_side+handle_width/2} ${handle_from_bottom-size_z/2+handle_height/2}" rpy="0 0 0"/>
       <axis xyz="0 0 1" />
       <parent link="${name}"/>

Commit message: Fix door not being insiede shelf

File: suturo_resources/urdf/urdf_components/suturo_shelf_openable.urdf.xacro (robot description, xacro)
@@ -141,5 +141,5 @@
     </joint>
     <joint name="${name}:joint" type="revolute">
-      <origin xyz="${shelf_x_size/-2} ${-wall_thickness} 0" rpy="0 0 0"/>
+      <origin xyz="${-shelf_x_size/2+wall_thickness/2} ${-wall_thickness} 0" rpy="0 0 0"/>
       <axis xyz="0 0 1" />
       <parent link="${parent}"/>
@@ -187,5 +187,5 @@
     </joint>
     <joint name="${name}:joint" type="revolute">
-      <origin xyz="${shelf_x_size/-2} ${wall_thickness} 0" rpy="0 0 0"/>
+      <origin xyz="${-shelf_x_size/2+wall_thickness/2} ${wall_thickness} 0" rpy="0 0 0"/>
       <axis xyz="0 0 1" />
       <parent link="${parent}"/>
