Commit message: fix: round_table in robocup semantic map

File: suturo_resources/urdf/urdf_components/suturo_round_table.urdf.xacro (robot description, xacro)
@@ -35,5 +35,5 @@
     </joint>
     <joint name="${name}:table_front_edge_center_joint" type="fixed">
-      <origin xyz="0 0 0" rpy="0 0 0" />
+      <origin xyz="0 0 ${length}" rpy="0 0 0" />
       <parent link="${name}:table_origin"/>
       <child link="${name}:table_front_edge_center"/>
