Commit message: fix table collision box pose

File: suturo_resources/urdf/urdf_components/suturo_table.urdf.xacro (robot description, xacro)
@@ -15,5 +15,5 @@
       </visual>
       <collision>
-        <origin xyz="0 0 0" rpy="0 0 0" />
+        <origin xyz="0 0 ${-(size_z)/2}" rpy="0 0 0" />
         <geometry>
           <box size="${size_x} ${size_y} ${size_z}" />

Commit message: - service definitions changed - pyhthon3 instead of python - added new color to table

File: suturo_resources/urdf/urdf_components/suturo_table.urdf.xacro (robot description, xacro)
@@ -1,6 +1,10 @@
 <?xml version="1.0"?>
 <robot name="suturo_table" xmlns:xacro="http://ros.org/wiki/xacro">
+  <!--<material name="table_grey">
+    <color rgba="0.8 0.8 0.8 1"/>
+  </material>
+  -->
   <material name="table_grey">
-    <color rgba="0.8 0.8 0.8 1"/>
+	<color rgba="0.255 0.62 0.223 1"/>
   </material>
   <xacro:macro name="suturo_table" params="name parent *origin size_x size_y size_z">
