Commit message: fixed some positions to match the real world objects

File: suturo_resources/urdf/urdf_components/suturo_kitchen.urdf.xacro (robot description, xacro)
@@ -1309,5 +1309,5 @@
   </joint>
   <joint name="kitchen_island_joint" type="fixed">
-    <origin rpy="0 0 0" xyz="0.2975 1.1292 0.421"/>
+    <origin rpy="0 0 0" xyz="0.2975 1.05 0.421"/>
     <parent link="kitchen_island_footprint"/>
     <child link="kitchen_island"/>
