Commit message: updated semantic map and added launch for simulation and vanessa deleted files

File: suturo_resources/urdf/urdf_components/suturo_environment_new.urdf.xacro (robot description, xacro)
@@ -39,6 +39,4 @@
     <xacro:property name="number_of_tables"
         value="${data.get('tables', dict(amount=0)).get('amount', 0)}" />
-    <xacro:property name="number_of_couches"
-        value="${data.get('couch', dict(amount=0)).get('amount', 0)}" />
     <xacro:property name="number_of_round_tables"
         value="${data.get('round_tables', dict(amount=0)).get('amount', 0)}" />
@@ -75,20 +73,4 @@
         </xacro:if>
     </xacro:macro>
-      <!--  ~~Couches~~  -->
-    <xacro:macro name="couch_loop" params="couch_number">
-        <xacro:suturo_couch
-            name="${data['couch'][couch_number]['name']}:${data['couch'][couch_number]['knowledge_role']}"
-            parent="${data['couch'][couch_number]['parent']}"
-            size_x="${data['couch'][couch_number]['depth']}"
-            size_y="${data['couch'][couch_number]['width']}"
-            size_z="${data['couch'][couch_number]['height']}">
-            <origin
-                xyz="${data['couch'][couch_number]['x_pos']} ${data['couch'][couch_number]['y_pos']} 0"
-                rpy="0 0 ${data['couch'][couch_number]['z_rot']}" />
-        </xacro:suturo_couch>
-        <xacro:if value="${(number_of_couches - 1) > couch_number}">
-            <xacro:couch_loop couch_number="${couch_number + 1}" />
-        </xacro:if>
-    </xacro:macro>
     <!--  ~~Round_tables~~  -->
     <xacro:macro name="round_table_loop" params="round_table_number">
@@ -288,7 +270,4 @@
         <xacro:table_loop table_number="0" />
     </xacro:if>
-    <xacro:if value="${number_of_couches > 0}">
-        <xacro:couch_loop couch_number="0" />
-    </xacro:if>
     <xacro:if value="${number_of_round_tables > 0}">
         <xacro:round_table_loop round_table_number="0" />

Commit message: new semantic map without the whole detailed kitchen

File: suturo_resources/urdf/urdf_components/suturo_environment_new.urdf.xacro (robot description, xacro)
@@ -30,6 +30,4 @@
     <xacro:include
         filename="$(find suturo_resources)/urdf/urdf_components/suturo_simple_drawer.urdf.xacro" />
-    <xacro:include
-        filename="$(find suturo_resources)/urdf/urdf_components/suturo_dishwasher.urdf.xacro" />
     <!-- general data -->
     <xacro:property name="number_of_drawers"
@@ -55,6 +53,6 @@
     <xacro:property name="number_of_paths"
         value="${data.get('paths', dict(amount=0)).get('amount', 0)}" />
-    <xacro:property name="number_of_dishwashers"
-        value="${data.get('dishwashers', dict(amount=0)).get('amount', 0)}" />
+    <!--<xacro:property name="number_of_dishwashers"
+        value="${data.get('dishwashers', dict(amount=0)).get('amount', 0)}" /> -->
     <!--  ~~Tables~~  -->
     <xacro:macro name="table_loop" params="table_number">
@@ -88,5 +86,6 @@
         </xacro:if>
     </xacro:macro>
-    <!--  ~~Dishwashers~~  -->
+    <!--
+     ~~Dishwashers~~
     <xacro:macro name="dishwasher_loop" params="dishwasher_number">
         <xacro:suturo_dishwasher
@@ -101,4 +100,5 @@
         </xacro:if>
     </xacro:macro>
+-->
     <!--  ~~Bucket~~  -->
     <xacro:macro name="bucket_loop" params="bucket_number">

File: suturo_resources/urdf/urdf_components/suturo_kitchen.urdf.xacro (robot description, xacro)
@@ -14,326 +14,9 @@
 	  <child link="kitchen_main"/>
     </joint>
-    <link name="sink_area_footprint">
-    <inertial>
-      <origin rpy="0 0 0" xyz="0.0 0.0 0.0"/>
-      <mass value="1"/>
-      <inertia ixx="1" ixy="0.0" ixz="0.0" iyy="1" iyz="0.0" izz="1"/>
-    </inertial>
-  </link>
-  <link name="sink_area">
-    <inertial>
-      <origin rpy="0 0 0" xyz="0.0 0.0 0.0"/>
-      <mass value="1"/>
-      <inertia ixx="1" ixy="0.0" ixz="0.0" iyy="1" iyz="0.0" izz="1"/>
-    </inertial>
-    <visual>
-      <origin rpy="0 0 0" xyz="0 0 0"/>
-      <geometry>
-        <mesh filename="package://iai_kitchen/meshes/racks/SinkArea.obj"/>
-      </geometry>
-    </visual>
-    <collision>
-      <origin rpy="0 0 0" xyz="0 0 0"/>
-      <geometry>
-        <mesh filename="package://iai_kitchen/meshes/racks/SinkArea.obj"/>
-      </geometry>
-    </collision>
-  </link>
-  <joint name="sink_area_footprint_joint" type="fixed">
-    <origin rpy="0 0 3.14159265359" xyz="1.825 1.32 0"/>
-    <child link="sink_area_footprint"/>
-    <parent link="kitchen_main"/>
-  </joint>
-  <joint name="sink_area_main_joint" type="fixed">
-    <origin rpy="0 0 0" xyz="0.29 1.03 0.41"/>
-    <parent link="sink_area_footprint"/>
-    <child link="sink_area"/>
-  </joint>
-  <link name="sink_area_surface">
-    <inertial>
-      <origin rpy="0 0 0" xyz="0.0 0.0 0.0"/>
-      <mass value="1"/>
-      <inertia ixx="1" ixy="0.0" ixz="0.0" iyy="1" iyz="0.0" izz="1"/>
-    </inertial>
-    <collision>
-      <origin rpy="0 0 0" xyz="0 -0.225 0"/>
-      <geometry>
-        <box size="0.575 1.6 0.02"/>
-      </geometry>
-    </collision>
-  </link>
-  <joint name="sink_area_surface_joint" type="fixed">
-    <origin rpy="0 0 0" xyz="0.0 0. 0.43"/>
-    <parent link="sink_area"/>
-    <child link="sink_area_surface"/>
-  </joint>
-  <link name="sink_area_sink">
-    <inertial>
-      <origin rpy="0 0 0" xyz="0.0 0.0 0.0"/>
-      <mass value="1"/>
-      <inertia ixx="1" ixy="0.0" ixz="0.0" iyy="1" iyz="0.0" izz="1"/>
-    </inertial>
-    <visual>
-      <origin rpy="0 0 0" xyz="0 0 0"/>
-      <geometry>
-        <mesh filename="package://iai_kitchen/meshes/misc/Sink.obj"/>
-      </geometry>
-    </visual>
-    <collision>
-      <origin rpy="0 0 0" xyz="0 0 0"/>
-      <geometry>
-        <mesh filename="package://iai_kitchen/meshes/misc/Sink.obj"/>
-      </geometry>
-    </collision>
-  </link>
-  <joint name="sink_area_sink_joint" type="fixed">
-    <origin rpy="0 0 0" xyz="0.005 0.47 0.4414"/>
-    <parent link="sink_area"/>
-    <child link="sink_area_sink"/>
-  </joint>
-  <link name="sink_area_right_panel">
-    <inertial>
-      <origin rpy="0 0 0" xyz="0.0 0.0 0.0"/>
-      <mass value="1"/>
-      <inertia ixx="1" ixy="0.0" ixz="0.0" iyy="1" iyz="0.0" izz="1"/>
-    </inertial>
-    <visual>
-      <origin rpy="0 0 0" xyz="0 0 0"/>
-      <geometry>
-        <mesh filename="package://iai_kitchen/meshes/drawers/Panel_60.obj"/>
-      </geometry>
-    </visual>
-    <collision>
-      <origin rpy="0 0 0" xyz="0 0 0"/>
-      <geometry>
-        <mesh filename="package://iai_kitchen/meshes/drawers/Panel_60.obj"/>
-      </geometry>
-    </collision>
-  </link>
-  <joint name="sink_area_right_panel_joint" type="fixed">
-    <origin rpy="0 0 0" xyz="0.28 0.7 0.355 "/>
-    <parent link="sink_area"/>
-    <child link="sink_area_right_panel"/>
-  </joint>
-  <link name="sink_area_trash_drawer_main">
-    <inertial>
-      <origin rpy="0 0 0" xyz="0.0 0.0 0.0"/>
-      <mass value="1"/>
-      <inertia ixx="1" ixy="0.0" ixz="0.0" iyy="1" iyz="0.0" izz="1"/>
-    </inertial>
-    <visual>
-      <origin rpy="0 0 0" xyz="0 0 0"/>
-      <geometry>
-        <mesh filename="package://iai_kitchen/meshes/drawers/Drawer_60_58.obj"/>
-      </geometry>
-    </visual>
-    <collision>
-      <origin rpy="0 0 0" xyz="0 0 0"/>
-      <geometry>
-        <mesh filename="package://iai_kitchen/meshes/drawers/Drawer_60_58.obj"/>
-      </geometry>
-    </collision>
-  </link>
-  <link name="sink_area_trash_drawer_handle">
-    <inertial>
-      <origin rpy="0 0 0" xyz="0.0 0.0 0.0"/>
-      <mass value="1"/>
-      <inertia ixx="1" ixy="0.0" ixz="0.0" iyy="1" iyz="0.0" izz="1"/>
-    </inertial>
-    <visual>
-      <origin rpy="0 0 0" xyz="0 0 0"/>
-      <geometry>
-        <mesh filename="package://iai_kitchen/meshes/handles/Handle60.obj"/>
-      </geometry>
-    </visual>
-    <collision>
-      <origin rpy="0 0 0" xyz="0 0 0"/>
-      <geometry>
-        <mesh filename="package://iai_kitchen/meshes/handles/Handle60.obj"/>
-      </geometry>
-    </collision>
-  </link>
-  <joint name="sink_area_trash_drawer_main_joint" type="prismatic">
-    <origin rpy="0 0 0" xyz="0.01 0.7 -0.015 "/>
-    <parent link="sink_area"/>
-    <child link="sink_area_trash_drawer_main"/>
-    <axis xyz="1. 0. 0.0"/>
-    <limit effort="300" lower="0" upper="0.48" velocity="10"/>
-    <!--
-    <limit effort="300" lower="0" upper="0" velocity="10"/>
--->
-  </joint>
-  <joint name="sink_area_trash_drawer_handle_joint" type="fixed">
-    <origin rpy="0 0 0" xyz="0.3325 0 0.2375"/>
-    <parent link="sink_area_trash_drawer_main"/>
-    <child link="sink_area_trash_drawer_handle"/>
-    <axis xyz="0 0 1"/>
-    <limit effort="300" lower="0" upper="1.57079632679" velocity="10"/>
-  </joint>
-  <link name="sink_area_left_upper_drawer_main">
-    <inertial>
-      <origin rpy="0 0 0" xyz="0.0 0.0 0.0"/>
-      <mass value="1"/>
-      <inertia ixx="1" ixy="0.0" ixz="0.0" iyy="1" iyz="0.0" izz="1"/>
-    </inertial>
-    <visual>
-      <origin rpy="0 0 0" xyz="0 0 0"/>
-      <geometry>
-        <mesh filename="package://iai_kitchen/meshes/drawers/Drawer_80_14.obj"/>
-      </geometry>
-    </visual>
-    <collision>
-      <origin rpy="0 0 0" xyz="0 0 0"/>
-      <geometry>
-        <mesh filename="package://iai_kitchen/meshes/drawers/Drawer_80_14.obj"/>
-      </geometry>
-    </collision>
-  </link>
-  <link name="sink_area_left_upper_drawer_handle">
-    <inertial>
-      <origin rpy="0 0 0" xyz="0.0 0.0 0.0"/>
-      <mass value="1"/>
-      <inertia ixx="1" ixy="0.0" ixz="0.0" iyy="1" iyz="0.0" izz="1"/>
-    </inertial>
-    <visual>
-      <origin rpy="0 0 0" xyz="0 0 0"/>
-      <geometry>
-        <mesh filename="package://iai_kitchen/meshes/handles/Handle80.obj"/>
-      </geometry>
-    </visual>
-    <collision>
-      <origin rpy="0 0 0" xyz="0 0 0"/>
-      <geometry>
-        <mesh filename="package://iai_kitchen/meshes/handles/Handle80.obj"/>
-      </geometry>
-    </collision>
-  </link>
-  <joint name="sink_area_left_upper_drawer_main_joint" type="prismatic">
-    <origin rpy="0 0 0" xyz="0.01 -0.6 0.345 "/>
-    <parent link="sink_area"/>
-    <child link="sink_area_left_upper_drawer_main"/>
-    <axis xyz="1. 0. 0.0"/>
-    <limit effort="300" lower="0" upper="0.48" velocity="10"/>
-    <!--
-    <limit effort="300" lower="0" upper="0" velocity="10"/>
--->
-  </joint>
-  <joint name="sink_area_left_upper_drawer_handle_joint" type="fixed">
-    <origin rpy="0 0 0" xyz="0.3325 0 0.0175"/>
-    <parent link="sink_area_left_upper_drawer_main"/>
-    <child link="sink_area_left_upper_drawer_handle"/>
-    <axis xyz="0 0 1"/>
-    <limit effort="300" lower="0" upper="1.57079632679" velocity="10"/>
-  </joint>
-  <link name="sink_area_left_middle_drawer_main">
-    <inertial>
-      <origin rpy="0 0 0" xyz="0.0 0.0 0.0"/>
-      <mass value="1"/>
-      <inertia ixx="1" ixy="0.0" ixz="0.0" iyy="1" iyz="0.0" izz="1"/>
-    </inertial>
-    <visual>
-      <origin rpy="0 0 0" xyz="0 0 0"/>
-      <geometry>
-        <mesh filename="package://iai_kitchen/meshes/drawers/Drawer_80_29.obj"/>
-      </geometry>
-    </visual>
-    <collision>
-      <origin rpy="0 0 0" xyz="0 0 0"/>
-      <geometry>
-        <mesh filename="package://iai_kitchen/meshes/drawers/Drawer_80_29.obj"/>
-      </geometry>
-    </collision>
-  </link>
-  <link name="sink_area_left_middle_drawer_handle">
-    <inertial>
-      <origin rpy="0 0 0" xyz="0.0 0.0 0.0"/>
-      <mass value="1"/>
-      <inertia ixx="1" ixy="0.0" ixz="0.0" iyy="1" iyz="0.0" izz="1"/>
-    </inertial>
-    <visual>
-      <origin rpy="0 0 0" xyz="0 0 0"/>
-      <geometry>
-        <mesh filename="package://iai_kitchen/meshes/handles/Handle80.obj"/>
-      </geometry>
-    </visual>
-    <collision>
-      <origin rpy="0 0 0" xyz="0 0 0"/>
-      <geometry>
-        <mesh filename="package://iai_kitchen/meshes/handles/Handle80.obj"/>
-      </geometry>
-    </collision>
-  </link>
-  <joint name="sink_area_left_middle_drawer_main_joint" type="prismatic">
-    <origin rpy="0 0 0" xyz="0.01 -0.6 0.12 "/>
-    <parent link="sink_area"/>
-    <child link="sink_area_left_middle_drawer_main"/>
-    <axis xyz="1. 0. 0.0"/>
-    <limit effort="300" lower="0" upper="0.48" velocity="10"/>
-    <!--
-    <limit effort="300" lower="0" upper="0" velocity="10"/>
--->
-  </joint>
-  <joint name="sink_area_left_middle_drawer_handle_joint" type="fixed">
-    <origin rpy="0 0 0" xyz="0.3325 0 0.11"/>
-    <parent link="sink_area_left_middle_drawer_main"/>
-    <child link="sink_area_left_middle_drawer_handle"/>
-    <axis xyz="0 0 1"/>
-    <limit effort="300" lower="0" upper="1.57079632679" velocity="10"/>
-  </joint>
-  <link name="sink_area_left_bottom_drawer_main">
-    <inertial>
-      <origin rpy="0 0 0" xyz="0.0 0.0 0.0"/>
-      <mass value="1"/>
-      <inertia ixx="1" ixy="0.0" ixz="0.0" iyy="1" iyz="0.0" izz="1"/>
-    </inertial>
-    <visual>
-      <origin rpy="0 0 0" xyz="0 0 0"/>
-      <geometry>
-        <mesh filename="package://iai_kitchen/meshes/drawers/Drawer_80_29.obj"/>
-      </geometry>
-    </visual>
-    <collision>
-      <origin rpy="0 0 0" xyz="0 0 0"/>
-      <geometry>
-        <mesh filename="package://iai_kitchen/meshes/drawers/Drawer_80_29.obj"/>
-      </geometry>
-    </collision>
-  </link>
-  <link name="sink_area_left_bottom_drawer_handle">
-    <inertial>
-      <origin rpy="0 0 0" xyz="0.0 0.0 0.0"/>
-      <mass value="1"/>
-      <inertia ixx="1" ixy="0.0" ixz="0.0" iyy="1" iyz="0.0" izz="1"/>
-    </inertial>
-    <visual>
-      <origin rpy="0 0 0" xyz="0 0 0"/>
-      <geometry>
-        <mesh filename="package://iai_kitchen/meshes/handles/Handle80.obj"/>
-      </geometry>
-    </visual>
-    <collision>
-      <origin rpy="0 0 0" xyz="0 0 0"/>
-      <geometry>
-        <mesh filename="package://iai_kitchen/meshes/handles/Handle80.obj"/>
-      </geometry>
-    </collision>
-  </link>
-  <joint name="sink_area_left_bottom_drawer_main_joint" type="prismatic">
-    <origin rpy="0 0 0" xyz="0.01 -0.6 -0.18 "/>
-    <parent link="sink_area"/>
-    <child link="sink_area_left_bottom_drawer_main"/>
-    <axis xyz="1. 0. 0.0"/>
-    <limit effort="300" lower="0" upper="0.48" velocity="10"/>
-    <!--
-    <limit effort="300" lower="0" upper="0" velocity="10"/>
--->
-  </joint>
-  <joint name="sink_area_left_bottom_drawer_handle_joint" type="fixed">
-    <origin rpy="0 0 0" xyz="0.3325 0 0.11"/>
-    <parent link="sink_area_left_bottom_drawer_main"/>
-    <child link="sink_area_left_bottom_drawer_handle"/>
-    <axis xyz="0 0 1"/>
-    <limit effort="300" lower="0" upper="1.57079632679" velocity="10"/>
-  </joint>
+    <joint name="kitchen_main_joint" type="fixed">
+	  <xacro:insert_block name="origin" />
+	  <parent link="kitchen_main"/>
+	  <child link="sink_area_dish_washer_main"/>
+    </joint>
   <link name="sink_area_dish_washer_main">
     <inertial>
@@ -393,15 +76,21 @@
     </collision>
   </link>
-  <!--
+  	<link name="dishwasher_tab"/>
+	<!--
     <xacro:if value="simulated"/>
     -->
+	<joint name="dishwasher_tab_joint" type="fixed">
+	  <origin xyz="-0.1 0.1 0.15" rpy="0 0 0" />
+	  <parent link="sink_area_dish_washer_door_handle"/>
+      <child link="dishwasher_tab"/>
+	</joint>
   <joint name="sink_area_dish_washer_main_joint" type="fixed"> <!-- was revolute before, changed to fixed -->
     <axis xyz="1 0 0" />
     <!-- <limit effort="300" lower="0" upper="0" velocity="10"/> -->
-    <origin rpy="0 0 0" xyz="0.01 0.1 0.044 "/>
-    <parent link="sink_area"/>
+    <origin rpy="0 0 0" xyz="0.08 -0.78 0.44 "/>
+    <parent link="kitchen_main"/>
     <child link="sink_area_dish_washer_main"/>
   </joint>
-  <joint name="sink_area_dish_washer_door_joint" type="revolute">
+ <joint name="sink_area_dish_washer_door_joint" type="revolute">
     <origin rpy="-1.57079632679 0.03 0" xyz="0.27 0. -0.325"/>
     <parent link="sink_area_dish_washer_main"/>
@@ -417,1584 +106,4 @@
     <child link="sink_area_dish_washer_door_handle"/>
   </joint>
-  <link name="oven_area_area_footprint">
-    <inertial>
-      <origin rpy="0 0 0" xyz="0.0 0.0 0.0"/>
-      <mass value="1"/>
-      <inertia ixx="1" ixy="0.0" ixz="0.0" iyy="1" iyz="0.0" izz="1"/>
-    </inertial>
-  </link>
-  <link name="oven_area_area">
-    <inertial>
-      <origin rpy="0 0 0" xyz="0.0 0.0 0.0"/>
-      <mass value="1"/>
-      <inertia ixx="1" ixy="0.0" ixz="0.0" iyy="1" iyz="0.0" izz="1"/>
-    </inertial>
-    <visual>
-      <origin rpy="0 0 0" xyz="0 0 0"/>
-      <geometry>
-        <mesh filename="package://iai_kitchen/meshes/racks/OvenArea.obj"/>
-      </geometry>
-    </visual>
-    <collision>
-      <origin rpy="0 0 0" xyz="0 0 0"/>
-      <geometry>
-        <mesh filename="package://iai_kitchen/meshes/racks/OvenArea.obj"/>
-      </geometry>
-    </collision>
-  </link>
-  <joint name="oven_area_footprint_joint" type="fixed">
-    <origin rpy="0 0 3.14159265359" xyz="1.805 2.52 0"/>
-    <child link="oven_area_area_footprint"/>
-    <parent link="kitchen_main"/>
-  </joint>
-  <joint name="oven_area_main_joint" type="fixed">
-    <origin rpy="0 0 0" xyz="0.29 0.6 0.755"/>
-    <parent link="oven_area_area_footprint"/>
-    <child link="oven_area_area"/>
-  </joint>
-  <!-- LINKS -->
-  <link name="oven_area_oven_main">
-    <inertial>
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