Commit message: change room urdf to use -

File: suturo_resources/urdf/urdf_components/suturo_room.urdf.xacro (robot description, xacro)
@@ -4,10 +4,10 @@
   <xacro:macro name="suturo_room" params="name parent num_of_corners corners_x_pos corners_y_pos center_x center_y color">
     <!-- define a central joint to wich every corner is connected -->
-    <joint name="world_${name}_room_joint" type="fixed">
+    <joint name="world_${name}-room_joint" type="fixed">
         <origin xyz="${center_x} ${center_y} 0 " rpy="0 0 0" />
         <parent link="${parent}"/>
-        <child link="${name}_room_center_link"/>
+        <child link="${name}-room_center_link"/>
     </joint>
-    <link name="${name}_room_center_link">
+    <link name="${name}-room_center_link">
       <visual>
         <geometry>
@@ -21,10 +21,10 @@
     <!-- room loop to create every corner -->
     <xacro:macro name="corner_loop" params="loop_number">
-      <joint name="${name}_room_joint_${loop_number}" type="fixed">
+      <joint name="${name}-room_joint_${loop_number}" type="fixed">
           <origin xyz="${corners_x_pos[loop_number] - center_x} ${corners_y_pos[loop_number] - center_y} 0 " rpy="0 0 0" />
-          <parent link="${name}_room_center_link"/>
-          <child link="${name}_room_corner_${loop_number}_link"/>
+          <parent link="${name}-room_center_link"/>
+          <child link="${name}-room_corner_${loop_number}_link"/>
       </joint>
-      <link name="${name}_room_corner_${loop_number}_link" />
+      <link name="${name}-room_corner_${loop_number}_link" />
       <xacro:if value="${(num_of_corners - 1) > loop_number}">
         <xacro:corner_loop loop_number="${loop_number + 1}" />

Commit message: move room urdf location down to prevent z-fighting

File: suturo_resources/urdf/urdf_components/suturo_room.urdf.xacro (robot description, xacro)
@@ -13,5 +13,5 @@
   <xacro:macro name="suturo_room" params="name parent center_x center_y color size_x size_y connections">
     <joint name="world_${name}:room_joint" type="fixed">
-        <origin xyz="${center_x} ${center_y} -0.01 " rpy="0 0 0" />
+        <origin xyz="${center_x} ${center_y} -0.05 " rpy="0 0 0" />
         <parent link="${parent}"/>
         <child link="${name}:room_center_link"/>

Commit message: fix room color for different rooms

File: suturo_resources/urdf/urdf_components/suturo_room.urdf.xacro (robot description, xacro)
@@ -22,5 +22,5 @@
           <box size="${size_x} ${size_y} 0.01" />
         </geometry>
-        <material name="color">
+        <material name="${name}:color">
           <color rgba="${color}"/>
         </material>

Commit message: [semantic map] remove collision of room links

File: suturo_resources/urdf/urdf_components/suturo_room.urdf.xacro (robot description, xacro)
@@ -26,14 +26,4 @@
         </material>
       </visual>
-      <collision>
-        <geometry>
-          <box size="${size_x} ${size_y} 0.01" />
-        </geometry>
-      </collision>
-      <inertial>
-        <origin xyz="0 0 0" rpy="0 0 0"/>
-        <mass value="1.0"/>
-        <inertia ixx="0.1" ixy="0.0" ixz="0.0" iyy="0.1" iyz="0.0" izz="0.1"/>
-      </inertial>
     </link>
     <xacro:property name="number_of_connections" value="${connections['amount']}" />

Commit message: Revert "[semantic map] remove collision of room links"
This reverts commit 3f4ed95b32aa120dbe481ed5683a294437aa5812.

Knowledge needs the collision links for loading the rooms.

File: suturo_resources/urdf/urdf_components/suturo_room.urdf.xacro (robot description, xacro)
@@ -26,4 +26,14 @@
         </material>
       </visual>
+      <collision>
+        <geometry>
+          <box size="${size_x} ${size_y} 0.01" />
+        </geometry>
+      </collision>
+      <inertial>
+        <origin xyz="0 0 0" rpy="0 0 0"/>
+        <mass value="1.0"/>
+        <inertia ixx="0.1" ixy="0.0" ixz="0.0" iyy="0.1" iyz="0.0" izz="0.1"/>
+      </inertial>
     </link>
     <xacro:property name="number_of_connections" value="${connections['amount']}" />
