Commit message: hohc change and first step of the semantic map (kitchen counter and dishwasher missing)

File: suturo_resources/urdf/urdf_components/suturo_shelf_hohc.urdf.xacro (robot description, xacro)
@@ -50,40 +50,40 @@
     <!-- door -->
     <xacro:if value="${door == 'left'}">
-      <xacro:suturo_shelf_left_door_openable name="${name}:shelf_door_left" parent="${name}:shelf_left_side"
+      <xacro:suturo_shelf_left_door_openable_h name="${name}:shelf_door_left" parent="${name}:shelf_left_side"
        wall_thickness="${wall_thickness}" door_height="${door_height}" size_y="${door_width}" size_z="${door_length}" shelf_x_size="${size_x}"
        handle_from_bottom="${handle_from_bottom}" handle_from_side="${handle_from_side}" handle_height="${handle_height}" handle_width="${handle_width}" handle_depth="${handle_depth}">
         <origin xyz="0 ${size_y*0.75} ${size_z/2}" rpy="0 0 0"/>
-      </xacro:suturo_shelf_left_door_openable>
+      </xacro:suturo_shelf_left_door_openable_h>
     </xacro:if>
     <xacro:if value="${door == 'right'}">
-      <xacro:suturo_shelf_right_door_openable name="${name}:shelf_door_right" parent="${name}:shelf_right_side"
+      <xacro:suturo_shelf_right_door_openable_h name="${name}:shelf_door_right" parent="${name}:shelf_right_side"
         wall_thickness="${wall_thickness}" door_height="${door_height}" size_y="${door_width}" size_z="${door_length}" shelf_x_size="${size_x}"
        handle_from_bottom="${handle_from_bottom}" handle_from_side="${handle_from_side}" handle_height="${handle_height}" handle_width="${handle_width}" handle_depth="${handle_depth}">
         <origin xyz="0 ${size_y*0.75} ${door_length/2}" rpy="0 0 0"/>
-      </xacro:suturo_shelf_right_door_openable>
+      </xacro:suturo_shelf_right_door_openable_h>
     </xacro:if>
     <xacro:if value="${door == 'both'}">
-       <xacro:suturo_shelf_right_door_openable name="${name}:shelf_door_right" parent="${name}:shelf_right_side"
+       <xacro:suturo_shelf_right_door_openable_h name="${name}:shelf_door_right" parent="${name}:shelf_right_side"
         wall_thickness="${wall_thickness}" door_height="${door_height}" size_y="${door_width}" size_z="${door_length}" shelf_x_size="${size_x}"
        handle_from_bottom="${handle_from_bottom}" handle_from_side="${handle_from_side}" handle_height="${handle_height}" handle_width="${handle_width}" handle_depth="${handle_depth}">
         <origin xyz="0 ${size_y} ${door_length/2}" rpy="0 0 0"/>
-       </xacro:suturo_shelf_right_door_openable>
-         <xacro:suturo_shelf_left_door_openable name="${name}:shelf_door_left" parent="${name}:shelf_left_side"
+       </xacro:suturo_shelf_right_door_openable_h>
+         <xacro:suturo_shelf_left_door_openable_h name="${name}:shelf_door_left" parent="${name}:shelf_left_side"
           wall_thickness="${wall_thickness}" door_height="${door_height}" size_y="${door_width}" size_z="${door_length}" shelf_x_size="${size_x}"
 	  handle_from_bottom="${handle_from_bottom}" handle_from_side="${handle_from_side}" handle_height="${handle_height}" handle_width="${handle_width}" handle_depth="${handle_depth}">
         <origin xyz="0 ${size_y} ${door_length/2}" rpy="0 0 0"/>
-      </xacro:suturo_shelf_left_door_openable>
+      </xacro:suturo_shelf_left_door_openable_h>
     </xacro:if>
     <xacro:if value="${door == 'both_open'}">
-       <xacro:suturo_shelf_right_door_openable name="${name}:shelf_door_right" parent="${name}:shelf_right_side"
+       <xacro:suturo_shelf_right_door_openable_h name="${name}:shelf_door_right" parent="${name}:shelf_right_side"
         wall_thickness="${wall_thickness}" door_height="${door_height}" size_y="${door_width}" size_z="${door_length}" shelf_x_size="${size_x}"
        handle_from_bottom="${handle_from_bottom}" handle_from_side="${handle_from_side}" handle_height="${handle_height}" handle_width="${handle_width}" handle_depth="${handle_depth}">
         <origin xyz="0 ${size_y} ${door_length/2}" rpy="0 0 0"/>
-       </xacro:suturo_shelf_right_door_openable>
-         <xacro:suturo_shelf_left_door_openable name="${name}:shelf_door_left" parent="${name}:shelf_left_side"
+       </xacro:suturo_shelf_right_door_openable_h>
+         <xacro:suturo_shelf_left_door_openable_h name="${name}:shelf_door_left" parent="${name}:shelf_left_side"
           wall_thickness="${wall_thickness}" door_height="${door_height}" size_y="${door_width}" size_z="${door_length}" shelf_x_size="${size_x}"
 	  handle_from_bottom="${handle_from_bottom}" handle_from_side="${handle_from_side}" handle_height="${handle_height}" handle_width="${handle_width}" handle_depth="${handle_depth}">
         <origin xyz="0 ${size_y} ${door_length/2}" rpy="0 0 0"/>
-      </xacro:suturo_shelf_left_door_openable>
+      </xacro:suturo_shelf_left_door_openable_h>
     </xacro:if>
   </xacro:macro>
@@ -119,5 +119,5 @@
     </joint>
   </xacro:macro>
-  <xacro:macro name="suturo_shelf_left_door_openable" params="name parent *origin wall_thickness door_height size_y size_z shelf_x_size handle_from_bottom handle_from_side handle_height handle_width handle_depth">
+  <xacro:macro name="suturo_shelf_left_door_openable_h" params="name parent *origin wall_thickness door_height size_y size_z shelf_x_size handle_from_bottom handle_from_side handle_height handle_width handle_depth">
     <xacro:property name="size_x" value="${wall_thickness}"/>
     <link name="${name}">
@@ -186,5 +186,5 @@
     </xacro:if>
   </xacro:macro>
-  <xacro:macro name="suturo_shelf_right_door_openable" params="name parent *origin wall_thickness door_height size_y size_z shelf_x_size handle_from_bottom handle_from_side handle_height handle_width handle_depth">
+  <xacro:macro name="suturo_shelf_right_door_openable_h" params="name parent *origin wall_thickness door_height size_y size_z shelf_x_size handle_from_bottom handle_from_side handle_height handle_width handle_depth">
     <xacro:property name="size_x" value="${wall_thickness}"/>
     <link name="${name}">
@@ -253,5 +253,5 @@
     </xacro:if>
   </xacro:macro>
-  <!-- <xacro:macro name="suturo_shelf_right_door_openable" params="name parent *origin size_x size_y size_z shelf_x_size"> -->
+  <!-- <xacro:macro name="suturo_shelf_right_door_openable_h" params="name parent *origin size_x size_y size_z shelf_x_size"> -->
   <!--   <link name="${name}:shelf_link"> -->
   <!--     <visual> -->
