Commit message: [Robocup] Semantic map adjusted with point cloud, more fixes needed

File: suturo_resources/urdf/urdf_components/suturo_dishwasher_robocup.urdf.xacro (robot description, xacro)
@@ -131,5 +131,5 @@
   </joint>
   <joint name="sink_area_dish_washer_door_handle_joint" type="fixed">
-    <origin rpy="-1.57079632679 0 0" xyz="0.0625 -0.6325 0."/>
+    <origin rpy="-1.57079632679 0 0" xyz="0.0625 -0.6625 0."/>
     <parent link="sink_area_dish_washer_door"/>
     <child link="sink_area_dish_washer_door_handle"/>
