Commit message: - no more table objects

File: suturo_resources/urdf/urdf_components/suturo_coathanger.urdf.xacro (robot description, xacro)
@@ -10,7 +10,7 @@
   <xacro:macro name="suturo_coathanger" params="name parent *origin size_x size_y size_z">
     <!-- LINKS -->
-    <link name="${name}:table_center">
+    <link name="${name}:coathanger_center">
       <visual>
-        <material name="table_grey"/>
+        <material name="coathanger_color"/>
         <origin xyz="0 0 ${-(size_z)/2}" rpy="0 0 0" />
         <geometry>
@@ -30,21 +30,21 @@
       </inertial>
     </link>
-    <link name="${name}:table_origin"/>
-    <link name="${name}:table_front_edge_center"/>
+    <link name="${name}:coathanger_origin"/>
+    <link name="${name}:coathanger_front_edge_center"/>
     <!-- JOINTS -->
-    <joint name="${name}:table_origin_joint" type="fixed">
+    <joint name="${name}:coathanger_origin_joint" type="fixed">
       <xacro:insert_block name="origin" />
       <parent link="${parent}"/>
-      <child link="${name}:table_origin"/>
+      <child link="${name}:coathanger_origin"/>
     </joint>
     <joint name="${name}:center_joint" type="fixed">
       <origin xyz="${size_x/2} ${size_y/2} ${size_z}" rpy="0 0 0" />
-      <parent link="${name}:table_origin"/>
-      <child link="${name}:table_center"/>
+      <parent link="${name}:coathanger_origin"/>
+      <child link="${name}:coathanger_center"/>
     </joint>
-    <joint name="${name}:table_front_edge_center_joint" type="fixed">
+    <joint name="${name}:coathanger_front_edge_center_joint" type="fixed">
       <origin xyz="0 ${size_y/2} ${size_z}" rpy="0 0 0" />
-      <parent link="${name}:table_origin"/>
-      <child link="${name}:table_front_edge_center"/>
+      <parent link="${name}:coathanger_origin"/>
+      <child link="${name}:coathanger_front_edge_center"/>
     </joint>
   </xacro:macro>

File: suturo_resources/urdf/urdf_components/suturo_trashbin.urdf.xacro (robot description, xacro)
@@ -1,12 +1,12 @@
 <?xml version="1.0"?>
 <robot name="suturo_trashbin" xmlns:xacro="http://ros.org/wiki/xacro">
-  <material name="trashbin_grey">
+  <material name="trashbin_color">
     <color rgba="0.8 0.8 0.8 1"/>
   </material>
   <xacro:macro name="suturo_trashbin" params="name parent *origin radius length">
     <!-- LINKS -->
-    <link name="${name}:table_center">
+    <link name="${name}:trashbin_center">
       <visual>
-        <material name="round_table_grey"/>
+        <material name="trashbin_color"/>
         <origin xyz="0 0 ${-(length)/2}" rpy="0 0 0" />
         <geometry>
@@ -26,21 +26,21 @@
       </inertial>
     </link>
-    <link name="${name}:table_origin"/>
-    <link name="${name}:table_front_edge_center"/>
+    <link name="${name}:trashbin_origin"/>
+    <link name="${name}:trashbin_front_edge_center"/>
     <!-- JOINTS -->
-    <joint name="${name}:table_origin_joint" type="fixed">
+    <joint name="${name}:trashbin_origin_joint" type="fixed">
       <xacro:insert_block name="origin" />
       <parent link="${parent}"/>
-      <child link="${name}:table_origin"/>
+      <child link="${name}:trashbin_origin"/>
     </joint>
     <joint name="${name}:center_joint" type="fixed">
       <origin xyz="${radius} 0 ${length}" rpy="0 0 0" />
-      <parent link="${name}:table_origin"/>
-      <child link="${name}:table_center"/>
+      <parent link="${name}:trashbin_origin"/>
+      <child link="${name}:trashbin_center"/>
     </joint>
-    <joint name="${name}:table_front_edge_center_joint" type="fixed">
+    <joint name="${name}:trashbin_front_edge_center_joint" type="fixed">
       <origin xyz="0 0 ${length}" rpy="0 0 0" />
-      <parent link="${name}:table_origin"/>
-      <child link="${name}:table_front_edge_center"/>
+      <parent link="${name}:trashbin_origin"/>
+      <child link="${name}:trashbin_front_edge_center"/>
     </joint>
   </xacro:macro>
