Commit message: [semantic map] couch model fix

File: suturo_resources/urdf/urdf_components/suturo_couch.urdf.xacro (robot description, xacro)
@@ -3,4 +3,10 @@
  <material name="color_grey">
     <color rgba="0.8 0.8 0.8 1"/>
+  </material>
+  <material name="color_red">
+    <color rgba="1 0 0 1"/>
+  </material>
+  <material name="color_blue">
+    <color rgba="0 0 1 1"/>
   </material>
   <xacro:macro name="suturo_couch" params="name parent *origin size_x size_y size_z">
@@ -9,5 +15,5 @@
       <visual>
         <material name="color_grey"/>
-        <origin xyz="0 0 ${-(size_z)/2}" rpy="0 0 0" />
+        <origin xyz="0 0 ${size_z/2}" rpy="0 0 0" />
         <geometry>
           <box size="${size_x} ${size_y} ${size_z}" />
@@ -15,5 +21,5 @@
       </visual>
       <collision>
-        <origin xyz="0 0 ${-(size_z)/2}" rpy="0 0 0" />
+        <origin xyz="0 0 0" rpy="0 0 0" />
         <geometry>
           <box size="${size_x} ${size_y} ${size_z}" />
@@ -23,12 +29,12 @@
     <link name="${name}:place2">
     <visual>
-        <material name="color_grey"/>
-        <origin xyz="0 ${-(size_y)/3} ${-(size_z)/2}" rpy="0 0 0" />
+        <material name="color_red"/>
+        <origin xyz="0 ${-(size_y)/4} ${(size_z)/2}" rpy="0 0 0" />
         <geometry>
-          <box size="${size_x} ${size_y} ${size_z}" />
+          <box size="${size_x} ${(size_y)/2} ${size_z}" />
         </geometry>
       </visual>
       <collision>
-        <origin xyz="0 0 ${-(size_z)/2}" rpy="0 0 0" />
+        <origin xyz="0 0 0" rpy="0 0 0" />
         <geometry>
           <box size="${size_x} ${size_y} ${size_z}" />
@@ -38,8 +44,8 @@
     <link name="${name}:place3">
     <visual>
-        <material name="color_grey"/>
-        <origin xyz="0 ${+(size_y)/3} ${-(size_z)/2}" rpy="0 0 0" />
+        <material name="color_blue"/>
+        <origin xyz="0 ${+(size_y)/4} ${(size_z)/2}" rpy="0 0 0" />
         <geometry>
-          <box size="${size_x} ${size_y} ${size_z}" />
+          <box size="${size_x} ${(size_y)/2} ${size_z}" />
         </geometry>
       </visual>
@@ -58,10 +64,10 @@
     </joint>
     <joint name="${name}:couch_left_joint" type="fixed">
-      <origin xyz="0 ${-(size_y)/3} ${-(size_z)/2}" rpy="0 0 0" />
+      <origin xyz="0 0 0" rpy="0 0 0" />
       <parent link="${name}:place1"/>
       <child link="${name}:place2"/>
     </joint>
     <joint name="${name}:couch_right_joint" type="fixed">
-      <origin xyz="0 ${+(size_y)/3} ${-(size_z)/2}" rpy="0 0 0" />
+      <origin xyz="0 0 0" rpy="0 0 0" />
       <parent link="${name}:place1"/>
       <child link="${name}:place3"/>

Commit message: [urdf_components]: added inertia to objects for gazebo

File: suturo_resources/urdf/urdf_components/suturo_couch.urdf.xacro (robot description, xacro)
@@ -26,4 +26,9 @@
         </geometry>
       </collision>
+      <inertial>
+        <origin xyz="0 0 0" rpy="0 0 0"/>
+        <mass value="1.0"/>
+        <inertia ixx="0.1" ixy="0.0" ixz="0.0" iyy="0.1" iyz="0.0" izz="0.1"/>
+      </inertial>
     </link>
     <link name="${name}:place2">
@@ -41,4 +46,9 @@
         </geometry>
       </collision>
+      <inertial>
+        <origin xyz="0 0 0" rpy="0 0 0"/>
+        <mass value="1.0"/>
+        <inertia ixx="0.1" ixy="0.0" ixz="0.0" iyy="0.1" iyz="0.0" izz="0.1"/>
+      </inertial>
     </link>
     <link name="${name}:place3">
@@ -56,4 +66,9 @@
         </geometry>
       </collision>
+      <inertial>
+        <origin xyz="0 0 0" rpy="0 0 0"/>
+        <mass value="1.0"/>
+        <inertia ixx="0.1" ixy="0.0" ixz="0.0" iyy="0.1" iyz="0.0" izz="0.1"/>
+      </inertial>
     </link>
      <!-- JOINTS -->

File: suturo_resources/urdf/urdf_components/suturo_door.urdf.xacro (robot description, xacro)
@@ -1,4 +1,7 @@
 <?xml version="1.0"?>
 <robot name="suturo_door" xmlns:xacro="http://ros.org/wiki/xacro">
+      <gazebo>
+   <gravity>0</gravity>
+</gazebo>
   <material name="door_green">
     <color rgba="0 0.31 0.22 1"/>
@@ -13,4 +16,5 @@
   <xacro:macro name="suturo_door" params="name parent height width depth x y z zrot door_turn_limit_lower door_turn_limit_max handle_x handle_z">
     <!-- LINKS -->
+    <!-- TODO: Remove gravity for door -->
     <link name="${name}:door_center">
       <visual>
@@ -27,4 +31,9 @@
         </geometry>
       </collision>
+      <inertial>
+        <origin xyz="0 0 0" rpy="0 0 0"/>
+        <mass value="1.0"/>
+        <inertia ixx="0.1" ixy="0.0" ixz="0.0" iyy="0.1" iyz="0.0" izz="0.1"/>
+      </inertial>
     </link>
     <link name="${name}:door_hinge">
@@ -42,4 +51,12 @@
         </geometry>
       </collision>
+      <inertial>
+        <origin xyz="0 0 0" rpy="0 0 0"/>
+        <mass value="1.0"/>
+        <inertia ixx="0.1" ixy="0.0" ixz="0.0" iyy="0.1" iyz="0.0" izz="0.1"/>
+      </inertial>
+            <gazebo>
+   <turnGravityOff>true</turnGravityOff>
+</gazebo>
     </link>
 	<link name="${name}:door_handle_link">
@@ -56,4 +73,12 @@
         </geometry>
       </collision>
+      <inertial>
+        <origin xyz="0 0 0" rpy="0 0 0"/>
+        <mass value="1.0"/>
+        <inertia ixx="0.1" ixy="0.0" ixz="0.0" iyy="0.1" iyz="0.0" izz="0.1"/>
+      </inertial>
+                  <gazebo>
+   <turnGravityOff>true</turnGravityOff>
+</gazebo>
     </link>
     <link name="${name}:door_handle_outside">
@@ -72,4 +97,12 @@
         </geometry>
       </collision>
+      <inertial>
+        <origin xyz="0 0 0" rpy="0 0 0"/>
+        <mass value="1.0"/>
+        <inertia ixx="0.1" ixy="0.0" ixz="0.0" iyy="0.1" iyz="0.0" izz="0.1"/>
+      </inertial>
+                        <gazebo>
+   <turnGravityOff>true</turnGravityOff>
+</gazebo>
     </link>
     <link name="${name}:door_handle_inside">
@@ -88,4 +121,12 @@
         </geometry>
       </collision>
+      <inertial>
+        <origin xyz="0 0 0" rpy="0 0 0"/>
+        <mass value="1.0"/>
+        <inertia ixx="0.1" ixy="0.0" ixz="0.0" iyy="0.1" iyz="0.0" izz="0.1"/>
+      </inertial>
+      <gazebo>
+   <turnGravityOff>true</turnGravityOff>
+</gazebo>
     </link>
     <!-- JOINTS -->

File: suturo_resources/urdf/urdf_components/suturo_shelf_hohc.urdf.xacro (robot description, xacro)
@@ -106,4 +106,9 @@
         </geometry>
       </collision>
+      <inertial>
+        <origin xyz="0 0 0" rpy="0 0 0"/>
+        <mass value="1.0"/>
+        <inertia ixx="0.1" ixy="0.0" ixz="0.0" iyy="0.1" iyz="0.0" izz="0.1"/>
+      </inertial>
     </link>
     <!-- JOINT -->
@@ -130,4 +135,9 @@
         </geometry>
       </collision>
+      <inertial>
+        <origin xyz="0 0 0" rpy="0 0 0"/>
+        <mass value="1.0"/>
+        <inertia ixx="0.1" ixy="0.0" ixz="0.0" iyy="0.1" iyz="0.0" izz="0.1"/>
+      </inertial>
     </link>
     <link name="${name}:handle">
@@ -145,4 +155,9 @@
         </geometry>
       </collision>
+      <inertial>
+        <origin xyz="0 0 0" rpy="0 0 0"/>
+        <mass value="1.0"/>
+        <inertia ixx="0.1" ixy="0.0" ixz="0.0" iyy="0.1" iyz="0.0" izz="0.1"/>
+      </inertial>
     </link>
     <joint name="${name}:handle_joint" type="fixed">
@@ -187,4 +202,9 @@
         </geometry>
       </collision>
+      <inertial>
+        <origin xyz="0 0 0" rpy="0 0 0"/>
+        <mass value="1.0"/>
+        <inertia ixx="0.1" ixy="0.0" ixz="0.0" iyy="0.1" iyz="0.0" izz="0.1"/>
+      </inertial>
     </link>
     <link name="${name}:handle">
@@ -202,4 +222,9 @@
         </geometry>
       </collision>
+      <inertial>
+        <origin xyz="0 0 0" rpy="0 0 0"/>
+        <mass value="1.0"/>
+        <inertia ixx="0.1" ixy="0.0" ixz="0.0" iyy="0.1" iyz="0.0" izz="0.1"/>
+      </inertial>
     </link>
     <joint name="${name}:handle_joint" type="fixed">

Commit message: [semantic map] fix suturo_couch.urdf.xacro
- removed visual and collision of center link

- moved side links to center of their seats

File: suturo_resources/urdf/urdf_components/suturo_couch.urdf.xacro (robot description, xacro)
@@ -12,28 +12,29 @@
   <xacro:macro name="suturo_couch" params="name parent *origin size_x size_y size_z">
     <!-- LINKS -->
+    <!-- Center of the couch, should not have a collision/visual to not overlap with the other two links -->
     <link name="${name}:place1">
-      <visual>
-        <material name="color_grey"/>
-        <origin xyz="0 0 ${size_z/2}" rpy="0 0 0" />
-        <geometry>
-          <box size="${size_x} ${size_y} ${size_z}" />
-        </geometry>
-      </visual>
-      <collision>
-        <origin xyz="0 0 0" rpy="0 0 0" />
-        <geometry>
-          <box size="${size_x} ${size_y} ${size_z}" />
-        </geometry>
-      </collision>
-      <inertial>
-        <origin xyz="0 0 0" rpy="0 0 0"/>
-        <mass value="1.0"/>
-        <inertia ixx="0.1" ixy="0.0" ixz="0.0" iyy="0.1" iyz="0.0" izz="0.1"/>
-      </inertial>
+      <!-- <visual> -->
+      <!--   <material name="color_grey"/> -->
+      <!--   <origin xyz="0 0 ${size_z/2}" rpy="0 0 0" /> -->
+      <!--   <geometry> -->
+      <!--     <box size="${size_x} ${size_y} ${size_z}" /> -->
+      <!--   </geometry> -->
+      <!-- </visual> -->
+      <!-- <collision> -->
+      <!--   <origin xyz="0 0 0" rpy="0 0 0" /> -->
+      <!--   <geometry> -->
+      <!--     <box size="${size_x} ${size_y} ${size_z}" /> -->
+      <!--   </geometry> -->
+      <!-- </collision> -->
+      <!-- <inertial> -->
+      <!--   <origin xyz="0 0 0" rpy="0 0 0"/> -->
+      <!--   <mass value="1.0"/> -->
+      <!--   <inertia ixx="0.1" ixy="0.0" ixz="0.0" iyy="0.1" iyz="0.0" izz="0.1"/> -->
+      <!-- </inertial> -->
     </link>
     <link name="${name}:place2">
     <visual>
         <material name="color_red"/>
-        <origin xyz="0 ${-(size_y)/4} ${(size_z)/2}" rpy="0 0 0" />
+        <origin xyz="0 0 0" rpy="0 0 0" />
         <geometry>
           <box size="${size_x} ${(size_y)/2} ${size_z}" />
@@ -43,5 +44,5 @@
         <origin xyz="0 0 0" rpy="0 0 0" />
         <geometry>
-          <box size="${size_x} ${size_y} ${size_z}" />
+          <box size="${size_x} ${(size_y)/2} ${size_z}" />
         </geometry>
       </collision>
@@ -55,5 +56,5 @@
     <visual>
         <material name="color_blue"/>
-        <origin xyz="0 ${+(size_y)/4} ${(size_z)/2}" rpy="0 0 0" />
+        <origin xyz="0 0 0" rpy="0 0 0" />
         <geometry>
           <box size="${size_x} ${(size_y)/2} ${size_z}" />
@@ -61,7 +62,7 @@
       </visual>
       <collision>
-        <origin xyz="0 0 ${-(size_z)/2}" rpy="0 0 0" />
+        <origin xyz="0 0 0" rpy="0 0 0" />
         <geometry>
-          <box size="${size_x} ${size_y} ${size_z}" />
+          <box size="${size_x} ${(size_y)/2} ${size_z}" />
         </geometry>
       </collision>
@@ -79,10 +80,10 @@
     </joint>
     <joint name="${name}:couch_left_joint" type="fixed">
-      <origin xyz="0 0 0" rpy="0 0 0" />
+      <origin xyz="0 ${-(size_y)/4} ${(size_z)/2}" rpy="0 0 0" />
       <parent link="${name}:place1"/>
       <child link="${name}:place2"/>
     </joint>
     <joint name="${name}:couch_right_joint" type="fixed">
-      <origin xyz="0 0 0" rpy="0 0 0" />
+      <origin xyz="0 ${+(size_y)/4} ${(size_z)/2}" rpy="0 0 0" />
       <parent link="${name}:place1"/>
       <child link="${name}:place3"/>

Commit message: added walls and fixes for the couch and dishwasher

File: suturo_resources/urdf/urdf_components/suturo_couch.urdf.xacro (robot description, xacro)
@@ -13,38 +13,38 @@
     <!-- LINKS -->
     <!-- Center of the couch, should not have a collision/visual to not overlap with the other two links -->
-    <link name="${name}:place1">
-      <!-- <visual> -->
-      <!--   <material name="color_grey"/> -->
-      <!--   <origin xyz="0 0 ${size_z/2}" rpy="0 0 0" /> -->
-      <!--   <geometry> -->
-      <!--     <box size="${size_x} ${size_y} ${size_z}" /> -->
-      <!--   </geometry> -->
-      <!-- </visual> -->
-      <!-- <collision> -->
-      <!--   <origin xyz="0 0 0" rpy="0 0 0" /> -->
-      <!--   <geometry> -->
-      <!--     <box size="${size_x} ${size_y} ${size_z}" /> -->
-      <!--   </geometry> -->
-      <!-- </collision> -->
-      <!-- <inertial> -->
-      <!--   <origin xyz="0 0 0" rpy="0 0 0"/> -->
-      <!--   <mass value="1.0"/> -->
-      <!--   <inertia ixx="0.1" ixy="0.0" ixz="0.0" iyy="0.1" iyz="0.0" izz="0.1"/> -->
-      <!-- </inertial> -->
+    <link name="${name}:place_one">
+       <visual>
+         <material name="color_grey"/>
+         <origin xyz="0 0 ${size_z/2}" rpy="0 0 0" />
+         <geometry>
+           <box size="${size_x} ${size_y} ${size_z}" />
+         </geometry>
+       </visual>
+       <collision>
+         <origin xyz="0 0 0" rpy="0 0 0" />
+         <geometry>
+           <box size="${size_x} ${size_y} ${size_z}" />
+         </geometry>
+       </collision>
+       <inertial>
+         <origin xyz="0 0 0" rpy="0 0 0"/>
+         <mass value="1.0"/>
+         <inertia ixx="0.1" ixy="0.0" ixz="0.0" iyy="0.1" iyz="0.0" izz="0.1"/>
+       </inertial>
     </link>
-    <link name="${name}:place2">
-    <visual>
-        <material name="color_red"/>
-        <origin xyz="0 0 0" rpy="0 0 0" />
-        <geometry>
-          <box size="${size_x} ${(size_y)/2} ${size_z}" />
-        </geometry>
-      </visual>
-      <collision>
-        <origin xyz="0 0 0" rpy="0 0 0" />
-        <geometry>
-          <box size="${size_x} ${(size_y)/2} ${size_z}" />
-        </geometry>
-      </collision>
+    <link name="${name}:place_two">
+    <!--<visual> -->
+    <!--    <material name="color_red"/> -->
+    <!--    <origin xyz="0 0 0" rpy="0 0 0" /> -->
+    <!--    <geometry> -->
+    <!--      <box size="${size_x} ${(size_y)/2} ${size_z}" /> -->
+    <!--    </geometry> -->
+    <!--  </visual> -->
+      <!--<collision>-->
+      <!--  <origin xyz="0 0 0" rpy="0 0 0" />-->
+      <!--  <geometry>-->
+      <!--    <box size="${size_x} ${(size_y)/2} ${size_z}" />-->
+      <!--  </geometry>-->
+      <!--</collision> -->
       <inertial>
         <origin xyz="0 0 0" rpy="0 0 0"/>
@@ -53,18 +53,18 @@
       </inertial>
     </link>
-    <link name="${name}:place3">
-    <visual>
-        <material name="color_blue"/>
-        <origin xyz="0 0 0" rpy="0 0 0" />
-        <geometry>
-          <box size="${size_x} ${(size_y)/2} ${size_z}" />
-        </geometry>
-      </visual>
-      <collision>
-        <origin xyz="0 0 0" rpy="0 0 0" />
-        <geometry>
-          <box size="${size_x} ${(size_y)/2} ${size_z}" />
-        </geometry>
-      </collision>
+    <link name="${name}:place_three">
+    <!--<visual> -->
+    <!--    <material name="color_blue"/> -->
+    <!--    <origin xyz="0 0 0" rpy="0 0 0" /> -->
+    <!--    <geometry> -->
+    <!--      <box size="${size_x} ${(size_y)/2} ${size_z}" /> -->
+    <!--    </geometry> -->
+    <!--  </visual> -->
+      <!--<collision> -->
+      <!--  <origin xyz="0 0 0" rpy="0 0 0" /> -->
+      <!--  <geometry> -->
+      <!--    <box size="${size_x} ${(size_y)/2} ${size_z}" /> -->
+      <!--  </geometry> -->
+      <!--</collision> -->
       <inertial>
         <origin xyz="0 0 0" rpy="0 0 0"/>
@@ -77,15 +77,15 @@
       <xacro:insert_block name="origin" />
       <parent link="${parent}"/>
-      <child link="${name}:place1"/>
+      <child link="${name}:place_one"/>
     </joint>
     <joint name="${name}:couch_left_joint" type="fixed">
       <origin xyz="0 ${-(size_y)/4} ${(size_z)/2}" rpy="0 0 0" />
-      <parent link="${name}:place1"/>
-      <child link="${name}:place2"/>
+      <parent link="${name}:place_one"/>
+      <child link="${name}:place_two"/>
     </joint>
     <joint name="${name}:couch_right_joint" type="fixed">
       <origin xyz="0 ${+(size_y)/4} ${(size_z)/2}" rpy="0 0 0" />
-      <parent link="${name}:place1"/>
-      <child link="${name}:place3"/>
+      <parent link="${name}:place_one"/>
+      <child link="${name}:place_three"/>
     </joint>
   </xacro:macro>

File: suturo_resources/urdf/urdf_components/suturo_dishwasher_robocup.urdf.xacro (robot description, xacro)
@@ -67,5 +67,5 @@
   <link name="sink_area_dish_washer_door_handle">
     <inertial>
-      <origin rpy="0 0 0" xyz="0.1 0.0 0.0"/>
+      <origin rpy="0 0 0" xyz="0.1 0 0.0"/>
       <mass value="1"/>
       <inertia ixx="1" ixy="0.0" ixz="0.0" iyy="1" iyz="0.0" izz="1"/>
@@ -88,5 +88,5 @@
   </gazebo>
   <link name="dishwasher_tab"/>
-  <link name="dishwasher_table:d_table:table_origin"/>
+  <link name="dishwasher_table:d_table:d_table_origin"/>
   <link name="dishwasher_table:d_table:table_front_edge_center"/>
   <link name="dishwasher_table:d_table:table_center">
@@ -139,14 +139,14 @@
     <origin rpy="0 0 ${pi}" xyz="0.0 0.0 0.3971"/>
     <parent link="sink_area_dish_washer_main"/>
-    <child link="dishwasher_table:d_table:table_origin"/>
+    <child link="dishwasher_table:d_table:d_table_origin"/>
   </joint>
   <joint name="dish_washer_table_center_joint" type="fixed">
     <origin rpy="0 0 0" xyz="-0.3 0 0"/>
-    <parent link="dishwasher_table:d_table:table_origin"/>
+    <parent link="dishwasher_table:d_table:d_table_origin"/>
     <child link="dishwasher_table:d_table:table_front_edge_center"/>
   </joint>
   <joint name="dish_washer_table_edge_joint" type="fixed">
     <origin rpy="0 0 0" xyz="0 0 0"/>
-    <parent link="dishwasher_table:d_table:table_origin"/>
+    <parent link="dishwasher_table:d_table:d_table_origin"/>
     <child link="dishwasher_table:d_table:table_center"/>
   </joint>
