Commit message: fix typo

File: suturo_resources/urdf/urdf_components/suturo_door.urdf.xacro (robot description, xacro)
@@ -94,5 +94,5 @@
       <limit effort="1" lower="0" upper="1.5708" velocity="1"/>
       <origin xyz="${0.9 * width} ${-1.25 * depth} -0.13" rpy="0 0 0" />
-      <parent link="${name}_center"/>
+      <parent link="${name}_door_center"/>
       <child link="${name}_door_handle_inside"/>
     </joint>

Commit message: removing the - of death...

File: suturo_resources/urdf/urdf_components/suturo_door.urdf.xacro (robot description, xacro)
@@ -38,5 +38,5 @@
       <collision>
         <origin xyz="0 0 0" rpy="0 0 0" />
-        <geometry>-
+        <geometry>
           <box size="0.05 0.05 ${height}" />
         </geometry>
@@ -64,5 +64,5 @@
 	<material name="handle_blue"/>
         <origin xyz="0 0 0" rpy="${half_pi} 0 ${pi}" />
-        <geometry>-
+        <geometry>
           <box size="0.15 0.025 0.015" />
         </geometry>

Commit message: Changed icp values

File: suturo_resources/urdf/urdf_components/suturo_door.urdf.xacro (robot description, xacro)
@@ -100,5 +100,5 @@
       <axis xyz="0 0 0"/>
       <limit effort="1" lower="0" upper="1.5708" velocity="1"/>
-      <origin xyz="${0.9 * width} ${1.25 * depth} -0.13" rpy="0 0 0" />
+      <origin xyz="${0.9 * width} ${depth} -0.13" rpy="0 0 0" />
       <parent link="${name}_door_center"/>
       <child link="${name}_door_handle_outside"/>

Commit message: remapping the base_scan and adjusting the handle

File: suturo_resources/urdf/urdf_components/suturo_door.urdf.xacro (robot description, xacro)
@@ -93,5 +93,5 @@
       <axis xyz="0 0 0"/>
       <limit effort="1" lower="0" upper="1.5708" velocity="1"/>
-      <origin xyz="${0.9 * width} ${-1.25 * depth} -0.13" rpy="0 0 0" />
+      <origin xyz="${0.88 * width} ${-1.25 * depth} -0.13" rpy="0 0 0" />
       <parent link="${name}_door_center"/>
       <child link="${name}_door_handle_inside"/>
@@ -100,5 +100,5 @@
       <axis xyz="0 0 0"/>
       <limit effort="1" lower="0" upper="1.5708" velocity="1"/>
-      <origin xyz="${0.9 * width} ${depth} -0.13" rpy="0 0 0" />
+      <origin xyz="${0.88 * width} ${depth} -0.13" rpy="0 0 0" />
       <parent link="${name}_door_center"/>
       <child link="${name}_door_handle_outside"/>

Commit message: added base_scan_limiter to the starting process. This node republishes the base_scan to base_scan_unlimited

File: suturo_resources/urdf/urdf_components/suturo_door.urdf.xacro (robot description, xacro)
@@ -49,5 +49,5 @@
         <origin xyz="0 0 0" rpy="${half_pi} 0 ${pi}" />
         <geometry>
-          <box size="0.15 0.025 0.015" />
+          <box size="0.15 0.008 0.015" />
         </geometry>
       </visual>
@@ -55,5 +55,5 @@
         <origin xyz="0 0 0" rpy="${half_pi} 0 ${pi}" />
         <geometry>
-          <box size="0.15 0.025 0.015" />
+          <box size="0.15 0.008 0.015" />
         </geometry>
       </collision>
@@ -65,5 +65,5 @@
         <origin xyz="0 0 0" rpy="${half_pi} 0 ${pi}" />
         <geometry>
-          <box size="0.15 0.025 0.015" />
+          <box size="0.15 0.01 0.015" />
         </geometry>
       </visual>
@@ -71,5 +71,5 @@
         <origin xyz="0 0 0" rpy="${half_pi} 0 ${pi}" />
         <geometry>
-          <box size="0.15 0.025 0.015" />
+          <box size="0.15 0.01 0.015" />
         </geometry>
       </collision>
@@ -93,5 +93,5 @@
       <axis xyz="0 0 0"/>
       <limit effort="1" lower="0" upper="1.5708" velocity="1"/>
-      <origin xyz="${0.9 * width} ${-1.25 * depth} -0.13" rpy="0 0 0" />
+      <origin xyz="${0.88 * width} ${-1.25 * depth} -0.12" rpy="0 0 0" />
       <parent link="${name}:door_center"/>
       <child link="${name}:door_handle_inside"/>
@@ -100,5 +100,5 @@
       <axis xyz="0 0 0"/>
       <limit effort="1" lower="0" upper="1.5708" velocity="1"/>
-      <origin xyz="${0.9 * width} ${depth} -0.13" rpy="0 0 0" />
+      <origin xyz="${0.88 * width} ${depth} -0.12" rpy="0 0 0" />
       <parent link="${name}:door_center"/>
       <child link="${name}:door_handle_outside"/>

Commit message: fix door handle frame to makex point inwards

File: suturo_resources/urdf/urdf_components/suturo_door.urdf.xacro (robot description, xacro)
@@ -47,13 +47,13 @@
       <visual>
 	<material name="handle_blue"/>
-        <origin xyz="0 0 0" rpy="${half_pi} 0 ${pi}" />
+        <origin xyz="0 0 0" rpy="0 0 0" />
         <geometry>
-          <box size="0.15 0.008 0.015" />
+          <box size="0.015 0.15 0.01" />
         </geometry>
       </visual>
       <collision>
-        <origin xyz="0 0 0" rpy="${half_pi} 0 ${pi}" />
+        <origin xyz="0 0 0" rpy="0 0 0" />
         <geometry>
-          <box size="0.15 0.008 0.015" />
+          <box size="0.015 0.15 0.01" />
         </geometry>
       </collision>
@@ -63,13 +63,13 @@
       <visual>
 	<material name="handle_blue"/>
-        <origin xyz="0 0 0" rpy="${half_pi} 0 ${pi}" />
+        <origin xyz="0 0 0" rpy="0 0 0" />
         <geometry>
-          <box size="0.15 0.01 0.015" />
+          <box size="0.015 0.15 0.01" />
         </geometry>
       </visual>
       <collision>
-        <origin xyz="0 0 0" rpy="${half_pi} 0 ${pi}" />
+        <origin xyz="0 0 0" rpy="0 0 0" />
         <geometry>
-          <box size="0.15 0.01 0.015" />
+          <box size="0.015 0.15 0.01" />
         </geometry>
       </collision>
@@ -93,5 +93,5 @@
       <axis xyz="0 0 0"/>
       <limit effort="1" lower="0" upper="1.5708" velocity="1"/>
-      <origin xyz="${0.88 * width} ${-1.25 * depth} -0.12" rpy="0 0 0" />
+      <origin xyz="${0.88 * width} ${-1.25 * depth} -0.12" rpy="0 0 ${pi/2}" />
       <parent link="${name}:door_center"/>
       <child link="${name}:door_handle_inside"/>
@@ -100,5 +100,5 @@
       <axis xyz="0 0 0"/>
       <limit effort="1" lower="0" upper="1.5708" velocity="1"/>
-      <origin xyz="${0.88 * width} ${depth} -0.12" rpy="0 0 0" />
+      <origin xyz="${0.88 * width} ${depth} -0.12" rpy="0 0 ${-pi/2}" />
       <parent link="${name}:door_center"/>
       <child link="${name}:door_handle_outside"/>

Commit message: changed door urdf: added link + joint for revolute handle added python.urdf.xacro for giskard testing

File: suturo_resources/urdf/urdf_components/suturo_door.urdf.xacro (robot description, xacro)
@@ -40,4 +40,18 @@
         <geometry>
           <box size="0.05 0.05 ${height}" />
+        </geometry>
+      </collision>
+    </link>
+	<link name="${name}:door_handle_link">
+      <visual >
+        <origin xyz="0.0 0.0 0.0" rpy="0 0 0" />
+        <geometry name="handle_blue">
+          <cylinder radius="0.013" length="0.15" />
+        </geometry>
+      </visual>
+      <collision >
+        <origin xyz="0.0 0.0 0.0" rpy="0 0 0" />
+        <geometry name="handle_collision_geom">
+          <cylinder radius="0.013" length="0.15" />
         </geometry>
       </collision>
@@ -90,16 +104,19 @@
       <child link="${name}:door_hinge"/>
     </joint>
+    <joint name="${name}:door_handle_joint" type="revolute" >
+      <axis xyz="0 0 1"/>
+      <limit effort="1" lower="0" upper="${pi/5}" velocity="1"/>
+      <origin xyz="${0.92 * width} 0 0.05" rpy="${pi/2} 0 0" />
+      <parent link="${name}:door_center"/>
+	  <child link="${name}:door_handle_link"/>
+    </joint>
     <joint name="${name}:door_handle_inside_joint" type="fixed">
-      <axis xyz="0 0 0"/>
-      <limit effort="1" lower="0" upper="1.5708" velocity="1"/>
-      <origin xyz="${0.88 * width} ${-1.25 * depth} -0.12" rpy="0 0 ${pi/2}" />
-      <parent link="${name}:door_center"/>
+      <origin xyz="-0.075 0 0.075" rpy="0 0 ${pi/2}" />
+      <parent link="${name}:door_handle_link"/>
       <child link="${name}:door_handle_inside"/>
     </joint>
     <joint name="${name}:door_handle_outside_joint" type="fixed">
-      <axis xyz="0 0 0"/>
-      <limit effort="1" lower="0" upper="1.5708" velocity="1"/>
-      <origin xyz="${0.88 * width} ${depth} -0.12" rpy="0 0 ${-pi/2}" />
-      <parent link="${name}:door_center"/>
+      <origin xyz="-0.075 0 -0.075" rpy="0 0 ${-pi/2}" />
+      <parent link="${name}:door_handle_link"/>
       <child link="${name}:door_handle_outside"/>
     </joint>

Commit message: [Map/semantixc map] changes from friday

File: suturo_resources/urdf/urdf_components/suturo_door.urdf.xacro (robot description, xacro)
@@ -112,5 +112,5 @@
     </joint>
     <joint name="${name}:door_handle_inside_joint" type="fixed">
-      <origin xyz="-0.06 0 0.035" rpy="0 0 ${pi/2}" />
+      <origin xyz="-0.06 0 0.06" rpy="0 0 ${pi/2}" />
       <parent link="${name}:door_handle_link"/>
       <child link="${name}:door_handle_inside"/>

File: suturo_resources/urdf/urdf_components/suturo_kitchen.urdf.xacro (robot description, xacro)
@@ -1305,5 +1305,5 @@
   </link>
   <joint name="kitchen_island_footprint_joint" type="fixed">
-    <origin rpy="0 0 0" xyz="-1.365 0.59 0"/>
+    <origin rpy="0 0 0" xyz="-1.365 0.64 0"/>
     <child link="kitchen_island_footprint"/>
     <parent link="kitchen_main"/>

Commit message: [semantic map] door handle moved to right

File: suturo_resources/urdf/urdf_components/suturo_door.urdf.xacro (robot description, xacro)
@@ -112,5 +112,5 @@
     </joint>
     <joint name="${name}:door_handle_inside_joint" type="fixed">
-      <origin xyz="-0.06 0 0.06" rpy="0 0 ${pi/2}" />
+      <origin xyz="-0.04 0 0.06" rpy="0 0 ${pi/2}" />
       <parent link="${name}:door_handle_link"/>
       <child link="${name}:door_handle_inside"/>

Commit message: [semantic map] door handle inertia and dampening

File: suturo_resources/urdf/urdf_components/suturo_door.urdf.xacro (robot description, xacro)
@@ -34,4 +34,9 @@
       </inertial>
     </link>
+    <gazebo reference="${name}:door_center">
+      <turnGravityOff>true</turnGravityOff>
+      <!-- this value is not accurate, but for now it should be enough for the simulation -->
+      <dampingFactor>0.000001</dampingFactor>
+    </gazebo>
     <link name="${name}:door_hinge">
       <visual>
@@ -69,10 +74,12 @@
       <inertial>
         <origin xyz="0 0 0" rpy="0 0 0"/>
-        <mass value="1.0"/>
-        <inertia ixx="0.1" ixy="0.0" ixz="0.0" iyy="0.1" iyz="0.0" izz="0.1"/>
+        <mass value="0.1"/>
+        <inertia ixx="0.001" ixy="0.0" ixz="0.0" iyy="0.001" iyz="0.0" izz="0.001"/>
       </inertial>
     </link>
     <gazebo reference="${name}:door_handle_link">
       <turnGravityOff>true</turnGravityOff>
+      <!-- this value is not accurate, but for now it should be enough for the simulation -->
+      <dampingFactor>0.005</dampingFactor>
     </gazebo>
     <link name="${name}:door_handle_outside">
@@ -93,6 +100,6 @@
       <inertial>
         <origin xyz="0 0 0" rpy="0 0 0"/>
-        <mass value="1.0"/>
-        <inertia ixx="0.1" ixy="0.0" ixz="0.0" iyy="0.1" iyz="0.0" izz="0.1"/>
+        <mass value="0.1"/>
+        <inertia ixx="0.001" ixy="0.0" ixz="0.0" iyy="0.001" iyz="0.0" izz="0.001"/>
       </inertial>
     </link>
@@ -117,6 +124,6 @@
       <inertial>
         <origin xyz="0 0 0" rpy="0 0 0"/>
-        <mass value="1.0"/>
-        <inertia ixx="0.1" ixy="0.0" ixz="0.0" iyy="0.1" iyz="0.0" izz="0.1"/>
+        <mass value="0.1"/>
+        <inertia ixx="0.001" ixy="0.0" ixz="0.0" iyy="0.001" iyz="0.0" izz="0.001"/>
       </inertial>
     </link>

Commit message: door fixes

File: suturo_resources/urdf/urdf_components/suturo_door.urdf.xacro (robot description, xacro)
@@ -147,5 +147,5 @@
     </joint>
     <joint name="${name}:door_handle_inside_joint" type="fixed">
-      <origin xyz="-0.04 0 0.06" rpy="0 0 ${pi/2}" />
+      <origin xyz="-0.069 0 0.06" rpy="0 0 ${pi/2}" />
       <parent link="${name}:door_handle_link"/>
       <child link="${name}:door_handle_inside"/>

Commit message: changed coordinate system for outside door handle to work better for door opening.

File: suturo_resources/urdf/urdf_components/suturo_door.urdf.xacro (robot description, xacro)
@@ -152,5 +152,5 @@
     </joint>
     <joint name="${name}:door_handle_outside_joint" type="fixed">
-      <origin xyz="-0.075 0 -0.05" rpy="0 0 ${-pi/2}" />
+      <origin xyz="-0.069 0 -0.06" rpy="0 ${pi} ${pi/2}" />
       <parent link="${name}:door_handle_link"/>
       <child link="${name}:door_handle_outside"/>

Commit message: changed door handle pose

File: suturo_resources/urdf/urdf_components/suturo_door.urdf.xacro (robot description, xacro)
@@ -147,10 +147,10 @@
     </joint>
     <joint name="${name}:door_handle_inside_joint" type="fixed">
-      <origin xyz="-0.069 0 0.06" rpy="0 0 ${pi/2}" />
+      <origin xyz="-0.0635 0 0.06" rpy="0 0 ${pi/2}" />
       <parent link="${name}:door_handle_link"/>
       <child link="${name}:door_handle_inside"/>
     </joint>
     <joint name="${name}:door_handle_outside_joint" type="fixed">
-      <origin xyz="-0.069 0 -0.06" rpy="0 ${pi} ${pi/2}" />
+      <origin xyz="-0.0635 0 -0.06" rpy="0 ${pi} ${pi/2}" />
       <parent link="${name}:door_handle_link"/>
       <child link="${name}:door_handle_outside"/>
