Commit message: Added dishwasher to map 2023 and fixed frames

File: suturo_resources/urdf/urdf_components/suturo_dishwasher.urdf.xacro (robot description, xacro)
@@ -6,5 +6,5 @@
       <xacro:sphere_inertia radius="0" mass="0"/>
       <visual>
-        <origin xyz="0 0 0" rpy="0 0 0" />
+        <origin xyz="0 0 0" rpy="0 0 ${pi}" />
         <geometry>
           <mesh filename="package://iai_kitchen/meshes/misc/DishWasher.dae"/>
@@ -36,5 +36,5 @@
       <xacro:sphere_inertia radius="0" mass="0"/>
       <visual>
-        <origin xyz="0 0 0" rpy="0 0 0" />
+        <origin xyz="0 0 0" rpy="0 ${pi} 0" />
         <geometry>
           <mesh filename="package://iai_kitchen/meshes/handles/Handle60.dae"/>
@@ -42,5 +42,5 @@
       </visual>
       <collision>
-        <origin xyz="0 0 0" rpy="0 0 0" />
+        <origin xyz="0 0 0" rpy="0 ${pi} 0" />
         <geometry>
           <mesh filename="package://iai_kitchen/meshes/handles/Handle60.obj"/>
@@ -72,5 +72,5 @@
     -->
     <joint name="${name}_door_joint" type="revolute">
-      <origin xyz="0.27 0. -0.285" rpy="${-0.5*pi} 0 0" />
+      <origin xyz="-0.27 0. -0.285" rpy="${-0.5*pi} 0 0" />
       <parent link="${name}_main"/>
       <child link="${name}_door"/>
@@ -79,5 +79,5 @@
       <limit lower="0" upper="${0.5*pi}" effort="300" velocity="10"/>
       -->
-      <limit lower="0" upper="${0.5*pi}" effort="300" velocity="10"/>
+      <limit lower="${-0.5*pi}" upper="0" effort="300" velocity="10"/>
     </joint>
     <!--
@@ -85,5 +85,5 @@
   -->
     <joint name="${name}_door_handle_joint" type="fixed">
-      <origin xyz="0.085 -0.575 0.0" rpy="${-0.5*pi} 0 0" />
+      <origin xyz="-0.065 -0.575 0.0" rpy="${pi/2} 0 0" />
       <parent link="${name}_door"/>
       <child link="${name}_door_handle"/>
@@ -99,5 +99,5 @@
       <child link="${name}_bottom"/>
       <axis xyz="1 0 0"/>
-      <limit lower="0" upper="0.48" effort="300" velocity="10"/>
+      <limit lower="-0.33" upper="0" effort="300" velocity="10"/>
     </joint>
     <link name="${name}_bottom">
@@ -172,15 +172,15 @@
     </joint>
     <joint name="${name}_bottom_back" type="fixed">
-      <origin xyz="-0.16 0 0.075"/>
+      <origin xyz="0.16 0 0.075"/>
       <child link="${name}_back_side" />
       <parent link="${name}_bottom"/>
     </joint>
     <joint name="${name}_bottom_front" type="fixed">
-      <origin xyz="0.16 0 0.075"/>
+      <origin xyz="-0.16 0 0.075" rpy="0 0 0"/>
       <child link="${name}_front_side" />
       <parent link="${name}_bottom"/>
     </joint>
     <xacro:tray_handle name="${name}_handle" parent="${name}_front_side">
-      <origin xyz="0.06 -0.1 -0.02"/>
+      <origin xyz="-0.03 -0.1 -0.02"/>
     </xacro:tray_handle>
   </xacro:macro>
@@ -228,10 +228,10 @@
     </link>
     <joint name="${name}_front_left_joint" type="fixed">
-      <origin xyz="-0.01 -0.1 0"/>
+      <origin xyz="0.01 -0.1 0"/>
       <child link="${name}_left_side" />
       <parent link="${name}_front_side"/>
     </joint>
     <joint name="${name}_front_right_joint" type="fixed">
-      <origin xyz="-0.01 0.1 0"/>
+      <origin xyz="0.01 0.1 0"/>
       <child link="${name}_right_side" />
       <parent link="${name}_front_side"/>

Commit message: Added second tray to dishwasher

File: suturo_resources/urdf/urdf_components/suturo_dishwasher.urdf.xacro (robot description, xacro)
@@ -92,4 +92,7 @@
       <origin xyz="-0.08 0 0.15"/>
     </xacro:dishwasher_tray>
+    <xacro:dishwasher_tray name="${name}_tray_2" parent="${name}_main">
+      <origin xyz="-0.08 0 -0.15"/>
+    </xacro:dishwasher_tray>
   </xacro:macro>
   <xacro:macro name="dishwasher_tray" params="name parent *origin">
@@ -185,4 +188,96 @@
     </xacro:tray_handle>
   </xacro:macro>
+    <xacro:macro name="dishwasher_tray_2" params="name parent *origin">
+    <joint name="${name}_main_2" type="prismatic">
+      <xacro:insert_block name="origin"/>
+      <parent link="${parent}"/>
+      <child link="${name}_bottom_2"/>
+      <axis xyz="1 0 0"/>
+      <limit lower="-0.33" upper="0" effort="300" velocity="10"/>
+    </joint>
+    <link name="${name}_bottom_2">
+      <visual>
+        <geometry>
+          <box size="0.32 0.5 0.05"/>
+        </geometry>
+      </visual>
+      <collision>
+        <geometry>
+          <box size="0.32 0.5 0.05"/>
+        </geometry>
+      </collision>
+    </link>
+    <link name="${name}_left_side_2">
+      <visual>
+        <geometry>
+          <box size="0.32 0.005 0.17"/>
+        </geometry>
+      </visual>
+      <collision>
+        <geometry>
+          <box size="0.32 0.005 0.17"/>
+        </geometry>
+      </collision>
+    </link>
+    <link name="${name}_right_side_2">
+      <visual>
+        <geometry>
+          <box size="0.32 0.005 0.17"/>
+        </geometry>
+      </visual>
+      <collision>
+        <geometry>
+          <box size="0.32 0.005 0.17"/>
+        </geometry>
+      </collision>
+    </link>
+    <link name="${name}_back_side_2">
+      <visual>
+        <geometry>
+          <box size="0.005 0.5 0.17"/>
+        </geometry>
+      </visual>
+      <collision>
+        <geometry>
+          <box size="0.005 0.5 0.17"/>
+        </geometry>
+      </collision>
+    </link>
+    <link name="${name}_front_side_2">
+      <visual>
+        <geometry>
+          <box size="0.005 0.5 0.17"/>
+        </geometry>
+      </visual>
+      <collision>
+        <geometry>
+          <box size="0.005 0.5 0.17"/>
+        </geometry>
+      </collision>
+    </link>
+    <joint name="${name}_bottom_left_2" type="fixed">
+      <origin xyz="-0.0 -0.25 -0.075"/>
+      <child link="${name}_left_side_2" />
+      <parent link="${name}_bottom_2"/>
+    </joint>
+    <joint name="${name}_bottom_right_2" type="fixed">
+      <origin xyz="-0.0 0.25 -0.075"/>
+      <child link="${name}_right_side_2" />
+      <parent link="${name}_bottom_2"/>
+    </joint>
+    <joint name="${name}_bottom_back" type="fixed">
+      <origin xyz="0.16 0 -0.075"/>
+      <child link="${name}_back_side_2" />
+      <parent link="${name}_bottom_2"/>
+    </joint>
+    <joint name="${name}_bottom_front" type="fixed">
+      <origin xyz="-0.16 0 -0.075" rpy="0 0 0"/>
+      <child link="${name}_front_side_2" />
+      <parent link="${name}_bottom_2"/>
+    </joint>
+    <xacro:tray_handle name="${name}_handle_2" parent="${name}_front_side_2">
+      <origin xyz="-0.03 -0.1 -0.02"/>
+    </xacro:tray_handle>
+  </xacro:macro>
   <xacro:macro name="tray_handle" params="name parent *origin">
     <joint name="${name}_joint" type="fixed">

Commit message: Robocup dishwasher changes

File: suturo_resources/urdf/urdf_components/suturo_dishwasher.urdf.xacro (robot description, xacro)
@@ -8,5 +8,5 @@
         <origin xyz="0 0 0" rpy="0 0 ${pi}" />
         <geometry>
-          <mesh filename="package://iai_kitchen/meshes/misc/DishWasher.dae"/>
+          <mesh filename="package://iai_kitchen/meshes/misc/DishWasher.dae" scale="1.1 1.2 1"/>
         </geometry>
       </visual>
@@ -14,5 +14,5 @@
         <origin xyz="0 0 0" rpy="0 0 0" />
         <geometry>
-          <mesh filename="package://iai_kitchen/meshes/misc/DishWasher.obj"/>
+          <mesh filename="package://iai_kitchen/meshes/misc/DishWasher.obj"  scale="1.1 1.2 1"/>
         </geometry>
       </collision>

Commit message: Refact: adjust dishwasher tray height to RoboCup 2023 dishwasher

File: suturo_resources/urdf/urdf_components/suturo_dishwasher.urdf.xacro (robot description, xacro)
@@ -90,8 +90,8 @@
     </joint>
     <xacro:dishwasher_tray name="${name}:dishwasher_tray" parent="${name}:dishwasher_main">
-      <origin xyz="-0.08 0 0.15"/>
+      <origin xyz="-0.08 0 0.26"/>
     </xacro:dishwasher_tray>
     <xacro:dishwasher_tray name="${name}:dishwasher_tray_2" parent="${name}:dishwasher_main">
-      <origin xyz="-0.08 0 -0.15"/>
+      <origin xyz="-0.08 0 -0.07"/>
     </xacro:dishwasher_tray>
   </xacro:macro>

Commit message: add dishwasher_tab_joint

File: suturo_resources/urdf/urdf_components/suturo_dishwasher.urdf.xacro (robot description, xacro)
@@ -48,7 +48,13 @@
       </collision>
     </link>
-    <!--
+	<link name="${name}:dishwasher_tab"/>
+	<!--
     <xacro:if value="simulated"/>
     -->
+	<joint name="${name}:dishwasher_tab_joint" type="fixed">
+	  <origin xyz="0.18 -0.33 0.1775" rpy="0 0 0" />
+	  <parent link="${name}:dishwasher_door"/>
+      <child link="${name}:dishwasher_tab"/>
+	</joint>
     <joint name="${name}:dishwasher_main_joint" type="fixed">
       <xacro:insert_block name="origin" />

Commit message: remove duplicate joint from dishwasher

File: suturo_resources/urdf/urdf_components/suturo_dishwasher.urdf.xacro (robot description, xacro)
@@ -17,9 +17,11 @@
 	  <child link="dishwasher_main"/>
     </joint>
-    <joint name="dishwasher_main_joint" type="fixed">
-	  <xacro:insert_block name="origin" />
-	  <parent link="dishwasher_main"/>
-	  <child link="sink_area_dish_washer_main"/>
-    </joint>
+	<!-- Below there is another joint connecting these two links,
+		 which breaks giskards ability to work with this -->
+    <!-- <joint name="dishwasher_main_joint" type="fixed"> -->
+	<!--   <xacro:insert_block name="origin" /> -->
+	<!--   <parent link="dishwasher_main"/> -->
+	<!--   <child link="sink_area_dish_washer_main"/> -->
+    <!-- </joint> -->
   <link name="sink_area_dish_washer_main">
     <inertial>

Commit message: WIP: add mass and forces to semantic map to allow good gazebo simulation

File: suturo_resources/urdf/urdf_components/suturo_dishwasher.urdf.xacro (robot description, xacro)
@@ -47,5 +47,5 @@
       <origin rpy="0 0 0" xyz="0.0 0.0 0.0"/>
       <mass value="1"/>
-      <inertia ixx="1" ixy="0.0" ixz="0.0" iyy="1" iyz="0.0" izz="1"/>
+      <inertia ixx="0.03" ixy="0.0" ixz="0.0" iyy="0.07" iyz="0.0" izz="0.041"/>
     </inertial>
     <visual>
@@ -62,9 +62,13 @@
     </collision>
   </link>
+ <gazebo reference="sink_area_dish_washer_door">
+   <gravity>false</gravity>
+   <dampingFactor>0.01</dampingFactor>
+ </gazebo>
   <link name="sink_area_dish_washer_door_handle">
     <inertial>
       <origin rpy="0 0 0" xyz="0.0 0.0 0.0"/>
-      <mass value="1"/>
-      <inertia ixx="1" ixy="0.0" ixz="0.0" iyy="1" iyz="0.0" izz="1"/>
+      <mass value="0.1"/>
+      <inertia ixx="0.0025" ixy="0.0" ixz="0.0" iyy="0.0025" iyz="0.0" izz="0.000125"/>
     </inertial>
     <visual>
@@ -81,4 +85,8 @@
     </collision>
   </link>
+ <gazebo reference="sink_area_dish_washer_door_handle">
+   <gravity>false</gravity>
+   <dampingFactor>0.01</dampingFactor>
+ </gazebo>
   <link name="dishwasher_tab"/>
   <link name="dishwasher_table:d_table:table_origin"/>
@@ -122,5 +130,5 @@
     <!-- TODO Fix Limits to be able to open dishwasher-->
     <limit effort="300" lower="0.0" upper="1.57079632679" velocity="10"/>
-  </joint>
+ </joint>
   <joint name="sink_area_dish_washer_door_handle_joint" type="fixed">
     <origin rpy="-1.57079632679 0 0" xyz="0.0625 -0.6325 0."/>

File: suturo_resources/urdf/urdf_components/suturo_door.urdf.xacro (robot description, xacro)
@@ -56,7 +56,4 @@
         <inertia ixx="0.1" ixy="0.0" ixz="0.0" iyy="0.1" iyz="0.0" izz="0.1"/>
       </inertial>
-            <gazebo>
-   <turnGravityOff>true</turnGravityOff>
-</gazebo>
     </link>
 	<link name="${name}:door_handle_link">
@@ -78,7 +75,4 @@
         <inertia ixx="0.1" ixy="0.0" ixz="0.0" iyy="0.1" iyz="0.0" izz="0.1"/>
       </inertial>
-                  <gazebo>
-   <turnGravityOff>true</turnGravityOff>
-</gazebo>
     </link>
     <link name="${name}:door_handle_outside">
@@ -102,7 +96,4 @@
         <inertia ixx="0.1" ixy="0.0" ixz="0.0" iyy="0.1" iyz="0.0" izz="0.1"/>
       </inertial>
-                        <gazebo>
-   <turnGravityOff>true</turnGravityOff>
-</gazebo>
     </link>
     <link name="${name}:door_handle_inside">
@@ -126,7 +117,4 @@
         <inertia ixx="0.1" ixy="0.0" ixz="0.0" iyy="0.1" iyz="0.0" izz="0.1"/>
       </inertial>
-      <gazebo>
-   <turnGravityOff>true</turnGravityOff>
-</gazebo>
     </link>
     <!-- JOINTS -->
@@ -152,4 +140,8 @@
 	  <child link="${name}:door_handle_link"/>
     </joint>
+    <gazebo reference="${name}:door_handle_joint">
+      <springReference>-${pi}</springReference>
+      <springStiffness>1</springStiffness>
+    </gazebo>
     <joint name="${name}:door_handle_inside_joint" type="fixed">
       <origin xyz="-0.04 0 0.06" rpy="0 0 ${pi/2}" />

Commit message: [semantic map] dishwasher door inertia and dampening

File: suturo_resources/urdf/urdf_components/suturo_dishwasher.urdf.xacro (robot description, xacro)
@@ -47,5 +47,5 @@
       <origin rpy="0 0 0" xyz="0.0 0.0 0.0"/>
       <mass value="1"/>
-      <inertia ixx="1" ixy="0.0" ixz="0.0" iyy="1" iyz="0.0" izz="1"/>
+      <inertia ixx="0.03" ixy="0.0" ixz="0.0" iyy="0.07" iyz="0.0" izz="0.041"/>
     </inertial>
     <visual>
@@ -64,10 +64,12 @@
   <gazebo reference="sink_area_dish_washer_door">
     <turnGravityOff>true</turnGravityOff>
+    <!-- this value is not accurate, but for now it should be enough for the simulation -->
+    <dampingFactor>0.005</dampingFactor>
   </gazebo>
   <link name="sink_area_dish_washer_door_handle">
     <inertial>
       <origin rpy="0 0 0" xyz="0.0 0.0 0.0"/>
-      <mass value="1"/>
-      <inertia ixx="1" ixy="0.0" ixz="0.0" iyy="1" iyz="0.0" izz="1"/>
+      <mass value="0.1"/>
+      <inertia ixx="0.0025" ixy="0.0" ixz="0.0" iyy="0.0025" iyz="0.0" izz="0.000125"/>
     </inertial>
     <visual>

Commit message: semantic map adjust dishwasher position

File: suturo_resources/urdf/urdf_components/suturo_dishwasher.urdf.xacro (robot description, xacro)
@@ -116,5 +116,5 @@
     <axis xyz="1 0 0" />
     <!-- <limit effort="300" lower="0" upper="0" velocity="10"/> -->
-    <origin rpy="0 0 0" xyz="0.08 -0.78 0.44 "/>
+    <origin rpy="0 0 0" xyz="0.08 -0.78 0.455 "/>
     <parent link="dishwasher_main"/>
     <child link="sink_area_dish_washer_main"/>

Commit message: [semantic map] dishwasher table frame direction fixed. X is now away from the room

File: suturo_resources/urdf/urdf_components/suturo_dishwasher.urdf.xacro (robot description, xacro)
@@ -136,10 +136,10 @@
   <!-- from here for dishwasher_table -->
   <joint name="dish_washer_table_main_joint" type="fixed">
-    <origin rpy="0.0 0 0" xyz="0.0 0.0 0.39"/>
+    <origin rpy="0 0 ${pi}" xyz="0.0 0.0 0.39"/>
     <parent link="sink_area_dish_washer_main"/>
     <child link="dishwasher_table:d_table:table_origin"/>
   </joint>
   <joint name="dish_washer_table_center_joint" type="fixed">
-    <origin rpy="0 0 0" xyz="0.3 0 0"/>
+    <origin rpy="0 0 0" xyz="-0.3 0 0"/>
     <parent link="dishwasher_table:d_table:table_origin"/>
     <child link="dishwasher_table:d_table:table_front_edge_center"/>

Commit message: added apartment dishwasher changes

File: suturo_resources/urdf/urdf_components/suturo_dishwasher.urdf.xacro (robot description, xacro)
@@ -2,5 +2,5 @@
 <robot name="suturo_dishwasher" xmlns:xacro="http://ros.org/wiki/xacro">
   <material name="dishwasher_table_color">
-	<color rgba="0.255 0.62 0.223 1"/>
+	<color rgba="1 0.62 0.223 1"/>
   </material>
   <xacro:macro name="suturo_dishwasher" params="name parent *origin">
@@ -116,5 +116,5 @@
     <axis xyz="1 0 0" />
     <!-- <limit effort="300" lower="0" upper="0" velocity="10"/> -->
-    <origin rpy="0 0 0" xyz="0.08 -0.78 0.455 "/>
+    <origin rpy="0 0 0" xyz="0.08 -0.78 0.555 "/>
     <parent link="dishwasher_main"/>
     <child link="sink_area_dish_washer_main"/>
@@ -129,6 +129,7 @@
     <limit effort="300" lower="0.0" upper="1.57079632679" velocity="10"/>
   </joint>
+  <!--x,y,z Handle position change-->
   <joint name="sink_area_dish_washer_door_handle_joint" type="fixed">
-    <origin rpy="-1.57079632679 0 0" xyz="0.0625 -0.6325 0."/>
+    <origin rpy="-1.57079632679 0 0" xyz="0.05 -0.6325 0."/>
     <parent link="sink_area_dish_washer_door"/>
     <child link="sink_area_dish_washer_door_handle"/>
@@ -136,5 +137,5 @@
   <!-- from here for dishwasher_table -->
   <joint name="dish_washer_table_main_joint" type="fixed">
-    <origin rpy="0 0 ${pi}" xyz="0.0 0.0 0.39"/>
+    <origin rpy="0 0 ${pi}" xyz="0.0 0.0 0.37"/>
     <parent link="sink_area_dish_washer_main"/>
     <child link="dishwasher_table:d_table:table_origin"/>

Commit message: little Dishwasher handle adjustment

File: suturo_resources/urdf/urdf_components/suturo_dishwasher.urdf.xacro (robot description, xacro)
@@ -131,5 +131,5 @@
   <!--x,y,z Handle position change-->
   <joint name="sink_area_dish_washer_door_handle_joint" type="fixed">
-    <origin rpy="-1.57079632679 0 0" xyz="0.05 -0.6325 0."/>
+    <origin rpy="-1.57079632679 0 0" xyz="0.035 -0.6325 0."/>
     <parent link="sink_area_dish_washer_door"/>
     <child link="sink_area_dish_washer_door_handle"/>

Commit message: old dishwasher

File: suturo_resources/urdf/urdf_components/suturo_dishwasher.urdf.xacro (robot description, xacro)
@@ -2,5 +2,5 @@
 <robot name="suturo_dishwasher" xmlns:xacro="http://ros.org/wiki/xacro">
   <material name="dishwasher_table_color">
-	<color rgba="1 0.62 0.223 1"/>
+	<color rgba="0.255 0.62 0.223 1"/>
   </material>
   <xacro:macro name="suturo_dishwasher" params="name parent *origin">
@@ -116,5 +116,5 @@
     <axis xyz="1 0 0" />
     <!-- <limit effort="300" lower="0" upper="0" velocity="10"/> -->
-    <origin rpy="0 0 0" xyz="0.08 -0.78 0.555 "/>
+    <origin rpy="0 0 0" xyz="0.08 -0.78 0.455 "/>
     <parent link="dishwasher_main"/>
     <child link="sink_area_dish_washer_main"/>
@@ -131,5 +131,5 @@
   <!--x,y,z Handle position change-->
   <joint name="sink_area_dish_washer_door_handle_joint" type="fixed">
-    <origin rpy="-1.57079632679 0 0" xyz="0.035 -0.6325 0."/>
+    <origin rpy="-1.57079632679 0 0" xyz="0.0625 -0.6325 0."/>
     <parent link="sink_area_dish_washer_door"/>
     <child link="sink_area_dish_washer_door_handle"/>
@@ -137,5 +137,5 @@
   <!-- from here for dishwasher_table -->
   <joint name="dish_washer_table_main_joint" type="fixed">
-    <origin rpy="0 0 ${pi}" xyz="0.0 0.0 0.37"/>
+    <origin rpy="0 0 ${pi}" xyz="0.0 0.0 0.39"/>
     <parent link="sink_area_dish_washer_main"/>
     <child link="dishwasher_table:d_table:table_origin"/>

Commit message: more changes for dishwasher opening, to be able to have a smaller gap in dishwasher

File: suturo_resources/urdf/urdf_components/suturo_dishwasher.urdf.xacro (robot description, xacro)
@@ -50,5 +50,5 @@
     </inertial>
     <visual>
-      <origin rpy="1.57079632679 0 0" xyz="0 0 0"/>
+      <origin rpy="1.57079632679 0 0" xyz="0 0.05 0"/>
       <geometry>
         <mesh filename="package://iai_kitchen/meshes/misc/DishWasherDoor.obj"/>
@@ -56,5 +56,5 @@
     </visual>
     <collision>
-      <origin rpy="1.57079632679 0 0" xyz="0 0 0"/>
+      <origin rpy="1.57079632679 0 0" xyz="0 0.05 0"/>
       <geometry>
         <mesh filename="package://iai_kitchen/meshes/misc/DishWasherDoor.obj"/>

Commit message: adjusted some positions for the dishwasher

File: suturo_resources/urdf/urdf_components/suturo_dishwasher.urdf.xacro (robot description, xacro)
@@ -50,5 +50,5 @@
     </inertial>
     <visual>
-      <origin rpy="1.57079632679 0 0" xyz="0 0.05 0"/>
+      <origin rpy="1.57079632679 0 0" xyz="0 0.07 0"/>
       <geometry>
         <mesh filename="package://iai_kitchen/meshes/misc/DishWasherDoor.obj"/>
